Commit message: Fix formatting (tab->spaces, etc.)

File: wamv_description/urdf/cpu_cases.xacro (robot description, xacro)
@@ -2,34 +2,34 @@
 <robot xmlns:xacro="http://ros.org/wiki/xacro" name="wam-v-cpu_cases">
 <xacro:macro name="cpu_cases" params="position:='0 0 0' orientation:='0 0 0'">
-    <link name="cpu_cases_link">
-      <visual name="cpu_cases_visual">
-        <origin xyz="0.073 0 -1.53" rpy="0 0 0"/>
-        <geometry>
-	  <mesh filename="package://vrx_gazebo/models/cpu_cases/mesh/cpu_cases.dae"/>
-	</geometry>
-      </visual>
-      <collision name="cpu_cases_collision">
-        <origin xyz="0 0 0" rpy="0 0 0"/>
-        <geometry>
-           <box size="0.97 0.83 .47"/>
-        </geometry>
-      </collision>
-      <inertial>
-        <origin xyz="0 0 0" rpy="0 0 0"/>
-	<mass value="20"/>
-	<inertia
-	  ixx="1.51633333333333"
-          iyy="1.93633333333333"
-	  izz="2.71633333333333"
-	  ixy="0"
-	  ixz="0"
-	  iyz="0"/>
-      </inertial>
-    </link>
-    <joint name ="chasis_cpu_cases_joint" type="fixed">
-      <origin xyz="${position}" rpy="${orientation}"/>
-      <parent link="base_link"/>
-      <child link="cpu_cases_link"/>
-    </joint>
+  <link name="cpu_cases_link">
+    <visual name="cpu_cases_visual">
+      <origin xyz="0.073 0 -1.53" rpy="0 0 0"/>
+      <geometry>
+        <mesh filename="package://vrx_gazebo/models/cpu_cases/mesh/cpu_cases.dae"/>
+      </geometry>
+    </visual>
+    <collision name="cpu_cases_collision">
+      <origin xyz="0 0 0" rpy="0 0 0"/>
+      <geometry>
+         <box size="0.97 0.83 0.47"/>
+      </geometry>
+    </collision>
+    <inertial>
+      <origin xyz="0 0 0" rpy="0 0 0"/>
+      <mass value="20"/>
+      <inertia
+        ixx="1.51633333333333"
+        iyy="1.93633333333333"
+        izz="2.71633333333333"
+        ixy="0"
+        ixz="0"
+        iyz="0"/>
+    </inertial>
+  </link>
+  <joint name ="chasis_cpu_cases_joint" type="fixed">
+    <origin xyz="${position}" rpy="${orientation}"/>
+    <parent link="base_link"/>
+    <child link="cpu_cases_link"/>
+  </joint>
 </xacro:macro>
 </robot>

Commit message: Move boxes forward to prevent collision with gps

File: wamv_description/urdf/cpu_cases.xacro (robot description, xacro)
@@ -12,5 +12,5 @@
       <origin xyz="0 0 0" rpy="0 0 0"/>
       <geometry>
-         <box size="0.97 0.83 0.47"/>
+        <box size="0.97 0.83 0.47"/>
       </geometry>
     </collision>

File: wamv_gazebo/urdf/wamv_gazebo.urdf.xacro (robot description, xacro)
@@ -15,5 +15,5 @@
   <!-- === CPU Cases === -->
   <xacro:include filename="$(find wamv_description)/urdf/cpu_cases.xacro" />
-  <xacro:cpu_cases position="-0.3 0 1.53" orientation="0 0 0"/>
+  <xacro:cpu_cases position="-0.15 0 1.53" orientation="0 0 0"/>
   <!-- === Thrusters === -->
   <xacro:property name="thruster_conf" value="$(arg thruster_config)"/> -->

Commit message: Change cpu case collision box from 1 box to 2 boxes

File: wamv_description/urdf/cpu_cases.xacro (robot description, xacro)
@@ -9,12 +9,17 @@
       </geometry>
     </visual>
-    <collision name="cpu_cases_collision">
-      <origin xyz="0 0 0" rpy="0 0 0"/>
+    <collision name="cpu_case_1_collision">
+      <origin xyz="0.185 0 0" rpy="0 0 0"/>
       <geometry>
-        <box size="0.97 0.83 0.47"/>
+        <box size="0.595 0.83 0.47"/>
+      </geometry>
+    </collision>
+    <collision name="cpu_case_2_collision">
+      <origin xyz="-0.3 0 -0.092" rpy="0 0 0"/>
+      <geometry>
+        <box size="0.375 0.64 0.28"/>
       </geometry>
     </collision>
     <inertial>
-      <origin xyz="0 0 0" rpy="0 0 0"/>
       <mass value="20"/>
       <inertia
