Commit message: incremental

File: wamv_description/urdf/sensors.xacro (robot description, xacro)
@@ -8,11 +8,2 @@
   <!-- === wamv_p3d === -->
   <xacro:wamv_p3d name="p3d_wamv" />
-  <!-- === wamv_camera === -->
-  <xacro:wamv_camera y="0.3" x="0.75" z="2" name="front_camera" P="${radians(15)}" />
-  <xacro:wamv_camera y="0.1" x="0.75" name="front_left_camera" P="${radians(15)}" />
-  <xacro:wamv_camera y="-0.1" x="0.75" name="front_right_camera" P="${radians(15)}" />
-  <xacro:wamv_camera y="0.1" x="0.75" name="middle_right_camera" P="${radians(15)}" />
-  <!-- === wamv_3d_lidar === -->
-  <xacro:wamv_3d_lidar P="${radians(8)}" name="lidar_wamv" />
-</xacro:macro>
-</robot>

Commit message: incremental

File: wamv_description/urdf/sensors.xacro (robot description, xacro)
@@ -8,2 +8,11 @@
   <!-- === wamv_p3d === -->
   <xacro:wamv_p3d name="p3d_wamv" />
+  <!-- === wamv_camera === -->
+  <xacro:wamv_camera y="0.3" x="0.75" z="2" name="front_camera" P="${radians(15)}" />
+  <xacro:wamv_camera y="0.1" x="0.75" name="front_left_camera" P="${radians(15)}" />
+  <xacro:wamv_camera y="-0.1" x="0.75" name="front_right_camera" P="${radians(15)}" />
+  <xacro:wamv_camera y="0.1" x="0.75" name="middle_right_camera" P="${radians(15)}" />
+  <!-- === wamv_3d_lidar === -->
+  <xacro:wamv_3d_lidar P="${radians(8)}" name="lidar_wamv" />
+</xacro:macro>
+</robot>

Commit message: changed directory, added launch file support

File: wamv_description/urdf/sensors.xacro (robot description, xacro)
@@ -7,5 +7,5 @@
   <xacro:wamv_gps P="0" R="0" name="gps_wamv" Y="0" x="-0.85" z="1.28" y="0" />
   <!-- === wamv_p3d === -->
-  <xacro:wamv_p3d name="ground_truth_odometry" />
+  <xacro:wamv_p3d name="p3d_wamv" />
   <!-- === wamv_camera === -->
   <xacro:wamv_camera P="${radians(15)}" R="0" name="front_camera" Y="0" x="0.75" z="2" y="0.3" />
@@ -15,4 +15,4 @@
   <!-- === wamv_3d_lidar === -->
   <xacro:wamv_3d_lidar max_range="100" noise_stddev="0.01" vertical_lasers="16" P="${radians(8)}" min_vertical_angle="${-pi/12}" Y="0" max_angle="${pi}" name="lidar_wamv" R="0" update_rate="10" samples="1800" y="0" x="0.7" z="1.45" resolution="0.1" max_vertical_angle="${pi/12}" min_angle="${-pi}" />
-</xacro:macro>
+  </xacro:macro>
 </robot>

Commit message: fixed styling problems with flake8, updated readme

File: wamv_description/urdf/sensors.xacro (robot description, xacro)
@@ -1,5 +1,5 @@
 <?xml version="1.0"?>
 <robot xmlns:xacro="http://ros.org/wiki/xacro" name="wam-v-sensors">
-<xacro:macro name="sensors">
+  <xacro:macro name="sensors">
   <!-- === wamv_imu === -->
   <xacro:wamv_imu P="0" R="0" name="imu_wamv" Y="0" x="0" z="1.3" y="-0.2" />
