Commit message: Implement turnable thruster joint

File: wamv_description/urdf/engine.xacro (robot description, xacro)
@@ -43,5 +43,7 @@
       </inertial>
     </link>
-    <joint name="${prefix}_chasis_engine_joint" type="fixed">
+    <joint name="${prefix}_chasis_engine_joint" type="revolute">
+      <axis xyz="0 0 1"/>
+      <limit lower="${-pi}" upper="${pi}" effort="10" velocity="10"/>
       <origin xyz="${position}" rpy="${orientation}"/>
       <parent link="base_link"/>

File: wamv_gazebo/urdf/thruster_layouts/wamv_gazebo_thruster_config.xacro (robot description, xacro)
@@ -5,4 +5,5 @@
       <linkName>${name}_propeller_link</linkName>
       <propJointName>${name}_engine_propeller_joint</propJointName>
+      <engineJointName>${name}_chasis_engine_joint</engineJointName>
       <cmdTopic>${name}_thrust_cmd</cmdTopic>
       <angleTopic>${name}_thrust_angle</angleTopic>
