Commit message: More modular model with spinning propellers.

File: wamv_description/urdf/wamv_base.urdf.xacro (robot description, xacro)
@@ -1,7 +1,142 @@
 <?xml version="1.0"?>
-<!-- Basic model of the 16' WAM-V USV -->
 <robot xmlns:xacro="http://ros.org/wiki/xacro" name="wam-v">
+  <!-- Macro for creating the main collisions as simple shapes. -->
+  <xacro:macro name="main_collisions" params="prefix reflect:=1">
+    <!-- Main float -->
+    <collision name="${prefix}_float">
+      <origin xyz="-0.4 ${1.03*reflect} 0.2" rpy="${0*reflect} 1.57 0" />
+      <geometry>
+        <cylinder length="4" radius="0.2" />
+      </geometry>
+    </collision>
+    <collision name="${prefix}_mid_float">
+      <origin xyz="1.85 ${1.03*reflect} 0.3" rpy="${0*reflect} 1.38 0" />
+      <geometry>
+        <cylinder length="0.5" radius="0.17" />
+      </geometry>
+    </collision>
+    <collision name="l${prefix}_front_float">
+      <origin xyz="2.3 ${1.03*reflect} 0.4" rpy="${0*reflect} 1.3 0" />
+      <geometry>
+        <cylinder length="0.45" radius="0.12" />
+      </geometry>
+    </collision>
+    <!-- Front beam -->
+    <collision name="front_${prefix}_beam_lower">
+      <origin xyz="0.9 ${0.85*reflect} 1" rpy="${0.78*reflect} 0 0" />
+      <geometry>
+        <cylinder length="0.5" radius="0.04" />
+      </geometry>
+    </collision>
+    <collision name="front_${prefix}_beam_upper">
+      <origin xyz="0.9 ${0.6*reflect} 1.18" rpy="${1.35*reflect} 0 0" />
+      <geometry>
+        <cylinder length="0.2" radius="0.04" />
+      </geometry>
+    </collision>
+    <!-- Mid beam -->
+    <collision name="mid_l${prefix}_beam_lower">
+      <origin xyz="-0.65 ${0.99*reflect} 0.7" rpy="${0.1*reflect} 0.25 0" />
+      <geometry>
+        <cylinder length="0.45" radius="0.03" />
+      </geometry>
+    </collision>
+    <collision name="mid_${prefix}_beam_medium">
+      <origin xyz="-0.57 ${0.87*reflect} 1.05" rpy="${0.75*reflect} 0.25 0" />
+      <geometry>
+        <cylinder length="0.32" radius="0.03" />
+      </geometry>
+    </collision>
+    <collision name="mid_l${prefix}_beam_upper">
+      <origin xyz="-0.55 ${0.65*reflect} 1.17" rpy="${1.35*reflect} 0.25 0" />
+      <geometry>
+        <cylinder length="0.3" radius="0.03" />
+      </geometry>
+    </collision>
+    <!-- Rear beam -->
+    <collision name="rear_${prefix}_beam_lower">
+      <origin xyz="-0.74 ${1.03*reflect} 0.7" rpy="${0*reflect} -0.15 0" />
+      <geometry>
+        <cylinder length="0.45" radius="0.03" />
+      </geometry>
+    </collision>
+    <collision name="rear_${prefix}_beam_medium">
+      <origin xyz="-0.79 ${0.91*reflect} 1.05" rpy="${0.75*reflect} -0.15 0" />
+      <geometry>
+        <cylinder length="0.32" radius="0.03" />
+      </geometry>
+    </collision>
+    <collision name="rear_${prefix}_beam_upper">
+      <origin xyz="-0.81 ${0.67*reflect} 1.18" rpy="${1.45*reflect} -0.15 0" />
+      <geometry>
+        <cylinder length="0.3" radius="0.03" />
+      </geometry>
+    </collision>
+    <!-- Joint -->
+    <collision name="${prefix}_joint">
+      <origin xyz="0.58 ${1.03*reflect} 0.6" rpy="${0*reflect} -0.6 0" />
+      <geometry>
+        <box size="0.65 0.2 0.1" />
+      </geometry>
+    </collision>
+  </xacro:macro>
+  <!-- Macro for inserting an engine with its propeller. -->
+  <xacro:macro name="engine" params="prefix position:='0 0 0' orientation:='0 0 0'">
+    <link name="${prefix}_engine_link">
+      <visual>
+        <geometry>
+          <mesh filename="package://wamv_description/mesh/engine.dae"/>
+        </geometry>
+      </visual>
+      <collision name="${prefix}_engine_vertical_axis_collision">
+        <origin xyz="-0.16 0 -0.24" rpy="0 0 0" />
+        <geometry>
+          <box size="0.2 0.15 0.83" />
+        </geometry>
+      </collision>
+      <collision name="${prefix}_engine_rear_end_collision">
+        <origin xyz="-0.34 0 0.12" rpy="0 0 0" />
+        <geometry>
+          <box size="0.12 0.15 0.12" />
+        </geometry>
+      </collision>
+      <inertial>
+        <mass value="15"/>
+        <inertia ixx="0.889245" ixy="0.0" ixz="0.0" iyy="0.911125" iyz="0.0" izz="0.078125"/>
+      </inertial>
+    </link>
+    <link name="${prefix}_propeller_link">
+      <visual>
+        <geometry>
+          <mesh filename="package://wamv_description/mesh/propeller.dae"/>
+        </geometry>
+      </visual>
+      <collision name="${prefix}_propeller_collision">
+        <origin xyz="-0.08 0 0" rpy="0 1.57 0" />
+        <geometry>
+          <cylinder length="0.18" radius="0.24" />
+        </geometry>
+      </collision>
+      <inertial>
+        <mass value="0.5"/>
+        <inertia ixx="0.008545" ixy="0.0" ixz="0.0" iyy="0.008545" iyz="0.0" izz="0.0144"/>
+      </inertial>
+    </link>
+    <joint name="${prefix}_chasis_engine_joint" type="fixed">
+      <origin xyz="${position}" rpy="${orientation}"/>
+      <parent link="base_link"/>
+      <child link="${prefix}_engine_link"/>
+    </joint>
+    <joint name="${prefix}_engine_propeller_joint" type="continuous">
+      <axis rpy="0 0 0" xyz="1 0 0"/>
+      <parent link="${prefix}_engine_link"/>
+      <child link="${prefix}_propeller_link"/>
+      <origin rpy="0 0 0" xyz="-0.278156 0 -0.509371"/>
+      <limit effort="100" velocity="100" />
+      <dynamics friction="0.05" damping="0.05" />
+    </joint>
+  </xacro:macro>
+  <!-- Basic model of the 16' WAM-V USV -->
   <link name="base_link">
-    <wind>true</wind>
     <visual>
       <geometry>
@@ -9,81 +144,9 @@
       </geometry>
     </visual>
-    <!-- Left float -->
-    <collision name="left_float">
-      <origin xyz="-0.4 1.03 0.2" rpy="0 1.57 0" />
-      <geometry>
-        <cylinder length="4" radius="0.2" />
-      </geometry>
-    </collision>
-    <collision name="left_mid_float">
-      <origin xyz="1.85 1.03 0.3" rpy="0 1.38 0" />
-      <geometry>
-        <cylinder length="0.5" radius="0.17" />
-      </geometry>
-    </collision>
-    <collision name="left_front_float">
-      <origin xyz="2.3 1.03 0.4" rpy="0 1.3 0" />
-      <geometry>
-        <cylinder length="0.45" radius="0.12" />
-      </geometry>
-    </collision>
-    <!-- Left engine upper -->
-    <collision name="left_engine_vertical_axis">
-      <origin xyz="-2.55 1.03 0.09" rpy="0 0 0" />
-      <geometry>
-        <box size="0.2 0.15 0.83" />
-      </geometry>
-    </collision>
-    <collision name="left_engine_rear_end">
-      <origin xyz="-2.71 1.03 0.45" rpy="0 0 0" />
-      <geometry>
-        <box size="0.12 0.15 0.12" />
-      </geometry>
-    </collision>
-    <collision name="left_propeller">
-      <origin xyz="-2.73 1.03 -0.2" rpy="0 1.57 0" />
-      <geometry>
-        <cylinder length="0.18" radius="0.24" />
-      </geometry>
-    </collision>
-    <!-- Right float -->
-    <collision name="left_float">
-      <origin xyz="-0.4 -1.03 0.2" rpy="0 1.57 0" />
-      <geometry>
-        <cylinder length="4" radius="0.2" />
-      </geometry>
-    </collision>
-    <collision name="left_mid_float">
-      <origin xyz="1.85 -1.03 0.3" rpy="0 1.38 0" />
-      <geometry>
-        <cylinder length="0.5" radius="0.17" />
-      </geometry>
-    </collision>
-    <collision name="left_front_float">
-      <origin xyz="2.3 -1.03 0.4" rpy="0 1.3 0" />
-      <geometry>
-        <cylinder length="0.45" radius="0.12" />
-      </geometry>
-    </collision>
-    <!-- Right engine upper -->
-    <collision name="left_engine_vertical_axis">
-      <origin xyz="-2.55 -1.03 0.09" rpy="0 0 0" />
-      <geometry>
-        <box size="0.2 0.15 0.83" />
-      </geometry>
-    </collision>
-    <collision name="left_engine_rear_end">
-      <origin xyz="-2.71 -1.03 0.45" rpy="0 0 0" />
-      <geometry>
-        <box size="0.12 0.15 0.12" />
-      </geometry>
-    </collision>
-    <collision name="left_propeller">
-      <origin xyz="-2.73 -1.03 -0.2" rpy="0 1.57 0" />
-      <geometry>
-        <cylinder length="0.18" radius="0.24" />
-      </geometry>
-    </collision>
-    <!-- Base -->
+    <!-- Left base collisions -->
+    <xacro:main_collisions prefix="left" reflect="1" />
+    <!-- Right side collisions -->
+    <xacro:main_collisions prefix="right" reflect="-1" />
+     <!-- Top base -->
     <collision name="top_base">
       <origin xyz="0 -0 1.25" rpy="0 0 0" />
@@ -92,128 +155,13 @@
       </geometry>
     </collision>
-    <!-- Front left beam -->
-    <collision name="front_left_beam_lower">
-      <origin xyz="0.9 0.85 1" rpy="0.78 0 0" />
-      <geometry>
-        <cylinder length="0.5" radius="0.04" />
-      </geometry>
-    </collision>
-    <collision name="front_left_beam_upper">
-      <origin xyz="0.9 0.6 1.18" rpy="1.35 0 0" />
-      <geometry>
-        <cylinder length="0.2" radius="0.04" />
-      </geometry>
-    </collision>
-    <!-- Front right beam -->
-    <collision name="front_right_beam_lower">
-      <origin xyz="0.9 -0.85 1" rpy="-0.78 0 0" />
-      <geometry>
-        <cylinder length="0.5" radius="0.04" />
-      </geometry>
-    </collision>
-    <collision name="front_right_beam_upper">
-      <origin xyz="0.9 -0.6 1.18" rpy="-1.35 0 0" />
-      <geometry>
-        <cylinder length="0.2" radius="0.04" />
-      </geometry>
-    </collision>
-    <!-- Mid left beam -->
-    <collision name="mid_left_beam_lower">
-      <origin xyz="-0.65 0.99 0.7" rpy="0.1 0.25 0" />
-      <geometry>
-        <cylinder length="0.45" radius="0.03" />
-      </geometry>
-    </collision>
-    <collision name="mid_left_beam_medium">
-      <origin xyz="-0.57 0.87 1.05" rpy="0.75 0.25 0" />
-      <geometry>
-        <cylinder length="0.32" radius="0.03" />
-      </geometry>
-    </collision>
-    <collision name="mid_left_beam_upper">
-      <origin xyz="-0.55 0.65 1.17" rpy="1.35 0.25 0" />
-      <geometry>
-        <cylinder length="0.3" radius="0.03" />
-      </geometry>
-    </collision>
-    <!-- Mid right beam -->
-    <collision name="mid_right_beam_lower">
-      <origin xyz="-0.65 -0.99 0.7" rpy="-0.1 0.25 0" />
-      <geometry>
-        <cylinder length="0.45" radius="0.03" />
-      </geometry>
-    </collision>
-    <collision name="mid_right_beam_medium">
-      <origin xyz="-0.57 -0.87 1.05" rpy="-0.75 0.25 0" />
-      <geometry>
-        <cylinder length="0.32" radius="0.03" />
-      </geometry>
-    </collision>
-    <collision name="mid_right_beam_upper">
-      <origin xyz="-0.55 -0.65 1.17" rpy="-1.35 0.25 0" />
-      <geometry>
-        <cylinder length="0.3" radius="0.03" />
-      </geometry>
-    </collision>
-    <!-- Rear left beam -->
-    <collision name="rear_left_beam_lower">
-      <origin xyz="-0.74 1.03 0.7" rpy="0 -0.15 0" />
-      <geometry>
-        <cylinder length="0.45" radius="0.03" />
-      </geometry>
-    </collision>
-    <collision name="rear_left_beam_medium">
-      <origin xyz="-0.79 0.91 1.05" rpy="0.75 -0.15 0" />
-      <geometry>
-        <cylinder length="0.32" radius="0.03" />
-      </geometry>
-    </collision>
-    <collision name="rear_left_beam_upper">
-      <origin xyz="-0.81 0.67 1.18" rpy="1.45 -0.15 0" />
-      <geometry>
-        <cylinder length="0.3" radius="0.03" />
-      </geometry>
-    </collision>
-    <!-- Rear right beam -->
-    <collision name="rear_right_beam_lower">
-      <origin xyz="-0.74 -1.03 0.7" rpy="0 -0.15 0" />
-      <geometry>
-        <cylinder length="0.45" radius="0.03" />
-      </geometry>
-    </collision>
-    <collision name="rear_right_beam_medium">
-      <origin xyz="-0.79 -0.91 1.05" rpy="-0.75 -0.15 0" />
-      <geometry>
-        <cylinder length="0.32" radius="0.03" />
-      </geometry>
-    </collision>
-    <collision name="rear_right_beam_upper">
-      <origin xyz="-0.81 -0.67 1.18" rpy="-1.45 -0.15 0" />
-      <geometry>
-        <cylinder length="0.3" radius="0.03" />
-      </geometry>
-    </collision>
-    <collision name="left_joint">
-      <origin xyz="0.58 1.03 0.6" rpy="0 -0.6 0" />
-      <geometry>
-        <box size="0.65 0.2 0.1" />
-      </geometry>
-    </collision>
-    <collision name="right_joint">
-      <origin xyz="0.58 -1.03 0.6" rpy="0 -0.6 0" />
-      <geometry>
-        <box size="0.65 0.2 0.1" />
-      </geometry>
-    </collision>
     <inertial>
-      <mass value="180.0"/> <!-- From WAM-V spec sheet -->
+      <!-- From WAM-V spec sheet -->
+      <mass value="180.0"/>
       <inertia ixx="120.0" ixy="0.0" ixz="0.0" iyy="393" iyz="0.0" izz="446.0"/>
     </inertial>
   </link>
-  <joint name="base_link_joint" type="fixed">
-    <origin xyz="0 0 0"/>
-    <parent link="base_footprint"/>
-    <child link="base_link"/>
-  </joint>
-  <link name="base_footprint"/>
+  <!-- Left engine-->
+  <xacro:engine prefix="left" position="-2.373776 1.027135 0.318237" />
+  <!-- Right engine-->
+  <xacro:engine prefix="right" position="-2.373776 -1.027135 0.318237" />
 </robot>

File: wamv_gazebo/urdf/wamv_gazebo_thrust_plugin.xacro (robot description, xacro)
@@ -19,4 +19,6 @@
       <maxForceRev>-100.0</maxForceRev>
       <cmdTimeout>1.0</cmdTimeout>
+      <left_propeller_joint>left_engine_propeller_joint</left_propeller_joint>
+      <right_propeller_joint>right_engine_propeller_joint</right_propeller_joint>
       </plugin>
     </gazebo>

Commit message: Split the wamv xacro file.

File: wamv_description/urdf/wamv_base.urdf.xacro (robot description, xacro)
@@ -16,5 +16,5 @@
       </geometry>
     </collision>
-    <collision name="l${prefix}_front_float">
+    <collision name="${prefix}_front_float">
       <origin xyz="2.3 ${1.03*reflect} 0.4" rpy="${0*reflect} 1.3 0" />
       <geometry>
@@ -36,5 +36,5 @@
     </collision>
     <!-- Mid beam -->
-    <collision name="mid_l${prefix}_beam_lower">
+    <collision name="mid_${prefix}_beam_lower">
       <origin xyz="-0.65 ${0.99*reflect} 0.7" rpy="${0.1*reflect} 0.25 0" />
       <geometry>
@@ -48,5 +48,5 @@
       </geometry>
     </collision>
-    <collision name="mid_l${prefix}_beam_upper">
+    <collision name="mid_${prefix}_beam_upper">
       <origin xyz="-0.55 ${0.65*reflect} 1.17" rpy="${1.35*reflect} 0.25 0" />
       <geometry>
@@ -81,60 +81,4 @@
     </collision>
   </xacro:macro>
-  <!-- Macro for inserting an engine with its propeller. -->
-  <xacro:macro name="engine" params="prefix position:='0 0 0' orientation:='0 0 0'">
-    <link name="${prefix}_engine_link">
-      <visual>
-        <geometry>
-          <mesh filename="package://wamv_description/mesh/engine.dae"/>
-        </geometry>
-      </visual>
-      <collision name="${prefix}_engine_vertical_axis_collision">
-        <origin xyz="-0.16 0 -0.24" rpy="0 0 0" />
-        <geometry>
-          <box size="0.2 0.15 0.83" />
-        </geometry>
-      </collision>
-      <collision name="${prefix}_engine_rear_end_collision">
-        <origin xyz="-0.34 0 0.12" rpy="0 0 0" />
-        <geometry>
-          <box size="0.12 0.15 0.12" />
-        </geometry>
-      </collision>
-      <inertial>
-        <mass value="15"/>
-        <inertia ixx="0.889245" ixy="0.0" ixz="0.0" iyy="0.911125" iyz="0.0" izz="0.078125"/>
-      </inertial>
-    </link>
-    <link name="${prefix}_propeller_link">
-      <visual>
-        <geometry>
-          <mesh filename="package://wamv_description/mesh/propeller.dae"/>
-        </geometry>
-      </visual>
-      <collision name="${prefix}_propeller_collision">
-        <origin xyz="-0.08 0 0" rpy="0 1.57 0" />
-        <geometry>
-          <cylinder length="0.18" radius="0.24" />
-        </geometry>
-      </collision>
-      <inertial>
-        <mass value="0.5"/>
-        <inertia ixx="0.008545" ixy="0.0" ixz="0.0" iyy="0.008545" iyz="0.0" izz="0.0144"/>
-      </inertial>
-    </link>
-    <joint name="${prefix}_chasis_engine_joint" type="fixed">
-      <origin xyz="${position}" rpy="${orientation}"/>
-      <parent link="base_link"/>
-      <child link="${prefix}_engine_link"/>
-    </joint>
-    <joint name="${prefix}_engine_propeller_joint" type="continuous">
-      <axis rpy="0 0 0" xyz="1 0 0"/>
-      <parent link="${prefix}_engine_link"/>
-      <child link="${prefix}_propeller_link"/>
-      <origin rpy="0 0 0" xyz="-0.278156 0 -0.509371"/>
-      <limit effort="100" velocity="100" />
-      <dynamics friction="0.05" damping="0.05" />
-    </joint>
-  </xacro:macro>
   <!-- Basic model of the 16' WAM-V USV -->
   <link name="base_link">
@@ -161,7 +105,3 @@
     </inertial>
   </link>
-  <!-- Left engine-->
-  <xacro:engine prefix="left" position="-2.373776 1.027135 0.318237" />
-  <!-- Right engine-->
-  <xacro:engine prefix="right" position="-2.373776 -1.027135 0.318237" />
 </robot>

File: wamv_gazebo/urdf/wamv_gazebo.urdf.xacro (robot description, xacro)
@@ -4,5 +4,5 @@
        name="WAM-V">
   <!-- Defines the base vehicle -->
-  <xacro:include filename="$(find wamv_description)/urdf/wamv_base.urdf.xacro" />
+  <xacro:include filename="$(find wamv_description)/urdf/wamv_two_engines.urdf.xacro" />
   <!-- Attach hydrodynamics plugin -->
   <xacro:include filename="$(find wamv_gazebo)/urdf/wamv_gazebo_dynamics_plugin.xacro" />

Commit message: Add sail link and joint

File: wamv_description/urdf/wamv_base.urdf.xacro (robot description, xacro)
@@ -1,4 +1,9 @@
 <?xml version="1.0"?>
 <robot xmlns:xacro="http://ros.org/wiki/xacro" name="wam-v">
+  <xacro:property name="platform_z" value="1.2965"/>
+  <xacro:property name="sail_length_x" value="1"/>
+  <xacro:property name="sail_length_y" value="0.2"/>
+  <xacro:property name="sail_length_z" value="1"/>
+  <xacro:property name="sail_z" value="${platform_z+sail_length_z/2}"/>
   <!-- Macro for creating the main collisions as simple shapes. -->
   <xacro:macro name="main_collisions" params="prefix reflect:=1">
@@ -87,4 +92,27 @@
     <child link="dummy_link"/>
   </joint>
+  <joint name="sail_joint" type="revolute">
+    <parent link="base_link"/>
+    <child link="sail_link"/>
+    <axis xyz="0 0 1"/>
+    <limit lower="${-pi}" upper="${pi}" effort="10" velocity="10"/>
+    <origin xyz="0 0 ${sail_z}" rpy="0 0 0"/>
+  </joint>
+  <link name="sail_link">
+    <visual>
+      <geometry>
+        <box size="1 0.25 1" />
+      </geometry>
+    </visual>
+    <collision>
+      <geometry>
+        <box size="1 0.25 1" />
+      </geometry>
+    </collision>
+    <inertial>
+      <mass value="1"/>
+      <inertia ixx="1" iyy="1" izz="1" ixy="0" ixz="0" iyz="0" />
+    </inertial>
+  </link>
   <!-- Basic model of the 16' WAM-V USV -->
   <link name="dummy_link">

Commit message: Add sail and rudder link to wamv base, as well as turn post to wind direction arrow

File: wamv_description/urdf/wamv_base.urdf.xacro (robot description, xacro)
@@ -4,6 +4,11 @@
   <xacro:property name="sail_length_x" value="1"/>
   <xacro:property name="sail_length_y" value="0.2"/>
-  <xacro:property name="sail_length_z" value="1"/>
+  <xacro:property name="sail_length_z" value="2"/>
   <xacro:property name="sail_z" value="${platform_z+sail_length_z/2}"/>
+  <xacro:property name="rudder_length_x" value="2"/>
+  <xacro:property name="rudder_length_y" value="0.2"/>
+  <xacro:property name="rudder_length_z" value="0.2"/>
+  <xacro:property name="rudder_x" value="-1"/>
+  <xacro:property name="rudder_z" value="${platform_z-1}"/>
   <!-- Macro for creating the main collisions as simple shapes. -->
   <xacro:macro name="main_collisions" params="prefix reflect:=1">
@@ -102,10 +107,33 @@
     <visual>
       <geometry>
-        <box size="1 0.25 1" />
+        <box size="${sail_length_x} ${sail_length_y} ${sail_length_z}" />
       </geometry>
     </visual>
     <collision>
       <geometry>
-        <box size="1 0.25 1" />
+        <box size="${sail_length_x} ${sail_length_y} ${sail_length_z}" />
+      </geometry>
+    </collision>
+    <inertial>
+      <mass value="1"/>
+      <inertia ixx="1" iyy="1" izz="1" ixy="0" ixz="0" iyz="0" />
+    </inertial>
+  </link>
+  <joint name="rudder_joint" type="revolute">
+    <parent link="base_link"/>
+    <child link="rudder_link"/>
+    <axis xyz="0 0 1"/>
+    <limit lower="${-pi}" upper="${pi}" effort="10" velocity="10"/>
+    <origin xyz="${rudder_x} 0 ${rudder_z}" rpy="0 0 0"/>
+  </joint>
+  <link name="rudder_link">
+    <visual>
+      <geometry>
+        <box size="${rudder_length_x} ${rudder_length_y} ${rudder_length_z}" />
+      </geometry>
+    </visual>
+    <collision>
+      <geometry>
+        <box size="${rudder_length_x} ${rudder_length_y} ${rudder_length_z}" />
       </geometry>
     </collision>

Commit message: Move rudder farther back

File: wamv_description/urdf/wamv_base.urdf.xacro (robot description, xacro)
@@ -9,5 +9,5 @@
   <xacro:property name="rudder_length_y" value="0.2"/>
   <xacro:property name="rudder_length_z" value="0.2"/>
-  <xacro:property name="rudder_x" value="-1"/>
+  <xacro:property name="rudder_x" value="-4"/>
   <xacro:property name="rudder_z" value="${platform_z-1}"/>
   <!-- Macro for creating the main collisions as simple shapes. -->

Commit message: Melodic compatibility - added namespace arg to wamv_base.urdf.xacro and removed tf_prefix

File: wamv_description/urdf/wamv_base.urdf.xacro (robot description, xacro)
@@ -1,4 +1,7 @@
 <?xml version="1.0"?>
 <robot xmlns:xacro="http://ros.org/wiki/xacro" name="wam-v">
+  <!-- Required arg for melodic and kinetic... -->
+  <xacro:arg name="namespace" default="wamv"/>
+  <xacro:property name="namespace" value="$(arg namespace)" scope="global" />
   <!-- Macro for creating the main collisions as simple shapes. -->
   <xacro:macro name="main_collisions" params="prefix reflect:=1">
