Commit message: Migrate to Noetic and Gazebo11 (#247)
Migrate to Noetic and Gazebo11.

File: wamv_description/urdf/battery.xacro (robot description, xacro)
@@ -2,5 +2,5 @@
 <robot xmlns:xacro="http://ros.org/wiki/xacro" name="wam-v-batteries">
   <xacro:macro name="battery" params="prefix position:='0 0 0' orientation:='0 0 0'">
-    <link name="${prefix}_battery_link">
+    <link name="${namespace}/${prefix}_battery_link">
       <visual name="${prefix}_battery_visual">
         <origin xyz="0 -1.03 -.45" rpy="0 0 0"/>
@@ -27,8 +27,8 @@
       </inertial>
     </link>
-    <joint name ="${prefix}_chasis_battery_joint" type="fixed">
+    <joint name ="${namespace}/${prefix}_chasis_battery_joint" type="fixed">
       <origin xyz="${position}" rpy="${orientation}"/>
-      <parent link="base_link"/>
-      <child link="${prefix}_battery_link"/>
+      <parent link="${namespace}/base_link"/>
+      <child link="${namespace}/${prefix}_battery_link"/>
     </joint>
   </xacro:macro>

File: wamv_description/urdf/cpu_cases.xacro (robot description, xacro)
@@ -2,5 +2,5 @@
 <robot xmlns:xacro="http://ros.org/wiki/xacro" name="wam-v-cpu_cases">
 <xacro:macro name="cpu_cases" params="position:='0 0 0' orientation:='0 0 0'">
-  <link name="cpu_cases_link">
+  <link name="${namespace}/cpu_cases_link">
     <visual name="cpu_cases_visual">
       <origin xyz="0.073 0 -1.53" rpy="0 0 0"/>
@@ -32,8 +32,8 @@
     </inertial>
   </link>
-  <joint name ="chasis_cpu_cases_joint" type="fixed">
+  <joint name ="${namespace}/chasis_cpu_cases_joint" type="fixed">
     <origin xyz="${position}" rpy="${orientation}"/>
-    <parent link="base_link"/>
-    <child link="cpu_cases_link"/>
+    <parent link="${namespace}/base_link"/>
+    <child link="${namespace}/cpu_cases_link"/>
   </joint>
 </xacro:macro>

File: wamv_description/urdf/thrusters/engine.xacro (robot description, xacro)
@@ -3,5 +3,5 @@
   <!-- Macro for inserting an engine with its propeller. -->
   <xacro:macro name="engine" params="prefix position:='0 0 0' orientation:='0 0 0'">
-    <link name="${prefix}_engine_link">
+    <link name="${namespace}/${prefix}_engine_link">
       <visual>
         <geometry>
@@ -26,5 +26,5 @@
       </inertial>
     </link>
-    <link name="${prefix}_propeller_link">
+    <link name="${namespace}/${prefix}_propeller_link">
       <visual>
         <geometry>
@@ -43,15 +43,15 @@
       </inertial>
     </link>
-    <joint name="${prefix}_chasis_engine_joint" type="revolute">
+    <joint name="${namespace}/${prefix}_chasis_engine_joint" type="revolute">
       <axis xyz="0 0 1"/>
       <limit lower="${-pi}" upper="${pi}" effort="10" velocity="10"/>
       <origin xyz="${position}" rpy="${orientation}"/>
-      <parent link="base_link"/>
-      <child link="${prefix}_engine_link"/>
+      <parent link="${namespace}/base_link"/>
+      <child link="${namespace}/${prefix}_engine_link"/>
     </joint>
-    <joint name="${prefix}_engine_propeller_joint" type="continuous">
+    <joint name="${namespace}/${prefix}_engine_propeller_joint" type="continuous">
       <axis rpy="0 0 0" xyz="1 0 0"/>
-      <parent link="${prefix}_engine_link"/>
-      <child link="${prefix}_propeller_link"/>
+      <parent link="${namespace}/${prefix}_engine_link"/>
+      <child link="${namespace}/${prefix}_propeller_link"/>
       <origin rpy="0 0 0" xyz="-0.278156 0 -0.509371"/>
       <limit effort="100" velocity="100" />

File: wamv_description/urdf/wamv_base.urdf.xacro (robot description, xacro)
@@ -1,4 +1,7 @@
 <?xml version="1.0"?>
 <robot xmlns:xacro="http://ros.org/wiki/xacro" name="wam-v">
+  <!-- Required arg for melodic and kinetic... -->
+  <xacro:arg name="namespace" default="wamv"/>
+  <xacro:property name="namespace" value="$(arg namespace)" scope="global" />
   <!-- Macro for creating the main collisions as simple shapes. -->
   <xacro:macro name="main_collisions" params="prefix reflect:=1">
@@ -81,12 +84,12 @@
     </collision>
   </xacro:macro>
-  <link name="base_link">
+  <link name="${namespace}/base_link">
   </link>
-  <joint name="dummy_joint" type = "fixed">
-    <parent link="base_link"/>
-    <child link="dummy_link"/>
+  <joint name="${namespace}/dummy_joint" type = "fixed">
+    <parent link="${namespace}/base_link"/>
+    <child link="${namespace}/dummy_link"/>
   </joint>
   <!-- Basic model of the 16' WAM-V USV -->
-  <link name="dummy_link">
+  <link name="${namespace}/dummy_link">
     <visual>
       <geometry>

File: wamv_gazebo/urdf/sensors/wamv_3d_lidar.xacro (robot description, xacro)
@@ -36,5 +36,5 @@
     <xacro:property name="post_arm_to_lidar_z" value="0.05"/>
     <!-- 3d lidar sensor -->
-    <link name="${name}_link">
+    <link name="${namespace}/${name}_link">
       <visual name="${name}_visual">
         <origin xyz="0 0 -0.035" rpy="0 0 0"/>
@@ -65,5 +65,5 @@
     <xacro:property name="post_radius" value="0.0076"/>
     <!-- Sensor post -->
-    <link name="${name}_post_link">
+    <link name="${namespace}/${name}_post_link">
       <visual>
         <geometry>
@@ -91,5 +91,5 @@
     </link>
     <!-- Sensor post arm -->
-    <link name="${name}_post_arm_link">
+    <link name="${namespace}/${name}_post_arm_link">
       <visual name="${name}_post_arm_visual">
         <origin xyz="-0.038 0 -0.003" rpy="${radians(-60)} 0 ${-pi/2}"/>
@@ -119,20 +119,20 @@
     <xacro:property name="post_z" value="${platform_z+post_length/2}"/>
     <xacro:property name="post_to_lidar_x" value="${post_to_post_arm_x+post_arm_to_lidar_x}"/>
-    <joint name="base_to_${name}_post_joint" type="fixed">
+    <joint name="${namespace}/base_to_${name}_post_joint" type="fixed">
       <origin xyz="${x-(post_to_lidar_x)*cos(post_Y)} ${y-(post_to_lidar_x)*sin(post_Y)} ${post_z}" rpy="0 0 ${post_Y}" />
-      <parent link="base_link" />
-      <child link="${name}_post_link" />
+      <parent link="${namespace}/base_link" />
+      <child link="${namespace}/${name}_post_link" />
     </joint>
     <!-- Sensor post to sensor post arm joint -->
-    <joint name="${name}_post_to_${name}_post_arm_joint" type="fixed">
+    <joint name="${namespace}/${name}_post_to_${name}_post_arm_joint" type="fixed">
       <origin xyz="${post_to_post_arm_x} 0 ${z-post_z-post_arm_to_lidar_z}" rpy="0 0 0" />
-      <parent link="${name}_post_link" />
-      <child link="${name}_post_arm_link" />
+      <parent link="${namespace}/${name}_post_link" />
+      <child link="${namespace}/${name}_post_arm_link" />
     </joint>
     <!-- Sensor post arm to lidar joint -->
-    <joint name="${name}_post_arm_to_${name}_joint" type="fixed">
+    <joint name="${namespace}/${name}_post_arm_to_${name}_joint" type="fixed">
       <origin xyz="${post_arm_to_lidar_x} 0 ${post_arm_to_lidar_z}" rpy="${R} ${P} ${Y-post_Y}" />
-      <parent link="${name}_post_arm_link" />
-      <child link="${name}_link" />
+      <parent link="${namespace}/${name}_post_arm_link" />
+      <child link="${namespace}/${name}_link" />
     </joint>
     <gazebo reference="${name}_link">
@@ -172,5 +172,5 @@
     </gazebo>
     <!-- Set color of post -->
-    <gazebo reference="${name}_post_link">
+    <gazebo reference="${namespace}/${name}_post_link">
       <material>Gazebo/Black</material>
     </gazebo>

File: wamv_gazebo/urdf/sensors/wamv_camera.xacro (robot description, xacro)
@@ -8,5 +8,5 @@
     <xacro:property name="post_arm_to_camera_z" value="0.027"/>
     <!-- Monocular Camera -->
-    <link name="${name}_link">
+    <link name="${namespace}/${name}_link">
       <visual name="${name}_visual">
         <origin xyz="-0.033 0 0" rpy="0 0 ${pi/2}"/>
@@ -41,5 +41,5 @@
     <!-- Define a link for the optical frame.  This will match the sensor frame and
          be oriented in the camera convention. -->
-    <link name="${name}_link_optical">
+    <link name="${namespace}/${name}_link_optical">
     </link>
     <!-- Define post length and mass based on desired z position of sensor -->
@@ -49,5 +49,5 @@
     <xacro:property name="post_radius" value="0.0076"/>
     <!-- Sensor post -->
-    <link name="${name}_post_link">
+    <link name="${namespace}/${name}_post_link">
       <visual>
         <geometry>
@@ -75,5 +75,5 @@
     </link>
     <!-- Sensor post arm -->
-    <link name="${name}_post_arm_link">
+    <link name="${namespace}/${name}_post_arm_link">
       <visual name="${name}_post_arm_visual">
         <origin xyz="-0.038 0 -0.003" rpy="${radians(-60)} 0 ${-pi/2}"/>
@@ -103,30 +103,30 @@
     <xacro:property name="post_z" value="${platform_z+post_length/2}"/>
     <xacro:property name="post_to_camera_x" value="${post_to_post_arm_x+post_arm_to_camera_x}"/>
-    <joint name="base_to_${name}_post_joint" type="fixed">
+    <joint name="${namespace}/base_to_${name}_post_joint" type="fixed">
       <origin xyz="${x-(post_to_camera_x)*cos(post_Y)} ${y-(post_to_camera_x)*sin(post_Y)} ${post_z}" rpy="0 0 ${post_Y}" />
-      <parent link="base_link" />
-      <child link="${name}_post_link" />
+      <parent link="${namespace}/base_link" />
+      <child link="${namespace}/${name}_post_link" />
     </joint>
     <!-- Sensor post to sensor post arm joint -->
-    <joint name="${name}_post_to_${name}_post_arm_joint" type="fixed">
+    <joint name="${namespace}/${name}_post_to_${name}_post_arm_joint" type="fixed">
       <origin xyz="${post_to_post_arm_x} 0 ${z-post_z-post_arm_to_camera_z}" rpy="0 0 0" />
-      <parent link="${name}_post_link" />
-      <child link="${name}_post_arm_link" />
+      <parent link="${namespace}/${name}_post_link" />
+      <child link="${namespace}/${name}_post_arm_link" />
     </joint>
     <!-- Sensor post arm to camera joint -->
-    <joint name="${name}_post_arm_to_${name}_joint" type="fixed">
+    <joint name="${namespace}/${name}_post_arm_to_${name}_joint" type="fixed">
       <origin xyz="${post_arm_to_camera_x} 0 ${post_arm_to_camera_z}" rpy="${R} ${P} ${Y-post_Y}" />
-      <parent link="${name}_post_arm_link" />
-      <child link="${name}_link" />
+      <parent link="${namespace}/${name}_post_arm_link" />
+      <child link="${namespace}/${name}_link" />
     </joint>
     <!-- Camera to optical frame joint.  This is oriented to convert between ENU
          and camera conventions -->
-    <joint name="${name}_to_${name}_link_optical_joint" type="fixed">
+    <joint name="${namespace}/${name}_to_${name}_link_optical_joint" type="fixed">
       <origin xyz="0 0 0" rpy="${-pi/2} 0 ${-pi/2}" />
-      <parent link="${name}_link" />
-      <child link="${name}_link_optical" />
+      <parent link="${namespace}/${name}_link" />
+      <child link="${namespace}/${name}_link_optical" />
     </joint>
     <!-- Gazebo camera setup -->
-    <gazebo reference="${name}_link">
+    <gazebo reference="${namespace}/${name}_link">
       <sensor type="camera" name="${name}_sensor">
         <update_rate>30.0</update_rate>

File: wamv_gazebo/urdf/sensors/wamv_gps.xacro (robot description, xacro)
@@ -2,5 +2,5 @@
 <robot xmlns:xacro="http://ros.org/wiki/xacro">
   <xacro:macro name="wamv_gps" params="name:=gps x:=0.3 y:=0 z:=1.3 R:=0 P:=0 Y:=0 lat:=21.30996 lon:=-157.8901 elev:=0.0 update_rate:=15">
-    <link name="${name}_link">
+    <link name="${namespace}/${name}_link">
       <visual name="${name}_visual">
         <geometry>
@@ -25,10 +25,10 @@
       </inertial>
     </link>
-    <joint name="${name}_joint" type="revolute">
+    <joint name="${namespace}/${name}_joint" type="revolute">
       <axis xyz="0 0 1"/>
       <limit effort="1000.0" lower="0.0" upper="0" velocity="0"/>
       <origin xyz="${x} ${y} ${z}" rpy="${R} ${P} ${Y}" />
-      <parent link="base_link" />
-      <child link="${name}_link" />
+      <parent link="${namespace}/base_link" />
+      <child link="${namespace}/${name}_link" />
     </joint>
     <gazebo>
@@ -36,5 +36,5 @@
         <updateRate>${update_rate}</updateRate>
         <alwaysOn>true</alwaysOn>
-        <bodyName>${name}_link</bodyName>
+        <bodyName>${namespace}/${name}_link</bodyName>
         <!-- Manually prepend namespace to tf frame. -->
         <frameId>${namespace}/${name}_link</frameId>

File: wamv_gazebo/urdf/sensors/wamv_imu.xacro (robot description, xacro)
@@ -2,5 +2,5 @@
 <robot xmlns:xacro="http://ros.org/wiki/xacro">
   <xacro:macro name="wamv_imu" params="name:=imu x:=0.3 y:=0.5 z:=1.3 R:=0 P:=0 Y:=0 update_rate:=15">
-    <link name="${name}_link">
+    <link name="${namespace}/${name}_link">
       <visual name="${name}_visual">>
         <geometry>
@@ -16,15 +16,15 @@
       </inertial>
     </link>
-    <joint name="${name}_joint" type="revolute">
+    <joint name="${namespace}/${name}_joint" type="revolute">
       <axis xyz="0 0 1"/>
       <limit effort="1000.0" lower="0.0" upper="0" velocity="0"/>
       <origin xyz="${x} ${y} ${z}" rpy="${R} ${P} ${Y}"/>
-      <parent link="base_link"/>
-      <child link="${name}_link"/>
+      <parent link="${namespace}/base_link"/>
+      <child link="${namespace}/${name}_link"/>
     </joint>
     <gazebo>
       <plugin name="imu_plugin_${name}" filename="libhector_gazebo_ros_imu.so">
         <updateRate>${update_rate}</updateRate>
-        <bodyName>${name}_link</bodyName>
+        <bodyName>${namespace}/${name}_link</bodyName>
         <topicName>${namespace}/${sensor_namespace}imu/imu/data</topicName>
         <serviceName>${namespace}/${sensor_namespace}imu_service</serviceName>

File: wamv_gazebo/urdf/sensors/wamv_pinger.xacro (robot description, xacro)
@@ -2,5 +2,5 @@
 <robot xmlns:xacro="http://ros.org/wiki/xacro">
   <xacro:macro name="wamv_pinger" params="name:='pinger' frameId:='wamv/pinger' position:='0 0 0' orientation:='0 0 0'">
-    <link name="${name}">
+    <link name="${namespace}/${name}">
       <visual>
         <origin xyz="0 0 0" rpy="0 0 0" />
@@ -16,8 +16,8 @@
       </collision>
     </link>
-    <joint name="${name}_pinger_joint" type="fixed">
+    <joint name="${namespace}/${name}_pinger_joint" type="fixed">
       <origin xyz="${position}" rpy="${orientation}"/>
-      <parent link="base_link"/>
-      <child link="${name}"/>
+      <parent link="${namespace}/base_link"/>
+      <child link="${namespace}/${name}"/>
     </joint>
     <gazebo>

Commit message: Migrated wamv_description to ROS 2.

File: wamv_description/urdf/battery.xacro (robot description, xacro)
@@ -6,5 +6,5 @@
         <origin xyz="0 -1.03 -.45" rpy="0 0 0"/>
         <geometry>
-          <mesh filename="package://vrx_gazebo/models/battery/mesh/battery.dae"/>
+          <mesh filename="file://$(find vrx_gazebo)/models/battery/mesh/battery.dae"/>
         </geometry>
       </visual>

File: wamv_description/urdf/cpu_cases.xacro (robot description, xacro)
@@ -6,5 +6,5 @@
       <origin xyz="0.073 0 -1.53" rpy="0 0 0"/>
       <geometry>
-        <mesh filename="package://vrx_gazebo/models/cpu_cases/mesh/cpu_cases.dae"/>
+        <mesh filename="file://$(find vrx_gazebo)/models/cpu_cases/mesh/cpu_cases.dae"/>
       </geometry>
     </visual>

File: wamv_description/urdf/thrusters/engine.xacro (robot description, xacro)
@@ -6,5 +6,5 @@
       <visual>
         <geometry>
-          <mesh filename="package://wamv_description/models/engine/mesh/engine.dae"/>
+          <mesh filename="file://$(find wamv_description)/models/engine/mesh/engine.dae"/>
         </geometry>
       </visual>
@@ -29,5 +29,5 @@
       <visual>
         <geometry>
-          <mesh filename="package://wamv_description/models/propeller/mesh/propeller.dae"/>
+          <mesh filename="file://$(find wamv_description)/models/propeller/mesh/propeller.dae"/>
         </geometry>
       </visual>

File: wamv_description/urdf/wamv_base.urdf.xacro (robot description, xacro)
@@ -94,5 +94,5 @@
     <visual>
       <geometry>
-        <mesh filename="package://wamv_description/models/WAM-V-Base/mesh/WAM-V-Base.dae"/>
+        <mesh filename="file://$(find wamv_description)/models/WAM-V-Base/mesh/WAM-V-Base.dae"/>
       </geometry>
     </visual>
