Commit message: Remove references to the Gazebo 8 wind plugin.

File: robotx_gazebo/worlds/sandisland.xacro (robot description, xacro)
@@ -2,5 +2,5 @@
 <!-- Macro to insert the sandisland into the world -->
 <world xmlns:xacro="http://ros.org/wiki/xacro">
-  <xacro:macro name="sandisland" params="wind_velocity:='10 0 0'">
+  <xacro:macro name="sandisland">
     <scene>
       <sky>
@@ -10,7 +10,4 @@
       </sky>
     </scene>
-    <wind>
-      <linear_velocity>${wind_velocity}</linear_velocity> <!-- Wind linear velocity -->
-    </wind>
     <!-- A global light source -->
     <include>

File: wamv_description/urdf/wamv_base.urdf.xacro (robot description, xacro)
@@ -83,5 +83,4 @@
   <!-- Basic model of the 16' WAM-V USV -->
   <link name="base_link">
-    <wind>true</wind>
     <visual>
       <geometry>
