Commit message: Fix multibeam laser xacro

File: wamv_gazebo/urdf/sensors/wamv_multibeam_laser.xacro (robot description, xacro)
@@ -1,5 +1,5 @@
 <?xml version="1.0" encoding="UTF-8"?>
 <robot xmlns:xacro="http://ros.org/wiki/xacro">
-  <xacro:macro name="wamv_multibeam_laser" params="name x:=0.5 y:=0 z:=1.35 R:=0 P:=0 Y:=0">
+  <xacro:macro name="wamv_multibeam_laser" params="name x:=0.5 y:=0 z:=2 R:=0 P:=0 Y:=0">
     <link name="${name}_link">
       <visual name="${name}_visual">>
@@ -17,7 +17,6 @@
       <child link="${name}_link" />
     </joint>
-    <gazebo reference="scan">
+    <gazebo reference="${name}_link">
       <sensor type="gpu_ray" name="multibeam_sensor_${name}">
-        <visualize>true</visualize>
         <update_rate>10</update_rate>
         <ray>
@@ -41,5 +40,5 @@
         <plugin name="multibeam_simulator" filename="libgazebo_ros_gpu_laser.so">
           <topicName>${name}/scan</topicName>
-          <frameName>${name}</frameName>
+          <frameName>${name}_link</frameName>
         </plugin>
       </sensor>
