Commit message: Add 3D Lidar mesh and put it on WAM-V

File: wamv_gazebo/urdf/sensors/wamv_3d_lidar.xacro (robot description, xacro)
@@ -13,5 +13,5 @@
     noise_stddev: Standard deviation of gaussian noise applied to output pointcloud
   -->
-  <xacro:macro name="wamv_3d_lidar" params="name x:=0.7 y:=0 z:=1.45 R:=0 P:=0 Y:=0
+  <xacro:macro name="wamv_3d_lidar" params="name x:=0.7 y:=0 z:=1.33 R:=0 P:=0 Y:=0
                                             update_rate:=10 vertical_lasers:=16 samples:=1800 resolution:=0.1
                                             min_angle:=${-pi} max_angle:=${pi}
@@ -19,12 +19,27 @@
                                             max_range:=100 noise_stddev:=0.01">
     <link name="${name}_link">
-      <visual name="${name}_visual">>
+      <visual name="${name}_visual">
+        <origin xyz="0 0 -0.035" rpy="0 0 0"/>
         <geometry>
-          <cylinder radius="0.025" length="0.1" />
+          <mesh filename="package://vrx_gazebo/models/3d_lidar/mesh/3d_lidar.dae"/>
         </geometry>
-        <material name="${name}_visual_material">
-          <color rgba="0.5 1.0 0.5 1.0" />
-        </material>
       </visual>
+      <collision name="${name}_collision">
+        <origin xyz="0 0 0" rpy="0 0 0"/>
+        <geometry>
+          <cylinder radius="0.055" length="0.075"/>
+        </geometry>
+      </collision>
+      <inertial>
+        <origin xyz="0 0 0" rpy="0 0 0"/>
+        <mass value="1"/>
+        <inertia
+          ixx="0.00109375"
+          iyy="0.00109375"
+          izz="0.00125"
+          ixy="0"
+          ixz="0"
+          iyz="0"/>
+      </inertial>
     </link>
     <joint name="${name}_joint" type="fixed">

File: wamv_gazebo/urdf/wamv_gazebo.urdf.xacro (robot description, xacro)
@@ -68,5 +68,5 @@
   <!-- Add 3D LIDAR -->
   <xacro:if value="$(arg lidar_enabled)">
-    <xacro:wamv_3d_lidar name="lidar_wamv" y="-0.3" />
+    <xacro:wamv_3d_lidar name="lidar_wamv" y="0" />
   </xacro:if>
   <!-- Add P3D ground truth -->

Commit message: Add sensor post to 3d lidar on WAM-V, including height parameter

File: wamv_gazebo/urdf/sensors/wamv_3d_lidar.xacro (robot description, xacro)
@@ -13,9 +13,10 @@
     noise_stddev: Standard deviation of gaussian noise applied to output pointcloud
   -->
-  <xacro:macro name="wamv_3d_lidar" params="name x:=0.7 y:=0 z:=1.33 R:=0 P:=0 Y:=0
+  <xacro:macro name="wamv_3d_lidar" params="name x:=0.7 y:=0 z:=1.545 R:=0 P:=0 Y:=${-pi/2} height:=0
                                             update_rate:=10 vertical_lasers:=16 samples:=1800 resolution:=0.1
                                             min_angle:=${-pi} max_angle:=${pi}
                                             min_vertical_angle:=${-pi/12} max_vertical_angle:=${pi/12}
                                             max_range:=100 noise_stddev:=0.01">
+    <!-- 3d lidar sensor -->
     <link name="${name}_link">
       <visual name="${name}_visual">
@@ -26,5 +27,4 @@
       </visual>
       <collision name="${name}_collision">
-        <origin xyz="0 0 0" rpy="0 0 0"/>
         <geometry>
           <cylinder radius="0.055" length="0.075"/>
@@ -32,5 +32,4 @@
       </collision>
       <inertial>
-        <origin xyz="0 0 0" rpy="0 0 0"/>
         <mass value="1"/>
         <inertia
@@ -43,7 +42,70 @@
       </inertial>
     </link>
-    <joint name="${name}_joint" type="fixed">
+    <!-- Sensor post -->
+    <link name="${name}_post_link">
+      <visual name="${name}_post_visual">
+        <origin xyz="0 0 -0.2515" rpy="${pi/2} 0 0"/>
+        <geometry>
+          <mesh filename="package://vrx_gazebo/models/sensor_post/mesh/sensor_post.dae"/>
+        </geometry>
+      </visual>
+      <collision name="${name}_post_collision">
+        <geometry>
+          <cylinder radius="0.0076" length="0.503"/>
+        </geometry>
+      </collision>
+      <inertial>
+        <mass value="0.5"/>
+        <inertia
+          ixx="0.010549261666667"
+          iyy="0.010549261666667"
+          izz="0.000014440000000"
+          ixy="0"
+          ixz="0"
+          iyz="0"/>
+      </inertial>
+    </link>
+    <!-- Sensor post arm -->
+    <link name="${name}_post_arm_link">
+      <visual name="${name}_post_arm_visual">
+        <origin xyz="0 -0.016 -0.035" rpy="0 0 0"/>
+        <geometry>
+          <mesh filename="package://vrx_gazebo/models/sensor_post/mesh/sensor_post_arm.dae"/>
+        </geometry>
+      </visual>
+      <collision name="${name}_post_arm_collision">
+        <origin xyz="0 0 0" rpy="${-pi/20} 0 0"/>
+        <geometry>
+          <cylinder radius="0.008" length="0.065"/>
+        </geometry>
+      </collision>
+      <inertial>
+        <origin xyz="0 0 0" rpy="${-pi/20} 0 0"/>
+        <mass value="0.1"/>
+        <inertia
+          ixx="0.00003680833"
+          iyy="0.00003680833"
+          izz="0.00000320000"
+          ixy="0"
+          ixz="0"
+          iyz="0"/>
+      </inertial>
+    </link>
+    <!-- Base to sensor post joint -->
+    <joint name="base_to_${name}_post_joint" type="fixed">
       <origin xyz="${x} ${y} ${z}" rpy="${R} ${P} ${Y}" />
       <parent link="base_link" />
+      <child link="${name}_post_link" />
+    </joint>
+    <!-- Sensor post to sensor post arm joint -->
+    <joint name="${name}_post_to_${name}_post_arm_joint" type="fixed">
+      <origin xyz="0 0.03 ${height}" rpy="${-pi/3} 0 0" />
+      <parent link="${name}_post_link" />
+      <child link="${name}_post_arm_link" />
+    </joint>
+    <!-- Sensor post arm to lidar joint -->
+    <joint name="${name}_post_arm_to_${name}_lidar_joint" type="fixed">
+      <origin xyz="0 -0.025 0.055" rpy="${pi/3} 0 0" />
+      <parent link="${name}_post_arm_link" />
       <child link="${name}_link" />
     </joint>

File: wamv_gazebo/urdf/wamv_gazebo.urdf.xacro (robot description, xacro)
@@ -68,5 +68,5 @@
   <!-- Add 3D LIDAR -->
   <xacro:if value="$(arg lidar_enabled)">
-    <xacro:wamv_3d_lidar name="lidar_wamv"/>
+    <xacro:wamv_3d_lidar name="lidar_wamv" height="0.25"/>
   </xacro:if>
   <!-- Add P3D ground truth -->
@@ -86,5 +86,5 @@
     <xacro:wamv_imu name="imu_wamv" y="-0.2" />
     <!-- Add 3D LIDAR -->
-    <xacro:wamv_3d_lidar name="lidar_wamv"/>
+    <xacro:wamv_3d_lidar name="lidar_wamv" height="0.25"/>
   </xacro:if>
 </robot>

Commit message: Add sensor_post_arm.dae

File: wamv_gazebo/urdf/sensors/wamv_3d_lidar.xacro (robot description, xacro)
@@ -13,5 +13,5 @@
     noise_stddev: Standard deviation of gaussian noise applied to output pointcloud
   -->
-  <xacro:macro name="wamv_3d_lidar" params="name x:=0.7 y:=0 z:=1.545 R:=0 P:=0 Y:=${-pi/2} height:=0
+  <xacro:macro name="wamv_3d_lidar" params="name x:=0.7 y:=0 z:=1.545 R:=0 P:=0 Y:=${-pi/2} height:=0.25
                                             update_rate:=10 vertical_lasers:=16 samples:=1800 resolution:=0.1
                                             min_angle:=${-pi} max_angle:=${pi}

Commit message: Fix issue with lidar seeing itself and set default lidar angle downwards towards water

File: wamv_gazebo/urdf/sensors/wamv_3d_lidar.xacro (robot description, xacro)
@@ -106,5 +106,6 @@
     <!-- Sensor post arm to lidar joint -->
     <joint name="${name}_post_arm_to_${name}_lidar_joint" type="fixed">
-      <origin xyz="0 -0.025 0.055" rpy="${pi/3} 0 0" />
+      <!-- rpy="${pi/3} 0 0" for flat lidar -->
+      <origin xyz="0 -0.025 0.055" rpy="${pi/3-radians(15)} 0 0" />
       <parent link="${name}_post_arm_link" />
       <child link="${name}_link" />
@@ -129,5 +130,5 @@
           </scan>
           <range>
-            <min>0.05</min>
+            <min>0.1</min>
             <max>${max_range}</max>
           </range>

Commit message: Add adjustment link and joint to make the lidar frame better match base frame

File: wamv_gazebo/urdf/sensors/wamv_3d_lidar.xacro (robot description, xacro)
@@ -13,5 +13,5 @@
     noise_stddev: Standard deviation of gaussian noise applied to output pointcloud
   -->
-  <xacro:macro name="wamv_3d_lidar" params="name x:=0.7 y:=0 z:=1.545 R:=0 P:=0 Y:=${-pi/2} height:=0.25
+  <xacro:macro name="wamv_3d_lidar" params="name x:=0.7 y:=0 z:=1.545 R:=0 P:=0 Y:=0 height:=0.25
                                             update_rate:=10 vertical_lasers:=16 samples:=1800 resolution:=0.1
                                             min_angle:=${-pi} max_angle:=${pi}
@@ -94,5 +94,5 @@
     <!-- Base to sensor post joint -->
     <joint name="base_to_${name}_post_joint" type="fixed">
-      <origin xyz="${x} ${y} ${z}" rpy="${R} ${P} ${Y}" />
+      <origin xyz="${x} ${y} ${z}" rpy="${R} ${P} ${Y-pi/2}" />
       <parent link="base_link" />
       <child link="${name}_post_link" />
@@ -100,13 +100,20 @@
     <!-- Sensor post to sensor post arm joint -->
     <joint name="${name}_post_to_${name}_post_arm_joint" type="fixed">
-      <origin xyz="0 0.03 ${height}" rpy="${-pi/3} 0 0" />
+      <origin xyz="0 0.035 ${height}" rpy="${-radians(70)} 0 0" />
       <parent link="${name}_post_link" />
       <child link="${name}_post_arm_link" />
+    </joint>
+    <!-- Adjustment joint -->
+    <link name="adjustment_link"/>
+    <joint name="adjustment_joint" type="fixed">
+      <origin xyz="0 0 0" rpy="${radians(70)} 0 0" />
+      <parent link="${name}_post_arm_link" />
+      <child link="adjustment_link" />
     </joint>
     <!-- Sensor post arm to lidar joint -->
     <joint name="${name}_post_arm_to_${name}_lidar_joint" type="fixed">
       <!-- rpy="${pi/3} 0 0" for flat lidar -->
-      <origin xyz="0 -0.025 0.055" rpy="${pi/3-radians(15)} 0 0" />
-      <parent link="${name}_post_arm_link" />
+      <origin xyz="0 0.035 0.045" rpy="${radians(-15)} 0 0" />
+      <parent link="adjustment_link" />
       <child link="${name}_link" />
     </joint>

Commit message: Add second adjustment link to perfectly match sensor and base frames

File: wamv_gazebo/urdf/sensors/wamv_3d_lidar.xacro (robot description, xacro)
@@ -13,5 +13,5 @@
     noise_stddev: Standard deviation of gaussian noise applied to output pointcloud
   -->
-  <xacro:macro name="wamv_3d_lidar" params="name x:=0.7 y:=0 z:=1.545 R:=0 P:=0 Y:=0 height:=0.25
+  <xacro:macro name="wamv_3d_lidar" params="name x:=0.7 y:=0 z:=1.545 R:=0 P:=0 Y:=0 height:=0.24
                                             update_rate:=10 vertical_lasers:=16 samples:=1800 resolution:=0.1
                                             min_angle:=${-pi} max_angle:=${pi}
@@ -105,15 +105,22 @@
     </joint>
     <!-- Adjustment joint -->
-    <link name="adjustment_link"/>
-    <joint name="adjustment_joint" type="fixed">
+    <link name="adjustment_1_link"/>
+    <joint name="adjustment_1_joint" type="fixed">
       <origin xyz="0 0 0" rpy="${radians(70)} 0 0" />
       <parent link="${name}_post_arm_link" />
-      <child link="adjustment_link" />
+      <child link="adjustment_1_link" />
+    </joint>
+    <!-- Adjustment 2 joint -->
+    <link name="adjustment_2_link"/>
+    <joint name="adjustment_2_joint" type="fixed">
+      <origin xyz="0 0 0" rpy="0 0 ${pi/2}" />
+      <parent link="adjustment_link" />
+      <child link="adjustment_2_link" />
     </joint>
     <!-- Sensor post arm to lidar joint -->
     <joint name="${name}_post_arm_to_${name}_lidar_joint" type="fixed">
       <!-- rpy="${pi/3} 0 0" for flat lidar -->
-      <origin xyz="0 0.035 0.045" rpy="${radians(-15)} 0 0" />
-      <parent link="adjustment_link" />
+      <origin xyz="0.04 0 0.045" rpy="0 ${radians(15)} 0" />
+      <parent link="adjustment_2_link" />
       <child link="${name}_link" />
     </joint>

File: wamv_gazebo/urdf/wamv_gazebo.urdf.xacro (robot description, xacro)
@@ -72,5 +72,5 @@
   <!-- Add 3D LIDAR -->
   <xacro:if value="$(arg lidar_enabled)">
-    <xacro:wamv_3d_lidar name="lidar_wamv" height="0.25"/>
+    <xacro:wamv_3d_lidar name="lidar_wamv" height="0.24"/>
   </xacro:if>
   <!-- Add P3D ground truth -->
@@ -93,5 +93,5 @@
     <xacro:wamv_imu name="imu_wamv" y="-0.2" />
     <!-- Add 3D LIDAR -->
-    <xacro:wamv_3d_lidar name="lidar_wamv" height="0.25"/>
+    <xacro:wamv_3d_lidar name="lidar_wamv" height="0.24"/>
   </xacro:if>
 </robot>

Commit message: Temporary test setting xyz of lidar, next need to change frames to simplify all of this

File: wamv_gazebo/urdf/sensors/wamv_3d_lidar.xacro (robot description, xacro)
@@ -13,5 +13,5 @@
     noise_stddev: Standard deviation of gaussian noise applied to output pointcloud
   -->
-  <xacro:macro name="wamv_3d_lidar" params="name x:=0.7 y:=0 z:=1.545 R:=0 P:=0 Y:=0 height:=0.24
+  <xacro:macro name="wamv_3d_lidar" params="name x:=0.7 y:=0 z:=1.8 R:=0 P:=0 Y:=0 post_Y:=0
                                             update_rate:=10 vertical_lasers:=16 samples:=1800 resolution:=0.1
                                             min_angle:=${-pi} max_angle:=${pi}
@@ -94,33 +94,39 @@
     <!-- Base to sensor post joint -->
     <joint name="base_to_${name}_post_joint" type="fixed">
-      <origin xyz="${x} ${y} ${z}" rpy="${R} ${P} ${Y-pi/2}" />
+      <origin xyz="${x-0.04-0.035} ${y} 1.545" rpy="0 0 ${post_Y-pi/2}" />
       <parent link="base_link" />
       <child link="${name}_post_link" />
     </joint>
+    <!-- Adjustment 1 joint -->
+    <link name="adjustment_1_link"/>
+    <joint name="adjustment_1_joint" type="fixed">
+      <origin xyz="0 0 0" rpy="0 0 ${pi/2}" />
+      <parent link="${name}_post_link" />
+      <child link="adjustment_1_link" />
+    </joint>
     <!-- Sensor post to sensor post arm joint -->
     <joint name="${name}_post_to_${name}_post_arm_joint" type="fixed">
-      <origin xyz="0 0.035 ${height}" rpy="${-radians(70)} 0 0" />
-      <parent link="${name}_post_link" />
+      <origin xyz="0.035 0 ${z-1.545-0.045}" rpy="${-radians(70)} 0 ${-pi/2}" />
+      <parent link="adjustment_1_link" />
       <child link="${name}_post_arm_link" />
-    </joint>
-    <!-- Adjustment joint -->
-    <link name="adjustment_1_link"/>
-    <joint name="adjustment_1_joint" type="fixed">
-      <origin xyz="0 0 0" rpy="${radians(70)} 0 0" />
-      <parent link="${name}_post_arm_link" />
-      <child link="adjustment_1_link" />
     </joint>
     <!-- Adjustment 2 joint -->
     <link name="adjustment_2_link"/>
     <joint name="adjustment_2_joint" type="fixed">
+      <origin xyz="0 0 0" rpy="${radians(70)} 0 0" />
+      <parent link="${name}_post_arm_link" />
+      <child link="adjustment_2_link" />
+    </joint>
+    <!-- Adjustment 3 joint -->
+    <link name="adjustment_3_link"/>
+    <joint name="adjustment_3_joint" type="fixed">
       <origin xyz="0 0 0" rpy="0 0 ${pi/2}" />
-      <parent link="adjustment_link" />
-      <child link="adjustment_2_link" />
+      <parent link="adjustment_2_link" />
+      <child link="adjustment_3_link" />
     </joint>
     <!-- Sensor post arm to lidar joint -->
     <joint name="${name}_post_arm_to_${name}_lidar_joint" type="fixed">
-      <!-- rpy="${pi/3} 0 0" for flat lidar -->
-      <origin xyz="0.04 0 0.045" rpy="0 ${radians(15)} 0" />
-      <parent link="adjustment_2_link" />
+      <origin xyz="0.04 0 0.045" rpy="${R} ${P} ${Y}" />
+      <parent link="adjustment_3_link" />
       <child link="${name}_link" />
     </joint>

File: wamv_gazebo/urdf/wamv_gazebo.urdf.xacro (robot description, xacro)
@@ -72,5 +72,5 @@
   <!-- Add 3D LIDAR -->
   <xacro:if value="$(arg lidar_enabled)">
-    <xacro:wamv_3d_lidar name="lidar_wamv" height="0.24"/>
+    <xacro:wamv_3d_lidar name="lidar_wamv"/>
   </xacro:if>
   <!-- Add P3D ground truth -->
@@ -93,5 +93,6 @@
     <xacro:wamv_imu name="imu_wamv" y="-0.2" />
     <!-- Add 3D LIDAR -->
-    <xacro:wamv_3d_lidar name="lidar_wamv" height="0.24"/>
+    <xacro:wamv_3d_lidar name="lidar_wamv" x="0.7" y="0" z="1.4" R="0" P="${radians(15)}" Y="0" post_Y="0"/>
+    <xacro:wamv_camera name="test_camera" x="0.7" y="0" z="1.4" R="0" P="${radians(15)}" Y="0" />
   </xacro:if>
 </robot>

Commit message: Redo sensor post to lidar joints to cleaner (x,y,z,r,p,y) coordinates

File: wamv_gazebo/urdf/sensors/wamv_3d_lidar.xacro (robot description, xacro)
@@ -92,7 +92,13 @@
       </inertial>
     </link>
+    <!-- Base to lidar joint -->
+    <joint name="base_to_${name}_joint" type="fixed">
+      <origin xyz="${x} ${y} ${z}" rpy="${R} ${P} ${Y}" />
+      <parent link="base_link" />
+      <child link="${name}_link" />
+    </joint>
     <!-- Base to sensor post joint -->
     <joint name="base_to_${name}_post_joint" type="fixed">
-      <origin xyz="${x-0.04-0.035} ${y} 1.545" rpy="0 0 ${post_Y-pi/2}" />
+      <origin xyz="${x-0.07} ${y} 1.545" rpy="0 0 ${-pi/2}" />
       <parent link="base_link" />
       <child link="${name}_post_link" />
@@ -107,27 +113,7 @@
     <!-- Sensor post to sensor post arm joint -->
     <joint name="${name}_post_to_${name}_post_arm_joint" type="fixed">
-      <origin xyz="0.035 0 ${z-1.545-0.045}" rpy="${-radians(70)} 0 ${-pi/2}" />
-      <parent link="adjustment_1_link" />
-      <child link="${name}_post_arm_link" />
-    </joint>
-    <!-- Adjustment 2 joint -->
-    <link name="adjustment_2_link"/>
-    <joint name="adjustment_2_joint" type="fixed">
-      <origin xyz="0 0 0" rpy="${radians(70)} 0 0" />
-      <parent link="${name}_post_arm_link" />
-      <child link="adjustment_2_link" />
-    </joint>
-    <!-- Adjustment 3 joint -->
-    <link name="adjustment_3_link"/>
-    <joint name="adjustment_3_joint" type="fixed">
-      <origin xyz="0 0 0" rpy="0 0 ${pi/2}" />
-      <parent link="adjustment_2_link" />
-      <child link="adjustment_3_link" />
-    </joint>
-    <!-- Sensor post arm to lidar joint -->
-    <joint name="${name}_post_arm_to_${name}_lidar_joint" type="fixed">
-      <origin xyz="0.04 0 0.045" rpy="${R} ${P} ${Y}" />
-      <parent link="adjustment_3_link" />
-      <child link="${name}_link" />
+      <origin xyz="0.028 0 ${z-1.545-0.05}" rpy="${radians(-50)} 0 ${-pi/2}"/>
+      <parent link="adjustment_1_link"/>
+      <child link="${name}_post_arm_link"/>
     </joint>
     <gazebo reference="${name}_link">

File: wamv_gazebo/urdf/wamv_gazebo.urdf.xacro (robot description, xacro)
@@ -72,5 +72,5 @@
   <!-- Add 3D LIDAR -->
   <xacro:if value="$(arg lidar_enabled)">
-    <xacro:wamv_3d_lidar name="lidar_wamv"/>
+    <xacro:wamv_3d_lidar name="lidar_wamv" x="0.7" y="0" z="1.8" R="0" P="${radians(10)}" Y="0"/>
   </xacro:if>
   <!-- Add P3D ground truth -->
@@ -93,6 +93,5 @@
     <xacro:wamv_imu name="imu_wamv" y="-0.2" />
     <!-- Add 3D LIDAR -->
-    <xacro:wamv_3d_lidar name="lidar_wamv" x="0.7" y="0" z="1.4" R="0" P="${radians(15)}" Y="0" post_Y="0"/>
-    <xacro:wamv_camera name="test_camera" x="0.7" y="0" z="1.4" R="0" P="${radians(15)}" Y="0" />
+    <xacro:wamv_3d_lidar name="lidar_wamv" x="0.7" y="0" z="1.8" R="0" P="${radians(10)}" Y="0"/>
   </xacro:if>
 </robot>

Commit message: Implement post_Y parameter that allows the post to be rotated in the yaw direction

File: wamv_gazebo/urdf/sensors/wamv_3d_lidar.xacro (robot description, xacro)
@@ -100,19 +100,19 @@
     <!-- Base to sensor post joint -->
     <joint name="base_to_${name}_post_joint" type="fixed">
-      <origin xyz="${x-0.07} ${y} 1.545" rpy="0 0 ${-pi/2}" />
+      <origin xyz="${x-0.07*cos(post_Y)} ${y-0.07*sin(post_Y)} 1.545" rpy="0 0 ${post_Y-pi/2}" />
       <parent link="base_link" />
       <child link="${name}_post_link" />
     </joint>
-    <!-- Adjustment 1 joint -->
-    <link name="adjustment_1_link"/>
-    <joint name="adjustment_1_joint" type="fixed">
+    <!-- Adjustment joint -->
+    <link name="adjustment_link"/>
+    <joint name="adjustment_joint" type="fixed">
       <origin xyz="0 0 0" rpy="0 0 ${pi/2}" />
       <parent link="${name}_post_link" />
-      <child link="adjustment_1_link" />
+      <child link="adjustment_link" />
     </joint>
     <!-- Sensor post to sensor post arm joint -->
     <joint name="${name}_post_to_${name}_post_arm_joint" type="fixed">
       <origin xyz="0.028 0 ${z-1.545-0.05}" rpy="${radians(-50)} 0 ${-pi/2}"/>
-      <parent link="adjustment_1_link"/>
+      <parent link="adjustment_link"/>
       <child link="${name}_post_arm_link"/>
     </joint>

File: wamv_gazebo/urdf/wamv_gazebo.urdf.xacro (robot description, xacro)
@@ -72,5 +72,5 @@
   <!-- Add 3D LIDAR -->
   <xacro:if value="$(arg lidar_enabled)">
-    <xacro:wamv_3d_lidar name="lidar_wamv" x="0.7" y="0" z="1.8" R="0" P="${radians(10)}" Y="0"/>
+    <xacro:wamv_3d_lidar name="lidar_wamv" x="0.7" y="0" z="1.8" R="0" P="${radians(15)}" Y="0" post_Y="0"/>
   </xacro:if>
   <!-- Add P3D ground truth -->
@@ -93,5 +93,5 @@
     <xacro:wamv_imu name="imu_wamv" y="-0.2" />
     <!-- Add 3D LIDAR -->
-    <xacro:wamv_3d_lidar name="lidar_wamv" x="0.7" y="0" z="1.8" R="0" P="${radians(10)}" Y="0"/>
+    <xacro:wamv_3d_lidar name="lidar_wamv" x="0.7" y="0" z="1.8" R="0" P="${radians(15)}" Y="0" post_Y="0"/>
   </xacro:if>
 </robot>
