Commit message: Simplify all transformations: base->post->arm->lidar

File: wamv_gazebo/urdf/sensors/wamv_3d_lidar.xacro (robot description, xacro)
@@ -69,5 +69,5 @@
     <link name="${name}_post_arm_link">
       <visual name="${name}_post_arm_visual">
-        <origin xyz="0 -0.016 -0.035" rpy="0 0 0"/>
+        <origin xyz="-0.038 0 -0.003" rpy="${radians(-60)} 0 ${-pi/2}"/>
         <geometry>
           <mesh filename="package://vrx_gazebo/models/sensor_post/mesh/sensor_post_arm.dae"/>
@@ -75,5 +75,5 @@
       </visual>
       <collision name="${name}_post_arm_collision">
-        <origin xyz="0 0 0" rpy="${-pi/20} 0 0"/>
+        <origin xyz="0 0 0" rpy="${radians(-60)-pi/20} 0 ${-pi/2}"/>
         <geometry>
           <cylinder radius="0.008" length="0.065"/>
@@ -81,5 +81,5 @@
       </collision>
       <inertial>
-        <origin xyz="0 0 0" rpy="${-pi/20} 0 0"/>
+        <origin xyz="0 0 0" rpy="${radians(-60)-pi/20} 0 ${-pi/2}"/>
         <mass value="0.1"/>
         <inertia
@@ -92,28 +92,21 @@
       </inertial>
     </link>
-    <!-- Base to lidar joint -->
-    <joint name="base_to_${name}_joint" type="fixed">
-      <origin xyz="${x} ${y} ${z}" rpy="${R} ${P} ${Y}" />
-      <parent link="base_link" />
-      <child link="${name}_link" />
-    </joint>
     <!-- Base to sensor post joint -->
     <joint name="base_to_${name}_post_joint" type="fixed">
-      <origin xyz="${x-0.07*cos(post_Y)} ${y-0.07*sin(post_Y)} 1.545" rpy="0 0 ${post_Y-pi/2}" />
+      <origin xyz="${x-(0.03+0.04)*cos(post_Y)} ${y-(0.03+0.04)*sin(post_Y)} 1.545" rpy="0 0 ${post_Y}" />
       <parent link="base_link" />
       <child link="${name}_post_link" />
     </joint>
-    <!-- Adjustment joint -->
-    <link name="adjustment_link"/>
-    <joint name="adjustment_joint" type="fixed">
-      <origin xyz="0 0 0" rpy="0 0 ${pi/2}" />
-      <parent link="${name}_post_link" />
-      <child link="adjustment_link" />
-    </joint>
     <!-- Sensor post to sensor post arm joint -->
     <joint name="${name}_post_to_${name}_post_arm_joint" type="fixed">
-      <origin xyz="0.028 0 ${z-1.545-0.05}" rpy="${radians(-50)} 0 ${-pi/2}"/>
-      <parent link="adjustment_link"/>
-      <child link="${name}_post_arm_link"/>
+      <origin xyz="0.03 0 ${z-1.545-0.05}" rpy="0 0 0" />
+      <parent link="${name}_post_link" />
+      <child link="${name}_post_arm_link" />
+    </joint>
+    <!-- Sensor post arm to lidar joint -->
+    <joint name="${name}_post_arm_to_${name}_joint" type="fixed">
+      <origin xyz="0.04 0 0.05" rpy="${R} ${P} ${Y-post_Y}" />
+      <parent link="${name}_post_arm_link" />
+      <child link="${name}_link" />
     </joint>
     <gazebo reference="${name}_link">

Commit message: Tweaked comments.

File: wamv_gazebo/urdf/sensors/wamv_3d_lidar.xacro (robot description, xacro)
@@ -2,8 +2,16 @@
 <robot xmlns:xacro="http://ros.org/wiki/xacro">
   <!-- Macro to insert a 3D scanning LIDAR with ROS integration
+    name: Prefix used for naming.
+    x: X position of the laser (from the base_link).
+    y: Y position of the laser (from the base_link).
+    z: Z position of the laser (from the base_link).
+    R: Roll orientation of the laser (from the laser's origin).
+    P: Pitch orientation of the laser (from the laser's origin).
+    Y: Yaw orientation of the laser (from the laser's origin).
+    post_Y: Yaw orientation of the post (from the post's origin).
     update_rate: frequency to publish output, hz
     vertical_lasers: number of vertical lasers which spin about Z to generate output
     samples: number of samples during spin, higher is more dense but slows down simulation
-    resolution: proportion of samples to actually simulate, rest are interprolated. Ex: 0.1 means 9/10 samples are interprolated
+    resolution: This number is multiplied by samples to determine the number of range data points returned.
     min_angle: the horizontal angle that the scan begins at
     max_angle: the angle that the scan ends at
@@ -13,5 +21,8 @@
     noise_stddev: Standard deviation of gaussian noise applied to output pointcloud
   -->
-  <xacro:macro name="wamv_3d_lidar" params="name x:=0.7 y:=0 z:=1.8 R:=0 P:=0 Y:=0 post_Y:=0
+  <xacro:macro name="wamv_3d_lidar" params="name
+                                            x:=0.7 y:=0 z:=1.8
+                                            R:=0 P:=0 Y:=0
+                                            post_Y:=0
                                             update_rate:=10 vertical_lasers:=16 samples:=1800 resolution:=0.1
                                             min_angle:=${-pi} max_angle:=${pi}

Commit message: Implement varying length lidar pole

File: wamv_gazebo/urdf/sensors/wamv_3d_lidar.xacro (robot description, xacro)
@@ -29,4 +29,9 @@
                                             min_vertical_angle:=${-pi/12} max_vertical_angle:=${pi/12}
                                             max_range:=100 noise_stddev:=0.01">
+    <!-- Define length variables for link positioning -->
+    <xacro:property name="platform_z" value="1.2965"/>
+    <xacro:property name="post_to_post_arm_x" value="0.03"/>
+    <xacro:property name="post_arm_to_lidar_x" value="0.04"/>
+    <xacro:property name="post_arm_to_lidar_z" value="0.05"/>
     <!-- 3d lidar sensor -->
     <link name="${name}_link">
@@ -53,23 +58,30 @@
       </inertial>
     </link>
+    <!-- Define post length and mass based on desired z position of sensor -->
+    <xacro:property name="post_length" value="${z-platform_z-post_arm_to_lidar_z}"/>
+    <xacro:property name="post_mass_per_meter" value="0.9"/>
+    <xacro:property name="post_mass" value="${post_mass_per_meter * post_length}"/>
+    <xacro:property name="post_radius" value="0.0076"/>
     <!-- Sensor post -->
     <link name="${name}_post_link">
-      <visual name="${name}_post_visual">
-        <origin xyz="0 0 -0.2515" rpy="${pi/2} 0 0"/>
+      <visual>
         <geometry>
-          <mesh filename="package://vrx_gazebo/models/sensor_post/mesh/sensor_post.dae"/>
+          <cylinder radius="${post_radius}" length="${post_length}"/>
         </geometry>
+        <material name="${name}_post_material">
+          <color rgba="0.0 0.0 0.0 1.0"/>
+        </material>
       </visual>
       <collision name="${name}_post_collision">
         <geometry>
-          <cylinder radius="0.0076" length="0.503"/>
+          <cylinder radius="${post_radius}" length="${post_length}"/>
         </geometry>
       </collision>
       <inertial>
-        <mass value="0.5"/>
+        <mass value="${post_mass}"/>
         <inertia
-          ixx="0.010549261666667"
-          iyy="0.010549261666667"
-          izz="0.000014440000000"
+          ixx="${(post_mass/12) * (3*post_radius*post_radius + post_length*post_length)}"
+          iyy="${(post_mass/12) * (3*post_radius*post_radius + post_length*post_length)}"
+          izz="${(post_mass/2) * (post_radius*post_radius)}"
           ixy="0"
           ixz="0"
@@ -104,6 +116,7 @@
     </link>
     <!-- Base to sensor post joint -->
+    <xacro:property name="post_z" value="${platform_z+post_length/2}"/>
     <joint name="base_to_${name}_post_joint" type="fixed">
-      <origin xyz="${x-(0.03+0.04)*cos(post_Y)} ${y-(0.03+0.04)*sin(post_Y)} 1.545" rpy="0 0 ${post_Y}" />
+      <origin xyz="${x-(post_to_post_arm_x+post_arm_to_lidar_x)*cos(post_Y)} ${y-(post_to_post_arm_x+post_arm_to_lidar_x)*sin(post_Y)} ${post_z}" rpy="0 0 ${post_Y}" />
       <parent link="base_link" />
       <child link="${name}_post_link" />
@@ -111,5 +124,5 @@
     <!-- Sensor post to sensor post arm joint -->
     <joint name="${name}_post_to_${name}_post_arm_joint" type="fixed">
-      <origin xyz="0.03 0 ${z-1.545-0.05}" rpy="0 0 0" />
+      <origin xyz="${post_to_post_arm_x} 0 ${z-post_z-post_arm_to_lidar_z}" rpy="0 0 0" />
       <parent link="${name}_post_link" />
       <child link="${name}_post_arm_link" />
@@ -117,5 +130,5 @@
     <!-- Sensor post arm to lidar joint -->
     <joint name="${name}_post_arm_to_${name}_joint" type="fixed">
-      <origin xyz="0.04 0 0.05" rpy="${R} ${P} ${Y-post_Y}" />
+      <origin xyz="${post_arm_to_lidar_x} 0 ${post_arm_to_lidar_z}" rpy="${R} ${P} ${Y-post_Y}" />
       <parent link="${name}_post_arm_link" />
       <child link="${name}_link" />
@@ -156,4 +169,8 @@
       </sensor>
     </gazebo>
+    <!-- Set color of post -->
+    <gazebo reference="${name}_post_link">
+      <material>Gazebo/Black</material>
+    </gazebo>
   </xacro:macro>
 </robot>

File: wamv_gazebo/urdf/sensors/wamv_camera.xacro (robot description, xacro)
@@ -48,5 +48,5 @@
       <visual>
         <geometry>
-          <cylinder radius="0.0076" length="${post_length}"/>
+          <cylinder radius="${post_radius}" length="${post_length}"/>
         </geometry>
         <material name="${name}_post_material">

Commit message: Clarify link relative position calculation

File: wamv_gazebo/urdf/sensors/wamv_3d_lidar.xacro (robot description, xacro)
@@ -117,6 +117,7 @@
     <!-- Base to sensor post joint -->
     <xacro:property name="post_z" value="${platform_z+post_length/2}"/>
+    <xacro:property name="post_to_lidar_x" value="${post_to_post_arm_x+post_arm_to_lidar_x}"/>
     <joint name="base_to_${name}_post_joint" type="fixed">
-      <origin xyz="${x-(post_to_post_arm_x+post_arm_to_lidar_x)*cos(post_Y)} ${y-(post_to_post_arm_x+post_arm_to_lidar_x)*sin(post_Y)} ${post_z}" rpy="0 0 ${post_Y}" />
+      <origin xyz="${x-(post_to_lidar_x)*cos(post_Y)} ${y-(post_to_lidar_x)*sin(post_Y)} ${post_z}" rpy="0 0 ${post_Y}" />
       <parent link="base_link" />
       <child link="${name}_post_link" />

File: wamv_gazebo/urdf/sensors/wamv_camera.xacro (robot description, xacro)
@@ -98,6 +98,7 @@
     <!-- Base to sensor post joint -->
     <xacro:property name="post_z" value="${platform_z+post_length/2}"/>
+    <xacro:property name="post_to_camera_x" value="${post_to_post_arm_x+post_arm_to_camera_x}"/>
     <joint name="base_to_${name}_post_joint" type="fixed">
-      <origin xyz="${x-(post_to_post_arm_x+post_arm_to_camera_x)*cos(post_Y)} ${y-(post_to_post_arm_x+post_arm_to_camera_x)*sin(post_Y)} ${post_z}" rpy="0 0 ${post_Y}" />
+      <origin xyz="${x-(post_to_camera_x)*cos(post_Y)} ${y-(post_to_camera_x)*sin(post_Y)} ${post_z}" rpy="0 0 ${post_Y}" />
       <parent link="base_link" />
       <child link="${name}_post_link" />

Commit message: Modify xacro files to add further topic subnamespaces to sensor models

File: wamv_gazebo/urdf/sensors/wamv_3d_lidar.xacro (robot description, xacro)
@@ -164,5 +164,5 @@
         </ray>
         <plugin name="${name}_plugin" filename="libgazebo_ros_velodyne_gpu_laser.so">
-          <topicName>${sensor_namespace}${name}/points</topicName>
+          <topicName>${sensor_namespace}lidar/${name}/points</topicName>
           <frameName>${name}_link</frameName>
           <min_intensity>0</min_intensity>

File: wamv_gazebo/urdf/sensors/wamv_gps.xacro (robot description, xacro)
@@ -35,6 +35,7 @@
         <alwaysOn>true</alwaysOn>
         <bodyName>${name}_link</bodyName>
-        <frameId>${name}_link</frameId>
-        <topicName>${sensor_namespace}gps/fix</topicName>
+        <!-- Manually prepend namespace to tf frame. -->
+        <frameId>${namespace}/${name}_link</frameId>
+        <topicName>${sensor_namespace}gps/gps/fix</topicName>
         <!-- Note that the hector_gazebo_ros_gps plugin uses NWU coordinates
              for reporting velocities.  This may cause problems if localization
@@ -42,5 +43,5 @@
              See Issue #64 in VRX project for details
              https://bitbucket.org/osrf/vrx/issues/64 -->
-        <velocityTopicName>${sensor_namespace}gps/fix_velocity</velocityTopicName>
+        <velocityTopicName>${sensor_namespace}gps/gps/fix_velocity</velocityTopicName>
         <!-- Location of origin of Gazebo Sand Island map -->
         <referenceLatitude>21.30996</referenceLatitude>

File: wamv_gazebo/urdf/sensors/wamv_imu.xacro (robot description, xacro)
@@ -21,7 +21,8 @@
         <updateRate>15.0</updateRate>
         <bodyName>${name}_link</bodyName>
-        <topicName>${sensor_namespace}imu/data</topicName>
+        <topicName>${sensor_namespace}imu/imu/data</topicName>
         <serviceName>${sensor_namespace}imu_service</serviceName>
-        <frameId>${name}_link</frameId>
+        <!-- Manually prepend namespace to tf frame. -->
+        <frameId>${namespace}/${name}_link</frameId>
         <alwaysOn>true</alwaysOn>
         <accelOffset>0.0 0.0 0.0</accelOffset>

File: wamv_gazebo/urdf/sensors/wamv_p3d.xacro (robot description, xacro)
@@ -7,5 +7,5 @@
         <frameName>map</frameName>
         <updateRate>10.0</updateRate>
-        <topicName>${sensor_namespace}${name}</topicName>
+        <topicName>${sensor_namespace}position/${name}</topicName>
         <xyzOffset>0 0 0</xyzOffset>
         <rpyOffset>0 0 0</rpyOffset>

File: wamv_gazebo/urdf/sensors/wamv_planar_lidar.xacro (robot description, xacro)
@@ -39,5 +39,5 @@
         </ray>
         <plugin name="multibeam_simulator" filename="libgazebo_ros_gpu_laser.so">
-          <topicName>${sensor_namespace}${name}/scan</topicName>
+          <topicName>${sensor_namespace}lidar/${name}/scan</topicName>
           <frameName>${name}_link</frameName>
         </plugin>

File: wamv_gazebo/urdf/wamv_gazebo.urdf.xacro (robot description, xacro)
@@ -14,7 +14,11 @@
   <xacro:arg name="camera_namespace" default="cameras/"/>
   <xacro:arg name="sensor_namespace" default="sensors/"/>
+  <!-- Note: this is only used for some sensors that do not correctly use the
+  robotNamespace parameter -->
+  <xacro:arg name="namespace" default="wamv"/>
   <xacro:property name="thruster_namespace" value="$(arg thruster_namespace)" scope="global" />
   <xacro:property name="camera_namespace" value="$(arg camera_namespace)" scope="global" />
   <xacro:property name="sensor_namespace" value="$(arg sensor_namespace)" scope="global" />
+  <xacro:property name="namespace" value="$(arg namespace)" scope="global" />
   <!-- Sensor yaml file -->
   <xacro:arg name="yaml_sensor_generation" default="false"/>
