Commit message: VRX namespaces.

File: wamv_gazebo/urdf/sensors/wamv_pinger.xacro (robot description, xacro)
@@ -23,5 +23,7 @@
     <gazebo>
       <plugin name="pinger_plugin" filename="libusv_gazebo_acoustic_pinger_plugin.so">
-        <frameId>pinger_wamv</frameId>
+        <frameId>wamv/pinger</frameId>
+        <topicName>${namespace}/${sensor_namespace}${pinger_namespace}${name}/range_bearing</topicName>
+        <setPositionTopicName>${namespace}/${sensor_namespace}${pinger_namespace}${name}/set_pinger_position</setPositionTopicName>
         <rangeNoise>
           <noise>

File: wamv_gazebo/urdf/wamv_gazebo.urdf.xacro (robot description, xacro)
@@ -15,4 +15,5 @@
   <xacro:arg name="camera_namespace" default="cameras/"/>
   <xacro:arg name="sensor_namespace" default="sensors/"/>
+  <xacro:arg name="pinger_namespace" default="pingers/"/>
   <!-- Note: this is only used for some sensors that do not correctly use the
   robotNamespace parameter -->
@@ -21,4 +22,5 @@
   <xacro:property name="camera_namespace" value="$(arg camera_namespace)" scope="global" />
   <xacro:property name="sensor_namespace" value="$(arg sensor_namespace)" scope="global" />
+  <xacro:property name="pinger_namespace" value="$(arg pinger_namespace)" scope="global" />
   <xacro:property name="namespace" value="$(arg namespace)" scope="global" />
   <!-- Sensor yaml file -->
@@ -115,5 +117,5 @@
     <!-- Add pinger -->
     <xacro:if value="$(arg pinger_enabled)">
-      <xacro:wamv_pinger name="pinger_wamv" position="1.0 0 -1.0" />
+      <xacro:wamv_pinger name="pinger" position="1.0 0 -1.0" />
     </xacro:if>
     <!-- ==== VRX sensor configuration ==== -->
@@ -134,5 +136,5 @@
       <xacro:lidar name="lidar_wamv" type="16_beam"/>
       <!-- Add pinger -->
-      <xacro:wamv_pinger name="pinger_wamv" position="1.0 0 -1.0" />
+      <xacro:wamv_pinger name="pinger" position="1.0 0 -1.0" />
     </xacro:if>
   </xacro:unless>

Commit message: Parametrize frameId in wamv_pinger xacro macro.
Signed-off-by: Carlos Agüero <caguero@openrobotics.org>

File: wamv_gazebo/urdf/sensors/wamv_pinger.xacro (robot description, xacro)
@@ -1,5 +1,5 @@
 <?xml version="1.0"?>
 <robot xmlns:xacro="http://ros.org/wiki/xacro">
-  <xacro:macro name="wamv_pinger" params="name:='pinger' position:='0 0 0' orientation:='0 0 0'">
+  <xacro:macro name="wamv_pinger" params="name:='pinger' frameId:='wamv/pinger' position:='0 0 0' orientation:='0 0 0'">
     <link name="${name}">
       <visual>
@@ -23,5 +23,5 @@
     <gazebo>
       <plugin name="pinger_plugin" filename="libusv_gazebo_acoustic_pinger_plugin.so">
-        <frameId>wamv/pinger</frameId>
+        <frameId>${frameId}</frameId>
         <topicName>${namespace}/${sensor_namespace}${pinger_namespace}${name}/range_bearing</topicName>
         <setPositionTopicName>${namespace}/${sensor_namespace}${pinger_namespace}${name}/set_pinger_position</setPositionTopicName>
