Commit message: Fix macro

File: wamv_gazebo/urdf/sensors/lidar.xacro (robot description, xacro)
@@ -1,16 +1,19 @@
 <?xml version="1.0" encoding="UTF-8"?>
 <robot xmlns:xacro="http://ros.org/wiki/xacro">
-  <xacro:macro name="lidar" params = "type:='16_beam'
-                                      name
-				      x:=0.7 y:=0 z:=1.8
-                                      R:=0 P:=0 Y:=0
-                                      post_Y:=0">
-    <xacro:include filename="$(find wamv_gazebo)/urdf/sensors/wamv_3d_lidar.xacro"/>
+  <xacro:include filename="$(find wamv_gazebo)/urdf/sensors/wamv_3d_lidar.xacro"/>
+  <xacro:macro name="lidar"
+               params = "type:='16_beam'
+                         name
+                         x:=0.7 y:=0 z:=1.8
+                         R:=0 P:=0 Y:=0
+                         post_Y:=0">
     <xacro:if value="${type == '16_beam'}">
       <xacro:wamv_3d_lidar name="${name}"
                            x="${x}" y="${y}" z="${z}"
                            R="${R}" P="${P}" Y="${Y}"
-			   vertical_lasers="16"/>
-      <!--specs for 16 beam lidar are implimneted by default. See wamv_3d_lidar for those-->
+                           post_Y="${post_Y}"
+                           vertical_lasers="16"/>
+      <!--specs for 16 beam lidar are implemented by default.
+          See wamv_3d_lidar for those-->
     </xacro:if>
     <xacro:if value="${type == '32_beam'}">
@@ -18,7 +21,9 @@
                            x="${x}" y="${y}" z="${z}"
                            R="${R}" P="${P}" Y="${Y}"
-			   vertical_lasers="32"
-			   samples="2187"
-			   min_vertical_angle="0.54" max_vertical_angle="-0.186"/>
+                           post_Y="${post_Y}"
+                           vertical_lasers="32"
+                           samples="2187"
+                           min_vertical_angle="0.54"
+                           max_vertical_angle="-0.186"/>
     </xacro:if>
   </xacro:macro>

Commit message: Adding extra parameter to set the height of the post's base.
Signed-off-by: Carlos Agüero <caguero@openrobotics.org>

File: wamv_gazebo/urdf/sensors/lidar.xacro (robot description, xacro)
@@ -7,10 +7,10 @@
                          x:=0.7 y:=0 z:=1.8
                          R:=0 P:=0 Y:=0
-                         post_Y:=0">
+                         post_Y:=0 post_z_from:=1.2965">
     <xacro:if value="${type == '16_beam'}">
       <xacro:wamv_3d_lidar name="${name}"
                            x="${x}" y="${y}" z="${z}"
                            R="${R}" P="${P}" Y="${Y}"
-                           post_Y="${post_Y}"
+                           post_Y="${post_Y}" post_z_from="${post_z_from}"
                            vertical_lasers="16"/>
       <!--specs for 16 beam lidar are implemented by default.
@@ -21,5 +21,5 @@
                            x="${x}" y="${y}" z="${z}"
                            R="${R}" P="${P}" Y="${Y}"
-                           post_Y="${post_Y}"
+                           post_Y="${post_Y}" post_z_from="${post_z_from}"
                            vertical_lasers="32"
                            samples="2187"

File: wamv_gazebo/urdf/sensors/wamv_3d_lidar.xacro (robot description, xacro)
@@ -10,4 +10,5 @@
     Y: Yaw orientation of the laser (from the laser's origin).
     post_Y: Yaw orientation of the post (from the post's origin).
+    post_z_from: Z position of the post's base.
     update_rate: frequency to publish output, hz
     vertical_lasers: number of vertical lasers which spin about Z to generate output
@@ -24,5 +25,5 @@
                                             x:=0.7 y:=0 z:=1.8
                                             R:=0 P:=0 Y:=0
-                                            post_Y:=0
+                                            post_Y:=0 post_z_from:=1.2965
                                             update_rate:=10 vertical_lasers:=16 samples:=1875 resolution:=0.1
                                             min_angle:=${-pi} max_angle:=${pi}
@@ -30,5 +31,5 @@
                                             max_range:=130 noise_stddev:=0.01">
     <!-- Define length variables for link positioning -->
-    <xacro:property name="platform_z" value="1.2965"/>
+    <xacro:property name="platform_z" value="${post_z_from}"/>
     <xacro:property name="post_to_post_arm_x" value="0.03"/>
     <xacro:property name="post_arm_to_lidar_x" value="0.04"/>

File: wamv_gazebo/urdf/sensors/wamv_camera.xacro (robot description, xacro)
@@ -1,7 +1,7 @@
 <?xml version="1.0"?>
 <robot xmlns:xacro="http://ros.org/wiki/xacro">
-  <xacro:macro name="wamv_camera" params="name x:=0.5 y:=0 z:=1.5 R:=0 P:=0 Y:=0 post_Y:=0">
+  <xacro:macro name="wamv_camera" params="name x:=0.5 y:=0 z:=1.5 post_z_from:=1.2965  R:=0 P:=0 Y:=0 post_Y:=0">
     <!-- Define length variables for link positioning -->
-    <xacro:property name="platform_z" value="1.2965"/>
+    <xacro:property name="platform_z" value="${post_z_from}"/>
     <xacro:property name="post_to_post_arm_x" value="0.03"/>
     <xacro:property name="post_arm_to_camera_x" value="0.02"/>
