Commit message: Adding gps mesh, collisions and inertia.

File: wamv_gazebo/urdf/sensors/wamv_gps.xacro (robot description, xacro)
@@ -3,21 +3,25 @@
   <xacro:macro name="wamv_gps" params="name:=gps x:=0 y:=0 z:=1.3 R:=0 P:=0 Y:=0">
     <link name="${name}_link">
-      <visual name="${name}_visual_base">
+      <visual name="{name}_visual">
         <geometry>
-          <box size="0.1 0.1 0.025" />
+          <mesh filename="package://wamv_gazebo/mesh/gps.dae"/>
         </geometry>
-        <material name="${name}_visual_base_material">
-          <color rgba="1.0 1.0 1.0 1.0" />
-        </material>
       </visual>
-      <visual name="${name}_visual_antenna">
-        <origin xyz="0 0 0.025" />
+      <collision name="collision_stick">
+        <origin xyz="0 0 0.4" rpy="0 0 0" />
         <geometry>
-          <sphere radius="0.03" />
+          <cylinder length="0.8" radius="0.05" />
         </geometry>
-        <material name="${name}_visual_antenna_material">
-          <color rgba="0.7 0.7 0.7 1.0" />
-        </material>
-      </visual>
+      </collision>
+      <collision name="collision_antenna">
+        <origin xyz="0 -0.05 0.85" rpy="0 0 0" />
+        <geometry>
+          <cylinder length="0.1" radius="0.15" />
+        </geometry>
+      </collision>
+      <inertial>
+        <mass value="1"/>
+        <inertia ixx="0.0684" ixy="0.0" ixz="0.0" iyy="0.0684" iyz="0.0" izz="0.0018"/>
+      </inertial>
     </link>
     <joint name="${name}_joint" type="fixed">

File: wamv_gazebo/urdf/wamv_gazebo.urdf.xacro (robot description, xacro)
@@ -82,5 +82,5 @@
     <xacro:wamv_camera name="middle_right_camera" y="-0.45" P="${radians(15)}" Y="${radians(-90)}" />
     <!-- Add simulated GPS -->
-    <xacro:wamv_gps name="gps_wamv" y="0.2" />
+    <xacro:wamv_gps name="gps_wamv" x="-0.75" />
     <!-- Add Simulated IMU -->
     <xacro:wamv_imu name="imu_wamv" y="-0.2" />

Commit message: Tweak names.

File: wamv_gazebo/urdf/sensors/wamv_gps.xacro (robot description, xacro)
@@ -3,10 +3,10 @@
   <xacro:macro name="wamv_gps" params="name:=gps x:=0 y:=0 z:=1.3 R:=0 P:=0 Y:=0">
     <link name="${name}_link">
-      <visual name="{name}_visual">
+      <visual name="${name}_visual">
         <geometry>
           <mesh filename="package://wamv_gazebo/mesh/gps.dae"/>
         </geometry>
       </visual>
-      <collision name="collision_stick">
+      <collision name="${name}_collision_base">
         <origin xyz="0 0 0.4" rpy="0 0 0" />
         <geometry>
@@ -14,5 +14,5 @@
         </geometry>
       </collision>
-      <collision name="collision_antenna">
+      <collision name="${name}_collision_antenna">
         <origin xyz="0 -0.05 0.85" rpy="0 0 0" />
         <geometry>

Commit message: Lower mast.

File: wamv_gazebo/urdf/sensors/wamv_gps.xacro (robot description, xacro)
@@ -1,5 +1,5 @@
 <?xml version="1.0" encoding="UTF-8"?>
 <robot xmlns:xacro="http://ros.org/wiki/xacro">
-  <xacro:macro name="wamv_gps" params="name:=gps x:=0 y:=0 z:=1.3 R:=0 P:=0 Y:=0">
+  <xacro:macro name="wamv_gps" params="name:=gps x:=0 y:=0 z:=1.28 R:=0 P:=0 Y:=0">
     <link name="${name}_link">
       <visual name="${name}_visual">
@@ -9,11 +9,11 @@
       </visual>
       <collision name="${name}_collision_base">
-        <origin xyz="0 0 0.4" rpy="0 0 0" />
+        <origin xyz="0 0 0.025" rpy="0 0 0" />
         <geometry>
-          <cylinder length="0.8" radius="0.05" />
+          <cylinder length="0.05" radius="0.015" />
         </geometry>
       </collision>
       <collision name="${name}_collision_antenna">
-        <origin xyz="0 -0.05 0.85" rpy="0 0 0" />
+        <origin xyz="0 0 0.11" rpy="0 0 0" />
         <geometry>
           <cylinder length="0.1" radius="0.15" />
@@ -22,5 +22,5 @@
       <inertial>
         <mass value="1"/>
-        <inertia ixx="0.0684" ixy="0.0" ixz="0.0" iyy="0.0684" iyz="0.0" izz="0.0018"/>
+        <inertia ixx="0.006458" ixy="0.0" ixz="0.0" iyy="0.006458" iyz="0.0" izz="0.01125"/>
       </inertial>
     </link>

File: wamv_gazebo/urdf/wamv_gazebo.urdf.xacro (robot description, xacro)
@@ -60,5 +60,5 @@
   <!-- Add simulated GPS -->
   <xacro:if value="$(arg gps_enabled)">
-    <xacro:wamv_gps name="gps_wamv" y="0.2" />
+    <xacro:wamv_gps name="gps_wamv" x="-0.85" />
   </xacro:if>
   <!-- Add Simulated IMU -->
@@ -82,5 +82,5 @@
     <xacro:wamv_camera name="middle_right_camera" y="-0.45" P="${radians(15)}" Y="${radians(-90)}" />
     <!-- Add simulated GPS -->
-    <xacro:wamv_gps name="gps_wamv" x="-0.75" />
+    <xacro:wamv_gps name="gps_wamv" x="-0.85" />
     <!-- Add Simulated IMU -->
     <xacro:wamv_imu name="imu_wamv" y="-0.2" />

Commit message: Added allowences for post_Y and moved wamv_imu, wamv_gps default locations to be within compliance

File: wamv_gazebo/urdf/sensors/wamv_gps.xacro (robot description, xacro)
@@ -1,5 +1,5 @@
 <?xml version="1.0" encoding="UTF-8"?>
 <robot xmlns:xacro="http://ros.org/wiki/xacro">
-  <xacro:macro name="wamv_gps" params="name:=gps x:=0 y:=0 z:=1.28 R:=0 P:=0 Y:=0">
+  <xacro:macro name="wamv_gps" params="name:=gps x:=0.3 y:=0.5 z:=1.3 R:=0 P:=0 Y:=0">
     <link name="${name}_link">
       <visual name="${name}_visual">

File: wamv_gazebo/urdf/sensors/wamv_imu.xacro (robot description, xacro)
@@ -1,5 +1,5 @@
 <?xml version="1.0"?>
 <robot xmlns:xacro="http://ros.org/wiki/xacro">
-  <xacro:macro name="wamv_imu" params="name:=imu x:=0 y:=0 z:=1.3 R:=0 P:=0 Y:=0">
+  <xacro:macro name="wamv_imu" params="name:=imu x:=0.3 y:=0.5 z:=1.3 R:=0 P:=0 Y:=0">
     <link name="${name}_link">
       <visual name="${name}_visual">>

Commit message: Using 16 beam lasers

File: wamv_gazebo/urdf/sensors/wamv_gps.xacro (robot description, xacro)
@@ -1,5 +1,5 @@
 <?xml version="1.0" encoding="UTF-8"?>
 <robot xmlns:xacro="http://ros.org/wiki/xacro">
-  <xacro:macro name="wamv_gps" params="name:=gps x:=0.3 y:=0.5 z:=1.3 R:=0 P:=0 Y:=0">
+  <xacro:macro name="wamv_gps" params="name:=gps x:=0.3 y:=0 z:=1.3 R:=0 P:=0 Y:=0">
     <link name="${name}_link">
       <visual name="${name}_visual">

File: wamv_gazebo/urdf/wamv_gazebo.urdf.xacro (robot description, xacro)
@@ -93,5 +93,5 @@
     <!-- Add 3D LIDAR -->
     <xacro:if value="$(arg lidar_enabled)">
-      <xacro:lidar name="lidar_wamv" y="-0.3" type="32_beam"/>
+      <xacro:lidar name="lidar_wamv" y="-0.3" type="16_beam"/>
     </xacro:if>
     <!-- Add P3D ground truth -->
@@ -114,5 +114,5 @@
       <xacro:wamv_imu name="imu_wamv" y="-0.2" />
       <!-- Add 3D LIDAR -->
-      <xacro:wamv_3d_lidar name="lidar_wamv" P="${radians(8)}" />
+      <xacro:lidar name="lidar_wamv" type="16_beam"/>
     </xacro:if>
   </xacro:unless>

Commit message: Create links where the GPS and IMU sensors are attached.

File: wamv_gazebo/urdf/sensors/wamv_gps.xacro (robot description, xacro)
@@ -25,5 +25,7 @@
       </inertial>
     </link>
-    <joint name="${name}_joint" type="fixed">
+    <joint name="${name}_joint" type="revolute">
+      <axis xyz="0 0 0"/>
+      <limit effort="1000.0" lower="0.0" upper="0" velocity="0"/>
       <origin xyz="${x} ${y} ${z}" rpy="${R} ${P} ${Y}" />
       <parent link="base_link" />

File: wamv_gazebo/urdf/sensors/wamv_imu.xacro (robot description, xacro)
@@ -11,6 +11,12 @@
         </material>
       </visual>
+      <inertial>
+        <mass value="0.1"/>
+        <inertia ixx="0.000083" ixy="0.0" ixz="0.0" iyy="0.000083" iyz="0.0" izz="0.0125"/>
+      </inertial>
     </link>
-    <joint name="${name}_joint" type="fixed">
+    <joint name="${name}_joint" type="revolute">
+      <axis xyz="0 0 0"/>
+      <limit effort="1000.0" lower="0.0" upper="0" velocity="0"/>
       <origin xyz="${x} ${y} ${z}" rpy="${R} ${P} ${Y}"/>
       <parent link="base_link"/>

Commit message: Switch to 0 0 1 in axis.

File: wamv_gazebo/urdf/sensors/wamv_gps.xacro (robot description, xacro)
@@ -26,5 +26,5 @@
     </link>
     <joint name="${name}_joint" type="revolute">
-      <axis xyz="0 0 0"/>
+      <axis xyz="0 0 1"/>
       <limit effort="1000.0" lower="0.0" upper="0" velocity="0"/>
       <origin xyz="${x} ${y} ${z}" rpy="${R} ${P} ${Y}" />

File: wamv_gazebo/urdf/sensors/wamv_imu.xacro (robot description, xacro)
@@ -17,5 +17,5 @@
     </link>
     <joint name="${name}_joint" type="revolute">
-      <axis xyz="0 0 0"/>
+      <axis xyz="0 0 1"/>
       <limit effort="1000.0" lower="0.0" upper="0" velocity="0"/>
       <origin xyz="${x} ${y} ${z}" rpy="${R} ${P} ${Y}"/>

Commit message: Added lat/lon/elev parameters to wamv_gps.xacro input parms

File: wamv_gazebo/urdf/sensors/wamv_gps.xacro (robot description, xacro)
@@ -1,5 +1,5 @@
 <?xml version="1.0" encoding="UTF-8"?>
 <robot xmlns:xacro="http://ros.org/wiki/xacro">
-  <xacro:macro name="wamv_gps" params="name:=gps x:=0.3 y:=0 z:=1.3 R:=0 P:=0 Y:=0">
+  <xacro:macro name="wamv_gps" params="name:=gps x:=0.3 y:=0 z:=1.3 R:=0 P:=0 Y:=0 lat:=21.30996 lon:=-157.8901 elev:=0.0">
     <link name="${name}_link">
       <visual name="${name}_visual">
@@ -47,7 +47,7 @@
         <velocityTopicName>${namespace}/${sensor_namespace}gps/gps/fix_velocity</velocityTopicName>
         <!-- Location of origin of Gazebo Sand Island map -->
-        <referenceLatitude>21.30996</referenceLatitude>
-        <referenceLongitude>-157.8901</referenceLongitude>
-        <referenceAltitude>0</referenceAltitude>
+        <referenceLatitude>${lat}</referenceLatitude>
+        <referenceLongitude>${lon}</referenceLongitude>
+        <referenceAltitude>${elev}</referenceAltitude>
         <referenceHeading>90</referenceHeading>
         <offset>0.0 0.0 0.0</offset>

Commit message: Add update_rate parameters to wamv_imu and wamv_gps.
Signed-off-by: Carlos Agüero <caguero@openrobotics.org>

File: wamv_gazebo/urdf/sensors/wamv_gps.xacro (robot description, xacro)
@@ -1,5 +1,5 @@
 <?xml version="1.0" encoding="UTF-8"?>
 <robot xmlns:xacro="http://ros.org/wiki/xacro">
-  <xacro:macro name="wamv_gps" params="name:=gps x:=0.3 y:=0 z:=1.3 R:=0 P:=0 Y:=0 lat:=21.30996 lon:=-157.8901 elev:=0.0">
+  <xacro:macro name="wamv_gps" params="name:=gps x:=0.3 y:=0 z:=1.3 R:=0 P:=0 Y:=0 lat:=21.30996 lon:=-157.8901 elev:=0.0 update_rate:=15">
     <link name="${name}_link">
       <visual name="${name}_visual">
@@ -34,5 +34,5 @@
     <gazebo>
       <plugin name="gps_plugin_${name}" filename="libhector_gazebo_ros_gps.so">
-        <updateRate>15.0</updateRate>
+        <updateRate>${update_rate}</updateRate>
         <alwaysOn>true</alwaysOn>
         <bodyName>${name}_link</bodyName>

File: wamv_gazebo/urdf/sensors/wamv_imu.xacro (robot description, xacro)
@@ -1,5 +1,5 @@
 <?xml version="1.0"?>
 <robot xmlns:xacro="http://ros.org/wiki/xacro">
-  <xacro:macro name="wamv_imu" params="name:=imu x:=0.3 y:=0.5 z:=1.3 R:=0 P:=0 Y:=0">
+  <xacro:macro name="wamv_imu" params="name:=imu x:=0.3 y:=0.5 z:=1.3 R:=0 P:=0 Y:=0 update_rate:=15">
     <link name="${name}_link">
       <visual name="${name}_visual">>
@@ -25,5 +25,5 @@
     <gazebo>
       <plugin name="imu_plugin_${name}" filename="libhector_gazebo_ros_imu.so">
-        <updateRate>15.0</updateRate>
+        <updateRate>${update_rate}</updateRate>
         <bodyName>${name}_link</bodyName>
         <topicName>${namespace}/${sensor_namespace}imu/imu/data</topicName>
