Commit message: Added namespace to gazebo references, re-add color, fix wamv_planar_lidar links and joints

File: wamv_gazebo/urdf/sensors/wamv_planar_lidar.xacro (robot description, xacro)
@@ -2,5 +2,5 @@
 <robot xmlns:xacro="http://ros.org/wiki/xacro">
   <xacro:macro name="wamv_multibeam_laser" params="name x:=0.5 y:=0 z:=2 R:=0 P:=0 Y:=0">
-    <link name="${name}_link">
+    <link name="${namespace}/${name}_link">
       <visual name="${name}_visual">>
         <geometry>
@@ -12,10 +12,10 @@
       </visual>
     </link>
-    <joint name="${name}_joint" type="fixed">
+    <joint name="${namespace}/${name}_joint" type="fixed">
       <origin xyz="${x} ${y} ${z}" rpy="${R} ${P} ${Y}" />
-      <parent link="base_link" />
-      <child link="${name}_link" />
+      <parent link="${namespace}/base_link" />
+      <child link="${namespace}/${name}_link" />
     </joint>
-    <gazebo reference="${name}_link">
+    <gazebo reference="${namespace}/${name}_link">
       <sensor type="gpu_ray" name="multibeam_sensor_${name}">
         <update_rate>10</update_rate>
@@ -40,5 +40,5 @@
         <plugin name="multibeam_simulator" filename="libgazebo_ros_gpu_laser.so">
           <topicName>${namespace}/${sensor_namespace}lidars/${name}/scan</topicName>
-          <frameName>${name}_link</frameName>
+          <frameName>${namespace}/${name}_link</frameName>
         </plugin>
       </sensor>
