Commit message: Add optical frame for proper camera visualization

File: wamv_gazebo/urdf/sensors/wamv_camera.xacro (robot description, xacro)
@@ -7,4 +7,10 @@
       <parent link="base_link"/>
       <child link="${name}_link"/>
+    </joint>
+    <link name="${name}_link_optical" />
+    <joint name="${name}_optical_joint" type="fixed">
+      <origin xyz="0 0 0" rpy="${-pi/2} 0 ${-pi/2}" />
+      <parent link="${name}_link"/>
+      <child link="${name}_link_optical"/>
     </joint>
     <gazebo reference="${name}_link">
@@ -37,5 +43,5 @@
           <imageTopicName>image_raw</imageTopicName>
           <cameraInfoTopicName>camera_info</cameraInfoTopicName>
-          <frameName>${name}_link</frameName>
+          <frameName>${name}_link_optical</frameName>
           <hackBaseline>0.07</hackBaseline>
           <distortionK1>0.0</distortionK1>

Commit message: Add simple visuals for sensors

File: wamv_gazebo/urdf/sensors/wamv_camera.xacro (robot description, xacro)
@@ -2,5 +2,16 @@
 <robot xmlns:xacro="http://ros.org/wiki/xacro">
   <xacro:macro name="wamv_camera" params="name x:=0.5 y:=0 z:=1.5 R:=0 P:=0 Y:=0">
-    <link name="${name}_link"/>
+    <link name="${name}_link">
+      <visual name="${name}_visual">
+        <xacro:property name="visual_length" value="0.05" />
+        <origin xyz="-${visual_length/2.0} 0 0" rpy="0 1.57 0" />
+        <geometry>
+          <cylinder radius="0.01" length="${visual_length}" />
+        </geometry>
+        <material name="${name}_visual_material">
+          <color rgba="1.0 1.0 0.0 1.0" />
+        </material>
+      </visual>
+    </link>
     <joint name="${name}_joint" type="fixed">
       <origin xyz="${x} ${y} ${z}" rpy="${R} ${P} ${Y}"/>

File: wamv_gazebo/urdf/sensors/wamv_gps.xacro (robot description, xacro)
@@ -1,6 +1,24 @@
 <?xml version="1.0" encoding="UTF-8"?>
 <robot xmlns:xacro="http://ros.org/wiki/xacro">
-  <xacro:macro name="wamv_gps" params="name:=gps x:=0 y:=0 z:=1.5 R:=0 P:=0 Y:=0">
-    <link name="${name}_link" />
+  <xacro:macro name="wamv_gps" params="name:=gps x:=0 y:=0 z:=1.3 R:=0 P:=0 Y:=0">
+    <link name="${name}_link">
+      <visual name="${name}_visual_base">
+        <geometry>
+          <box size="0.1 0.1 0.025" />
+        </geometry>
+        <material name="${name}_visual_base_material">
+          <color rgba="1.0 1.0 1.0 1.0" />
+        </material>
+      </visual>
+      <visual name="${name}_visual_antenna">
+        <origin xyz="0 0 0.025" />
+        <geometry>
+          <sphere radius="0.03" />
+        </geometry>
+        <material name="${name}_visual_antenna_material">
+          <color rgba="0.7 0.7 0.7 1.0" />
+        </material>
+      </visual>
+    </link>
     <joint name="${name}_joint" type="fixed">
       <origin xyz="${x} ${y} ${z}" rpy="${R} ${P} ${Y}" />

File: wamv_gazebo/urdf/sensors/wamv_imu.xacro (robot description, xacro)
@@ -1,6 +1,15 @@
 <?xml version="1.0"?>
 <robot xmlns:xacro="http://ros.org/wiki/xacro">
-  <xacro:macro name="wamv_imu" params="name:=imu x:=0 y:=0 z:=1.5 R:=0 P:=0 Y:=0">
-    <link name="${name}_link"/>
+  <xacro:macro name="wamv_imu" params="name:=imu x:=0 y:=0 z:=1.3 R:=0 P:=0 Y:=0">
+    <link name="${name}_link">
+      <visual name="${name}_visual">>
+        <geometry>
+          <box size="0.05 0.025 0.005" />
+        </geometry>
+        <material name="${name}_visual_material">
+          <color rgba="1.0 0.0 00 1.0" />
+        </material>
+      </visual>
+    </link>
     <joint name="${name}_joint" type="fixed">
       <origin xyz="${x} ${y} ${z}" rpy="${R} ${P} ${Y}"/>

File: wamv_gazebo/urdf/sensors/wamv_multibeam_laser.xacro (robot description, xacro)
@@ -1,6 +1,15 @@
 <?xml version="1.0" encoding="UTF-8"?>
 <robot xmlns:xacro="http://ros.org/wiki/xacro">
-  <xacro:macro name="wamv_multibeam_laser" params="name x:=0 y:=0 z:=0.5 R:=0 P:=0 Y:=0">
-      <link name="${name}_link" />
+  <xacro:macro name="wamv_multibeam_laser" params="name x:=0.5 y:=0 z:=1.35 R:=0 P:=0 Y:=0">
+    <link name="${name}_link">
+      <visual name="${name}_visual">>
+        <geometry>
+          <cylinder radius="0.025" length="0.1" />
+        </geometry>
+        <material name="${name}_visual_material">
+          <color rgba="0.5 1.0 0.5 1.0" />
+        </material>
+      </visual>
+    </link>
     <joint name="${name}_joint" type="fixed">
       <origin xyz="${x} ${y} ${z}" rpy="${R} ${P} ${Y}" />

Commit message: Red placards and rearrange a bit the sensors.

File: wamv_gazebo/urdf/sensors/wamv_camera.xacro (robot description, xacro)
@@ -1,5 +1,5 @@
 <?xml version="1.0"?>
 <robot xmlns:xacro="http://ros.org/wiki/xacro">
-  <xacro:macro name="wamv_camera" params="name x:=0.5 y:=0 z:=1.5 R:=0 P:=0 Y:=0">
+  <xacro:macro name="wamv_camera" params="name x:=0.5 y:=0 z:=1.4 R:=0 P:=0 Y:=0">
     <link name="${name}_link">
       <visual name="${name}_visual">

File: wamv_gazebo/urdf/sensors/wamv_planar_lidar.xacro (robot description, xacro)
@@ -1,5 +1,5 @@
 <?xml version="1.0" encoding="UTF-8"?>
 <robot xmlns:xacro="http://ros.org/wiki/xacro">
-  <xacro:macro name="wamv_multibeam_laser" params="name x:=0.5 y:=0 z:=1.5 R:=0 P:=0 Y:=0">
+  <xacro:macro name="wamv_multibeam_laser" params="name x:=1 y:=0 z:=1.5 R:=0 P:=0 Y:=0">
     <link name="${name}_link">
       <visual name="${name}_visual">>

File: wamv_gazebo/urdf/wamv_gazebo.urdf.xacro (robot description, xacro)
@@ -59,6 +59,6 @@
   <xacro:wamv_multibeam_laser name="planar_lidar" />
   <!-- Add simulated GPS -->
-  <xacro:wamv_gps name="gps_wamv" y="0.2" />
+  <!-- <xacro:wamv_gps name="gps_wamv" y="0.2" /> -->
   <!-- Add Simulated IMU -->
-  <xacro:wamv_imu name="imu_wamv" y="-0.2" />
+  <!-- <xacro:wamv_imu name="imu_wamv" y="-0.2" /> -->
 </robot>

Commit message: Add mono_camera mesh to urdf file and onto WAM-V

File: wamv_gazebo/urdf/sensors/wamv_camera.xacro (robot description, xacro)
@@ -1,16 +1,35 @@
 <?xml version="1.0"?>
 <robot xmlns:xacro="http://ros.org/wiki/xacro">
-  <xacro:macro name="wamv_camera" params="name x:=0.5 y:=0 z:=1.5 R:=0 P:=0 Y:=0">
+  <xacro:macro name="wamv_camera" params="name x:=0.5 y:=0 z:=1.5 R:=0 P:=0 Y:=${-pi/2}">
     <link name="${name}_link">
       <visual name="${name}_visual">
-        <xacro:property name="visual_length" value="0.05" />
-        <origin xyz="-${visual_length/2.0} 0 0" rpy="0 1.57 0" />
+        <origin xyz="0 -0.033 0" rpy="0 0 ${pi}"/>
         <geometry>
-          <cylinder radius="0.01" length="${visual_length}" />
+          <mesh filename="package://vrx_gazebo/models/mono_camera/mesh/mono_camera.dae"/>
         </geometry>
-        <material name="${name}_visual_material">
-          <color rgba="1.0 1.0 0.0 1.0" />
-        </material>
       </visual>
+      <collision name="${name}_lens_collision">
+        <origin xyz="0 0.018 0" rpy="1.57 0 0"/>
+        <geometry>
+          <cylinder radius="0.015" length="0.042"/>
+        </geometry>
+      </collision>
+      <collision name="${name}_box_collision">
+        <origin xyz="0 -0.0205 0" rpy="0 0 0"/>
+        <geometry>
+          <box size="0.03 0.036 0.03"/>
+        </geometry>
+      </collision>
+      <!-- Model inertia as box with <size>0.03 0.078 0.03</size> -->
+      <inertial>
+        <mass value="0.3"/>
+        <inertia
+          ixx="0.0001746"
+          iyy="0.0000450"
+          izz="0.0001746"
+          ixy="0"
+          ixz="0"
+          iyz="0"/>
+      </inertial>
     </link>
     <joint name="${name}_joint" type="fixed">

File: wamv_gazebo/urdf/wamv_gazebo.urdf.xacro (robot description, xacro)
@@ -60,5 +60,5 @@
   <!-- Add a front camera -->
   <xacro:if value="$(arg camera_enabled)">
-    <xacro:wamv_camera name="front_camera" y="0.3" x="0.75" P="${radians(15)}" />
+    <xacro:wamv_camera name="front_camera"/>
   </xacro:if>
   <!-- Add simulated GPS -->

Commit message: Integrate sensor post to camera urdf, with height parameter

File: wamv_gazebo/urdf/sensors/wamv_camera.xacro (robot description, xacro)
@@ -1,5 +1,6 @@
 <?xml version="1.0"?>
 <robot xmlns:xacro="http://ros.org/wiki/xacro">
-  <xacro:macro name="wamv_camera" params="name x:=0.5 y:=0 z:=1.5 R:=0 P:=0 Y:=${-pi/2}">
+  <xacro:macro name="wamv_camera" params="name x:=0.5 y:=0 z:=1.5 R:=0 P:=0 Y:=${-pi/2} height:=0.25">
+    <!-- Monocular Camera -->
     <link name="${name}_link">
       <visual name="${name}_visual">
@@ -33,14 +34,72 @@
       </inertial>
     </link>
-    <joint name="${name}_joint" type="fixed">
-      <origin xyz="${x} ${y} ${z}" rpy="${R} ${P} ${Y}"/>
-      <parent link="base_link"/>
-      <child link="${name}_link"/>
+    <!-- Sensor post -->
+    <link name="${name}_post_link">
+      <visual name="${name}_post_visual">
+        <origin xyz="0 0 -0.2515" rpy="${pi/2} 0 0"/>
+        <geometry>
+          <mesh filename="package://vrx_gazebo/models/sensor_post/mesh/sensor_post.dae"/>
+        </geometry>
+      </visual>
+      <collision name="${name}_post_collision">
+        <geometry>
+          <cylinder radius="0.0076" length="0.503"/>
+        </geometry>
+      </collision>
+      <inertial>
+        <mass value="0.5"/>
+        <inertia
+          ixx="0.010549261666667"
+          iyy="0.010549261666667"
+          izz="0.000014440000000"
+          ixy="0"
+          ixz="0"
+          iyz="0"/>
+      </inertial>
+    </link>
+    <!-- Sensor post arm -->
+    <link name="${name}_post_arm_link">
+      <visual name="${name}_post_arm_visual">
+        <origin xyz="0 -0.016 -0.035" rpy="0 0 0"/>
+        <geometry>
+          <mesh filename="package://vrx_gazebo/models/sensor_post/mesh/sensor_post_arm.dae"/>
+        </geometry>
+      </visual>
+      <collision name="${name}_post_arm_collision">
+        <origin xyz="0 0 0" rpy="${-pi/20} 0 0"/>
+        <geometry>
+          <cylinder radius="0.008" length="0.065"/>
+        </geometry>
+      </collision>
+      <inertial>
+        <origin xyz="0 0 0" rpy="${-pi/20} 0 0"/>
+        <mass value="0.1"/>
+        <inertia
+          ixx="0.00003680833"
+          iyy="0.00003680833"
+          izz="0.00000320000"
+          ixy="0"
+          ixz="0"
+          iyz="0"/>
+      </inertial>
+    </link>
+    <!-- Base to sensor post joint -->
+    <joint name="base_to_${name}_post_joint" type="fixed">
+      <origin xyz="${x} ${y} ${z}" rpy="${R} ${P} ${Y}" />
+      <parent link="base_link" />
+      <child link="${name}_post_link" />
     </joint>
-    <link name="${name}_link_optical" />
-    <joint name="${name}_optical_joint" type="fixed">
-      <origin xyz="0 0 0" rpy="${-pi/2} 0 ${-pi/2}" />
-      <parent link="${name}_link"/>
-      <child link="${name}_link_optical"/>
+    <!-- Sensor post to sensor post arm joint -->
+    <joint name="${name}_post_to_${name}_post_arm_joint" type="fixed">
+      <origin xyz="0 0.03 ${height}" rpy="${-pi/3} 0 0" />
+      <parent link="${name}_post_link" />
+      <child link="${name}_post_arm_link" />
+    </joint>
+    <!-- Sensor post arm to camera joint -->
+    <joint name="${name}_post_arm_to_${name}_lidar_joint" type="fixed">
+      <!-- rpy="${pi/3} 0 0" for flat camera -->
+      <origin xyz="0 -0.015 0.035" rpy="${pi/3-radians(15)} 0 0" />
+      <parent link="${name}_post_arm_link" />
+      <child link="${name}_link" />
     </joint>
     <gazebo reference="${name}_link">

File: wamv_gazebo/urdf/wamv_gazebo.urdf.xacro (robot description, xacro)
@@ -84,8 +84,8 @@
     <xacro:cpu_cases position="-0.15 0 1.53" orientation="0 0 0"/>
     <!-- Add a stereo camera pair -->
-    <xacro:wamv_camera name="front_left_camera" y="0.1" x="0.75" P="${radians(15)}" />
-    <xacro:wamv_camera name="front_right_camera" y="-0.1" x="0.75" P="${radians(15)}" />
+    <xacro:wamv_camera name="front_left_camera" y="0.1" x="0.75"/>
+    <xacro:wamv_camera name="front_right_camera" y="-0.1" x="0.75"/>
     <!-- Add a camera facing right -->
-    <xacro:wamv_camera name="middle_right_camera" y="-0.45" P="${radians(15)}" Y="${radians(-90)}" />
+    <xacro:wamv_camera name="middle_right_camera" y="-0.45" Y="${radians(-90)}" />
     <!-- Add simulated GPS -->
     <xacro:wamv_gps name="gps_wamv" x="-0.85" />

Commit message: Add adjustment link and joint to make the camera frame match base frame

File: wamv_gazebo/urdf/sensors/wamv_camera.xacro (robot description, xacro)
@@ -96,9 +96,16 @@
       <child link="${name}_post_arm_link" />
     </joint>
+    <!-- Adjustment joint -->
+    <link name="adjustment_link"/>
+    <joint name="adjustment_joint" type="fixed">
+      <origin xyz="0 0 0" rpy="${pi/3} 0 0" />
+      <parent link="${name}_post_arm_link" />
+      <child link="adjustment_link" />
+    </joint>
     <!-- Sensor post arm to camera joint -->
     <joint name="${name}_post_arm_to_${name}_lidar_joint" type="fixed">
       <!-- rpy="${pi/3} 0 0" for flat camera -->
-      <origin xyz="0 -0.015 0.035" rpy="${pi/3-radians(15)} 0 0" />
-      <parent link="${name}_post_arm_link" />
+      <origin xyz="0 0.02 0.03" rpy="${-radians(15)} 0 ${pi}" />
+      <parent link="adjustment_link" />
       <child link="${name}_link" />
     </joint>

Commit message: Simplify all transformations: base->post->arm->camera

File: wamv_gazebo/urdf/sensors/wamv_camera.xacro (robot description, xacro)
@@ -1,9 +1,9 @@
 <?xml version="1.0"?>
 <robot xmlns:xacro="http://ros.org/wiki/xacro">
-  <xacro:macro name="wamv_camera" params="name x:=0.5 y:=0 z:=1.5 R:=0 P:=0 Y:=${-pi/2} height:=0.25">
+  <xacro:macro name="wamv_camera" params="name x:=0.5 y:=0 z:=1.5 R:=0 P:=0 Y:=0 post_Y:=0">
     <!-- Monocular Camera -->
     <link name="${name}_link">
       <visual name="${name}_visual">
-        <origin xyz="0 -0.033 0" rpy="0 0 ${pi}"/>
+        <origin xyz="-0.033 0 0" rpy="0 0 ${pi/2}"/>
         <geometry>
           <mesh filename="package://vrx_gazebo/models/mono_camera/mesh/mono_camera.dae"/>
@@ -11,5 +11,5 @@
       </visual>
       <collision name="${name}_lens_collision">
-        <origin xyz="0 0.018 0" rpy="1.57 0 0"/>
+        <origin xyz="0.018 0 0" rpy="0 ${pi/2} 0"/>
         <geometry>
           <cylinder radius="0.015" length="0.042"/>
@@ -17,15 +17,15 @@
       </collision>
       <collision name="${name}_box_collision">
-        <origin xyz="0 -0.0205 0" rpy="0 0 0"/>
+        <origin xyz="-0.0205 0 0" rpy="0 0 0"/>
         <geometry>
-          <box size="0.03 0.036 0.03"/>
+          <box size="0.036 0.03 0.03"/>
         </geometry>
       </collision>
-      <!-- Model inertia as box with <size>0.03 0.078 0.03</size> -->
+      <!-- Model inertia as box with <size>0.078 0.03 0.03</size> -->
       <inertial>
         <mass value="0.3"/>
         <inertia
-          ixx="0.0001746"
-          iyy="0.0000450"
+          ixx="0.0000450"
+          iyy="0.0001746"
           izz="0.0001746"
           ixy="0"
@@ -61,5 +61,5 @@
     <link name="${name}_post_arm_link">
       <visual name="${name}_post_arm_visual">
-        <origin xyz="0 -0.016 -0.035" rpy="0 0 0"/>
+        <origin xyz="-0.038 0 -0.003" rpy="${radians(-60)} 0 ${-pi/2}"/>
         <geometry>
           <mesh filename="package://vrx_gazebo/models/sensor_post/mesh/sensor_post_arm.dae"/>
@@ -67,5 +67,5 @@
       </visual>
       <collision name="${name}_post_arm_collision">
-        <origin xyz="0 0 0" rpy="${-pi/20} 0 0"/>
+        <origin xyz="0 0 0" rpy="${radians(-60)-pi/20} 0 ${-pi/2}"/>
         <geometry>
           <cylinder radius="0.008" length="0.065"/>
@@ -73,5 +73,5 @@
       </collision>
       <inertial>
-        <origin xyz="0 0 0" rpy="${-pi/20} 0 0"/>
+        <origin xyz="0 0 0" rpy="${radians(-60)-pi/20} 0 ${-pi/2}"/>
         <mass value="0.1"/>
         <inertia
@@ -86,5 +86,5 @@
     <!-- Base to sensor post joint -->
     <joint name="base_to_${name}_post_joint" type="fixed">
-      <origin xyz="${x} ${y} ${z}" rpy="${R} ${P} ${Y}" />
+      <origin xyz="${x-(0.03+0.02)*cos(post_Y)} ${y-(0.03+0.02)*sin(post_Y)} 1.545" rpy="0 0 ${post_Y}" />
       <parent link="base_link" />
       <child link="${name}_post_link" />
@@ -92,20 +92,12 @@
     <!-- Sensor post to sensor post arm joint -->
     <joint name="${name}_post_to_${name}_post_arm_joint" type="fixed">
-      <origin xyz="0 0.03 ${height}" rpy="${-pi/3} 0 0" />
+      <origin xyz="0.03 0 ${z-1.545-0.05}" rpy="0 0 0" />
       <parent link="${name}_post_link" />
       <child link="${name}_post_arm_link" />
     </joint>
-    <!-- Adjustment joint -->
-    <link name="adjustment_link"/>
-    <joint name="adjustment_joint" type="fixed">
-      <origin xyz="0 0 0" rpy="${pi/3} 0 0" />
+    <!-- Sensor post arm to camera joint -->
+    <joint name="${name}_post_arm_to_${name}_joint" type="fixed">
+      <origin xyz="0.02 0 0.027" rpy="${R} ${P} ${Y-post_Y}" />
       <parent link="${name}_post_arm_link" />
-      <child link="adjustment_link" />
-    </joint>
-    <!-- Sensor post arm to camera joint -->
-    <joint name="${name}_post_arm_to_${name}_lidar_joint" type="fixed">
-      <!-- rpy="${pi/3} 0 0" for flat camera -->
-      <origin xyz="0 0.02 0.03" rpy="${-radians(15)} 0 ${pi}" />
-      <parent link="adjustment_link" />
       <child link="${name}_link" />
     </joint>

File: wamv_gazebo/urdf/wamv_gazebo.urdf.xacro (robot description, xacro)
@@ -60,5 +60,5 @@
   <!-- Add a front camera -->
   <xacro:if value="$(arg camera_enabled)">
-    <xacro:wamv_camera name="front_camera"/>
+    <xacro:wamv_camera name="front_camera" y="0.3" x="0.75" P="${radians(15)}"/>
   </xacro:if>
   <!-- Add simulated GPS -->
@@ -84,8 +84,8 @@
     <xacro:cpu_cases position="-0.15 0 1.53" orientation="0 0 0"/>
     <!-- Add a stereo camera pair -->
-    <xacro:wamv_camera name="front_left_camera" y="0.1" x="0.75"/>
-    <xacro:wamv_camera name="front_right_camera" y="-0.1" x="0.75"/>
+    <xacro:wamv_camera name="front_left_camera" y="0.1" x="0.75" P="${radians(15)}"/>
+    <xacro:wamv_camera name="front_right_camera" y="-0.1" x="0.75" P="${radians(15)}"/>
     <!-- Add a camera facing right -->
-    <xacro:wamv_camera name="middle_right_camera" y="-0.45" Y="${radians(-90)}" />
+    <xacro:wamv_camera name="middle_right_camera" y="-0.45" P="${radians(15)}" Y="${radians(-90)}" post_Y="${radians(-90)}"/>
     <!-- Add simulated GPS -->
     <xacro:wamv_gps name="gps_wamv" x="-0.85" />

Commit message: Scale post length to better match camera height

File: wamv_gazebo/urdf/sensors/wamv_camera.xacro (robot description, xacro)
@@ -2,4 +2,8 @@
 <robot xmlns:xacro="http://ros.org/wiki/xacro">
   <xacro:macro name="wamv_camera" params="name x:=0.5 y:=0 z:=1.5 R:=0 P:=0 Y:=0 post_Y:=0">
+    <xacro:property name="platform_z" value="1.2965"/>
+    <xacro:property name="post_arm_to_camera_z_offset" value="0.027"/>
+    <xacro:property name="mesh_post_length" value="0.503"/>
+    <xacro:property name="post_length" value="${z-platform_z-post_arm_to_camera_z_offset}"/>
     <!-- Monocular Camera -->
     <link name="${name}_link">
@@ -37,12 +41,12 @@
     <link name="${name}_post_link">
       <visual name="${name}_post_visual">
-        <origin xyz="0 0 -0.2515" rpy="${pi/2} 0 0"/>
+        <origin xyz="0 0 ${-0.2515*post_length/mesh_post_length}" rpy="${pi/2} 0 0"/>
         <geometry>
-          <mesh filename="package://vrx_gazebo/models/sensor_post/mesh/sensor_post.dae"/>
+          <mesh filename="package://vrx_gazebo/models/sensor_post/mesh/sensor_post.dae" scale="1 ${post_length/mesh_post_length} 1"/>
         </geometry>
       </visual>
       <collision name="${name}_post_collision">
         <geometry>
-          <cylinder radius="0.0076" length="0.503"/>
+          <cylinder radius="0.0076" length="${post_length}"/>
         </geometry>
       </collision>
@@ -85,6 +89,7 @@
     </link>
     <!-- Base to sensor post joint -->
+    <xacro:property name="post_z" value="${platform_z+post_length/2}"/>
     <joint name="base_to_${name}_post_joint" type="fixed">
-      <origin xyz="${x-(0.03+0.02)*cos(post_Y)} ${y-(0.03+0.02)*sin(post_Y)} 1.545" rpy="0 0 ${post_Y}" />
+      <origin xyz="${x-(0.03+0.02)*cos(post_Y)} ${y-(0.03+0.02)*sin(post_Y)} ${post_z}" rpy="0 0 ${post_Y}" />
       <parent link="base_link" />
       <child link="${name}_post_link" />
@@ -92,5 +97,5 @@
     <!-- Sensor post to sensor post arm joint -->
     <joint name="${name}_post_to_${name}_post_arm_joint" type="fixed">
-      <origin xyz="0.03 0 ${z-1.545-0.05}" rpy="0 0 0" />
+      <origin xyz="0.03 0 ${z-post_z-post_arm_to_camera_z_offset}" rpy="0 0 0" />
       <parent link="${name}_post_link" />
       <child link="${name}_post_arm_link" />
@@ -98,5 +103,5 @@
     <!-- Sensor post arm to camera joint -->
     <joint name="${name}_post_arm_to_${name}_joint" type="fixed">
-      <origin xyz="0.02 0 0.027" rpy="${R} ${P} ${Y-post_Y}" />
+      <origin xyz="0.02 0 ${post_arm_to_camera_z_offset}" rpy="${R} ${P} ${Y-post_Y}" />
       <parent link="${name}_post_arm_link" />
       <child link="${name}_link" />
