Commit message: Define positioning variables for improved clarity

File: wamv_gazebo/urdf/sensors/wamv_camera.xacro (robot description, xacro)
@@ -2,8 +2,12 @@
 <robot xmlns:xacro="http://ros.org/wiki/xacro">
   <xacro:macro name="wamv_camera" params="name x:=0.5 y:=0 z:=1.5 R:=0 P:=0 Y:=0 post_Y:=0">
+    <!-- Define length variables for link positioning -->
     <xacro:property name="platform_z" value="1.2965"/>
-    <xacro:property name="post_arm_to_camera_z_offset" value="0.027"/>
+    <xacro:property name="post_to_post_arm_x" value="0.03"/>
+    <xacro:property name="post_arm_to_camera_x" value="0.02"/>
+    <xacro:property name="post_arm_to_camera_z" value="0.027"/>
+    <!-- Define post length based on desired z position of sensor -->
+    <xacro:property name="post_length" value="${z-platform_z-post_arm_to_camera_z}"/>
     <xacro:property name="mesh_post_length" value="0.503"/>
-    <xacro:property name="post_length" value="${z-platform_z-post_arm_to_camera_z_offset}"/>
     <!-- Monocular Camera -->
     <link name="${name}_link">
@@ -91,5 +95,5 @@
     <xacro:property name="post_z" value="${platform_z+post_length/2}"/>
     <joint name="base_to_${name}_post_joint" type="fixed">
-      <origin xyz="${x-(0.03+0.02)*cos(post_Y)} ${y-(0.03+0.02)*sin(post_Y)} ${post_z}" rpy="0 0 ${post_Y}" />
+      <origin xyz="${x-(post_to_post_arm_x+post_arm_to_camera_x)*cos(post_Y)} ${y-(post_to_post_arm_x+post_arm_to_camera_x)*sin(post_Y)} ${post_z}" rpy="0 0 ${post_Y}" />
       <parent link="base_link" />
       <child link="${name}_post_link" />
@@ -97,5 +101,5 @@
     <!-- Sensor post to sensor post arm joint -->
     <joint name="${name}_post_to_${name}_post_arm_joint" type="fixed">
-      <origin xyz="0.03 0 ${z-post_z-post_arm_to_camera_z_offset}" rpy="0 0 0" />
+      <origin xyz="${post_to_post_arm_x} 0 ${z-post_z-post_arm_to_camera_z}" rpy="0 0 0" />
       <parent link="${name}_post_link" />
       <child link="${name}_post_arm_link" />
@@ -103,5 +107,5 @@
     <!-- Sensor post arm to camera joint -->
     <joint name="${name}_post_arm_to_${name}_joint" type="fixed">
-      <origin xyz="0.02 0 ${post_arm_to_camera_z_offset}" rpy="${R} ${P} ${Y-post_Y}" />
+      <origin xyz="${post_arm_to_camera_x} 0 ${post_arm_to_camera_z}" rpy="${R} ${P} ${Y-post_Y}" />
       <parent link="${name}_post_arm_link" />
       <child link="${name}_link" />

Commit message: Change from visual mesh to cylinder, but color not working. Stil showing white

File: wamv_gazebo/urdf/sensors/wamv_camera.xacro (robot description, xacro)
@@ -45,8 +45,10 @@
     <link name="${name}_post_link">
       <visual name="${name}_post_visual">
-        <origin xyz="0 0 ${-0.2515*post_length/mesh_post_length}" rpy="${pi/2} 0 0"/>
         <geometry>
-          <mesh filename="package://vrx_gazebo/models/sensor_post/mesh/sensor_post.dae" scale="1 ${post_length/mesh_post_length} 1"/>
+          <cylinder radius="0.0076" length="${post_length}"/>
         </geometry>
+        <material name="${name}_post_material">
+          <color rgba="1.0 0.0 0.0 1.0"/>
+        </material>
       </visual>
       <collision name="${name}_post_collision">

Commit message: Add gazebo tag for color, still not working

File: wamv_gazebo/urdf/sensors/wamv_camera.xacro (robot description, xacro)
@@ -9,5 +9,4 @@
     <!-- Define post length based on desired z position of sensor -->
     <xacro:property name="post_length" value="${z-platform_z-post_arm_to_camera_z}"/>
-    <xacro:property name="mesh_post_length" value="0.503"/>
     <!-- Monocular Camera -->
     <link name="${name}_link">
@@ -49,5 +48,5 @@
         </geometry>
         <material name="${name}_post_material">
-          <color rgba="1.0 0.0 0.0 1.0"/>
+          <color rgba="0.0 0.0 0.0 1.0"/>
         </material>
       </visual>
@@ -152,4 +151,7 @@
       </sensor>
     </gazebo>
+    <gazebo reference="${name}_post_link">
+      <material>Gazebo/Black</material>
+    </gazebo>
   </xacro:macro>
 </robot>

Commit message: Fix post color issue by removing <visual> tag name

File: wamv_gazebo/urdf/sensors/wamv_camera.xacro (robot description, xacro)
@@ -43,5 +43,5 @@
     <!-- Sensor post -->
     <link name="${name}_post_link">
-      <visual name="${name}_post_visual">
+      <visual>
         <geometry>
           <cylinder radius="0.0076" length="${post_length}"/>
@@ -112,4 +112,5 @@
       <child link="${name}_link" />
     </joint>
+    <!-- Gazebo camera setup -->
     <gazebo reference="${name}_link">
       <sensor type="camera" name="${name}_sensor">
@@ -151,4 +152,5 @@
       </sensor>
     </gazebo>
+    <!-- Set color of post -->
     <gazebo reference="${name}_post_link">
       <material>Gazebo/Black</material>

Commit message: Vary post mass as length changes

File: wamv_gazebo/urdf/sensors/wamv_camera.xacro (robot description, xacro)
@@ -7,6 +7,4 @@
     <xacro:property name="post_arm_to_camera_x" value="0.02"/>
     <xacro:property name="post_arm_to_camera_z" value="0.027"/>
-    <!-- Define post length based on desired z position of sensor -->
-    <xacro:property name="post_length" value="${z-platform_z-post_arm_to_camera_z}"/>
     <!-- Monocular Camera -->
     <link name="${name}_link">
@@ -41,4 +39,9 @@
       </inertial>
     </link>
+    <!-- Define post length and mass based on desired z position of sensor -->
+    <xacro:property name="post_length" value="${z-platform_z-post_arm_to_camera_z}"/>
+    <xacro:property name="post_mass_per_meter" value="0.9"/>
+    <xacro:property name="post_mass" value="${post_mass_per_meter * post_length}"/>
+    <xacro:property name="post_radius" value="0.0076"/>
     <!-- Sensor post -->
     <link name="${name}_post_link">
@@ -53,13 +56,13 @@
       <collision name="${name}_post_collision">
         <geometry>
-          <cylinder radius="0.0076" length="${post_length}"/>
+          <cylinder radius="${post_radius}" length="${post_length}"/>
         </geometry>
       </collision>
       <inertial>
-        <mass value="0.5"/>
+        <mass value="${post_mass}"/>
         <inertia
-          ixx="0.010549261666667"
-          iyy="0.010549261666667"
-          izz="0.000014440000000"
+          ixx="${(post_mass/12) * (3*post_radius*post_radius + post_length*post_length)}"
+          iyy="${(post_mass/12) * (3*post_radius*post_radius + post_length*post_length)}"
+          izz="${(post_mass/2) * (post_radius*post_radius)}"
           ixy="0"
           ixz="0"

Commit message: Update sensor model with sensor optical frame *Add name_link_optical joint to match tf frame *Add joint that encodes transform between sensor and optical frame *Modify sensor frame to add namespace.  This ensures compatibility with localisation example

File: wamv_gazebo/urdf/sensors/wamv_camera.xacro (robot description, xacro)
@@ -38,4 +38,8 @@
           iyz="0"/>
       </inertial>
+    </link>
+    <!-- Define a link for the optical frame.  This will match the sensor frame and
+         be oriented in the camera convention. -->
+    <link name="${name}_link_optical">
     </link>
     <!-- Define post length and mass based on desired z position of sensor -->
@@ -116,4 +120,11 @@
       <child link="${name}_link" />
     </joint>
+    <!-- Camera to optical frame joint.  This is oriented to convert between ENU
+         and camera conventions -->
+    <joint name="${name}_to_${name}_link_optical_joint" type="fixed">
+      <origin xyz="0 0 0" rpy="${-pi/2} 0 ${-pi/2}" />
+      <parent link="${name}_link" />
+      <child link="${name}_link_optical" />
+    </joint>
     <!-- Gazebo camera setup -->
     <gazebo reference="${name}_link">
@@ -146,5 +157,5 @@
           <imageTopicName>image_raw</imageTopicName>
           <cameraInfoTopicName>camera_info</cameraInfoTopicName>
-          <frameName>${name}_link_optical</frameName>
+          <frameName>${namespace}/${name}_link_optical</frameName>
           <hackBaseline>0.07</hackBaseline>
           <distortionK1>0.0</distortionK1>

Commit message: Remove extra space
Signed-off-by: Carlos Agüero <caguero@openrobotics.org>

File: wamv_gazebo/urdf/sensors/wamv_camera.xacro (robot description, xacro)
@@ -1,5 +1,5 @@
 <?xml version="1.0"?>
 <robot xmlns:xacro="http://ros.org/wiki/xacro">
-  <xacro:macro name="wamv_camera" params="name x:=0.5 y:=0 z:=1.5 post_z_from:=1.2965  R:=0 P:=0 Y:=0 post_Y:=0">
+  <xacro:macro name="wamv_camera" params="name x:=0.5 y:=0 z:=1.5 post_z_from:=1.2965 R:=0 P:=0 Y:=0 post_Y:=0">
     <!-- Define length variables for link positioning -->
     <xacro:property name="platform_z" value="${post_z_from}"/>

Commit message: Extra parameter to set the height of the post's base in sensors (#221)
* Adding extra parameter to set the height of the post's base.

Signed-off-by: Carlos Agüero <caguero@openrobotics.org>

* Remove extra space

Signed-off-by: Carlos Agüero <caguero@openrobotics.org>

File: wamv_gazebo/urdf/sensors/wamv_camera.xacro (robot description, xacro)
@@ -1,7 +1,7 @@
 <?xml version="1.0"?>
 <robot xmlns:xacro="http://ros.org/wiki/xacro">
-  <xacro:macro name="wamv_camera" params="name x:=0.5 y:=0 z:=1.5 R:=0 P:=0 Y:=0 post_Y:=0">
+  <xacro:macro name="wamv_camera" params="name x:=0.5 y:=0 z:=1.5 post_z_from:=1.2965 R:=0 P:=0 Y:=0 post_Y:=0">
     <!-- Define length variables for link positioning -->
-    <xacro:property name="platform_z" value="1.2965"/>
+    <xacro:property name="platform_z" value="${post_z_from}"/>
     <xacro:property name="post_to_post_arm_x" value="0.03"/>
     <xacro:property name="post_arm_to_camera_x" value="0.02"/>

Commit message: Added namespace to gazebo references, return color to camera posts

File: wamv_gazebo/urdf/sensors/wamv_camera.xacro (robot description, xacro)
@@ -168,5 +168,5 @@
     </gazebo>
     <!-- Set color of post -->
-    <gazebo reference="${name}_post_link">
+    <gazebo reference="${namespace}/${name}_post_link">
       <material>Gazebo/Black</material>
     </gazebo>

File: wamv_gazebo/urdf/sensors/wamv_planar_lidar.xacro (robot description, xacro)
@@ -2,5 +2,5 @@
 <robot xmlns:xacro="http://ros.org/wiki/xacro">
   <xacro:macro name="wamv_multibeam_laser" params="name x:=0.5 y:=0 z:=2 R:=0 P:=0 Y:=0">
-    <link name="${name}_link">
+    <link name="${namespace}/${name}_link">
       <visual name="${name}_visual">>
         <geometry>
@@ -12,10 +12,10 @@
       </visual>
     </link>
-    <joint name="${name}_joint" type="fixed">
+    <joint name="${namespace}/${name}_joint" type="fixed">
       <origin xyz="${x} ${y} ${z}" rpy="${R} ${P} ${Y}" />
       <parent link="base_link" />
       <child link="${name}_link" />
     </joint>
-    <gazebo reference="${name}_link">
+    <gazebo reference="${namespace}/${name}_link">
       <sensor type="gpu_ray" name="multibeam_sensor_${name}">
         <update_rate>10</update_rate>
@@ -40,5 +40,5 @@
         <plugin name="multibeam_simulator" filename="libgazebo_ros_gpu_laser.so">
           <topicName>${namespace}/${sensor_namespace}lidars/${name}/scan</topicName>
-          <frameName>${name}_link</frameName>
+          <frameName>${namespace}/${name}_link</frameName>
         </plugin>
       </sensor>

Commit message: Adding xacro parameter to enable Gazebo camera visualization

File: wamv_gazebo/urdf/sensors/wamv_camera.xacro (robot description, xacro)
@@ -1,5 +1,5 @@
 <?xml version="1.0"?>
 <robot xmlns:xacro="http://ros.org/wiki/xacro">
-  <xacro:macro name="wamv_camera" params="name x:=0.5 y:=0 z:=1.5 post_z_from:=1.2965 R:=0 P:=0 Y:=0 post_Y:=0">
+  <xacro:macro name="wamv_camera" params="name x:=0.5 y:=0 z:=1.5 post_z_from:=1.2965 R:=0 P:=0 Y:=0 post_Y:=0 visualize:=False">
     <!-- Define length variables for link positioning -->
     <xacro:property name="platform_z" value="${post_z_from}"/>
@@ -131,4 +131,7 @@
       <sensor type="camera" name="${name}_sensor">
         <update_rate>30.0</update_rate>
+	<xacro:if value="${visualize}">
+	  <visualize>true</visualize>
+	</xacro:if>
         <camera name="${name}_camera">
           <horizontal_fov>1.3962634</horizontal_fov>
