Commit message: Vehicle locked during 'initial' and released during 'ready'.

File: vmrc_gazebo/worlds/navigation_task.world.xacro (robot description, xacro)
@@ -129,4 +129,12 @@
       <max_time>10</max_time>
       <vehicle>wamv</vehicle>
+      <release_joints>
+        <joint>
+          <name>wamv_external_pivot_joint</name>
+        </joint>
+        <joint>
+          <name>wamv_external_riser</name>
+        </joint>
+      </release_joints>
       <gates>
         <gate>
