Commit message: first prototype of station keeping plugin - blank for now

File: vmrc_gazebo/worlds/stationkeeping_task.world.xacro (robot description, xacro)
@@ -5,4 +5,20 @@
     <xacro:include filename="$(find vmrc_gazebo)/worlds/sandisland.xacro" />
     <xacro:sandisland />
+	<plugin name="stationkeeping_scoring_plugin"
+            filename="stationkeeping_scoring_plugin.so">
+      <vehicle>wamv</vehicle>
+      <task_name>navigation_course</task_name>
+      <initial_state_duration>10</initial_state_duration>
+      <ready_state_duration>10</ready_state_duration>
+      <running_state_duration>300</running_state_duration>
+      <release_joints>
+        <joint>
+          <name>wamv_external_pivot_joint</name>
+        </joint>
+        <joint>
+          <name>wamv_external_riser</name>
+        </joint>
+      </release_joints>
+    </plugin>
   </world>
 </sdf>
