Commit message: Checking the dock condition.

File: vmrc_gazebo/worlds/find_symbols_and_dock.world.xacro (robot description, xacro)
@@ -15,4 +15,32 @@
       <pose>60 -2.75 0 0 0 0</pose>
     </include>
+    <model name="activation_placard1">
+      <static>true</static>
+      <link name="link">
+        <visual name="visual">
+          <pose>72.75 0 0 0 0 0</pose>
+          <geometry>
+            <box>
+              <size>1.5 4 2</size>
+            </box>
+          </geometry>
+          <transparency>0.8</transparency>
+        </visual>
+      </link>
+    </model>
+    <model name="activation_placard2">
+      <static>true</static>
+      <link name="link">
+        <visual name="visual">
+          <pose>61.75 0 0 0 0 0</pose>
+          <geometry>
+            <box>
+              <size>1.5 4 2</size>
+            </box>
+          </geometry>
+          <transparency>0.8</transparency>
+        </visual>
+      </link>
+    </model>
     <!-- The scoring plugin -->
     <plugin name="scan_dock_scoring_plugin"
@@ -20,6 +48,6 @@
       <vehicle>wamv</vehicle>
       <task_name>scan_dock</task_name>
-      <initial_state_duration>10</initial_state_duration>
-      <ready_state_duration>10</ready_state_duration>
+      <initial_state_duration>3</initial_state_duration>
+      <ready_state_duration>3</ready_state_duration>
       <running_state_duration>300</running_state_duration>
       <release_joints>
@@ -31,9 +59,32 @@
         </joint>
       </release_joints>
-      <color_1>RED</color_1>
-      <color_2>GREEN</color_2>
-      <color_3>BLUE</color_3>
+      <color_1>red</color_1>
+      <color_2>green</color_2>
+      <color_3>blue</color_3>
       <robot_namespace>vrx</robot_namespace>
       <color_sequence_service>scan_dock/color_sequence</color_sequence_service>
+      <bay1_topic>/vrx/dock_2018/bay_1/contain</bay1_topic>
+      <bay2_topic>/vrx/dock_2018/bay_2/contain</bay2_topic>
+      <correct_bay_topic>/vrx/dock_2018/bay_2/contain</correct_bay_topic>
+    </plugin>
+    <plugin name="vehicle_docked_bay1" filename="libContainPlugin.so">
+      <entity>wamv::base_link</entity>
+      <namespace>vrx/dock_2018/bay_1</namespace>
+      <pose frame="robotx_dock_2018::dock_2018_placard1::placard::link">0 -5 -1.5 0 0 0</pose>
+      <geometry>
+        <box>
+          <size>4 1.5 2</size>
+        </box>
+      </geometry>
+    </plugin>
+    <plugin name="vehicle_docked_bay2" filename="libContainPlugin.so">
+      <entity>wamv::base_link</entity>
+      <namespace>vrx/dock_2018/bay_2</namespace>
+      <pose frame="robotx_dock_2018::dock_2018_placard2::placard::link">0 5 -1.5 0 0 0</pose>
+      <geometry>
+        <box>
+          <size>4 1.5 2</size>
+        </box>
+      </geometry>
     </plugin>
   </world>
