Commit message: Prototype of population plugin - only for a single object at a time.  Moves it back to original position when done

File: vrx_gazebo/worlds/perception_task.world.xacro (robot description, xacro)
@@ -2,172 +2,45 @@
 <!-- World containing sandisland model and some course challenges -->
 <sdf version="1.6" xmlns:xacro="http://ros.org/wiki/xacro">
-  <world name="robotx_example_course">
+  <world name="perception_task_example">
     <xacro:include filename="$(find vrx_gazebo)/worlds/sandisland.xacro" />
     <xacro:sandisland />
-    <!-- Starboard_border -->
-    <include>
-        <name>red_bound_0</name>
-        <pose>-29.8874 7.80274 0 0 -0 0</pose>
-        <uri>model://surmark950410</uri>
-      </include>
-    <include>
-      <name>red_bound_1</name>
-      <pose>-51.4227 1.0515 0 0 -0 0</pose>
-      <uri>model://surmark950410</uri>
-    </include>
-    <include>
-      <name>red_bound_2</name>
-      <pose>-64.574 -13.7242 0 0 -0 0</pose>
-      <uri>model://surmark950410</uri>
-    </include>
-    <include>
-      <name>red_bound_3</name>
-      <pose>-70.5798 -30.9289 0 0 -0 0</pose>
-      <uri>model://surmark950410</uri>
-    </include>
-    <include>
-      <name>red_bound_4</name>
-      <pose>-73.2084 -44.9953 0 0 -0 0</pose>
-      <uri>model://surmark950410</uri>
-    </include>
-    <include>
-      <name>red_bound_5</name>
-      <pose>-87.3051 -43.4804 0 0 -0 0</pose>
-      <uri>model://surmark950410</uri>
-    </include>
-    <include>
-      <name>red_bound_6</name>
-      <pose>-90.539 -28.0283 0 0 -0 0</pose>
-      <uri>model://surmark950410</uri>
-    </include>
-    <!-- Port_border -->
-    <include>
-      <name>green_bound_0</name>
-      <pose>-32.2914 -10.0761 -0.2 0 -0 0</pose>
-      <uri>model://surmark950400</uri>
-    </include>
-    <include>
-      <name>green_bound_1</name>
-      <pose>-47.3915 -11.2422 -0.2 0 -0 0</pose>
-      <uri>model://surmark950400</uri>
-    </include>
-    <include>
-      <name>green_bound_2</name>
-      <pose>-50.4509 -25.1164 -0.2 0 -0 0</pose>
-      <uri>model://surmark950400</uri>
-    </include>
-    <include>
-      <name>green_bound_3</name>
-      <pose>-58.7734 -39.351 -0.2 0 -0 0</pose>
-      <uri>model://surmark950400</uri>
-    </include>
-    <include>
-      <name>green_bound_4</name>
-      <pose>-70.9557 -57.7238 -0.2 0 -0 0</pose>
-      <uri>model://surmark950400</uri>
-    </include>
-    <include>
-      <name>green_bound_5</name>
-      <pose>-95.8278 -54.0979 -0.2 0 -0 0</pose>
-      <uri>model://surmark950400</uri>
-    </include>
-    <include>
-      <name>green_bound_6</name>
-      <pose>-107.643 -29.1729 -0.2 0 -0 0</pose>
-      <uri>model://surmark950400</uri>
-    </include>
-    <!-- Obstacles -->
-    <include>
-      <name>obstacle_1</name>
-      <pose>-57.283 -28.3719 -0.2 0 -0 0</pose>
-      <uri>model://polyform_a5</uri>
-    </include>
-    <include>
-      <name>obstacle_2</name>
-      <pose>-68.6471 -41.2087 -0.2 0 -0 0</pose>
-      <uri>model://polyform_a5</uri>
-    </include>
-    <include>
-      <name>obstacle_3</name>
-      <pose>-80.2333 -48.5559 -0.2 0 -0 0</pose>
-      <uri>model://polyform_a5</uri>
-    </include>
-    <include>
-      <name>obstacle_4</name>
-      <pose>-78.842 -55.2626 -0.2 0 -0 0</pose>
-      <uri>model://polyform_a5</uri>
-    </include>
-    <include>
-      <name>obstacle_5</name>
-      <pose>-84.9105 -53.4974 -0.2 0 -0 0</pose>
-      <uri>model://polyform_a5</uri>
-    </include>
-    <include>
-      <name>obstacle_6</name>
-      <pose>-98.5759 -42.8883 -0.2 0 -0 0</pose>
-      <uri>model://polyform_a5</uri>
-    </include>
-    <include>
-      <name>obstacle_7</name>
-      <pose>-95.2334 -39.1624 -0.2 0 -0 0</pose>
-      <uri>model://polyform_a5</uri>
-    </include>
-    <include>
-      <name>obstacle_8</name>
-      <pose>-100.506 -33.524 -0.2 0 -0 0</pose>
-      <uri>model://polyform_a5</uri>
-    </include>
-    <include>
-      <name>obstacle_9</name>
-      <pose>-56.0734 -9.21053 -0.2 0 -0 0</pose>
-      <uri>model://polyform_a7</uri>
-    </include>
-    <!-- The scoring plugin -->
-    <plugin name="navigation_scoring_plugin"
-            filename="libnavigation_scoring_plugin.so">
-      <vehicle>wamv</vehicle>
-      <task_name>navigation_course</task_name>
-      <initial_state_duration>10</initial_state_duration>
-      <ready_state_duration>10</ready_state_duration>
-      <running_state_duration>300</running_state_duration>
-      <release_joints>
-        <joint>
-          <name>wamv_external_pivot_joint</name>
-        </joint>
-        <joint>
-          <name>wamv_external_riser</name>
-        </joint>
-      </release_joints>
-      <gates>
-        <gate>
-          <left_marker>red_bound_0</left_marker>
-          <right_marker>green_bound_0</right_marker>
-        </gate>
-        <gate>
-          <left_marker>red_bound_1</left_marker>
-          <right_marker>green_bound_1</right_marker>
-        </gate>
-        <gate>
-          <left_marker>red_bound_2</left_marker>
-          <right_marker>green_bound_2</right_marker>
-        </gate>
-        <gate>
-          <left_marker>red_bound_3</left_marker>
-          <right_marker>green_bound_3</right_marker>
-        </gate>
-        <gate>
-          <left_marker>red_bound_4</left_marker>
-          <right_marker>green_bound_4</right_marker>
-        </gate>
-        <gate>
-          <left_marker>red_bound_5</left_marker>
-          <right_marker>green_bound_5</right_marker>
-        </gate>
-        <gate>
-          <left_marker>red_bound_6</left_marker>
-          <right_marker>green_bound_6</right_marker>
-        </gate>
-      </gates>
-    </plugin>
+	<!-- Include all the objects we plan to use for perception.
+		 Stash them out of the field of view for now -->
+	<include>
+	  <name>red_0</name>
+	  <pose>-10 0 1 0 0 0</pose>
+	  <uri>model://surmark950410</uri>
+	</include>
+	<include>
+	  <name>green_0</name>
+	  <pose>-11 0 1 0 0 0</pose>
+	  <uri>model://surmark950400</uri>
+	</include>
+	<include>
+	  <name>black_0</name>
+	  <pose>-12 0 1 0 0 0</pose>
+	  <uri>model://black_totem</uri>
+	</include>
+	<plugin filename="libpopulation_plugin.so" name="populate_plugin">
+	  <loop_forever>false</loop_forever>
+	  <frame>wamv</frame>
+	  <object_sequence>
+		<object>
+		  <time>5.0</time>
+		  <type>red</type>
+		  <pose>6 0 1 0 0 0</pose>
+		</object>
+		<object>
+		  <time>5.0</time>
+		  <type>green</type>
+		  <pose>6 6 1 0 0 0</pose>
+		</object>
+		<object>
+		  <time>5.0</time>
+		  <type>black</type>
+		  <pose>6 -6 1 0 0 0</pose>
+		</object>
+	  </object_sequence>
+	</plugin>
   </world>
 </sdf>
