Commit message: updates xacro

File: vrx_gazebo/worlds/sandisland.world.xacro (robot description, xacro)
@@ -7,5 +7,5 @@
     <!--wind for the wamv-->
     <xacro:include filename="$(find vrx_gazebo)/worlds/xacros/wamv_gazebo_wind_plugin.xacro"/>
-    <xacro:usv_wind_gazebo>
+    <xacro:usv_wind_gazebo n="1">
       <wind_objs>
         <wind_obj>

File: vrx_gazebo/worlds/xacros/wamv_gazebo_wind_plugin.xacro (robot description, xacro)
@@ -1,6 +1,5 @@
 <?xml version="1.0"?>
 <world xmlns:xacro="http://ros.org/wiki/xacro">
-	<xacro:macro name="usv_wind_gazebo" params="n:=0
-						    **wind_objs
+	<xacro:macro name="usv_wind_gazebo" params="**wind_objs
 						    direction:=270
 						    mean_vel:=10
@@ -13,5 +12,4 @@
     <plugin name="wind" filename="libusv_gazebo_wind_plugin.so">
         <!-- models to be effected by the wind -->
-	<models_n>${n}</models_n>
 	<xacro:insert_block name="wind_objs"/>
         <!-- Wind -->
