Commit message: Tweaks.

File: vrx_gazebo/worlds/scan_and_dock_a.world.xacro (robot description, xacro)
@@ -68,13 +68,17 @@
           <name>bay1</name>
           <activation_topic>/vrx/dock_2018/bay_1/contain</activation_topic>
+          <symbol_topic>/vrx/dock_2018_placard1/symbol</symbol_topic>
           <min_dock_time>10.0</min_dock_time>
           <dock_allowed>false</dock_allowed>
+          <symbol>red_circle</symbol>
         </bay>
         <bay>
           <name>bay2</name>
           <activation_topic>/vrx/dock_2018/bay_2/contain</activation_topic>
+          <symbol_topic>/vrx/dock_2018_placard2/symbol</symbol_topic>
           <min_dock_time>10.0</min_dock_time>
           <dock_allowed>true</dock_allowed>
-          <announce_symbol>red_circle</announce_symbol>
+          <announce_symbol>red_triangle</announce_symbol>
+          <symbol>red_triangle</symbol>
         </bay>
       </bays>

File: vrx_gazebo/worlds/scan_and_dock_b.world.xacro (robot description, xacro)
@@ -74,7 +74,7 @@
           <activation_topic>/vrx/dock_2018/bay_1/contain</activation_topic>
           <symbol_topic>/vrx/dock_2018_placard1/symbol</symbol_topic>
-	  <min_dock_time>10.0</min_dock_time>
-	  <dock_allowed>false</dock_allowed>
-	  <symbol>red_circle</symbol>
+	        <min_dock_time>10.0</min_dock_time>
+	        <dock_allowed>false</dock_allowed>
+	        <symbol>red_circle</symbol>
         </bay>
         <bay>
@@ -83,6 +83,6 @@
           <symbol_topic>/vrx/dock_2018_placard2/symbol</symbol_topic>
           <min_dock_time>10.0</min_dock_time>
-	  <dock_allowed>true</dock_allowed>
-	  <symbol>red_triangle</symbol>
+	        <dock_allowed>true</dock_allowed>
+	        <symbol>red_triangle</symbol>
         </bay>
       </bays>

File: vrx_gazebo/worlds/xacros/usv_wind_plugin.xacro (robot description, xacro)
@@ -1,24 +1,25 @@
 <?xml version="1.0"?>
 <world xmlns:xacro="http://ros.org/wiki/xacro">
-  <xacro:macro name="usv_wind_gazebo" params="**wind_objs
-						    direction:=270
-						    mean_vel:=10
-						    var_gain:=100
-						    var_time:=5
-						    seed:=''
-						    ros_update_rate:=1
-						    " >
+  <xacro:macro name="usv_wind_gazebo"
+               params="**wind_objs
+                         direction:=270
+                         mean_vel:=10
+                         var_gain:=100
+                         var_time:=5
+                         seed:=''
+                         ros_update_rate:=1
+                         " >
     <!--Gazebo Plugin for simulating WAM-V dynamics-->
     <plugin name="wind" filename="libusv_gazebo_wind_plugin.so">
-        <!-- models to be effected by the wind -->
-	<xacro:insert_block name="wind_objs"/>
-        <!-- Wind -->
-	<wind_direction>${direction}</wind_direction> <!-- in degrees -->
-	<wind_mean_velocity>${mean_vel}</wind_mean_velocity>
-	<var_wind_gain_constants>${var_gain}</var_wind_gain_constants>
-	<var_wind_time_constants>${var_time}</var_wind_time_constants>
-	<random_seed>${seed}</random_seed> <!-- set to zero/empty to randomize -->
-	<update_rate>${ros_update_rate}</update_rate>
-      </plugin>
+      <!-- models to be effected by the wind -->
+      <xacro:insert_block name="wind_objs"/>
+      <!-- Wind -->
+      <wind_direction>${direction}</wind_direction> <!-- in degrees -->
+      <wind_mean_velocity>${mean_vel}</wind_mean_velocity>
+      <var_wind_gain_constants>${var_gain}</var_wind_gain_constants>
+      <var_wind_time_constants>${var_time}</var_wind_time_constants>
+      <random_seed>${seed}</random_seed> <!-- set to zero/empty to randomize -->
+      <update_rate>${ros_update_rate}</update_rate>
+    </plugin>
   </xacro:macro>
 </world>
