Commit message: Custom tweaks

File: vrx_gazebo/worlds/example_course.world.xacro (robot description, xacro)
@@ -5,5 +5,5 @@
     <xacro:include filename="$(find vrx_gazebo)/worlds/sandisland.xacro" />
     <xacro:sandisland />
-    <include>
+    <!-- <include>
       <uri>model://robotx_navigation_challenge</uri>
       <pose>15 0 2 0 0 0</pose>
@@ -16,15 +16,15 @@
       <uri>model://robotx_2016_qualifying_pinger_transit</uri>
       <pose>55 -50 0 0 0 -1.3</pose>
-    </include>
+    </include> -->
     <!-- The 2016 dock with the three placards -->
     <include>
       <uri>model://dock_2016</uri>
-      <pose>80 -8.75 0 0 0 0</pose>
+      <pose>50 -1 0 0 0 0.15</pose>
     </include>
     <!-- The 2018 dock with the two placards -->
-    <include>
+    <!-- <include>
       <uri>model://dock_2018</uri>
       <pose>120 -2.75 0 0 0 0</pose>
-    </include>
+    </include> -->
   </world>
 </sdf>

File: wamv_gazebo/urdf/sensors/wamv_planar_lidar.xacro (robot description, xacro)
@@ -1,5 +1,5 @@
 <?xml version="1.0" encoding="UTF-8"?>
 <robot xmlns:xacro="http://ros.org/wiki/xacro">
-  <xacro:macro name="wamv_multibeam_laser" params="name x:=0.5 y:=0 z:=2 R:=0 P:=0 Y:=0">
+  <xacro:macro name="wamv_multibeam_laser" params="name x:=0.5 y:=0 z:=1.5 R:=0 P:=0 Y:=0">
     <link name="${name}_link">
       <visual name="${name}_visual">>

File: wamv_gazebo/urdf/wamv_gazebo.urdf.xacro (robot description, xacro)
@@ -55,7 +55,9 @@
   </xacro:if>
   <!-- Add a front camera -->
-  <xacro:if value="$(arg camera_enabled)">
+  <!-- <xacro:if value="$(arg camera_enabled)"> -->
     <xacro:wamv_camera name="front_camera" y="0.3" x="0.75" P="${radians(15)}" />
-  </xacro:if>
+  <!-- </xacro:if> -->
+  <!-- Add 2D LIDAR -->
+  <xacro:wamv_multibeam_laser name="planar_lidar" />
   <!-- Add simulated GPS -->
   <xacro:if value="$(arg gps_enabled)">
@@ -75,16 +77,16 @@
   </xacro:if>
   <!-- ==== VRX sensor configuration ==== -->
-  <xacro:if value="$(arg vrx_sensors_enabled)">
+ <!--  <xacro:if value="$(arg vrx_sensors_enabled)"> -->
     <!-- Add a stereo camera pair -->
-    <xacro:wamv_camera name="front_left_camera" y="0.1" x="0.75" P="${radians(15)}" />
-    <xacro:wamv_camera name="front_right_camera" y="-0.1" x="0.75" P="${radians(15)}" />
+    <!-- <xacro:wamv_camera name="front_left_camera" y="0.1" x="0.75" P="${radians(15)}" />
+    <xacro:wamv_camera name="front_right_camera" y="-0.1" x="0.75" P="${radians(15)}" /> -->
     <!-- Add a camera facing right -->
-    <xacro:wamv_camera name="middle_right_camera" y="-0.45" P="${radians(15)}" Y="${radians(-90)}" />
+    <!-- <xacro:wamv_camera name="middle_right_camera" y="-0.45" P="${radians(15)}" Y="${radians(-90)}" /> -->
     <!-- Add simulated GPS -->
-    <xacro:wamv_gps name="gps_wamv" y="0.2" />
+    <!-- <xacro:wamv_gps name="gps_wamv" y="0.2" /> -->
     <!-- Add Simulated IMU -->
-    <xacro:wamv_imu name="imu_wamv" y="-0.2" />
+    <!-- <xacro:wamv_imu name="imu_wamv" y="-0.2" /> -->
     <!-- Add 3D LIDAR -->
-    <xacro:wamv_3d_lidar name="lidar_wamv" P="${radians(8)}" />
-  </xacro:if>
+    <!-- <xacro:wamv_3d_lidar name="lidar_wamv" P="${radians(8)}" /> -->
+  <!-- </xacro:if> -->
 </robot>

Commit message: Sandisland texture, sensor meshes and extra objects.

File: vrx_gazebo/worlds/example_course.world.xacro (robot description, xacro)
@@ -7,9 +7,9 @@
     <include>
       <uri>model://robotx_navigation_challenge</uri>
-      <pose>15 0 2 0 0 0</pose>
+      <pose>58 68 2 0 0 0.4</pose>
     </include>
     <include>
       <uri>model://robotx_light_buoy</uri>
-      <pose>60 0 0.25 0 0 0</pose>
+      <pose>110 28 0.25 0 0 0</pose>
     </include>
     <include>
@@ -20,10 +20,10 @@
     <include>
       <uri>model://dock_2016</uri>
-      <pose>80 -8.75 0 0 0 0</pose>
+      <pose>75 22 0 0 0 -2.78</pose>
     </include>
     <!-- The 2018 dock with the two placards -->
     <include>
       <uri>model://dock_2018</uri>
-      <pose>120 -2.75 0 0 0 0</pose>
+      <pose>-2 -18 0 0 0 0.2</pose>
     </include>
   </world>

File: vrx_gazebo/worlds/sandisland.xacro (robot description, xacro)
@@ -9,4 +9,6 @@
         </clouds>
       </sky>
+      <grid>0</grid>
+      <origin_visual>0</origin_visual>
     </scene>
     <!-- Estimated latitude/longitude of sandisland from satellite imagery -->
@@ -26,5 +28,5 @@
     <gui fullscreen='0'>
       <camera name='user_camera'>
-        <pose frame=''>17.5798 4.82061 4.05674 0 0.216 -2.876</pose>
+        <pose frame=''>175.544 123.61 4.70958 0 0.168 -2.40718</pose>
         <view_controller>orbit</view_controller>
       </camera>
@@ -33,5 +35,5 @@
       <!-- Note - the pose tag doesn't seem to work for heightmaps, so you need
       to go into the model file to change the altitutde/height!-->
-      <pose> 0 0 0 0 0 0 </pose>
+      <pose>0 0 0 0 0 0</pose>
       <uri>model://sandisland</uri>
     </include>
@@ -39,6 +41,11 @@
     plugin configurations -->
     <include>
-      <pose> 0 0 0 0 0 0 </pose>
+      <pose>0 0 0 0 0 0</pose>
       <uri>model://ocean</uri>
+    </include>
+    <!-- The post for securing the WAM-V -->
+    <include>
+      <pose>168.07 111.75 0.333 0.046 -0.157 0</pose>
+      <uri>model://post</uri>
     </include>
   </xacro:macro>

File: wamv_description/urdf/wamv_base.urdf.xacro (robot description, xacro)
@@ -88,9 +88,14 @@
       </geometry>
     </visual>
+    <visual name="payload">
+      <geometry>
+        <mesh filename="package://wamv_gazebo/mesh/payload.dae"/>
+      </geometry>
+    </visual>
     <!-- Left base collisions -->
     <xacro:main_collisions prefix="left" reflect="1" />
     <!-- Right side collisions -->
     <xacro:main_collisions prefix="right" reflect="-1" />
-     <!-- Top base -->
+    <!-- Top base -->
     <collision name="top_base">
       <origin xyz="0 -0 1.25" rpy="0 0 0" />

File: wamv_gazebo/urdf/macros.xacro (robot description, xacro)
@@ -13,3 +13,4 @@
   <xacro:include filename="$(find wamv_gazebo)/urdf/sensors/wamv_3d_lidar.xacro" />
   <xacro:include filename="$(find wamv_gazebo)/urdf/sensors/wamv_p3d.xacro" />
+  <xacro:include filename="$(find wamv_gazebo)/urdf/wamv_payload.xacro" />
 </robot>

File: wamv_gazebo/urdf/sensors/wamv_3d_lidar.xacro (robot description, xacro)
@@ -19,11 +19,8 @@
                                             max_range:=100 noise_stddev:=0.01">
     <link name="${name}_link">
-      <visual name="${name}_visual">>
+      <visual name="{name}_visual">
         <geometry>
-          <cylinder radius="0.025" length="0.1" />
+          <mesh filename="package://wamv_gazebo/mesh/lidar_3d.dae"/>
         </geometry>
-        <material name="${name}_visual_material">
-          <color rgba="0.5 1.0 0.5 1.0" />
-        </material>
       </visual>
     </link>

File: wamv_gazebo/urdf/sensors/wamv_camera.xacro (robot description, xacro)
@@ -3,13 +3,8 @@
   <xacro:macro name="wamv_camera" params="name x:=0.5 y:=0 z:=1.5 R:=0 P:=0 Y:=0">
     <link name="${name}_link">
-      <visual name="${name}_visual">
-        <xacro:property name="visual_length" value="0.05" />
-        <origin xyz="-${visual_length/2.0} 0 0" rpy="0 1.57 0" />
+      <visual name="{name}_visual">
         <geometry>
-          <cylinder radius="0.01" length="${visual_length}" />
+          <mesh filename="package://wamv_gazebo/mesh/monocamera.dae"/>
         </geometry>
-        <material name="${name}_visual_material">
-          <color rgba="1.0 1.0 0.0 1.0" />
-        </material>
       </visual>
     </link>

File: wamv_gazebo/urdf/sensors/wamv_gps.xacro (robot description, xacro)
@@ -3,20 +3,8 @@
   <xacro:macro name="wamv_gps" params="name:=gps x:=0 y:=0 z:=1.3 R:=0 P:=0 Y:=0">
     <link name="${name}_link">
-      <visual name="${name}_visual_base">
+      <visual name="{name}_visual">
         <geometry>
-          <box size="0.1 0.1 0.025" />
+          <mesh filename="package://wamv_gazebo/mesh/gps.dae"/>
         </geometry>
-        <material name="${name}_visual_base_material">
-          <color rgba="1.0 1.0 1.0 1.0" />
-        </material>
-      </visual>
-      <visual name="${name}_visual_antenna">
-        <origin xyz="0 0 0.025" />
-        <geometry>
-          <sphere radius="0.03" />
-        </geometry>
-        <material name="${name}_visual_antenna_material">
-          <color rgba="0.7 0.7 0.7 1.0" />
-        </material>
       </visual>
     </link>

File: wamv_gazebo/urdf/wamv_gazebo.urdf.xacro (robot description, xacro)
@@ -14,5 +14,5 @@
   <xacro:include filename="$(find wamv_gazebo)/urdf/wamv_gazebo.xacro" />
   <!-- === Thrusters === -->
-  <xacro:property name="thruster_conf" value="$(arg thruster_config)"/> -->
+  <xacro:property name="thruster_conf" value="$(arg thruster_config)"/>
   <!-- Default WAM-V with two aft thrusters -->
   <xacro:if value="${thruster_conf == 'H'}">
@@ -77,14 +77,16 @@
   <xacro:if value="$(arg vrx_sensors_enabled)">
     <!-- Add a stereo camera pair -->
-    <xacro:wamv_camera name="front_left_camera" y="0.1" x="0.75" P="${radians(15)}" />
-    <xacro:wamv_camera name="front_right_camera" y="-0.1" x="0.75" P="${radians(15)}" />
+    <xacro:wamv_camera name="front_left_camera" y="0.1" x="0.75" R="${radians(15)}" Y="${radians(90)}" />
+    <xacro:wamv_camera name="front_right_camera" y="-0.1" x="0.75" R="${radians(15)}" Y="${radians(90)}" />
     <!-- Add a camera facing right -->
-    <xacro:wamv_camera name="middle_right_camera" y="-0.45" P="${radians(15)}" Y="${radians(-90)}" />
+    <xacro:wamv_camera name="middle_right_camera" y="-0.45" R="${radians(15)}" />
     <!-- Add simulated GPS -->
-    <xacro:wamv_gps name="gps_wamv" y="0.2" />
+    <xacro:wamv_gps name="gps_wamv" x="-0.75" y="0" />
     <!-- Add Simulated IMU -->
     <xacro:wamv_imu name="imu_wamv" y="-0.2" />
     <!-- Add 3D LIDAR -->
     <xacro:wamv_3d_lidar name="lidar_wamv" P="${radians(8)}" />
+    <!-- Batteries and CPU boxes -->
+    <!-- <xacro:wamv_payload name="wamv_payload" /> -->
   </xacro:if>
 </robot>

Commit message: Tweaks

File: vrx_gazebo/worlds/example_course.world.xacro (robot description, xacro)
@@ -34,5 +34,5 @@
           <link_name>base_link</link_name>
           <coeff_vector>.5 .5 .33</coeff_vector>
-	      </wind_obj>
+        </wind_obj>
       </wind_objs>
     </xacro:usv_wind_gazebo>

File: vrx_gazebo/worlds/sandisland.world.xacro (robot description, xacro)
@@ -13,5 +13,5 @@
           <link_name>base_link</link_name>
           <coeff_vector>0.5 0.5 0.33</coeff_vector>
-	      </wind_obj>
+        </wind_obj>
       </wind_objs>
     </xacro:usv_wind_gazebo>

File: vrx_gazebo/worlds/xacros/include_all_xacros.xacro (robot description, xacro)
@@ -1,6 +1,6 @@
 <?xml version="1.0"?>
 <world xmlns:xacro="http://ros.org/wiki/xacro">
-  <xacro:macro name="include_all_xacros">
-	<xacro:include filename="$(find vrx_gazebo)/worlds/xacros/sandisland.xacro" />
+    <xacro:macro name="include_all_xacros">
+    <xacro:include filename="$(find vrx_gazebo)/worlds/xacros/sandisland.xacro" />
     <xacro:include filename="$(find vrx_gazebo)/worlds/xacros/sandisland2.xacro" />
     <xacro:include filename="$(find vrx_gazebo)/worlds/xacros/nav_challenge.xacro" />

File: vrx_gazebo/worlds/xacros/scene_macro.xacro (robot description, xacro)
@@ -5,5 +5,5 @@
       <time>${time}</time>
       <clouds>
-	    <speed>${cloud_speed}</speed>
+      <speed>${cloud_speed}</speed>
       </clouds>
       </sky>
