Commit message: functional?

File: vrx_gazebo/worlds/dock.world.xacro (robot description, xacro)
@@ -5,4 +5,7 @@
     <xacro:include filename="$(find vrx_gazebo)/worlds/sandisland.xacro" />
     <xacro:sandisland />
+    <!--Waves-->
+    <xacro:include filename="$(find wave_gazebo)/world_models/ocean_waves/model.xacro"/>
+    <xacro:ocean_waves/>
     <!-- The 2018 dock with the two placards -->
     <include>

File: vrx_gazebo/worlds/example_course.world.xacro (robot description, xacro)
@@ -5,4 +5,7 @@
     <xacro:include filename="$(find vrx_gazebo)/worlds/sandisland.xacro" />
     <xacro:sandisland />
+    <!--Waves-->
+    <xacro:include filename="$(find wave_gazebo)/world_models/ocean_waves/model.xacro"/>
+    <xacro:ocean_waves/>
     <include>
       <uri>model://robotx_navigation_challenge</uri>

File: vrx_gazebo/worlds/navigation_task.world.xacro (robot description, xacro)
@@ -5,4 +5,7 @@
     <xacro:include filename="$(find vrx_gazebo)/worlds/sandisland.xacro" />
     <xacro:sandisland />
+    <!--Waves-->
+    <xacro:include filename="$(find wave_gazebo)/world_models/ocean_waves/model.xacro"/>
+    <xacro:ocean_waves/>
     <!--wind for the wamv-->
     <xacro:include filename="$(find vrx_gazebo)/worlds/xacros/usv_wind_plugin.xacro"/>

File: vrx_gazebo/worlds/perception_task.world.xacro (robot description, xacro)
@@ -5,4 +5,7 @@
     <xacro:include filename="$(find vrx_gazebo)/worlds/sandisland.xacro" />
     <xacro:sandisland />
+    <!--Waves-->
+    <xacro:include filename="$(find wave_gazebo)/world_models/ocean_waves/model.xacro"/>
+    <xacro:ocean_waves/>
     <!-- Include all the objects we plan to use for perception.
        Stash them out of the field of view for now -->

File: vrx_gazebo/worlds/sandisland.world.xacro (robot description, xacro)
@@ -5,4 +5,7 @@
     <xacro:include filename="$(find vrx_gazebo)/worlds/sandisland.xacro" />
     <xacro:sandisland />
+    <!--Waves-->
+    <xacro:include filename="$(find wave_gazebo)/world_models/ocean_waves/model.xacro"/>
+    <xacro:ocean_waves/>
     <!--Wind for the WAM-V. Note, wind parameters are set in the plug.-->
     <xacro:include filename="$(find vrx_gazebo)/worlds/xacros/usv_wind_plugin.xacro"/>

File: vrx_gazebo/worlds/sandisland.xacro (robot description, xacro)
@@ -38,10 +38,4 @@
       <pose> 0 0 0 0 0 0 </pose>
       <uri>model://sandisland</uri>
-    </include>
-    <!-- Should be at the same height as the water level in USV and buoyancy
-    plugin configurations -->
-    <include>
-      <pose> 0 0 0 0 0 0 </pose>
-      <uri>model://ocean_waves</uri>
     </include>
     <!-- The posts for securing the WAM-V -->

File: vrx_gazebo/worlds/scan_and_dock.world.xacro (robot description, xacro)
@@ -5,4 +5,7 @@
     <xacro:include filename="$(find vrx_gazebo)/worlds/sandisland.xacro" />
     <xacro:sandisland />
+    <!--Waves-->
+    <xacro:include filename="$(find wave_gazebo)/world_models/ocean_waves/model.xacro"/>
+    <xacro:ocean_waves/>>
     <!-- The light buoy -->
     <include>

File: vrx_gazebo/worlds/wayfinding_task.world.xacro (robot description, xacro)
@@ -5,4 +5,7 @@
     <xacro:include filename="$(find vrx_gazebo)/worlds/sandisland.xacro" />
     <xacro:sandisland />
+    <!--Waves-->
+    <xacro:include filename="$(find wave_gazebo)/world_models/ocean_waves/model.xacro"/>
+    <xacro:ocean_waves/>
     <plugin name="wayfinding_scoring_plugin"
             filename="libwayfinding_scoring_plugin.so">

File: vrx_gazebo/worlds/wind_test.world.xacro (robot description, xacro)
@@ -4,4 +4,7 @@
     <xacro:include filename="$(find vrx_gazebo)/worlds/sandisland.xacro" />
     <xacro:sandisland />
+    <!--Waves-->
+    <xacro:include filename="$(find wave_gazebo)/world_models/ocean_waves/model.xacro"/>
+    <xacro:ocean_waves/>
     <include>
       <uri>model://robotx_light_buoy</uri>

File: vrx_gazebo/worlds/xacros/dock.xacro (robot description, xacro)
@@ -2,11 +2,6 @@
 <!-- World containing sandisland model and some course challenges -->
 <sdf version="1.6" xmlns:xacro="http://ros.org/wiki/xacro">
-  <world name="robotx_scan_and_dock">
-    <xacro:macro name="scan_and_dock">
-      <!-- The light buoy -->$
-      <include>
-        <uri>model://robotx_light_buoy</uri>
-        <pose>90 70 0.25 0 0 0</pose>
-      </include>
+  <world name="robotx_dock">
+    <xacro:macro name="dock">
       <!-- The 2018 dock with the two placards -->
       <include>

File: vrx_gazebo/worlds/xacros/include_all_xacros.xacro (robot description, xacro)
@@ -3,12 +3,14 @@
     <xacro:macro name="include_all_xacros">
     <xacro:include filename="$(find vrx_gazebo)/worlds/sandisland.xacro" />
-    <xacro:include filename="$(find vrx_gazebo)/worlds/xacros/sandisland2.xacro" />
+    <xacro:include filename="$(find vrx_gazebo)/worlds/xacros/sandisland_minus_scene.xacro" />
+    <xacro:include filename="$(find vrx_gazebo)/worlds/xacros/scene.xacro" />
     <xacro:include filename="$(find vrx_gazebo)/worlds/xacros/nav_challenge.xacro" />
-    <xacro:include filename="$(find vrx_gazebo)/worlds/xacros/light_buoy.xacro" />
-    <xacro:include filename="$(find vrx_gazebo)/worlds/xacros/qualifying_pinger_transit_2016.xacro" />
-    <xacro:include filename="$(find vrx_gazebo)/worlds/xacros/dock_2016.xacro" />
-    <xacro:include filename="$(find vrx_gazebo)/worlds/xacros/dock_2018.xacro" />
-    <xacro:include filename="$(find vrx_gazebo)/worlds/xacros/scene_macro.xacro" />
     <xacro:include filename="$(find vrx_gazebo)/worlds/xacros/usv_wind_plugin.xacro" />
+    <xacro:include filename="$(find wave_gazebo)/world_models/ocean_waves/model.xacro"/>
+    <xacro:include filename="$(find vrx_gazebo)/worlds/xacros/perception.xacro" />
+    <xacro:include filename="$(find vrx_gazebo)/worlds/xacros/stationkeeping.xacro" />
+    <xacro:include filename="$(find vrx_gazebo)/worlds/xacros/dock.xacro" />
+    <xacro:include filename="$(find vrx_gazebo)/worlds/xacros/scan_and_dock.xacro" />
+    <xacro:include filename="$(find vrx_gazebo)/worlds/xacros/wayfinding.xacro" />
   </xacro:macro>
 </world>

File: vrx_gazebo/worlds/xacros/sandisland_minus_scene.xacro (robot description, xacro)
@@ -2,5 +2,5 @@
 <!-- Macro to insert the sandisland into the world -->
 <world xmlns:xacro="http://ros.org/wiki/xacro">
-  <xacro:macro name="sandisland2">
+  <xacro:macro name="sandisland_minus_scene">
     <!-- Estimated latitude/longitude of sandisland from satellite imagery -->
     <spherical_coordinates>
@@ -22,4 +22,5 @@
         <view_controller>orbit</view_controller>
       </camera>
+      <!--<plugin name="GUITaskWidget" filename="libgui_task_widget.so"/>-->
     </gui>
     <include>
@@ -28,10 +29,4 @@
       <pose> 0 0 0 0 0 0 </pose>
       <uri>model://sandisland</uri>
-    </include>
-    <!-- Should be at the same height as the water level in USV and buoyancy
-    plugin configurations -->
-    <include>
-      <pose> 0 0 0 0 0 0 </pose>
-      <uri>model://ocean</uri>
     </include>
     <!-- The posts for securing the WAM-V -->

File: vrx_gazebo/worlds/xacros/stationkeeping.xacro (robot description, xacro)
@@ -1,17 +1,11 @@
-<?xml version="1.0" ?>
-<!-- World containing sandisland model and some course challenges -->
-<sdf version="1.6" xmlns:xacro="http://ros.org/wiki/xacro">
-  <world name="robotx_stationkeeping">
-    <xacro:include filename="$(find vrx_gazebo)/worlds/sandisland.xacro" />
-    <xacro:sandisland />
-    <!--Waves-->
-    <xacro:include filename="$(find wave_gazebo)/world_models/ocean_waves/model.xacro"/>
-    <xacro:ocean_waves/>
-  <plugin name="stationkeeping_scoring_plugin"
+<?xml version="1.0"?>
+<world xmlns:xacro="http://ros.org/wiki/xacro">
+  <xacro:macro name="stationkeeping" params="lat:=21.31091 lon:=-157.88868 heading:=0.0">
+    <plugin name="stationkeeping_scoring_plugin"
           filename="libstationkeeping_scoring_plugin.so">
       <vehicle>wamv</vehicle>
       <task_name>stationkeeping</task_name>
       <!-- Goal as Latitude, Longitude, Yaw -->
-      <goal_pose>21.31091 -157.88868 0.0 </goal_pose>
+      <goal_pose>${lat} ${lon} ${heading} </goal_pose>
       <initial_state_duration>10</initial_state_duration>
       <ready_state_duration>10</ready_state_duration>
@@ -26,4 +20,4 @@
       </release_joints>
     </plugin>
-  </world>
-</sdf>
+  </xacro:macro>
+</world>

Commit message: Functional

File: vrx_gazebo/worlds/dock.world.xacro (robot description, xacro)
@@ -10,13 +10,17 @@
     <!-- The 2018 dock with the two placards -->
     <include>
-      <uri>model://dock_2018</uri>
+      <uri>model://dock_2018_dynamic</uri>
       <pose>60 -2.75 0 0 0 0</pose>
     </include>
     <!-- Uncomment to visualize the bay #1 activation zone -->
-    <!-- <model name="activation_placard1">
+    <!--
+    <model name="activation_placard1">
+      <pose frame="robotx_dock_2018::dock_2018_placard1::placard::link">
+        0 0 10 0 0 0 </pose>
       <static>true</static>
       <link name="link">
+        <pose frame="robotx_dock_2018::dock_2018_placard1::placard::link">
+        0 0 10 0 0 0 </pose>
         <visual name="visual">
-          <pose>72.75 0 0 0 0 0</pose>
           <geometry>
             <box>
@@ -24,8 +28,13 @@
             </box>
           </geometry>
-          <transparency>0.8</transparency>
+          <transparency>0.0</transparency>
         </visual>
       </link>
-    </model> -->
+      <joint name="act1" type="fixed">
+        <child>robotx_dock_2018::dock_2018_placard1::placard::link</child>
+        <parent>link</parent>
+      </joint>
+    </model>
+  -->
     <!-- Uncomment to visualize the bay #2 activation zone -->
     <!-- <model name="activation_placard2">
@@ -95,5 +104,5 @@
       <geometry>
         <box>
-          <size>40 15 20</size>
+          <size>4 1.5 2</size>
         </box>
       </geometry>
@@ -106,5 +115,5 @@
       <geometry>
         <box>
-          <size>40 15 20</size>
+          <size>4 1.5 2</size>
         </box>
       </geometry>

Commit message: removing activation zone viz from world.xacro

File: vrx_gazebo/worlds/dock.world.xacro (robot description, xacro)
@@ -13,43 +13,4 @@
       <pose>130 97 0 0 0 0</pose>
     </include>
-    <!-- Uncomment to visualize the bay #1 activation zone -->
-    <!--
-    <model name="activation_placard1">
-      <pose frame="robotx_dock_2018::dock_2018_placard1::placard::link">
-        0 0 10 0 0 0 </pose>
-      <static>true</static>
-      <link name="link">
-        <pose frame="robotx_dock_2018::dock_2018_placard1::placard::link">
-        0 0 10 0 0 0 </pose>
-        <visual name="visual">
-          <geometry>
-            <box>
-              <size>1.5 4 2</size>
-            </box>
-          </geometry>
-          <transparency>0.0</transparency>
-        </visual>
-      </link>
-      <joint name="act1" type="fixed">
-        <child>robotx_dock_2018::dock_2018_placard1::placard::link</child>
-        <parent>link</parent>
-      </joint>
-    </model>
-  -->
-    <!-- Uncomment to visualize the bay #2 activation zone -->
-    <!-- <model name="activation_placard2">
-      <static>true</static>
-      <link name="link">
-        <visual name="visual">
-          <pose>61.75 0 0 0 0 0</pose>
-          <geometry>
-            <box>
-              <size>1.5 4 2</size>
-            </box>
-          </geometry>
-          <transparency>0.8</transparency>
-        </visual>
-      </link>
-    </model> -->
     <!-- The scoring plugin -->
     <plugin name="scan_dock_scoring_plugin"

Commit message: Double activation zone.

File: vrx_gazebo/worlds/dock.world.xacro (robot description, xacro)
@@ -40,5 +40,6 @@
         <bay>
           <name>bay1</name>
-          <activation_topic>/vrx/dock_2018/bay_1/contain</activation_topic>
+          <internal_activation_topic>/vrx/dock_2018/bay_1_internal/contain</internal_activation_topic>
+          <external_activation_topic>/vrx/dock_2018/bay_1_external/contain</external_activation_topic>
           <symbol_topic>/vrx/dock_2018_placard1/symbol</symbol_topic>
           <min_dock_time>10.0</min_dock_time>
@@ -48,5 +49,6 @@
         <bay>
           <name>bay2</name>
-          <activation_topic>/vrx/dock_2018/bay_2/contain</activation_topic>
+          <internal_activation_topic>/vrx/dock_2018/bay_2_internal/contain</internal_activation_topic>
+          <external_activation_topic>/vrx/dock_2018/bay_2_external/contain</external_activation_topic>
           <symbol_topic>/vrx/dock_2018_placard2/symbol</symbol_topic>
           <min_dock_time>10.0</min_dock_time>
@@ -61,5 +63,5 @@
     <plugin name="vehicle_docked_bay1" filename="libContainPlugin.so">
       <entity>wamv::base_link</entity>
-      <namespace>vrx/dock_2018/bay_1</namespace>
+      <namespace>vrx/dock_2018/bay_1_internal</namespace>
       <pose frame="robotx_dock_2018::dock_2018_placard1::placard::link">0 -5 -1.5 0 0 0</pose>
       <geometry>
@@ -69,8 +71,19 @@
       </geometry>
     </plugin>
+    <!-- Triggers a message when the vehicle enters and exits the bay #1 -->
+    <plugin name="vehicle_docked_bay1_exterior" filename="libContainPlugin.so">
+      <entity>wamv::base_link</entity>
+      <namespace>vrx/dock_2018/bay_1_external</namespace>
+      <pose frame="robotx_dock_2018::dock_2018_placard1::placard::link">0 -10 -1.5 0 0 0</pose>
+      <geometry>
+        <box>
+          <size>8 1.5 2</size>
+        </box>
+      </geometry>
+    </plugin>
     <!-- Triggers a message when the vehicle enters and exits the bay #2 -->
     <plugin name="vehicle_docked_bay2" filename="libContainPlugin.so">
       <entity>wamv::base_link</entity>
-      <namespace>vrx/dock_2018/bay_2</namespace>
+      <namespace>vrx/dock_2018/bay_2_internal</namespace>
       <pose frame="robotx_dock_2018::dock_2018_placard2::placard::link">0 5 -1.5 0 0 0</pose>
       <geometry>
@@ -80,4 +93,15 @@
       </geometry>
     </plugin>
+    <!-- Triggers a message when the vehicle enters and exits the bay #1 -->
+    <plugin name="vehicle_docked_bay2_exterior" filename="libContainPlugin.so">
+      <entity>wamv::base_link</entity>
+      <namespace>vrx/dock_2018/bay_2_external</namespace>
+      <pose frame="robotx_dock_2018::dock_2018_placard1::placard::link">0 10 -1.5 0 0 0</pose>
+      <geometry>
+        <box>
+          <size>8 1.5 2</size>
+        </box>
+      </geometry>
+    </plugin>
   </world>
 </sdf>

File: vrx_gazebo/worlds/scan_and_dock.world.xacro (robot description, xacro)
@@ -75,5 +75,6 @@
         <bay>
           <name>bay1</name>
-          <activation_topic>/vrx/dock_2018/bay_1/contain</activation_topic>
+          <internal_activation_topic>/vrx/dock_2018/bay_1/contain</internal_activation_topic>
+          <external_activation_topic>/vrx/dock_2018/bay_1_exterior/contain</external_activation_topic>
           <symbol_topic>/vrx/dock_2018_placard1/symbol</symbol_topic>
 	        <min_dock_time>10.0</min_dock_time>
@@ -83,5 +84,6 @@
         <bay>
           <name>bay2</name>
-          <activation_topic>/vrx/dock_2018/bay_2/contain</activation_topic>
+          <internal_activation_topic>/vrx/dock_2018/bay_2/contain</internal_activation_topic>
+          <external_activation_topic>/vrx/dock_2018/bay_2_exterior/contain</external_activation_topic>
           <symbol_topic>/vrx/dock_2018_placard2/symbol</symbol_topic>
           <min_dock_time>10.0</min_dock_time>

File: vrx_gazebo/worlds/xacros/dock.xacro (robot description, xacro)
@@ -47,5 +47,6 @@
         <bay>
           <name>bay1</name>
-          <activation_topic>/vrx/dock_2018/bay_1/contain</activation_topic>
+          <internal_activation_topic>/vrx/dock_2018/bay_1_internal/contain</internal_activation_topic>
+          <external_activation_topic>/vrx/dock_2018/bay_1_external/contain</external_activation_topic>
           <symbol_topic>/vrx/dock_2018_placard1/symbol</symbol_topic>
           <min_dock_time>10.0</min_dock_time>
@@ -55,5 +56,6 @@
         <bay>
           <name>bay2</name>
-          <activation_topic>/vrx/dock_2018/bay_2/contain</activation_topic>
+          <internal_activation_topic>/vrx/dock_2018/bay_2_internal/contain</internal_activation_topic>
+          <external_activation_topic>/vrx/dock_2018/bay_2_external/contain</external_activation_topic>
           <symbol_topic>/vrx/dock_2018_placard2/symbol</symbol_topic>
           <min_dock_time>10.0</min_dock_time>
@@ -66,5 +68,5 @@
     <plugin name="vehicle_docked_bay1" filename="libContainPlugin.so">
       <entity>wamv::base_link</entity>
-      <namespace>vrx/dock_2018/bay_1</namespace>
+      <namespace>vrx/dock_2018/bay_1_internal</namespace>
       <pose frame="robotx_dock_2018::dock_2018_placard1::placard::link">0 -5 -1.5 0 0 0</pose>
       <geometry>
@@ -74,8 +76,19 @@
       </geometry>
     </plugin>
+    <!-- Triggers a message when the vehicle enters and exits the bay #1 -->
+    <plugin name="vehicle_docked_bay1_exterior" filename="libContainPlugin.so">
+      <entity>wamv::base_link</entity>
+      <namespace>vrx/dock_2018/bay_1_external</namespace>
+      <pose frame="robotx_dock_2018::dock_2018_placard1::placard::link">0 -10 -1.5 0 0 0</pose>
+      <geometry>
+        <box>
+          <size>8 1.5 2</size>
+        </box>
+      </geometry>
+    </plugin>
     <!-- Triggers a message when the vehicle enters and exits the bay #2 -->
     <plugin name="vehicle_docked_bay2" filename="libContainPlugin.so">
       <entity>wamv::base_link</entity>
-      <namespace>vrx/dock_2018/bay_2</namespace>
+      <namespace>vrx/dock_2018/bay_2_internal</namespace>
       <pose frame="robotx_dock_2018::dock_2018_placard2::placard::link">0 5 -1.5 0 0 0</pose>
       <geometry>
@@ -85,4 +98,15 @@
       </geometry>
     </plugin>
+    <!-- Triggers a message when the vehicle enters and exits the bay #1 -->
+    <plugin name="vehicle_docked_bay2_exterior" filename="libContainPlugin.so">
+      <entity>wamv::base_link</entity>
+      <namespace>vrx/dock_2018/bay_2_external</namespace>
+      <pose frame="robotx_dock_2018::dock_2018_placard1::placard::link">0 10 -1.5 0 0 0</pose>
+      <geometry>
+        <box>
+          <size>8 1.5 2</size>
+        </box>
+      </geometry>
+    </plugin>
   </xacro:macro>
 </world>

File: vrx_gazebo/worlds/xacros/scan_and_dock.xacro (robot description, xacro)
@@ -40,5 +40,6 @@
         <bay>
           <name>bay1</name>
-          <activation_topic>/vrx/dock_2018/bay_1/contain</activation_topic>
+          <internal_activation_topic>/vrx/dock_2018/bay_1/contain</internal_activation_topic>
+          <external_activation_topic>/vrx/dock_2018/bay_1_exterior/contain</external_activation_topic>
           <symbol_topic>/vrx/dock_2018_placard1/symbol</symbol_topic>
           <min_dock_time>10.0</min_dock_time>
@@ -48,5 +49,6 @@
         <bay>
           <name>bay2</name>
-          <activation_topic>/vrx/dock_2018/bay_2/contain</activation_topic>
+          <internal_activation_topic>/vrx/dock_2018/bay_2/contain</internal_activation_topic>
+          <external_activation_topic>/vrx/dock_2018/bay_2_exterior/contain</external_activation_topic>
           <symbol_topic>/vrx/dock_2018_placard2/symbol</symbol_topic>
           <min_dock_time>10.0</min_dock_time>
