Commit message: Update GPS datum to more closely match nautical chart
Signed-off-by: Roland Arsenault <roland@ccom.unh.edu>

File: vrx_gazebo/worlds/sandisland.xacro (robot description, xacro)
@@ -16,6 +16,6 @@
       <surface_model>EARTH_WGS84</surface_model>
       <world_frame_orientation>ENU</world_frame_orientation>
-      <latitude_deg>21.30996</latitude_deg>
-      <longitude_deg>-157.8901</longitude_deg>
+      <latitude_deg>21.31030</latitude_deg>
+      <longitude_deg>-157.8908</longitude_deg>
       <elevation>0.0</elevation>
       <!-- For legacy gazebo reasons, need to rotate -->

File: vrx_gazebo/worlds/stationkeeping_task.world.xacro (robot description, xacro)
@@ -24,5 +24,5 @@
       <task_name>stationkeeping</task_name>
       <!-- Goal as Latitude, Longitude, Yaw -->
-      <goal_pose>21.31091 -157.88868 0.0 </goal_pose>
+      <goal_pose>21.31125 -157.88938 0.0 </goal_pose>
       <initial_state_duration>10</initial_state_duration>
       <ready_state_duration>10</ready_state_duration>

File: vrx_gazebo/worlds/wayfinding_task.world.xacro (robot description, xacro)
@@ -27,13 +27,13 @@
         <!-- Approx. starting point of wamv -->
         <waypoint>
-          <pose>21.3109331464 -157.888576027 1.21756121843</pose>
+          <pose>21.3112720364 -157.889280727 1.21756121843</pose>
         </waypoint>
         <!-- A waypoint -->
         <waypoint>
-          <pose>21.30996 -157.8901 1.0</pose>
+          <pose>21.3103 -157.8908 1.0</pose>
         </waypoint>
         <!-- Another waypoint -->
         <waypoint>
-          <pose>21.31 -157.89 1.0</pose>
+          <pose>21.3103 -157.8907 1.0</pose>
         </waypoint>
       </waypoints>

File: vrx_gazebo/worlds/xacros/sandisland_minus_scene.xacro (robot description, xacro)
@@ -7,6 +7,6 @@
       <surface_model>EARTH_WGS84</surface_model>
       <world_frame_orientation>ENU</world_frame_orientation>
-      <latitude_deg>21.30996</latitude_deg>
-      <longitude_deg>-157.8901</longitude_deg>
+      <latitude_deg>21.31030</latitude_deg>
+      <longitude_deg>-157.8908</longitude_deg>
       <elevation>0.0</elevation>
       <!-- For legacy gazebo reasons, need to rotate -->

File: vrx_gazebo/worlds/xacros/stationkeeping.xacro (robot description, xacro)
@@ -1,5 +1,5 @@
 <?xml version="1.0"?>
 <world xmlns:xacro="http://ros.org/wiki/xacro">
-  <xacro:macro name="stationkeeping" params="**wp_markers lat:=21.31091 lon:=-157.88868 heading:=0.0 namespace:=wamv competition:=vrx">
+  <xacro:macro name="stationkeeping" params="**wp_markers lat:=21.31125 lon:=-157.88938 heading:=0.0 namespace:=wamv competition:=vrx">
     <plugin name="stationkeeping_scoring_plugin"
           filename="libstationkeeping_scoring_plugin.so">

File: wamv_gazebo/urdf/sensors/wamv_gps.xacro (robot description, xacro)
@@ -1,5 +1,5 @@
 <?xml version="1.0" encoding="UTF-8"?>
 <robot xmlns:xacro="http://ros.org/wiki/xacro">
-  <xacro:macro name="wamv_gps" params="name:=gps x:=0.3 y:=0 z:=1.3 R:=0 P:=0 Y:=0 lat:=21.30996 lon:=-157.8901 elev:=0.0 update_rate:=15">
+  <xacro:macro name="wamv_gps" params="name:=gps x:=0.3 y:=0 z:=1.3 R:=0 P:=0 Y:=0 lat:=21.3103 lon:=-157.8907 elev:=0.0 update_rate:=15">
     <link name="${name}_link">
       <visual name="${name}_visual">
