Commit message: Updating coords

File: vrx_gazebo/worlds/stationkeeping_task.world.xacro (robot description, xacro)
@@ -24,5 +24,5 @@
       <task_name>stationkeeping</task_name>
       <!-- Goal as Latitude, Longitude, Yaw -->
-      <goal_pose>21.31091 -157.88868 0.0 </goal_pose>
+      <goal_pose>-33.724223 150.679736 0.0 </goal_pose>
       <initial_state_duration>10</initial_state_duration>
       <ready_state_duration>10</ready_state_duration>
@@ -37,5 +37,5 @@
       </release_joints>
       <markers>
-        <scaling>0.2 0.2 2.0</scaling>
+        <scaling>20 20 20</scaling>
         <height>0.5</height>
       </markers>

File: vrx_gazebo/worlds/xacros/stationkeeping.xacro (robot description, xacro)
@@ -1,5 +1,5 @@
 <?xml version="1.0"?>
 <world xmlns:xacro="http://ros.org/wiki/xacro">
-  <xacro:macro name="stationkeeping" params="**wp_markers lat:=21.31091 lon:=-157.88868 heading:=0.0 namespace:=wamv competition:=vrx">
+  <xacro:macro name="stationkeeping" params="**wp_markers lat:=-33.724223 lon:=150.679736 heading:=0.0 namespace:=wamv competition:=vrx">
     <plugin name="stationkeeping_scoring_plugin"
           filename="libstationkeeping_scoring_plugin.so">

File: wamv_gazebo/urdf/sensors/wamv_gps.xacro (robot description, xacro)
@@ -1,5 +1,5 @@
 <?xml version="1.0" encoding="UTF-8"?>
 <robot xmlns:xacro="http://ros.org/wiki/xacro">
-  <xacro:macro name="wamv_gps" params="name:=gps x:=0.3 y:=0 z:=1.3 R:=0 P:=0 Y:=0 lat:=21.30996 lon:=-157.8901 elev:=0.0 update_rate:=15">
+  <xacro:macro name="wamv_gps" params="name:=gps x:=0.3 y:=0 z:=1.3 R:=0 P:=0 Y:=0 lat:=-33.722690 lon:=150.673795 elev:=0.0 update_rate:=15">
     <link name="${namespace}/${name}_link">
       <visual name="${name}_visual">
