Commit message: Updated wayfinding task waypoint locations

File: vrx_gazebo/worlds/wayfinding_task.world.xacro (robot description, xacro)
@@ -3,6 +3,6 @@
 <sdf version="1.6" xmlns:xacro="http://ros.org/wiki/xacro">
   <world name="robotx_wayfinding">
-    <xacro:include filename="$(find vrx_gazebo)/worlds/sandisland.xacro" />
-    <xacro:sandisland />
+    <xacro:include filename="$(find vrx_gazebo)/worlds/sydneyregatta.xacro" />
+    <xacro:sydneyregatta />
     <!--Waves-->
     <xacro:include filename="$(find wave_gazebo)/world_models/ocean_waves/model.xacro"/>
@@ -27,13 +27,13 @@
         <!-- Approx. starting point of wamv -->
         <waypoint>
-          <pose>21.3109331464 -157.888576027 1.21756121843</pose>
+          <pose>-33.7226766699 150.6740630167 1.21756121843</pose>
         </waypoint>
         <!-- A waypoint -->
         <waypoint>
-          <pose>21.30996 -157.8901 1.0</pose>
+          <pose>-33.7220832884 150.67379127877 1.0</pose>
         </waypoint>
         <!-- Another waypoint -->
         <waypoint>
-          <pose>21.31 -157.89 1.0</pose>
+          <pose>-33.7226013209 150.67504609858 1.0</pose>
         </waypoint>
       </waypoints>

File: wamv_gazebo/urdf/sensors/wamv_gps.xacro (robot description, xacro)
@@ -1,5 +1,5 @@
 <?xml version="1.0" encoding="UTF-8"?>
 <robot xmlns:xacro="http://ros.org/wiki/xacro">
-  <xacro:macro name="wamv_gps" params="name:=gps x:=0.3 y:=0 z:=1.3 R:=0 P:=0 Y:=0 lat:=21.30996 lon:=-157.8901 elev:=0.0 update_rate:=15">
+  <xacro:macro name="wamv_gps" params="name:=gps x:=0.3 y:=0 z:=1.3 R:=0 P:=0 Y:=0 lat:=-33.724223 lon:=150.679736 elev:=0.0 update_rate:=15">
     <link name="${namespace}/${name}_link">
       <visual name="${name}_visual">
