Commit message: Fix water scaling and wind.
Signed-off-by: Carlos Agüero <caguero@openrobotics.org>

File: vrx_gazebo/worlds/gymkhana.world.xacro (robot description, xacro)
@@ -2,10 +2,10 @@
 <!-- World containing sandisland model and some course challenges -->
 <sdf version="1.6" xmlns:xacro="http://ros.org/wiki/xacro">
-  <world name="gymkhana">
+  <world name="vrx_gymkhana">
     <xacro:include filename="$(find vrx_gazebo)/worlds/sydneyregatta.xacro" />
     <xacro:sydneyregatta />
     <!--Waves-->
     <xacro:include filename="$(find wave_gazebo)/world_models/ocean_waves/model.xacro"/>
-    <xacro:ocean_waves />
+    <xacro:ocean_waves scale="2.5"/>
     <!--Wind. Note, wind parameters are set in the plugin.-->
     <xacro:include filename="$(find vrx_gazebo)/worlds/xacros/usv_wind_plugin.xacro"/>

File: vrx_gazebo/worlds/perception_task.world.xacro (robot description, xacro)
@@ -2,10 +2,10 @@
 <!-- World containing sandisland model and some course challenges -->
 <sdf version="1.6" xmlns:xacro="http://ros.org/wiki/xacro">
-  <world name="perception_task_example">
+  <world name="vrx_perception">
     <xacro:include filename="$(find vrx_gazebo)/worlds/sydneyregatta.xacro" />
     <xacro:sydneyregatta />
     <!--Waves-->
     <xacro:include filename="$(find wave_gazebo)/world_models/ocean_waves/model.xacro"/>
-    <xacro:ocean_waves/>
+    <xacro:ocean_waves scale="2.5"/>
     <!-- Include all the objects we plan to use for perception.
        Stash them out of the field of view for now -->

File: vrx_gazebo/worlds/scan_dock_deliver.world.xacro (robot description, xacro)
@@ -2,10 +2,10 @@
 <!-- World containing sydneyregatta model and some course challenges -->
 <sdf version="1.6" xmlns:xacro="http://ros.org/wiki/xacro">
-  <world name="robotx_example_course">
+  <world name="vrx_scan_dock_deliver">
     <xacro:include filename="$(find vrx_gazebo)/worlds/sydneyregatta.xacro" />
     <xacro:sydneyregatta />
     <!--Waves-->
     <xacro:include filename="$(find wave_gazebo)/world_models/ocean_waves/model.xacro"/>
-    <xacro:ocean_waves/>
+    <xacro:ocean_waves scale="2.5"/>
     <!--wind for the wamv-->
     <xacro:include filename="$(find vrx_gazebo)/worlds/xacros/usv_wind_plugin.xacro"/>
@@ -14,5 +14,5 @@
         <wind_obj>
           <name>wamv</name>
-          <link_name>base_link</link_name>
+          <link_name>wamv/base_link</link_name>
           <coeff_vector>.5 .5 .33</coeff_vector>
         </wind_obj>
@@ -29,34 +29,4 @@
       <pose>554 -233 0 0 0 0</pose>
     </include>
-    <!-- Uncomment to visualize the bay #1 activation zone -->
-    <!-- <model name="activation_placard1">
-      <static>true</static>
-      <link name="link">
-        <visual name="visual">
-          <pose>72.75 0 0 0 0 0</pose>
-          <geometry>
-            <box>
-              <size>1.5 4 2</size>
-            </box>
-          </geometry>
-          <transparency>0.8</transparency>
-        </visual>
-      </link>
-    </model> -->
-    <!-- Uncomment to visualize the bay #2 activation zone -->
-    <!-- <model name="activation_placard2">
-      <static>true</static>
-      <link name="link">
-        <visual name="visual">
-          <pose>61.75 0 0 0 0 0</pose>
-          <geometry>
-            <box>
-              <size>1.5 4 2</size>
-            </box>
-          </geometry>
-          <transparency>0.8</transparency>
-        </visual>
-      </link>
-    </model> -->
   </world>
 </sdf>

File: vrx_gazebo/worlds/stationkeeping_task.world.xacro (robot description, xacro)
@@ -2,10 +2,10 @@
 <!-- World containing sandisland model and some course challenges -->
 <sdf version="1.6" xmlns:xacro="http://ros.org/wiki/xacro">
-  <world name="robotx_stationkeeping">
+  <world name="vrx_stationkeeping">
     <xacro:include filename="$(find vrx_gazebo)/worlds/sydneyregatta.xacro" />
     <xacro:sydneyregatta />
     <!--Waves-->
     <xacro:include filename="$(find wave_gazebo)/world_models/ocean_waves/model.xacro"/>
-    <xacro:ocean_waves/>
+    <xacro:ocean_waves scale="2.5"/>
     <!--wind for the wamv-->
     <xacro:include filename="$(find vrx_gazebo)/worlds/xacros/usv_wind_plugin.xacro"/>
@@ -14,5 +14,5 @@
         <wind_obj>
           <name>wamv</name>
-          <link_name>base_link</link_name>
+          <link_name>wamv/base_link</link_name>
           <coeff_vector>.5 .5 .33</coeff_vector>
         </wind_obj>

File: vrx_gazebo/worlds/wayfinding_task.world.xacro (robot description, xacro)
@@ -2,10 +2,10 @@
 <!-- World containing sandisland model and some course challenges -->
 <sdf version="1.6" xmlns:xacro="http://ros.org/wiki/xacro">
-  <world name="robotx_wayfinding">
+  <world name="vrx_wayfinding">
     <xacro:include filename="$(find vrx_gazebo)/worlds/sydneyregatta.xacro" />
     <xacro:sydneyregatta />
     <!--Waves-->
     <xacro:include filename="$(find wave_gazebo)/world_models/ocean_waves/model.xacro"/>
-    <xacro:ocean_waves/>
+    <xacro:ocean_waves scale="2.5"/>
     <!--wind for the wamv-->
     <xacro:include filename="$(find vrx_gazebo)/worlds/xacros/usv_wind_plugin.xacro"/>
@@ -14,5 +14,5 @@
         <wind_obj>
           <name>wamv</name>
-          <link_name>base_link</link_name>
+          <link_name>wamv/base_link</link_name>
           <coeff_vector>.5 .5 .33</coeff_vector>
         </wind_obj>

File: vrx_gazebo/worlds/wildlife_task.world.xacro (robot description, xacro)
@@ -2,10 +2,10 @@
 <!-- World containing sydneyregatta model and some course challenges -->
 <sdf version="1.6" xmlns:xacro="http://ros.org/wiki/xacro">
-  <world name="robotx_example_course">
+  <world name="vrx_wildlife">
     <xacro:include filename="$(find vrx_gazebo)/worlds/sydneyregatta.xacro" />
     <xacro:sydneyregatta />
     <!--Waves-->
     <xacro:include filename="$(find wave_gazebo)/world_models/ocean_waves/model.xacro"/>
-    <xacro:ocean_waves/>
+    <xacro:ocean_waves scale="2.5"/>
     <!--wind for the wamv-->
     <xacro:include filename="$(find vrx_gazebo)/worlds/xacros/usv_wind_plugin.xacro"/>
@@ -14,5 +14,5 @@
         <wind_obj>
           <name>wamv</name>
-          <link_name>base_link</link_name>
+          <link_name>wamv/base_link</link_name>
           <coeff_vector>.5 .5 .33</coeff_vector>
         </wind_obj>
