Commit message: Scoring for the 'Scan, dock and deliver' task.
Signed-off-by: Carlos Agüero <caguero@openrobotics.org>

File: vrx_gazebo/worlds/scan_dock_deliver.world.xacro (robot description, xacro)
@@ -14,5 +14,5 @@
         <wind_obj>
           <name>wamv</name>
-          <link_name>base_link</link_name>
+          <link_name>wamv/base_link</link_name>
           <coeff_vector>.5 .5 .33</coeff_vector>
         </wind_obj>
@@ -29,34 +29,237 @@
       <pose>554 -233 0 0 0 0</pose>
     </include>
-    <!-- Uncomment to visualize the bay #1 activation zone -->
-    <!-- <model name="activation_placard1">
-      <static>true</static>
-      <link name="link">
-        <visual name="visual">
-          <pose>72.75 0 0 0 0 0</pose>
-          <geometry>
-            <box>
-              <size>1.5 4 2</size>
-            </box>
-          </geometry>
-          <transparency>0.8</transparency>
-        </visual>
-      </link>
-    </model> -->
-    <!-- Uncomment to visualize the bay #2 activation zone -->
-    <!-- <model name="activation_placard2">
-      <static>true</static>
-      <link name="link">
-        <visual name="visual">
-          <pose>61.75 0 0 0 0 0</pose>
-          <geometry>
-            <box>
-              <size>1.5 4 2</size>
-            </box>
-          </geometry>
-          <transparency>0.8</transparency>
-        </visual>
-      </link>
-    </model> -->
+    <!-- Plugin to detect if the projectile entered the hole -->
+    <!-- Debug: Run this command to face this hole -->
+    <!-- gz model -m wamv -x 555.21 -y -229.75 -z 0 -Y 0 -->
+    <plugin name="contain_placard1_big_plugin" filename="libContainPlugin.so">
+      <enabled>true</enabled>
+      <entity>blue_projectile::link</entity>
+      <namespace>vrx/dock_2022_placard1_big_hole</namespace>
+      <pose frame="robotx_dock_2022::dock_2022_placard1::link_symbols">0.6 -0.27 1.33 0 0 0</pose>
+      <geometry>
+        <box>
+          <size>0.5 0.5 0.5</size>
+        </box>
+      </geometry>
+    </plugin>
+    <!-- Plugin to detect if the projectile entered the hole -->
+    <!-- Debug: Run this command to face this hole -->
+    <!-- gz model -m wamv -x 555.28 -y -230.32 -z 0 -Y -0.13 -->
+    <plugin name="contain_placard1_small_plugin" filename="libContainPlugin.so">
+      <enabled>true</enabled>
+      <entity>blue_projectile::link</entity>
+      <namespace>vrx/dock_2022_placard1_small_hole</namespace>
+      <pose frame="robotx_dock_2022::dock_2022_placard1::link_symbols">-0.6 -0.27 1.33 0 0 0</pose>
+      <geometry>
+        <box>
+          <size>0.25 0.5 0.25</size>
+        </box>
+      </geometry>
+    </plugin>
+    <!-- Plugin to detect if the projectile entered the hole -->
+    <!-- Debug: Run this command to face this hole -->
+    <!-- gz model -m wamv -x 555.21 -y -223.75 -z 0 -Y 0 -->
+    <plugin name="contain_placard2_big_plugin" filename="libContainPlugin.so">
+      <enabled>true</enabled>
+      <entity>blue_projectile::link</entity>
+      <namespace>vrx/dock_2022_placard2_big_hole</namespace>
+      <pose frame="robotx_dock_2022::dock_2022_placard2::link_symbols">0.6 -0.27 1.33 0 0 0</pose>
+      <geometry>
+        <box>
+          <size>0.5 0.5 0.5</size>
+        </box>
+      </geometry>
+    </plugin>
+    <!-- Plugin to detect if the projectile entered the hole -->
+    <!-- Debug: Run this command to face this hole -->
+    <!-- gz model -m wamv -x 555.25 -y -223.75 -z 0 -Y -0.23 -->
+    <plugin name="contain_placard2_small_plugin" filename="libContainPlugin.so">
+      <enabled>true</enabled>
+      <entity>blue_projectile::link</entity>
+      <namespace>vrx/dock_2022_placard2_small_hole</namespace>
+      <pose frame="robotx_dock_2022::dock_2022_placard2::link_symbols">-0.6 -0.27 1.33 0 0 0</pose>
+      <geometry>
+        <box>
+          <size>0.25 0.5 0.25</size>
+        </box>
+      </geometry>
+    </plugin>
+    <!-- Plugin to detect if the projectile entered the hole -->
+    <!-- Debug: Run this command to face this hole -->
+    <!-- gz model -m wamv -x 555.25 -y -217.75 -z 0 -Y 0 -->
+    <plugin name="contain_placard3_big_plugin" filename="libContainPlugin.so">
+      <enabled>true</enabled>
+      <entity>blue_projectile::link</entity>
+      <namespace>vrx/dock_2022_placard3_big_hole</namespace>
+      <pose frame="robotx_dock_2022::dock_2022_placard3::link_symbols">0.6 -0.27 1.33 0 0 0</pose>
+      <geometry>
+        <box>
+          <size>0.5 0.5 0.5</size>
+        </box>
+      </geometry>
+    </plugin>
+    <!-- Plugin to detect if the projectile entered the hole -->
+    <!-- Debug: Run this command to face this hole -->
+    <!-- gz model -m wamv -x 555.25 -y -217.75 -z 0 -Y -0.25 -->
+    <plugin name="contain_placard3_small_plugin" filename="libContainPlugin.so">
+      <enabled>true</enabled>
+      <entity>blue_projectile::link</entity>
+      <namespace>vrx/dock_2022_placard3_small_hole</namespace>
+      <pose frame="robotx_dock_2022::dock_2022_placard3::link_symbols">-0.6 -0.27 1.33 0 0 0</pose>
+      <geometry>
+        <box>
+          <size>0.25 0.5 0.25</size>
+        </box>
+      </geometry>
+    </plugin>
+    <!-- The scoring plugin -->
+    <plugin name="scan_dock__deliver_scoring_plugin"
+            filename="libscan_dock_scoring_plugin.so">
+      <!-- Parameters for scoring_plugin -->
+      <vehicle>wamv</vehicle>
+      <task_name>scan_dock_deliver</task_name>
+      <initial_state_duration>3</initial_state_duration>
+      <ready_state_duration>3</ready_state_duration>
+      <running_state_duration>3000</running_state_duration>
+      <release_joints>
+        <joint>
+          <name>wamv_external_pivot_joint</name>
+        </joint>
+        <joint>
+          <name>wamv_external_riser</name>
+        </joint>
+      </release_joints>
+      <!-- Color sequence checker -->
+      <robot_namespace>vrx</robot_namespace>
+      <color_sequence_service>scan_dock/color_sequence</color_sequence_service>
+      <color_1>blue</color_1>
+      <color_2>green</color_2>
+      <color_3>red</color_3>
+      <!-- Dock checkers -->
+      <dock_bonus_points>15</dock_bonus_points>
+      <correct_dock_bonus_points>20</correct_dock_bonus_points>
+      <bays>
+        <bay>
+          <name>bay1</name>
+          <internal_activation_topic>/vrx/dock_2022/bay_1/contain</internal_activation_topic>
+          <external_activation_topic>/vrx/dock_2022/bay_1_external/contain</external_activation_topic>
+          <symbol_topic>/vrx/dock_2022_placard1/symbol</symbol_topic>
+          <min_dock_time>10.0</min_dock_time>
+          <dock_allowed>false</dock_allowed>
+          <symbol>red_circle</symbol>
+        </bay>
+        <bay>
+          <name>bay2</name>
+          <internal_activation_topic>/vrx/dock_2022/bay_2/contain</internal_activation_topic>
+          <external_activation_topic>/vrx/dock_2022/bay_2_external/contain</external_activation_topic>
+          <symbol_topic>/vrx/dock_2022_placard2/symbol</symbol_topic>
+          <min_dock_time>10.0</min_dock_time>
+          <dock_allowed>true</dock_allowed>
+          <symbol>blue_circle</symbol>
+        </bay>
+        <bay>
+          <name>bay3</name>
+          <internal_activation_topic>/vrx/dock_2022/bay_3/contain</internal_activation_topic>
+          <external_activation_topic>/vrx/dock_2022/bay_3_external/contain</external_activation_topic>
+          <symbol_topic>/vrx/dock_2022_placard3/symbol</symbol_topic>
+          <min_dock_time>10.0</min_dock_time>
+          <dock_allowed>true</dock_allowed>
+          <symbol>yellow_rectangle</symbol>
+        </bay>
+      </bays>
+      <!-- Shooting targets -->
+      <targets>
+        <!-- Placard #1 -->
+        <target>
+          <topic>vrx/dock_2022_placard1_big_hole/contain</topic>
+          <bonus_points>5</bonus_points>
+        </target>
+        <target>
+          <topic>vrx/dock_2022_placard1_small_hole/contain</topic>
+          <bonus_points>10</bonus_points>
+        </target>
+        <!-- Placard #2 -->
+        <target>
+          <topic>vrx/dock_2022_placard2_big_hole/contain</topic>
+          <bonus_points>5</bonus_points>
+        </target>
+        <target>
+          <topic>vrx/dock_2022_placard2_small_hole/contain</topic>
+          <bonus_points>10</bonus_points>
+        </target>
+        <!-- Placard #3 -->
+        <target>
+          <topic>vrx/dock_2022_placard3_big_hole/contain</topic>
+          <bonus_points>5</bonus_points>
+        </target>
+        <target>
+          <topic>vrx/dock_2022_placard3_small_hole/contain</topic>
+          <bonus_points>10</bonus_points>
+        </target>
+      </targets>
+    </plugin>
+    <!-- Triggers a message when the vehicle enters and exits the bay #1 -->
+    <plugin name="vehicle_docked_bay1" filename="libContainPlugin.so">
+      <entity>wamv::wamv/base_link</entity>
+      <namespace>vrx/dock_2022/bay_1</namespace>
+      <pose frame="robotx_dock_2022::dock_2022_placard1::placard::link">0 -4.5 -1.5 0 0 0</pose>
+      <geometry>
+        <box>
+          <size>1.5 4 2</size>
+        </box>
+      </geometry>
+    </plugin>
+    <plugin name="vehicle_docked_bay1_exterior" filename="libContainPlugin.so">
+      <entity>wamv::wamv/base_link</entity>
+      <namespace>vrx/dock_2022/bay_1_external</namespace>
+      <pose frame="robotx_dock_2022::dock_2022_placard1::placard::link">0 -9.5 -1.5 0 0 0</pose>
+      <geometry>
+        <box>
+          <size>5.5 1.5 2</size>
+        </box>
+      </geometry>
+    </plugin>
+    <!-- Triggers a message when the vehicle enters and exits the bay #2 -->
+    <plugin name="vehicle_docked_bay2" filename="libContainPlugin.so">
+      <entity>wamv::wamv/base_link</entity>
+      <namespace>vrx/dock_2022/bay_2</namespace>
+      <pose frame="robotx_dock_2022::dock_2022_placard2::placard::link">0 -4.5 -1.5 0 0 0</pose>
+      <geometry>
+        <box>
+          <size>1.5 4 2</size>
+        </box>
+      </geometry>
+    </plugin>
+    <plugin name="vehicle_docked_bay2_exterior" filename="libContainPlugin.so">
+      <entity>wamv::wamv/base_link</entity>
+      <namespace>vrx/dock_2022/bay_2_external</namespace>
+      <pose frame="robotx_dock_2022::dock_2022_placard2::placard::link">0 -9.5 -1.5 0 0 0</pose>
+      <geometry>
+        <box>
+          <size>5.5 1.5 2</size>
+        </box>
+      </geometry>
+    </plugin>
+    <!-- Triggers a message when the vehicle enters and exits the bay #3 -->
+    <plugin name="vehicle_docked_bay3" filename="libContainPlugin.so">
+      <entity>wamv::wamv/base_link</entity>
+      <namespace>vrx/dock_2022/bay_3</namespace>
+      <pose frame="robotx_dock_2022::dock_2022_placard3::placard::link">0 -4.5 -1.5 0 0 0</pose>
+      <geometry>
+        <box>
+          <size>1.5 4 2</size>
+        </box>
+      </geometry>
+    </plugin>
+    <plugin filename="libContainPlugin.so" name="vehicle_docked_bay3_exterior">
+      <entity>wamv::wamv/base_link</entity>
+      <namespace>vrx/dock_2022/bay_3_external</namespace>
+      <pose frame="robotx_dock_2022::dock_2022_placard3::placard::link">0 -9.5 -1.5 0 0 0</pose>
+      <geometry>
+        <box>
+          <size>5.5 1.5 2</size>
+        </box>
+      </geometry>
+    </plugin>
   </world>
 </sdf>

File: vrx_gazebo/worlds/sydneyregatta.world.xacro (robot description, xacro)
@@ -14,5 +14,5 @@
         <wind_obj>
           <name>wamv</name>
-          <link_name>base_link</link_name>
+          <link_name>wamv/base_link</link_name>
           <coeff_vector>0.5 0.5 0.33</coeff_vector>
         </wind_obj>

File: wamv_gazebo/urdf/ball_shooter/ball_shooter.xacro (robot description, xacro)
@@ -46,5 +46,5 @@
           <pose>0.14 0 0.09 0 0 0</pose>
         </projectile>
-        <shot_force>250</shot_force>
+        <shot_force>300</shot_force>
         <topic>${namespace}/${shooter_namespace}${name}/fire</topic>
       </plugin>

File: wamv_gazebo/urdf/wamv_gazebo.urdf.xacro (robot description, xacro)
@@ -122,7 +122,7 @@
       <xacro:wamv_pinger name="pinger" position="1.0 0 -1.0" />
     </xacro:if>
-    <!-- Add ball shooter (default pitch angle: -15 deg) -->
+    <!-- Add ball shooter (default pitch angle: ~-60 deg) -->
     <xacro:if value="$(arg ball_shooter_enabled)">
-      <xacro:wamv_ball_shooter name="ball_shooter" position="0.54 0.30 1.296" orientation="0 -0.261799 0"/>
+      <xacro:wamv_ball_shooter name="ball_shooter" position="0.54 0.30 1.296" orientation="0 -1.04 0"/>
     </xacro:if>
     <!-- ==== VRX sensor configuration ==== -->
@@ -144,6 +144,6 @@
       <!-- Add pinger -->
       <xacro:wamv_pinger name="pinger" position="1.0 0 -1.0" />
-      <!-- Add ball shooter (default pitch angle: -15 deg) -->
-      <xacro:wamv_ball_shooter name="ball_shooter" position="0.54 0.30 1.296" orientation="0 -0.261799 0"/>
+      <!-- Add ball shooter (default pitch angle: ~-60 deg) -->
+      <xacro:wamv_ball_shooter name="ball_shooter" position="0.54 0.30 1.296" orientation="0 -1.04 0"/>
     </xacro:if>
   </xacro:unless>
