Commit message: New ball shooter plugin for the "Scan and Dock and Deliver" task (#311)
* Add ball shooter plugin.

Signed-off-by: Carlos Agüero <caguero@openrobotics.org>

File: vrx_gazebo/worlds/sydneyregatta.xacro (robot description, xacro)
@@ -76,4 +76,16 @@
       <uri>model://ground_station</uri>
     </include>
+    <!-- A bowl to hold the blue projectile -->
+    <include>
+      <name>bowl</name>
+      <pose>533 -146.44 1.71 0 0 0</pose>
+      <uri>model://bowl</uri>
+    </include>
+    <!-- The projectile for the ball shooter -->
+    <include>
+      <name>blue_projectile</name>
+      <pose>533 -146.44 1.74 0 0 0</pose>
+      <uri>model://blue_projectile</uri>
+    </include>
   </xacro:macro>
 </world>

File: wamv_gazebo/urdf/wamv_gazebo.urdf.xacro (robot description, xacro)
@@ -12,8 +12,10 @@
   <xacro:arg name="vrx_sensors_enabled" default="false" />
   <xacro:arg name="pinger_enabled" default="false" />
+  <xacro:arg name="ball_shooter_enabled" default="false" />
   <xacro:arg name="thruster_namespace" default="thrusters/"/>
   <xacro:arg name="camera_namespace" default="cameras/"/>
   <xacro:arg name="sensor_namespace" default="sensors/"/>
   <xacro:arg name="pinger_namespace" default="pingers/"/>
+  <xacro:arg name="shooter_namespace" default="shooters/"/>
   <!-- Note: this is only used for some sensors that do not correctly use the
   robotNamespace parameter -->
@@ -23,4 +25,5 @@
   <xacro:property name="sensor_namespace" value="$(arg sensor_namespace)" scope="global" />
   <xacro:property name="pinger_namespace" value="$(arg pinger_namespace)" scope="global" />
+  <xacro:property name="shooter_namespace" value="$(arg shooter_namespace)" scope="global" />
   <xacro:property name="namespace" value="$(arg namespace)" scope="global" />
   <!-- Sensor yaml file -->
@@ -119,4 +122,8 @@
       <xacro:wamv_pinger name="pinger" position="1.0 0 -1.0" />
     </xacro:if>
+    <!-- Add ball shooter -->
+    <xacro:if value="$(arg ball_shooter_enabled)">
+      <xacro:wamv_ball_shooter name="ball_shooter" position="2.0 0 -1.0" />
+    </xacro:if>
     <!-- ==== VRX sensor configuration ==== -->
     <xacro:if value="$(arg vrx_sensors_enabled)">
@@ -137,4 +144,6 @@
       <!-- Add pinger -->
       <xacro:wamv_pinger name="pinger" position="1.0 0 -1.0" />
+      <!-- Add ball shooter -->
+      <xacro:wamv_ball_shooter name="ball_shooter" position="0.55 0.35 1.4" orientation="0 -1.0472 0"/>
     </xacro:if>
   </xacro:unless>

Commit message: Updated GPS heading and coordinates for correct lat/lon orientation

File: vrx_gazebo/worlds/sydneyregatta.xacro (robot description, xacro)
@@ -20,5 +20,5 @@
       <elevation>0.0</elevation>
       <!-- For legacy gazebo reasons, need to rotate -->
-      <!--<heading_deg>180</heading_deg>-->
+      <heading_deg>180</heading_deg>
     </spherical_coordinates>
     <!-- A global light source -->

File: wamv_gazebo/urdf/sensors/wamv_gps.xacro (robot description, xacro)
@@ -1,5 +1,5 @@
 <?xml version="1.0" encoding="UTF-8"?>
 <robot xmlns:xacro="http://ros.org/wiki/xacro">
-  <xacro:macro name="wamv_gps" params="name:=gps x:=0.3 y:=0 z:=1.3 R:=0 P:=0 Y:=0 lat:=21.30996 lon:=-157.8901 elev:=0.0 update_rate:=15">
+  <xacro:macro name="wamv_gps" params="name:=gps x:=0.3 y:=0 z:=1.3 R:=0 P:=0 Y:=0 lat:=-33.724223 lon:=150.679736 elev:=0.0 update_rate:=15">
     <link name="${namespace}/${name}_link">
       <visual name="${name}_visual">
@@ -50,5 +50,5 @@
         <referenceLongitude>${lon}</referenceLongitude>
         <referenceAltitude>${elev}</referenceAltitude>
-        <referenceHeading>90</referenceHeading>
+        <referenceHeading>270</referenceHeading>
         <offset>0.0 0.0 0.0</offset>
         <drift>0.0 0.0 0.0</drift>

Commit message: Wildlife scoring plugin - part 2.
Signed-off-by: Carlos Agüero <caguero@openrobotics.org>

File: vrx_gazebo/worlds/sydneyregatta.xacro (robot description, xacro)
@@ -28,5 +28,5 @@
     <gui fullscreen='0'>
       <camera name='user_camera'>
-        <pose frame=''>478 -148.66 13.58 0 0.25 -0.21</pose>
+        <pose frame=''>550 -139 49 0 0.82 -2.45</pose>
         <view_controller>orbit</view_controller>
       </camera>

File: vrx_gazebo/worlds/wildlife_task.world.xacro (robot description, xacro)
@@ -9,5 +9,5 @@
     <xacro:ocean_waves/>
     <!--wind for the wamv-->
-    <xacro:include filename="$(find vrx_gazebo)/worlds/xacros/usv_wind_plugin.xacro"/>
+    <!-- <xacro:include filename="$(find vrx_gazebo)/worlds/xacros/usv_wind_plugin.xacro"/>
     <xacro:usv_wind_gazebo direction = "270" ros_update_rate="10">
       <wind_objs>
@@ -18,9 +18,9 @@
         </wind_obj>
       </wind_objs>
-    </xacro:usv_wind_gazebo>
+    </xacro:usv_wind_gazebo> -->
     <!-- The VRX animal buoys -->
     <include>
       <uri>model://animal_buoys</uri>
-      <pose>512 -170 0 0 0 0</pose>
+      <pose>512 -180 0 0 0 0</pose>
     </include>
     <!-- The scoring plugin -->
@@ -58,8 +58,14 @@
       </buoys>
       <animals_model_name>animal_buoys</animals_model_name>
-      <engagement_distance>10.0</engagement_distance>
+      <engagement_distance>15.0</engagement_distance>
       <obstacle_penalty>10.0</obstacle_penalty>
       <time_bonus>30.0</time_bonus>
       <animals_topic>/vrx/wildlife/animals/poses</animals_topic>
+      <markers>
+        <material>Gazebo/Red</material>
+        <scaling>0.2 0.2 2.0</scaling>
+        <height>0.5</height>
+        <!-- <initial_id>100</initial_id> -->
+      </markers>
     </plugin>
   </world>

Commit message: Tweaks
Signed-off-by: Carlos Agüero <caguero@openrobotics.org>

File: vrx_gazebo/worlds/sydneyregatta.xacro (robot description, xacro)
@@ -28,5 +28,5 @@
     <gui fullscreen='0'>
       <camera name='user_camera'>
-        <pose frame=''>550 -139 49 0 0.82 -2.45</pose>
+        <pose frame=''>478 -148.66 13.58 0 0.25 -0.21</pose>
         <view_controller>orbit</view_controller>
       </camera>

File: vrx_gazebo/worlds/wildlife_task.world.xacro (robot description, xacro)
@@ -71,13 +71,7 @@
         </buoy>
       </buoys>
-      <engagement_distance>15.0</engagement_distance>
+      <engagement_distance>10.0</engagement_distance>
       <time_bonus>30.0</time_bonus>
       <animals_topic>/vrx/wildlife/animals/poses</animals_topic>
-      <markers>
-        <material>Gazebo/Red</material>
-        <scaling>0.2 0.2 2.0</scaling>
-        <height>0.5</height>
-        <!-- <initial_id>100</initial_id> -->
-      </markers>
     </plugin>
   </world>

Commit message: Changing hector config to use Gazebo world SDF

File: vrx_gazebo/worlds/sydneyregatta.xacro (robot description, xacro)
@@ -12,5 +12,6 @@
       <origin_visual>0</origin_visual>
     </scene>
-    <!-- Estimated latitude/longitude of sydneyregatta from satellite imagery -->
+    <!-- Estimated latitude/longitude of sydneyregatta
+	 from satellite imagery -->
     <spherical_coordinates>
       <surface_model>EARTH_WGS84</surface_model>
@@ -19,6 +20,5 @@
       <longitude_deg>150.679736</longitude_deg>
       <elevation>0.0</elevation>
-      <!-- For legacy gazebo reasons, need to rotate -->
-      <heading_deg>180</heading_deg>
+      <heading_deg>0.0</heading_deg>
     </spherical_coordinates>
     <!-- A global light source -->

File: wamv_gazebo/urdf/sensors/wamv_gps.xacro (robot description, xacro)
@@ -1,5 +1,6 @@
 <?xml version="1.0" encoding="UTF-8"?>
 <robot xmlns:xacro="http://ros.org/wiki/xacro">
-  <xacro:macro name="wamv_gps" params="name:=gps x:=0.3 y:=0 z:=1.3 R:=0 P:=0 Y:=0 lat:=-33.724223 lon:=150.679736 elev:=0.0 update_rate:=15">
+  <xacro:macro name="wamv_gps" params="name:=gps x:=0.3 y:=0 z:=1.3
+				       R:=0 P:=0 Y:=0 update_rate:=15">
     <link name="${namespace}/${name}_link">
       <visual name="${name}_visual">
@@ -22,5 +23,6 @@
       <inertial>
         <mass value="1"/>
-        <inertia ixx="0.006458" ixy="0.0" ixz="0.0" iyy="0.006458" iyz="0.0" izz="0.01125"/>
+        <inertia ixx="0.006458" ixy="0.0" ixz="0.0"
+		 iyy="0.006458" iyz="0.0" izz="0.01125"/>
       </inertial>
     </link>
@@ -46,9 +48,9 @@
              https://bitbucket.org/osrf/vrx/issues/64 -->
         <velocityTopicName>${namespace}/${sensor_namespace}gps/gps/fix_velocity</velocityTopicName>
-        <!-- Location of origin of Gazebo Sand Island map -->
-        <referenceLatitude>${lat}</referenceLatitude>
-        <referenceLongitude>${lon}</referenceLongitude>
-        <referenceAltitude>${elev}</referenceAltitude>
-        <referenceHeading>270</referenceHeading>
+        <!-- Tell the plugin to use the spherical_coordiantes parameters
+	     from SDF.
+	     https://github.com/tu-darmstadt-ros-pkg/hector_gazebo/blob/melodic-devel/hector_gazebo_plugins/src/gazebo_ros_gps.cpp#L101
+	-->
+	<useWorldSphericalCoordinates>true</useWorldSphericalCoordinates>
         <offset>0.0 0.0 0.0</offset>
         <drift>0.0 0.0 0.0</drift>
