Commit message: incremental

File: vrx_gazebo/worlds/xacros/dock_2016.xacro (robot description, xacro)
@@ -1,6 +1,7 @@
 <?xml version="1.0"?>
 <world xmlns:xacro="http://ros.org/wiki/xacro">
-  <xacro:macro name="dock_2016" params="x:=72 y:=22 z:=0 R:=0 P:=0 Y:=-2.78">
+  <xacro:macro name="dock_2016" params=" name x:=72 y:=22 z:=0 R:=0 P:=0 Y:=-2.78">
     <include>
+      <name>${name}</name>
       <uri>model://dock_2016</uri>
       <pose>${x} ${y} ${z} ${R} ${P} ${Y}</pose>

File: vrx_gazebo/worlds/xacros/dock_2018.xacro (robot description, xacro)
@@ -1,6 +1,7 @@
 <?xml version="1.0"?>
 <world xmlns:xacro="http://ros.org/wiki/xacro">
-  <xacro:macro name="dock_2018" params="x:=-2 y:=-18 z:=0 R:=0 P:=0 Y:=0.2">
+  <xacro:macro name="dock_2018" params="name x:=-2 y:=-18 z:=0 R:=0 P:=0 Y:=0.2">
     <include>
+      <name>${name}</name>
       <uri>model://dock_2018</uri>
       <pose>${x} ${y} ${z} ${R} ${P} ${Y}</pose>

File: vrx_gazebo/worlds/xacros/light_buoy.xacro (robot description, xacro)
@@ -1,6 +1,7 @@
 <?xml version="1.0"?>
 <world xmlns:xacro="http://ros.org/wiki/xacro">
-  <xacro:macro name="light_buoy" params="x:=110 y:=28 z:=0.25 R:=0 P:=0 Y:=0">
+  <xacro:macro name="light_buoy" params="name x:=110 y:=28 z:=0.25 R:=0 P:=0 Y:=0">
     <include>
+      <name>${name}</name>
       <uri>model://robotx_light_buoy</uri>
       <pose>${x} ${y} ${z} ${R} ${P} ${Y}</pose>

File: vrx_gazebo/worlds/xacros/nav_challenge.xacro (robot description, xacro)
@@ -1,6 +1,7 @@
 <?xml version="1.0"?>
 <world xmlns:xacro="http://ros.org/wiki/xacro">
-  <xacro:macro name="nav_challenge" params="x:=58 y:=68 z:=2 R:=0 P:=0 Y:=0.4">
+  <xacro:macro name="nav_challenge" params="name x:=58 y:=68 z:=2 R:=0 P:=0 Y:=0.4">
     <include>
+      <name>${name}</name>
       <uri>model://robotx_navigation_challenge</uri>
       <pose>${x} ${y} ${z} ${R} ${P} ${Y}</pose>

File: vrx_gazebo/worlds/xacros/qualifying_pinger_transit_2016.xacro (robot description, xacro)
@@ -1,6 +1,7 @@
 <?xml version="1.0"?>
 <world xmlns:xacro="http://ros.org/wiki/xacro">
-  <xacro:macro name="qualifying_pinger_transit_2016" params="x:=55 y:=-50 z:=0 R:=0 P:=0 Y:=-1.3">
+  <xacro:macro name="qualifying_pinger_transit_2016" params="name x:=55 y:=-50 z:=0 R:=0 P:=0 Y:=-1.3">
     <include>
+      <name>${name}</name>
       <uri>model://robotx_2016_qualifying_pinger_transit</uri>
       <pose>${x} ${y} ${z} ${R} ${P} ${Y}</pose>
