Commit message: Incremental

File: vrx_gazebo/worlds/xacros/usv_wind_plugin.xacro (robot description, xacro)
@@ -1,5 +1,5 @@
 <?xml version="1.0"?>
 <world xmlns:xacro="http://ros.org/wiki/xacro">
-	<xacro:macro name="usv_wind_gazebo" params="**wind_objs
+  <xacro:macro name="usv_wind_gazebo" params="**wind_objs
 						    direction:=270
 						    mean_vel:=10
