Commit message: Add nav_challenge scoring plugin and gates

File: vrx_gazebo/worlds/xacros/nav_challenge.xacro (robot description, xacro)
@@ -1,5 +1,5 @@
 <?xml version="1.0"?>
 <world xmlns:xacro="http://ros.org/wiki/xacro">
-  <xacro:macro name="nav_challenge" params="name x:=58 y:=68 z:=2 R:=0 P:=0 Y:=0.4">
+  <xacro:macro name="nav_challenge" params="name x:=58 y:=68 z:=2 R:=0 P:=0 Y:=0.4 **gates">
     <include>
       <name>${name}</name>
@@ -7,4 +7,27 @@
       <pose>${x} ${y} ${z} ${R} ${P} ${Y}</pose>
     </include>
+    <!-- The scoring plugin -->
+    <plugin name="navigation_scoring_plugin"
+            filename="libnavigation_scoring_plugin.so">
+      <vehicle>wamv</vehicle>
+      <task_name>navigation_course</task_name>
+      <initial_state_duration>10</initial_state_duration>
+      <ready_state_duration>10</ready_state_duration>
+      <running_state_duration>300</running_state_duration>
+      <collision_buffer>10</collision_buffer>
+      <release_joints>
+        <joint>
+          <name>wamv_external_pivot_joint</name>
+        </joint>
+        <joint>
+          <name>wamv_external_riser</name>
+        </joint>
+      </release_joints>
+      <course_name>vrx_navigation_course</course_name>
+      <obstacle_penalty>10.0</obstacle_penalty>
+      <gates>
+        <xacro:insert_block name="gates"/>
+      </gates>
+    </plugin>
   </xacro:macro>
 </world>

Commit message: added scoring plugin to the nav_challenge xacro for world generation

File: vrx_gazebo/worlds/xacros/nav_challenge.xacro (robot description, xacro)
@@ -1,10 +1,60 @@
 <?xml version="1.0"?>
 <world xmlns:xacro="http://ros.org/wiki/xacro">
-  <xacro:macro name="nav_challenge" params="name x:=58 y:=68 z:=2 R:=0 P:=0 Y:=0.4">
+  <xacro:macro name="nav_challenge" params="name='nav_challenge' uri:=navigation_course x:=58 y:=68 z:=2 R:=0 P:=0 Y:=0.4">
+    <!-- The VRX navigation course -->
     <include>
       <name>${name}</name>
-      <uri>model://robotx_navigation_challenge</uri>
+      <uri>model://${uri}</uri>
       <pose>${x} ${y} ${z} ${R} ${P} ${Y}</pose>
     </include>
+    <!-- The scoring plugin -->
+    <plugin name="navigation_scoring_plugin"
+            filename="libnavigation_scoring_plugin.so">
+      <vehicle>wamv</vehicle>
+      <initial_state_duration>10</initial_state_duration>
+      <ready_state_duration>10</ready_state_duration>
+      <running_state_duration>300</running_state_duration>
+      <collision_buffer>10</collision_buffer>
+      <release_joints>
+        <joint>
+          <name>wamv_external_pivot_joint</name>
+        </joint>
+        <joint>
+          <name>wamv_external_riser</name>
+        </joint>
+      </release_joints>
+      <course_name>${name}</course_name>
+      <obstacle_penalty>10.0</obstacle_penalty>
+      <gates>
+        <gate>
+          <left_marker>red_bound_0</left_marker>
+          <right_marker>green_bound_0</right_marker>
+        </gate>
+        <gate>
+          <left_marker>red_bound_1</left_marker>
+          <right_marker>green_bound_1</right_marker>
+        </gate>
+        <gate>
+          <left_marker>red_bound_2</left_marker>
+          <right_marker>green_bound_2</right_marker>
+        </gate>
+        <gate>
+          <left_marker>red_bound_3</left_marker>
+          <right_marker>green_bound_3</right_marker>
+        </gate>
+        <gate>
+          <left_marker>red_bound_4</left_marker>
+          <right_marker>green_bound_4</right_marker>
+        </gate>
+        <gate>
+          <left_marker>red_bound_5</left_marker>
+          <right_marker>green_bound_5</right_marker>
+        </gate>
+        <gate>
+          <left_marker>red_bound_6</left_marker>
+          <right_marker>green_bound_6</right_marker>
+        </gate>
+      </gates>
+    </plugin>
   </xacro:macro>
 </world>

Commit message: Adding running_duration parameter to the nav_challenge.xacro.

File: vrx_gazebo/worlds/xacros/nav_challenge.xacro (robot description, xacro)
@@ -1,5 +1,5 @@
 <?xml version="1.0"?>
 <world xmlns:xacro="http://ros.org/wiki/xacro">
-  <xacro:macro name="nav_challenge" params="name='nav_challenge' uri:=navigation_course x:=58 y:=68 z:=2 R:=0 P:=0 Y:=0.4 **gates">
+  <xacro:macro name="nav_challenge" params="name='nav_challenge' uri:=navigation_course x:=58 y:=68 z:=2 R:=0 P:=0 Y:=0.4 running_duration:=300 **gates">
     <!-- The VRX navigation course -->
     <include>
@@ -15,5 +15,5 @@
       <initial_state_duration>10</initial_state_duration>
       <ready_state_duration>10</ready_state_duration>
-      <running_state_duration>300</running_state_duration>
+      <running_state_duration>${running_duration}</running_state_duration>
       <collision_buffer>10</collision_buffer>
       <release_joints>
