Commit message: adding insert blocks to generate debug markers for wayfinding and stationkeeping tasks

File: vrx_gazebo/worlds/xacros/stationkeeping.xacro (robot description, xacro)
@@ -1,5 +1,5 @@
 <?xml version="1.0"?>
 <world xmlns:xacro="http://ros.org/wiki/xacro">
-  <xacro:macro name="stationkeeping" params="lat:=21.31091 lon:=-157.88868 heading:=0.0">
+  <xacro:macro name="stationkeeping" params="**wp_markers lat:=21.31091 lon:=-157.88868 heading:=0.0">
     <plugin name="stationkeeping_scoring_plugin"
           filename="libstationkeeping_scoring_plugin.so">
@@ -19,4 +19,5 @@
         </joint>
       </release_joints>
+      <xacro:insert_block name="wp_markers" />
     </plugin>
   </xacro:macro>

File: vrx_gazebo/worlds/xacros/wayfinding.xacro (robot description, xacro)
@@ -1,5 +1,5 @@
 <?xml version="1.0"?>
 <world xmlns:xacro="http://ros.org/wiki/xacro">
-  <xacro:macro name="wayfinding" params="**waypoints">
+  <xacro:macro name="wayfinding" params="**wp_markers **waypoints">
     <plugin name="wayfinding_scoring_plugin"
             filename="libwayfinding_scoring_plugin.so">
@@ -21,4 +21,5 @@
         </joint>
       </release_joints>
+      <xacro:insert_block name="wp_markers" />
     </plugin>
   </xacro:macro>
