Commit message: fixed xacro insert block ordering issue

File: vrx_gazebo/worlds/xacros/dock.xacro (robot description, xacro)
@@ -1,76 +1,74 @@
 <?xml version="1.0" ?>
 <!-- World containing sandisland model and some course challenges -->
-<sdf version="1.6" xmlns:xacro="http://ros.org/wiki/xacro">
-  <world name="robotx_dock">
-    <xacro:macro name="dock">
-      <!-- The 2018 dock with the two placards -->
-      <include>
-        <uri>model://dock_2018</uri>
-        <pose>60 -2.75 0 0 0 0</pose>
-      </include>
-      <!-- The scoring plugin -->
-      <plugin name="scan_dock_scoring_plugin"
-              filename="libscan_dock_scoring_plugin.so">
-        <!-- Parameters for scoring_plugin -->
-        <vehicle>wamv</vehicle>
-        <task_name>scan_dock</task_name>
-        <initial_state_duration>3</initial_state_duration>
-        <ready_state_duration>3</ready_state_duration>
-        <running_state_duration>300</running_state_duration>
-        <release_joints>
-          <joint>
-            <name>wamv_external_pivot_joint</name>
-          </joint>
-          <joint>
-            <name>wamv_external_riser</name>
-          </joint>
-        </release_joints>
-        <!-- Color sequence checker -->
-        <robot_namespace>vrx</robot_namespace>
-        <color_sequence_service>scan_dock/color_sequence</color_sequence_service>
-        <color_1>red</color_1>
-        <color_2>green</color_2>
-        <color_3>blue</color_3>
-        <!-- Dock checkers -->
-        <bays>
-          <bay>
-            <name>bay1</name>
-            <activation_topic>/vrx/dock_2018/bay_1/contain</activation_topic>
-            <min_dock_time>10.0</min_dock_time>
-            <dock_allowed>false</dock_allowed>
-          </bay>
-          <bay>
-            <name>bay2</name>
-            <activation_topic>/vrx/dock_2018/bay_2/contain</activation_topic>
-            <min_dock_time>10.0</min_dock_time>
-            <dock_allowed>true</dock_allowed>
-            <announce_symbol>red_circle</announce_symbol>
-          </bay>
-        </bays>
-        <placard_color_shape>red_triangle</placard_color_shape>
-      </plugin>
-      <!-- Triggers a message when the vehicle enters and exits the bay #1 -->
-      <plugin name="vehicle_docked_bay1" filename="libContainPlugin.so">
-        <entity>wamv::base_link</entity>
-        <namespace>vrx/dock_2018/bay_1</namespace>
-        <pose frame="robotx_dock_2018::dock_2018_placard1::placard::link">0 -5 -1.5 0 0 0</pose>
-        <geometry>
-          <box>
-            <size>4 1.5 2</size>
-          </box>
-        </geometry>
-      </plugin>
-      <!-- Triggers a message when the vehicle enters and exits the bay #2 -->
-      <plugin name="vehicle_docked_bay2" filename="libContainPlugin.so">
-        <entity>wamv::base_link</entity>
-        <namespace>vrx/dock_2018/bay_2</namespace>
-        <pose frame="robotx_dock_2018::dock_2018_placard2::placard::link">0 5 -1.5 0 0 0</pose>
-        <geometry>
-          <box>
-            <size>4 1.5 2</size>
-          </box>
-        </geometry>
-      </plugin>
-    </xacro:macro>
-  </world>
-</sdf>
+<world xmlns:xacro="http://ros.org/wiki/xacro">
+  <xacro:macro name="dock">
+    <!-- The 2018 dock with the two placards -->
+    <include>
+      <uri>model://dock_2018</uri>
+      <pose>60 -2.75 0 0 0 0</pose>
+    </include>
+    <!-- The scoring plugin -->
+    <plugin name="scan_dock_scoring_plugin"
+            filename="libscan_dock_scoring_plugin.so">
+      <!-- Parameters for scoring_plugin -->
+      <vehicle>wamv</vehicle>
+      <task_name>scan_dock</task_name>
+      <initial_state_duration>3</initial_state_duration>
+      <ready_state_duration>3</ready_state_duration>
+      <running_state_duration>300</running_state_duration>
+      <release_joints>
+        <joint>
+          <name>wamv_external_pivot_joint</name>
+        </joint>
+        <joint>
+          <name>wamv_external_riser</name>
+        </joint>
+      </release_joints>
+      <!-- Color sequence checker -->
+      <robot_namespace>vrx</robot_namespace>
+      <color_sequence_service>scan_dock/color_sequence</color_sequence_service>
+      <color_1>red</color_1>
+      <color_2>green</color_2>
+      <color_3>blue</color_3>
+      <!-- Dock checkers -->
+      <bays>
+        <bay>
+          <name>bay1</name>
+          <activation_topic>/vrx/dock_2018/bay_1/contain</activation_topic>
+          <min_dock_time>10.0</min_dock_time>
+          <dock_allowed>false</dock_allowed>
+        </bay>
+        <bay>
+          <name>bay2</name>
+          <activation_topic>/vrx/dock_2018/bay_2/contain</activation_topic>
+          <min_dock_time>10.0</min_dock_time>
+          <dock_allowed>true</dock_allowed>
+          <announce_symbol>red_circle</announce_symbol>
+        </bay>
+      </bays>
+      <placard_color_shape>red_triangle</placard_color_shape>
+    </plugin>
+    <!-- Triggers a message when the vehicle enters and exits the bay #1 -->
+    <plugin name="vehicle_docked_bay1" filename="libContainPlugin.so">
+      <entity>wamv::base_link</entity>
+      <namespace>vrx/dock_2018/bay_1</namespace>
+      <pose frame="robotx_dock_2018::dock_2018_placard1::placard::link">0 -5 -1.5 0 0 0</pose>
+      <geometry>
+        <box>
+          <size>4 1.5 2</size>
+        </box>
+      </geometry>
+    </plugin>
+    <!-- Triggers a message when the vehicle enters and exits the bay #2 -->
+    <plugin name="vehicle_docked_bay2" filename="libContainPlugin.so">
+      <entity>wamv::base_link</entity>
+      <namespace>vrx/dock_2018/bay_2</namespace>
+      <pose frame="robotx_dock_2018::dock_2018_placard2::placard::link">0 5 -1.5 0 0 0</pose>
+      <geometry>
+        <box>
+          <size>4 1.5 2</size>
+        </box>
+      </geometry>
+    </plugin>
+  </xacro:macro>
+</world>

File: vrx_gazebo/worlds/xacros/include_all_xacros.xacro (robot description, xacro)
@@ -1,5 +1,5 @@
 <?xml version="1.0"?>
 <world xmlns:xacro="http://ros.org/wiki/xacro">
-    <xacro:macro name="include_all_xacros">
+  <xacro:macro name="include_all_xacros">
     <xacro:include filename="$(find vrx_gazebo)/worlds/sandisland.xacro" />
     <xacro:include filename="$(find vrx_gazebo)/worlds/xacros/sandisland_minus_scene.xacro" />

File: vrx_gazebo/worlds/xacros/scan_and_dock.xacro (robot description, xacro)
@@ -1,81 +1,79 @@
 <?xml version="1.0" ?>
 <!-- World containing sandisland model and some course challenges -->
-<sdf version="1.6" xmlns:xacro="http://ros.org/wiki/xacro">
-  <world name="robotx_scan_and_dock">
-    <xacro:macro name="scan_and_dock">
-      <!-- The light buoy -->$
-      <include>
-        <uri>model://robotx_light_buoy</uri>
-        <pose>90 70 0.25 0 0 0</pose>
-      </include>
-      <!-- The 2018 dock with the two placards -->
-      <include>
-        <uri>model://dock_2018</uri>
-        <pose>60 -2.75 0 0 0 0</pose>
-      </include>
-      <!-- The scoring plugin -->
-      <plugin name="scan_dock_scoring_plugin"
-              filename="libscan_dock_scoring_plugin.so">
-        <!-- Parameters for scoring_plugin -->
-        <vehicle>wamv</vehicle>
-        <task_name>scan_dock</task_name>
-        <initial_state_duration>3</initial_state_duration>
-        <ready_state_duration>3</ready_state_duration>
-        <running_state_duration>300</running_state_duration>
-        <release_joints>
-          <joint>
-            <name>wamv_external_pivot_joint</name>
-          </joint>
-          <joint>
-            <name>wamv_external_riser</name>
-          </joint>
-        </release_joints>
-        <!-- Color sequence checker -->
-        <robot_namespace>vrx</robot_namespace>
-        <color_sequence_service>scan_dock/color_sequence</color_sequence_service>
-        <color_1>red</color_1>
-        <color_2>green</color_2>
-        <color_3>blue</color_3>
-        <!-- Dock checkers -->
-        <bays>
-          <bay>
-            <name>bay1</name>
-            <activation_topic>/vrx/dock_2018/bay_1/contain</activation_topic>
-            <min_dock_time>10.0</min_dock_time>
-            <dock_allowed>false</dock_allowed>
-          </bay>
-          <bay>
-            <name>bay2</name>
-            <activation_topic>/vrx/dock_2018/bay_2/contain</activation_topic>
-            <min_dock_time>10.0</min_dock_time>
-            <dock_allowed>true</dock_allowed>
-            <announce_symbol>red_circle</announce_symbol>
-          </bay>
-        </bays>
-        <placard_color_shape>red_triangle</placard_color_shape>
-      </plugin>
-      <!-- Triggers a message when the vehicle enters and exits the bay #1 -->
-      <plugin name="vehicle_docked_bay1" filename="libContainPlugin.so">
-        <entity>wamv::base_link</entity>
-        <namespace>vrx/dock_2018/bay_1</namespace>
-        <pose frame="robotx_dock_2018::dock_2018_placard1::placard::link">0 -5 -1.5 0 0 0</pose>
-        <geometry>
-          <box>
-            <size>4 1.5 2</size>
-          </box>
-        </geometry>
-      </plugin>
-      <!-- Triggers a message when the vehicle enters and exits the bay #2 -->
-      <plugin name="vehicle_docked_bay2" filename="libContainPlugin.so">
-        <entity>wamv::base_link</entity>
-        <namespace>vrx/dock_2018/bay_2</namespace>
-        <pose frame="robotx_dock_2018::dock_2018_placard2::placard::link">0 5 -1.5 0 0 0</pose>
-        <geometry>
-          <box>
-            <size>4 1.5 2</size>
-          </box>
-        </geometry>
-      </plugin>
-    </xacro:macro>
-  </world>
-</sdf>
+<world xmlns:xacro="http://ros.org/wiki/xacro">
+  <xacro:macro name="scan_and_dock">
+    <!-- The light buoy -->$
+    <include>
+      <uri>model://robotx_light_buoy</uri>
+      <pose>90 70 0.25 0 0 0</pose>
+    </include>
+    <!-- The 2018 dock with the two placards -->
+    <include>
+      <uri>model://dock_2018</uri>
+      <pose>60 -2.75 0 0 0 0</pose>
+    </include>
+    <!-- The scoring plugin -->
+    <plugin name="scan_dock_scoring_plugin"
+            filename="libscan_dock_scoring_plugin.so">
+      <!-- Parameters for scoring_plugin -->
+      <vehicle>wamv</vehicle>
+      <task_name>scan_dock</task_name>
+      <initial_state_duration>3</initial_state_duration>
+      <ready_state_duration>3</ready_state_duration>
+      <running_state_duration>300</running_state_duration>
+      <release_joints>
+        <joint>
+          <name>wamv_external_pivot_joint</name>
+        </joint>
+        <joint>
+          <name>wamv_external_riser</name>
+        </joint>
+      </release_joints>
+      <!-- Color sequence checker -->
+      <robot_namespace>vrx</robot_namespace>
+      <color_sequence_service>scan_dock/color_sequence</color_sequence_service>
+      <color_1>red</color_1>
+      <color_2>green</color_2>
+      <color_3>blue</color_3>
+      <!-- Dock checkers -->
+      <bays>
+        <bay>
+          <name>bay1</name>
+          <activation_topic>/vrx/dock_2018/bay_1/contain</activation_topic>
+          <min_dock_time>10.0</min_dock_time>
+          <dock_allowed>false</dock_allowed>
+        </bay>
+        <bay>
+          <name>bay2</name>
+          <activation_topic>/vrx/dock_2018/bay_2/contain</activation_topic>
+          <min_dock_time>10.0</min_dock_time>
+          <dock_allowed>true</dock_allowed>
+          <announce_symbol>red_circle</announce_symbol>
+        </bay>
+      </bays>
+      <placard_color_shape>red_triangle</placard_color_shape>
+    </plugin>
+    <!-- Triggers a message when the vehicle enters and exits the bay #1 -->
+    <plugin name="vehicle_docked_bay1" filename="libContainPlugin.so">
+      <entity>wamv::base_link</entity>
+      <namespace>vrx/dock_2018/bay_1</namespace>
+      <pose frame="robotx_dock_2018::dock_2018_placard1::placard::link">0 -5 -1.5 0 0 0</pose>
+      <geometry>
+        <box>
+          <size>4 1.5 2</size>
+        </box>
+      </geometry>
+    </plugin>
+    <!-- Triggers a message when the vehicle enters and exits the bay #2 -->
+    <plugin name="vehicle_docked_bay2" filename="libContainPlugin.so">
+      <entity>wamv::base_link</entity>
+      <namespace>vrx/dock_2018/bay_2</namespace>
+      <pose frame="robotx_dock_2018::dock_2018_placard2::placard::link">0 5 -1.5 0 0 0</pose>
+      <geometry>
+        <box>
+          <size>4 1.5 2</size>
+        </box>
+      </geometry>
+    </plugin>
+  </xacro:macro>
+</world>

Commit message: incremental

File: vrx_gazebo/worlds/xacros/dock.xacro (robot description, xacro)
@@ -2,9 +2,8 @@
 <!-- World containing sandisland model and some course challenges -->
 <world xmlns:xacro="http://ros.org/wiki/xacro">
-  <xacro:macro name="dock">
-    <!-- The 2018 dock with the two placards -->
+  <xacro:macro name="dock" params="uri:=model://dock_2018 x:=60 y:=-2.75 z:=0 R:=0 P:=0 Y:=0">
     <include>
       <uri>model://dock_2018</uri>
-      <pose>60 -2.75 0 0 0 0</pose>
+      <pose>${x} ${y} ${z} ${R} ${P} ${Y}</pose>
     </include>
     <!-- The scoring plugin -->

File: vrx_gazebo/worlds/xacros/nav_challenge.xacro (robot description, xacro)
@@ -12,4 +12,5 @@
             filename="libnavigation_scoring_plugin.so">
       <vehicle>wamv</vehicle>
+      <task_name>navigation_course</task_name>
       <initial_state_duration>10</initial_state_duration>
       <ready_state_duration>10</ready_state_duration>

Commit message: dock xacro fixed

File: vrx_gazebo/worlds/xacros/dock.xacro (robot description, xacro)
@@ -2,5 +2,5 @@
 <!-- World containing sandisland model and some course challenges -->
 <world xmlns:xacro="http://ros.org/wiki/xacro">
-  <xacro:macro name="dock">
+  <xacro:macro name="dock" params="x:=60 y:=-2.75 z:=0 R:=0 P:=0 Y:=0">
     <!-- The 2018 dock with the two placards -->
     <include>

File: vrx_gazebo/worlds/xacros/scan_and_dock.xacro (robot description, xacro)
@@ -52,30 +52,9 @@
           <min_dock_time>10.0</min_dock_time>
           <dock_allowed>true</dock_allowed>
-          <symbol>blue_circle</symbol>
+          <announce_symbol>red_cross</announce_symbol>
+          <symbol>red_cross</symbol>
         </bay>
       </bays>
-      <placard_color_shape>red_triangle</placard_color_shape>
-    </plugin>
-    <!-- Triggers a message when the vehicle enters and exits the bay #1 -->
-    <plugin name="vehicle_docked_bay1" filename="libContainPlugin.so">
-      <entity>wamv::base_link</entity>
-      <namespace>vrx/dock_2018/bay_1</namespace>
-      <pose frame="robotx_dock_2018::dock_2018_placard1::placard::link">0 -5 -1.5 0 0 0</pose>
-      <geometry>
-        <box>
-          <size>4 1.5 2</size>
-        </box>
-      </geometry>
-    </plugin>
-    <!-- Triggers a message when the vehicle enters and exits the bay #2 -->
-    <plugin name="vehicle_docked_bay2" filename="libContainPlugin.so">
-      <entity>wamv::base_link</entity>
-      <namespace>vrx/dock_2018/bay_2</namespace>
-      <pose frame="robotx_dock_2018::dock_2018_placard2::placard::link">0 5 -1.5 0 0 0</pose>
-      <geometry>
-        <box>
-          <size>4 1.5 2</size>
-        </box>
-      </geometry>
+      <placard_color_shape>red_cross</placard_color_shape>
     </plugin>
   </xacro:macro>

Commit message: added more params to dock xacro

File: vrx_gazebo/worlds/xacros/dock.xacro (robot description, xacro)
@@ -2,9 +2,9 @@
 <!-- World containing sandisland model and some course challenges -->
 <world xmlns:xacro="http://ros.org/wiki/xacro">
-  <xacro:macro name="dock">
+  <xacro:macro name="dock" params="uri:=dock_2018 x:=60 y:=-2.75 z:=0 R:=0 P:=0 Y:=0">
     <!-- The 2018 dock with the two placards -->
     <include>
-      <uri>model://dock_2018</uri>
-      <pose>60 -2.75 0 0 0 0</pose>
+      <uri>model://${uri}</uri>
+      <pose>${x} ${y} ${z} ${R} ${P} ${Y}</pose>
     </include>
     <!-- The scoring plugin -->

Commit message: adding params to dock xacro for the benefit of automatically generating tasks

File: vrx_gazebo/worlds/xacros/dock.xacro (robot description, xacro)
@@ -2,5 +2,5 @@
 <!-- World containing sandisland model and some course challenges -->
 <world xmlns:xacro="http://ros.org/wiki/xacro">
-  <xacro:macro name="dock" params="uri:=dock_2018 x:=60 y:=-2.75 z:=0 R:=0 P:=0 Y:=0">
+  <xacro:macro name="dock" params="uri:=dock_2018 x:=60 y:=-2.75 z:=0 R:=0 P:=0 Y:=0 bay1_allowed:=false bay1_symbol:=red_circle bay2_allowed:=true bay2_symbol:=blue_cross">
     <!-- The 2018 dock with the two placards -->
     <include>
@@ -38,6 +38,7 @@
           <symbol_topic>/vrx/dock_2018_placard1/symbol</symbol_topic>
           <min_dock_time>10.0</min_dock_time>
-          <dock_allowed>false</dock_allowed>
-          <symbol>red_circle</symbol>
+          <dock_allowed>${bay1_allowed}</dock_allowed>
+          <announce_symbol>${bay1_symbol}</announce_symbol>
+          <symbol>${bay1_symbol}</symbol>
         </bay>
         <bay>
@@ -46,7 +47,7 @@
           <symbol_topic>/vrx/dock_2018_placard2/symbol</symbol_topic>
           <min_dock_time>10.0</min_dock_time>
-          <dock_allowed>true</dock_allowed>
-          <announce_symbol>red_cross</announce_symbol>
-          <symbol>red_cross</symbol>
+          <dock_allowed>${bay2_allowed}</dock_allowed>
+          <announce_symbol>${bay2_symbol}</announce_symbol>
+          <symbol>${bay2_symbol}</symbol>
         </bay>
       </bays>

Commit message: adds light buoys

File: vrx_gazebo/worlds/xacros/dock.xacro (robot description, xacro)
@@ -2,5 +2,9 @@
 <!-- World containing sandisland model and some course challenges -->
 <world xmlns:xacro="http://ros.org/wiki/xacro">
-  <xacro:macro name="dock" params="uri:=dock_2018 x:=60 y:=-2.75 z:=0 R:=0 P:=0 Y:=0 bay1_allowed:=false bay1_symbol:=red_circle bay2_allowed:=true bay2_symbol:=blue_cross">
+  <xacro:macro name="dock" params="uri:=dock_2018 x:=60 y:=-2.75 z:=0
+    R:=0 P:=0 Y:=0 bay1_allowed:=false bay1_symbol:=red_circle
+    bay2_allowed:=true bay2_symbol:=blue_cross
+    light_buoy_present:=false
+    lb_x:=90 lb_y:=70 lb_z:=0 lb_R:=0 lb_P:=0 lb_Y:=0">
     <!-- The 2018 dock with the two placards -->
     <include>
@@ -8,4 +12,11 @@
       <pose>${x} ${y} ${z} ${R} ${P} ${Y}</pose>
     </include>
+    <!-- Add a ligth buoy if doing Scan and Dock -->
+    <xacro:if value="${light_buoy_present}">
+      <include>
+        <uri>model://robotx_light_buoy</uri>
+        <pose>${lb_x} ${lb_y} ${lb_z} ${lb_R} ${lb_P} ${lb_Y}</pose>
+      </include>
+    </xacro:if>
     <!-- The scoring plugin -->
     <plugin name="scan_dock_scoring_plugin"

Commit message: adding model_name paramter to dock.xacro for flexibility in generating automated tasks

File: vrx_gazebo/worlds/xacros/dock.xacro (robot description, xacro)
@@ -2,5 +2,6 @@
 <!-- World containing sandisland model and some course challenges -->
 <world xmlns:xacro="http://ros.org/wiki/xacro">
-  <xacro:macro name="dock" params="uri:=dock_2018 x:=60 y:=-2.75 z:=0
+  <xacro:macro name="dock" params="model_name:=robotx_dock_2018
+    uri:=dock_2018 x:=60 y:=-2.75 z:=0
     R:=0 P:=0 Y:=0 bay1_allowed:=false bay1_symbol:=red_circle
     bay2_allowed:=true bay2_symbol:=blue_cross
@@ -69,5 +70,5 @@
       <entity>wamv::base_link</entity>
       <namespace>vrx/dock_2018/bay_1_internal</namespace>
-      <pose frame="robotx_dock_2018::dock_2018_placard1::placard::link">0 -5 -1.5 0 0 0</pose>
+      <pose frame="${model_name}::dock_2018_placard1::placard::link">0 -5 -1.5 0 0 0</pose>
       <geometry>
         <box>
@@ -80,5 +81,5 @@
       <entity>wamv::base_link</entity>
       <namespace>vrx/dock_2018/bay_1_external</namespace>
-      <pose frame="robotx_dock_2018::dock_2018_placard1::placard::link">0 -10 -1.5 0 0 0</pose>
+      <pose frame="${model_name}::dock_2018_placard1::placard::link">0 -10 -1.5 0 0 0</pose>
       <geometry>
         <box>
@@ -91,5 +92,5 @@
       <entity>wamv::base_link</entity>
       <namespace>vrx/dock_2018/bay_2_internal</namespace>
-      <pose frame="robotx_dock_2018::dock_2018_placard2::placard::link">0 5 -1.5 0 0 0</pose>
+      <pose frame="${model_name}::dock_2018_placard2::placard::link">0 5 -1.5 0 0 0</pose>
       <geometry>
         <box>
@@ -102,5 +103,5 @@
       <entity>wamv::base_link</entity>
       <namespace>vrx/dock_2018/bay_2_external</namespace>
-      <pose frame="robotx_dock_2018::dock_2018_placard1::placard::link">0 10 -1.5 0 0 0</pose>
+      <pose frame="${model_name}::dock_2018_placard1::placard::link">0 10 -1.5 0 0 0</pose>
       <geometry>
         <box>
