Commit message: port task preparation for vorc-docker
Signed-off-by: Mabel Zhang <mabel@openrobotics.org>

File: vrx_gazebo/worlds/xacros/perception.xacro (robot description, xacro)
@@ -3,10 +3,10 @@
   <xacro:macro name="perception" params="**model_includes
                                          **object_sequence
-                                         ">
+                                         namespace:=wamv">
     <xacro:insert_block name="model_includes"/>"
       <plugin filename="libperception_scoring_plugin.so"
               name="perception_scoring_plugin">
       <!-- Parameters for ScoringPlugin base class -->
-      <vehicle>wamv</vehicle>
+      <vehicle>${namespace}</vehicle>
       <task_name>perception</task_name>
       <initial_state_duration>10.0</initial_state_duration>
@@ -15,5 +15,5 @@
       <!-- Parameters for PopulationPlugin -->
       <loop_forever>false</loop_forever>
-      <frame>wamv</frame>
+      <frame>${namespace}</frame>
       <!-- Pose of each object is expressed relative to the body frame
            of the object named in the frame field - i.e., relative to

File: vrx_gazebo/worlds/xacros/scene.xacro (robot description, xacro)
@@ -9,5 +9,5 @@
       </sky>
       <grid>0</grid>
-      <origin_visual> 0 </origin_visual>
+      <origin_visual>0</origin_visual>
       <xacro:insert_block name="fog"/>
       <ambient>

File: vrx_gazebo/worlds/xacros/stationkeeping.xacro (robot description, xacro)
@@ -1,8 +1,8 @@
 <?xml version="1.0"?>
 <world xmlns:xacro="http://ros.org/wiki/xacro">
-  <xacro:macro name="stationkeeping" params="**wp_markers lat:=21.31091 lon:=-157.88868 heading:=0.0">
+  <xacro:macro name="stationkeeping" params="**wp_markers lat:=21.31091 lon:=-157.88868 heading:=0.0 namespace:=wamv">
     <plugin name="stationkeeping_scoring_plugin"
           filename="libstationkeeping_scoring_plugin.so">
-      <vehicle>wamv</vehicle>
+      <vehicle>${namespace}</vehicle>
       <task_name>stationkeeping</task_name>
       <!-- Goal as Latitude, Longitude, Yaw -->
@@ -13,8 +13,8 @@
       <release_joints>
         <joint>
-          <name>wamv_external_pivot_joint</name>
+          <name>${namespace}_external_pivot_joint</name>
         </joint>
         <joint>
-          <name>wamv_external_riser</name>
+          <name>${namespace}_external_riser</name>
         </joint>
       </release_joints>

File: vrx_gazebo/worlds/xacros/wayfinding.xacro (robot description, xacro)
@@ -1,8 +1,8 @@
 <?xml version="1.0"?>
 <world xmlns:xacro="http://ros.org/wiki/xacro">
-  <xacro:macro name="wayfinding" params="**wp_markers **waypoints">
+  <xacro:macro name="wayfinding" params="**wp_markers **waypoints namespace:=wamv">
     <plugin name="wayfinding_scoring_plugin"
             filename="libwayfinding_scoring_plugin.so">
-      <vehicle>wamv</vehicle>
+      <vehicle>${namespace}</vehicle>
       <task_name>wayfinding</task_name>
       <!-- Goal as Latitude, Longitude, Yaw -->
@@ -15,8 +15,8 @@
       <release_joints>
         <joint>
-          <name>wamv_external_pivot_joint</name>
+          <name>${namespace}_external_pivot_joint</name>
         </joint>
         <joint>
-          <name>wamv_external_riser</name>
+          <name>${namespace}_external_riser</name>
         </joint>
       </release_joints>

Commit message: add competition arg to xacro templates
Signed-off-by: Mabel Zhang <mabel@openrobotics.org>

File: vrx_gazebo/worlds/xacros/perception.xacro (robot description, xacro)
@@ -3,5 +3,6 @@
   <xacro:macro name="perception" params="**model_includes
                                          **object_sequence
-                                         namespace:=wamv">
+                                         namespace:=wamv
+                                         competition:=vrx">
     <xacro:insert_block name="model_includes"/>"
       <plugin filename="libperception_scoring_plugin.so"
@@ -13,4 +14,7 @@
       <ready_state_duration>10.0</ready_state_duration>
       <running_state_duration>300</running_state_duration>
+      <task_info_topic>/${competition}/task/info</task_info_topic>
+      <contact_debug_topic>/${competition}/debug/contact</contact_debug_topic>
+      <landmark_topic>/${competition}/perception/landmark</landmark_topic>
       <!-- Parameters for PopulationPlugin -->
       <loop_forever>false</loop_forever>

File: vrx_gazebo/worlds/xacros/stationkeeping.xacro (robot description, xacro)
@@ -1,11 +1,16 @@
 <?xml version="1.0"?>
 <world xmlns:xacro="http://ros.org/wiki/xacro">
-  <xacro:macro name="stationkeeping" params="**wp_markers lat:=21.31091 lon:=-157.88868 heading:=0.0 namespace:=wamv">
+  <xacro:macro name="stationkeeping" params="**wp_markers lat:=21.31091 lon:=-157.88868 heading:=0.0 namespace:=wamv competition:=vrx">
     <plugin name="stationkeeping_scoring_plugin"
           filename="libstationkeeping_scoring_plugin.so">
       <vehicle>${namespace}</vehicle>
       <task_name>stationkeeping</task_name>
+      <rms_error_topic>/${competition}/station_keeping/rms_error</rms_error_topic>
+      <pose_error_topic>/${competition}/station_keeping/pose_error</pose_error_topic>
+      <goal_topic>/${competition}/station_keeping/goal</goal_topic>
+      <task_info_topic>/${competition}/task/info</task_info_topic>
+      <contact_debug_topic>/${competition}/debug/contact</contact_debug_topic>
       <!-- Goal as Latitude, Longitude, Yaw -->
-      <goal_pose>${lat} ${lon} ${heading} </goal_pose>
+      <goal_pose>${lat} ${lon} ${heading}</goal_pose>
       <initial_state_duration>10</initial_state_duration>
       <ready_state_duration>10</ready_state_duration>

File: vrx_gazebo/worlds/xacros/wayfinding.xacro (robot description, xacro)
@@ -1,9 +1,17 @@
 <?xml version="1.0"?>
 <world xmlns:xacro="http://ros.org/wiki/xacro">
-  <xacro:macro name="wayfinding" params="**wp_markers **waypoints namespace:=wamv">
+  <xacro:macro name="wayfinding" params="**wp_markers
+                                         **waypoints
+                                         namespace:=wamv
+                                         competition:=vrx">
     <plugin name="wayfinding_scoring_plugin"
             filename="libwayfinding_scoring_plugin.so">
       <vehicle>${namespace}</vehicle>
       <task_name>wayfinding</task_name>
+      <min_errors_topic>/${competition}/wayfinding/min_errors</min_errors_topic>
+      <mean_error_topic>/${competition}/wayfinding/mean_error</mean_error_topic>
+      <waypoints_topic>/${competition}/wayfinding/waypoints</waypoints_topic>
+      <task_info_topic>/${competition}/task/info</task_info_topic>
+      <contact_debug_topic>/${competition}/debug/contact</contact_debug_topic>
       <!-- Goal as Latitude, Longitude, Yaw -->
       <waypoints>
