Commit message: fix macro name and include

File: vrx_gazebo/worlds/xacros/include_all_xacros.xacro (robot description, xacro)
@@ -4,4 +4,5 @@
     <xacro:include filename="$(find vrx_2019)/worlds/sandisland.xacro" />
     <xacro:include filename="$(find vrx_gazebo)/worlds/xacros/sandisland_minus_scene.xacro" />
+    <xacro:include filename="$(find vrx_gazebo)/worlds/xacros/sydneyregatta_minus_scene.xacro" />
     <xacro:include filename="$(find vrx_gazebo)/worlds/xacros/scene.xacro" />
     <xacro:include filename="$(find vrx_gazebo)/worlds/xacros/nav_challenge.xacro" />

File: vrx_gazebo/worlds/xacros/sydneyregatta_minus_scene.xacro (robot description, xacro)
@@ -2,5 +2,5 @@
 <!-- Macro to insert the sydneyregatta into the world -->
 <world xmlns:xacro="http://ros.org/wiki/xacro">
-  <xacro:macro name="sydneyregatta">
+  <xacro:macro name="sydneyregatta_minus_scene">
     <!-- Estimated latitude/longitude of sydneyregatta
 	 from satellite imagery -->
