Commit message: Restoring cameras and laser visuals and creating demo.launch

File: wamv_gazebo/urdf/dynamics/wamv_gazebo_wind_plugin.xacro (robot description, xacro)
@@ -7,5 +7,5 @@
         <bodyName>base_link</bodyName>
         <!-- Wind -->
-        <wind_direction>1 0 0 </wind_direction>
+        <wind_direction>-0.5 0.5 0 </wind_direction>
         <wind_coeff_vector>0.5 0.5 0.33 </wind_coeff_vector>
         <wind_mean_velocity>5 </wind_mean_velocity>

File: wamv_gazebo/urdf/sensors/wamv_3d_lidar.xacro (robot description, xacro)
@@ -19,8 +19,11 @@
                                             max_range:=100 noise_stddev:=0.01">
     <link name="${name}_link">
-      <visual name="{name}_visual">
+      <visual name="${name}_visual">>
         <geometry>
-          <mesh filename="package://wamv_gazebo/mesh/lidar_3d.dae"/>
+          <cylinder radius="0.025" length="0.1" />
         </geometry>
+        <material name="${name}_visual_material">
+          <color rgba="0.5 1.0 0.5 1.0" />
+        </material>
       </visual>
     </link>

File: wamv_gazebo/urdf/sensors/wamv_camera.xacro (robot description, xacro)
@@ -3,8 +3,13 @@
   <xacro:macro name="wamv_camera" params="name x:=0.5 y:=0 z:=1.5 R:=0 P:=0 Y:=0">
     <link name="${name}_link">
-      <visual name="{name}_visual">
+      <visual name="${name}_visual">
+        <xacro:property name="visual_length" value="0.05" />
+        <origin xyz="-${visual_length/2.0} 0 0" rpy="0 1.57 0" />
         <geometry>
-          <mesh filename="package://wamv_gazebo/mesh/monocamera.dae"/>
+          <cylinder radius="0.01" length="${visual_length}" />
         </geometry>
+        <material name="${name}_visual_material">
+          <color rgba="1.0 1.0 0.0 1.0" />
+        </material>
       </visual>
     </link>

File: wamv_gazebo/urdf/wamv_gazebo.urdf.xacro (robot description, xacro)
@@ -77,8 +77,8 @@
   <xacro:if value="$(arg vrx_sensors_enabled)">
     <!-- Add a stereo camera pair -->
-    <xacro:wamv_camera name="front_left_camera" y="0.1" x="0.75" R="${radians(15)}" Y="${radians(90)}" />
-    <xacro:wamv_camera name="front_right_camera" y="-0.1" x="0.75" R="${radians(15)}" Y="${radians(90)}" />
+    <xacro:wamv_camera name="front_left_camera" y="0.1" x="0.75" P="${radians(15)}" />
+    <xacro:wamv_camera name="front_right_camera" y="-0.1" x="0.75" P="${radians(15)}" />
     <!-- Add a camera facing right -->
-    <xacro:wamv_camera name="middle_right_camera" y="-0.45" R="${radians(15)}" />
+    <xacro:wamv_camera name="middle_right_camera" y="-0.45" P="${radians(15)}" Y="${radians(-90)}" />
     <!-- Add simulated GPS -->
     <xacro:wamv_gps name="gps_wamv" x="-0.75" y="0" />

Commit message: incremental(basic testing passed)

File: wamv_gazebo/urdf/dynamics/wamv_gazebo_wind_plugin.xacro (robot description, xacro)
@@ -1,18 +1,19 @@
 <?xml version="1.0"?>
-<robot xmlns:xacro="http://ros.org/wiki/xacro">
-  <xacro:macro name="usv_wind_gazebo" params="name">
+<world xmlns:xacro="http://ros.org/wiki/xacro">
+  <xacro:macro name="usv_wind_gazebo">
     <!--Gazebo Plugin for simulating WAM-V dynamics-->
-    <gazebo>
-      <plugin name="usv_wind_${name}" filename="libusv_gazebo_wind_plugin.so">
-        <bodyName>base_link</bodyName>
+    <plugin name="wind" filename="libusv_gazebo_wind_plugin.so">
+        <!-- models to be effected by the wind -->
+	<models_n>1</models_n>
+	<model_name_0>wamv</model_name_0>
+	<link_name_0>base_link</link_name_0>
+	<coeff_vector_0>0.5 0.5 0.33</coeff_vector_0>
         <!-- Wind -->
         <wind_direction>-0.5 0.5 0 </wind_direction>
-        <wind_coeff_vector>0.5 0.5 0.33 </wind_coeff_vector>
-        <wind_mean_velocity>0 </wind_mean_velocity>
+        <wind_mean_velocity>10</wind_mean_velocity>
         <var_wind_gain_constants>100</var_wind_gain_constants>
         <var_wind_time_constants>5</var_wind_time_constants>
         <random_seed></random_seed> <!-- set to zero/empty to randomize -->
       </plugin>
-    </gazebo>
   </xacro:macro>
-</robot>
+</world>

File: wamv_gazebo/urdf/wamv_gazebo.xacro (robot description, xacro)
@@ -11,6 +11,4 @@
     <!-- Attach hydrodynamics plugin -->
     <xacro:usv_dynamics_gazebo name="wamv_dynamics_plugin"/>
-    <!-- Attach wind plugin -->
-    <xacro:usv_wind_gazebo name="wamv_wind_plugin"/>
   </xacro:macro>
 </robot>
