Commit message: New model for monocromatic waves, adding xacro param for ocean wave model specification and adding .gitignore based on .hgignore

File: wamv_gazebo/urdf/dynamics/wamv_gazebo_dynamics_plugin.xacro (robot description, xacro)
@@ -1,5 +1,5 @@
 <?xml version="1.0"?>
 <robot xmlns:xacro="http://ros.org/wiki/xacro">
-  <xacro:macro name="usv_dynamics_gazebo" params="name">
+  <xacro:macro name="usv_dynamics_gazebo" params="name wave_model">
     <!--Gazebo Plugin for simulating WAM-V dynamics-->
     <gazebo>
@@ -31,5 +31,5 @@
         <length_n>2</length_n>
         <!-- Wave model -->
-        <wave_model>ocean_waves</wave_model>
+        <wave_model>"${wave_model}"</wave_model>
       </plugin>
     </gazebo>

File: wamv_gazebo/urdf/wamv_gazebo.urdf.xacro (robot description, xacro)
@@ -19,4 +19,5 @@
   robotNamespace parameter -->
   <xacro:arg name="namespace" default="wamv"/>
+  <xacro:arg name="wave_model" default="ocean_waves"/>
   <xacro:property name="thruster_namespace" value="$(arg thruster_namespace)" scope="global" />
   <xacro:property name="camera_namespace" value="$(arg camera_namespace)" scope="global" />
@@ -39,5 +40,6 @@
   <!-- Use thruster yaml file if given -->
   <xacro:if value="$(arg yaml_thruster_generation)">
-    <xacro:wamv_gazebo thruster_layout="$(arg thruster_xacro_file)"/>
+    <xacro:wamv_gazebo thruster_layout="$(arg thruster_xacro_file)"
+		       wave_model="$(arg wave_model)"/>
   </xacro:if>
   <!-- Otherwise, add thrusters based on thruster_config variable -->
@@ -46,13 +48,16 @@
     <!-- Default WAM-V with two aft thrusters -->
     <xacro:if value="${thruster_conf == 'H'}">
-       <xacro:wamv_gazebo thruster_layout="$(find wamv_gazebo)/urdf/thruster_layouts/wamv_aft_thrusters.xacro"/>
+      <xacro:wamv_gazebo thruster_layout="$(find wamv_gazebo)/urdf/thruster_layouts/wamv_aft_thrusters.xacro"
+			 wave_model="$(arg wave_model)"/>
     </xacro:if>
     <!-- WAMV with "T" thruster configuration -->
     <xacro:if value="${thruster_conf == 'T'}">
-      <xacro:wamv_gazebo thruster_layout="$(find wamv_gazebo)/urdf/thruster_layouts/wamv_t_thrusters.xacro"/>
+      <xacro:wamv_gazebo thruster_layout="$(find wamv_gazebo)/urdf/thruster_layouts/wamv_t_thrusters.xacro"
+			wave_model="$(arg wave_model)"/>
     </xacro:if>
     <!-- WAMV with "X" thruster configuration -->
     <xacro:if value="${thruster_conf == 'X'}">
-      <xacro:wamv_gazebo thruster_layout="$(find wamv_gazebo)/urdf/thruster_layouts/wamv_x_thrusters.xacro"/>
+      <xacro:wamv_gazebo thruster_layout="$(find wamv_gazebo)/urdf/thruster_layouts/wamv_x_thrusters.xacro"
+			  wave_model="$(arg wave_model)"/>
     </xacro:if>
   </xacro:unless>

File: wamv_gazebo/urdf/wamv_gazebo.xacro (robot description, xacro)
@@ -2,5 +2,5 @@
 <robot xmlns:xacro="http://ros.org/wiki/xacro">
   <!-- Macro to create a WAM-V with dyanmics plugins and a customizeable thruster layout -->
-  <xacro:macro  name="wamv_gazebo" params="thruster_layout">
+  <xacro:macro  name="wamv_gazebo" params="wave_model thruster_layout">
     <!-- Include macros for dynamics plugins -->
     <xacro:include filename="$(find wamv_gazebo)/urdf/macros.xacro" />
@@ -10,5 +10,6 @@
     <xacro:include filename="${thruster_layout}"/>
     <!-- Attach hydrodynamics plugin -->
-    <xacro:usv_dynamics_gazebo name="wamv_dynamics_plugin"/>
+    <xacro:usv_dynamics_gazebo name="wamv_dynamics_plugin"
+			       wave_model="${wave_model}"/>
   </xacro:macro>
 </robot>

File: wave_gazebo/world_models/ocean_waves_mono/model.xacro (robot description, xacro)
@@ -17,8 +17,8 @@
 -->
 <world xmlns:xacro="http://ros.org/wiki/xacro">
-  <xacro:macro name="ocean_waves" params="gain:=0.1 period:=5
-                     direction_x:=1.0 direction_y:=0.0
-                     angle:=0.4">
-  <model name='ocean_waves'>
+  <xacro:macro name="ocean_waves_mono" params="amplitude:=0.1 period:=5
+					       direction_x:=1.0 direction_y:=0.0">
+  <!-- Don't change the model name! -->
+  <model name='ocean_waves_mono'>
     <static>true</static>
     <plugin name="wavefield_plugin" filename="libWavefieldModelPlugin.so">
@@ -28,14 +28,14 @@
       <cell_count>50 50</cell_count>
       <wave>
-	<model>PMS</model>
+	<model>MONO</model>
         <period>${period}</period>
-        <number>3</number>
-        <scale>1.5</scale>
-	<gain>${gain}</gain>
+        <number>1</number>
+        <scale>-1</scale>
+	<gain>-1</gain>
         <direction>${direction_x} ${direction_y}</direction>
-        <angle>${angle}</angle>
+        <angle>-1</angle>
         <tau>2.0</tau>
-        <amplitude>0.0</amplitude>  <!-- No effect for the PMS model -->
-        <steepness>0.0</steepness>
+        <amplitude>${amplitude}</amplitude>
+        <steepness>-1</steepness>
       </wave>
     </plugin>
@@ -47,16 +47,16 @@
           <refractOpacity>0.2</refractOpacity>
           <reflectOpacity>0.2</reflectOpacity>
-          <wave>
-            <model>PMS</model>
+	  <wave>
+	    <model>MONO</model>
             <period>${period}</period>
-            <number>3</number>
-            <scale>1.5</scale>
-	    <gain>${gain}</gain>
+            <number>1</number>
+            <scale>-1</scale>
+	    <gain>-1</gain>
             <direction>${direction_x} ${direction_y}</direction>
-            <angle>${angle}</angle>
+            <angle>-1</angle>
             <tau>2.0</tau>
-            <amplitude>0.0</amplitude>  <!-- No effect for the PMS model -->
-            <steepness>0.0</steepness>
-          </wave>
+            <amplitude>${amplitude}</amplitude>
+            <steepness>-1</steepness>
+	  </wave>
         </plugin>
         <geometry>

Commit message: add boat size to dynamics xacro
Signed-off-by: Mabel Zhang <mabel@openrobotics.org>

File: wamv_gazebo/urdf/dynamics/wamv_gazebo_dynamics_plugin.xacro (robot description, xacro)
@@ -1,5 +1,5 @@
 <?xml version="1.0"?>
 <robot xmlns:xacro="http://ros.org/wiki/xacro">
-  <xacro:macro name="usv_dynamics_gazebo" params="name">
+  <xacro:macro name="usv_dynamics_gazebo" params="name width:=2.4 length:=4.9">
     <!--Gazebo Plugin for simulating WAM-V dynamics-->
     <gazebo>
@@ -26,6 +26,6 @@
         <!--<boatArea>2.2</boatArea>-->
         <hullRadius>0.213</hullRadius>
-        <boatWidth>2.4</boatWidth>
-        <boatLength>4.9</boatLength>
+        <boatWidth>${width}</boatWidth>
+        <boatLength>${length}</boatLength>
         <!-- Length discretization, AKA, "N" -->
         <length_n>2</length_n>
