Commit message: rotation bug fix

File: usv_gazebo_plugins/test/worlds/buoyancy_plugin_test.world.xacro (robot description, xacro)
@@ -107,5 +107,5 @@
       </link>
     </model>
-    <!-- test_1: floating box -->
+    <!-- test_1: basic shape drop test | no rotation -->
     <xacro:basic_shape name="1_box" static="false">
       <pose>0 0 2 0 0 0</pose>
@@ -130,4 +130,27 @@
       <xacro:cylinder_inertial mass="5" r="0.5" l="0.3" />
     </xacro:basic_shape>
+    <!-- test_2: basic shape drop test | rotation -->
+    <xacro:basic_shape name="2_box" static="false">
+      <pose>0 2 2 0 0 0</pose>
+      <box>
+        <size>1 1 1</size>
+      </box>
+      <xacro:box_inertial mass="5" x="1" y="1" z="1"/>
+    </xacro:basic_shape>
+    <xacro:basic_shape name="2_sphere" static="false">
+      <pose>2 2 2 0 0 0</pose>
+      <sphere>
+        <radius>0.5</radius>
+      </sphere>
+      <xacro:sphere_inertial mass="5" r="0.5"/>
+    </xacro:basic_shape>
+    <xacro:basic_shape name="2_cylinder" static="false">
+      <pose>4 2 2 0 0 0</pose>
+      <cylinder>
+        <radius>0.5</radius>
+        <length>0.3</length>
+      </cylinder>
+      <xacro:cylinder_inertial mass="5" r="0.5" l="0.3" />
+    </xacro:basic_shape>
   </world>
 </sdf>

Commit message: mass loaded

File: usv_gazebo_plugins/test/worlds/buoyancy_plugin_test.world.xacro (robot description, xacro)
@@ -22,5 +22,5 @@
         <fluid_density>1000</fluid_density>
         <fluid_level>0.0</fluid_level>
-        <fluid_drag>5.0</fluid_drag>
+        <fluid_drag>0.0</fluid_drag>
         <buoyancy name="buoyancy">
           <link_name>link</link_name>
@@ -48,5 +48,5 @@
   <xacro:macro name="sphere_inertial" params="mass r">
     <inertial>
-      <mass value="${mass}" />
+      <mass>${mass}</mass>
       <inertia>
         <ixx>${0.4 * mass * r * r}</ixx>
@@ -61,5 +61,5 @@
   <xacro:macro name="cylinder_inertial" params="mass r l">
     <inertial>
-      <mass value="${mass}" />
+      <mass>${mass}</mass>
       <inertia>
         <ixx>${0.0833333 * mass * (3 * r * r + l * l)}</ixx>

Commit message: drag implemented

File: usv_gazebo_plugins/test/worlds/buoyancy_plugin_test.world.xacro (robot description, xacro)
@@ -22,5 +22,6 @@
         <fluid_density>1000</fluid_density>
         <fluid_level>0.0</fluid_level>
-        <linear_drag>5.0</linear_drag>
+        <linear_drag>10.0</linear_drag>
+        <angular_drag>4.0</angular_drag>
         <buoyancy name="buoyancy">
           <link_name>link</link_name>
@@ -154,4 +155,27 @@
       <xacro:cylinder_inertial mass="2" r="0.1" l="0.159" />
     </xacro:basic_shape>
+    <!-- test_3: basic shape float test | rotation -->
+    <xacro:basic_shape name="3_box" static="false">
+      <pose>0.1 1.0 -0.5 1.0 0 0</pose>
+      <box>
+        <size>0.171 0.171 0.171</size>
+      </box>
+      <xacro:box_inertial mass="2" x="0.171" y="0.171" z="0.171"/>
+    </xacro:basic_shape>
+    <xacro:basic_shape name="3_sphere" static="false">
+      <pose>0.4 1.0 -0.5 1.0 0 0</pose>
+      <sphere>
+        <radius>0.106</radius>
+      </sphere>
+      <xacro:sphere_inertial mass="2" r="0.106"/>
+    </xacro:basic_shape>
+    <xacro:basic_shape name="3_cylinder" static="false">
+      <pose>0.7 1.0 -0.5 1.0 0 0</pose>
+      <cylinder>
+        <radius>0.1</radius>
+        <length>0.159</length>
+      </cylinder>
+      <xacro:cylinder_inertial mass="2" r="0.1" l="0.159" />
+    </xacro:basic_shape>
   </world>
 </sdf>
