Commit message: Style changes.

File: wamv_gazebo/urdf/wamv_gazebo.xacro (robot description, xacro)
@@ -12,9 +12,9 @@
     <xacro:usv_dynamics_gazebo name="wamv_dynamics_plugin"/>
     <!-- Add the force visualization plugin -->
-<!--    <gazebo>-->
-<!--      <plugin name="ForcePlugin" filename="libforce_visual_plugin.so">-->
-<!--        <scaling>20.0</scaling>-->
-<!--      </plugin>-->
-<!--    </gazebo>-->
-  </xacro:macro>
+    <!-- <gazebo>
+      <plugin name="ForcePlugin" filename="libforce_visual_plugin.so">
+        <scaling>20.0</scaling>
+      </plugin>
+    </gazebo>
+  </xacro:macro> -->
 </robot>

Commit message: Fix typo.

File: wamv_gazebo/urdf/wamv_gazebo.xacro (robot description, xacro)
@@ -16,5 +16,5 @@
         <scaling>20.0</scaling>
       </plugin>
-    </gazebo>
-  </xacro:macro> -->
+    </gazebo> -->
+  </xacro:macro>
 </robot>
