Commit message: Locking the WAM-V conditionally.

File: wamv_gazebo/urdf/wamv_gazebo.urdf.xacro (robot description, xacro)
@@ -3,6 +3,33 @@
 <robot xmlns:xacro="http://ros.org/wiki/xacro"
        name="WAM-V">
+  <xacro:arg name="locked" default="false" />
   <!-- Default WAM-V with two aft thrusters -->
   <xacro:include filename="$(find wamv_gazebo)/urdf/wamv_gazebo.xacro" />
   <xacro:wamv_gazebo thruster_layout="$(find wamv_gazebo)/urdf/thruster_layouts/wamv_aft_thrusters.xacro"/>
+  <xacro:if value="$(arg locked)">
+    <gazebo>
+      <link name="wamv_external_link"/>
+      <joint name="wamv_external_pivot_joint" type="universal">
+        <parent>wamv::base_link</parent>
+        <child>wamv_external_link</child>
+        <axis>
+          <xyz>1 0 0</xyz>
+        </axis>
+        <axis2>
+          <xyz>0 1 0</xyz>
+        </axis2>
+      </joint>
+      <joint name="wamv_external_riser" type="prismatic">
+        <parent>world</parent>
+        <child>wamv_external_link</child>
+        <axis>
+          <limit>
+            <lower>-3</lower>
+            <upper>3</upper>
+          </limit>
+          <xyz>0 0 1</xyz>
+        </axis>
+      </joint>
+    </gazebo>
+  </xacro:if>
 </robot>

File: wamv_gazebo/urdf/wamv_gazebo_t.urdf.xacro (robot description, xacro)
@@ -3,6 +3,33 @@
 <robot xmlns:xacro="http://ros.org/wiki/xacro"
        name="WAM-V">
+  <xacro:arg name="locked" default="false" />
   <!-- WAMV with "T" thruster configuration -->
   <xacro:include filename="$(find wamv_gazebo)/urdf/wamv_gazebo.xacro" />
   <xacro:wamv_gazebo thruster_layout="$(find wamv_gazebo)/urdf/thruster_layouts/wamv_t_thrusters.xacro"/>
+  <xacro:if value="$(arg locked)">
+    <gazebo>
+      <link name="wamv_external_link"/>
+      <joint name="wamv_external_pivot_joint" type="universal">
+        <parent>wamv::base_link</parent>
+        <child>wamv_external_link</child>
+        <axis>
+          <xyz>1 0 0</xyz>
+        </axis>
+        <axis2>
+          <xyz>0 1 0</xyz>
+        </axis2>
+      </joint>
+      <joint name="wamv_external_riser" type="prismatic">
+        <parent>world</parent>
+        <child>wamv_external_link</child>
+        <axis>
+          <limit>
+            <lower>-3</lower>
+            <upper>3</upper>
+          </limit>
+          <xyz>0 0 1</xyz>
+        </axis>
+      </joint>
+    </gazebo>
+  </xacro:if>
 </robot>

File: wamv_gazebo/urdf/wamv_gazebo_x.urdf.xacro (robot description, xacro)
@@ -3,5 +3,32 @@
 <robot xmlns:xacro="http://ros.org/wiki/xacro"
        name="WAM-V">
+  <xacro:arg name="locked" default="false" />
   <xacro:include filename="$(find wamv_gazebo)/urdf/wamv_gazebo.xacro" />
   <xacro:wamv_gazebo thruster_layout="$(find wamv_gazebo)/urdf/thruster_layouts/wamv_x_thrusters.xacro"/>
+  <xacro:if value="$(arg locked)">
+    <gazebo>
+      <link name="wamv_external_link"/>
+      <joint name="wamv_external_pivot_joint" type="universal">
+        <parent>wamv::base_link</parent>
+        <child>wamv_external_link</child>
+        <axis>
+          <xyz>1 0 0</xyz>
+        </axis>
+        <axis2>
+          <xyz>0 1 0</xyz>
+        </axis2>
+      </joint>
+      <joint name="wamv_external_riser" type="prismatic">
+        <parent>world</parent>
+        <child>wamv_external_link</child>
+        <axis>
+          <limit>
+            <lower>-3</lower>
+            <upper>3</upper>
+          </limit>
+          <xyz>0 0 1</xyz>
+        </axis>
+      </joint>
+    </gazebo>
+  </xacro:if>
 </robot>

Commit message: Simplify urdf files.

File: wamv_gazebo/urdf/wamv_gazebo.urdf.xacro (robot description, xacro)
@@ -4,7 +4,28 @@
        name="WAM-V">
   <xacro:arg name="locked" default="false" />
+  <xacro:arg name="thruster_config" default="H" />
+  <xacro:arg name="camera_enabled" default="false" />
+  <xacro:arg name="gps_enabled" default="false" />
+  <xacro:arg name="imu_enabled" default="false" />
+  <xacro:arg name="lidar_enabled" default="false" />
+  <xacro:arg name="ground_truth_enabled" default="false" />
+  <xacro:arg name="vmrc_sensors_enabled" default="false" />
+  <!-- === The WAM-V platform === -->
+  <xacro:include filename="$(find wamv_gazebo)/urdf/wamv_gazebo.xacro" />
+  <!-- === Thrusters === -->
+  <xacro:property name="thruster_conf" value="$(arg thruster_config)"/> -->
   <!-- Default WAM-V with two aft thrusters -->
-  <xacro:include filename="$(find wamv_gazebo)/urdf/wamv_gazebo.xacro" />
-  <xacro:wamv_gazebo thruster_layout="$(find wamv_gazebo)/urdf/thruster_layouts/wamv_aft_thrusters.xacro"/>
+  <xacro:if value="${thruster_conf == 'H'}">
+     <xacro:wamv_gazebo thruster_layout="$(find wamv_gazebo)/urdf/thruster_layouts/wamv_aft_thrusters.xacro"/>
+  </xacro:if>
+  <!-- WAMV with "T" thruster configuration -->
+  <xacro:if value="${thruster_conf == 'T'}">
+    <xacro:wamv_gazebo thruster_layout="$(find wamv_gazebo)/urdf/thruster_layouts/wamv_t_thrusters.xacro"/>
+  </xacro:if>
+  <!-- WAMV with "X" thruster configuration -->
+  <xacro:if value="${thruster_conf == 'X'}">
+    <xacro:wamv_gazebo thruster_layout="$(find wamv_gazebo)/urdf/thruster_layouts/wamv_x_thrusters.xacro"/>
+  </xacro:if>
+  <!-- Decide if we lock the robot to the world -->
   <xacro:if value="$(arg locked)">
     <gazebo>
@@ -33,3 +54,37 @@
     </gazebo>
   </xacro:if>
+  <!-- Add a front camera -->
+  <xacro:if value="$(arg camera_enabled)">
+    <xacro:wamv_camera name="front_camera" y="0.3" x="0.75" P="${radians(15)}" />
+  </xacro:if>
+  <!-- Add simulated GPS -->
+  <xacro:if value="$(arg gps_enabled)">
+    <xacro:wamv_gps name="gps_wamv" y="0.2" />
+  </xacro:if>
+  <!-- Add Simulated IMU -->
+  <xacro:if value="$(arg imu_enabled)">
+    <xacro:wamv_imu name="imu_wamv" y="-0.2" />
+  </xacro:if>
+  <!-- Add 3D LIDAR -->
+  <xacro:if value="$(arg lidar_enabled)">
+    <xacro:wamv_3d_lidar name="lidar_wamv" y="-0.3" />
+  </xacro:if>
+  <!-- Add P3D ground truth -->
+  <xacro:if value="$(arg ground_truth_enabled)">
+    <xacro:wamv_p3d name="p3d_wamv"/>
+  </xacro:if>
+  <!-- ==== VMRC sensor configuration ==== -->
+  <xacro:if value="$(arg vmrc_sensors_enabled)">
+    <!-- Add a stereo camera pair -->
+    <xacro:wamv_camera name="front_left_camera" y="0.1" x="0.75" P="${radians(15)}" />
+    <xacro:wamv_camera name="front_right_camera" y="-0.1" x="0.75" P="${radians(15)}" />
+    <!-- Add a camera facing right -->
+    <xacro:wamv_camera name="middle_right_camera" y="-0.45" P="${radians(15)}" Y="${radians(-90)}" />
+    <!-- Add simulated GPS -->
+    <xacro:wamv_gps name="gps_wamv" y="0.2" />
+    <!-- Add Simulated IMU -->
+    <xacro:wamv_imu name="imu_wamv" y="-0.2" />
+    <!-- Add 3D LIDAR -->
+    <xacro:wamv_3d_lidar name="lidar_wamv" P="${radians(8)}" />
+  </xacro:if>
 </robot>

Commit message: Added Batteries to vrx_gazebo/models(sdf format) and macro(urdf format) to place on wamv

File: wamv_gazebo/urdf/wamv_gazebo.urdf.xacro (robot description, xacro)
@@ -12,7 +12,11 @@
   <xacro:arg name="vrx_sensors_enabled" default="false" />
   <!-- === The WAM-V platform === -->
-  <xacro:include filename="$(find wamv_gazebo)/urdf/wamv_gazebo.xacro" />
+  <xacro:include filename="$(find wamv_gazebo)/urdf/wamv_gazebo.xacro"/>
+  <!-- === Batteries === -->
+  <xacro:include filename="$(find wamv_description)/urdf/battery.xacro"/>
+  <xacro:battery prefix="left" position="0 1 0.45" orientation="0 0 0"/>
+  <xacro:battery prefix="right" position="0 -1 0.45" orientation="0 0 0"/>
   <!-- === Thrusters === -->
-  <xacro:property name="thruster_conf" value="$(arg thruster_config)"/> -->
+  <xacro:property name="thruster_conf" value="$(arg thruster_config)"/>
   <!-- Default WAM-V with two aft thrusters -->
   <xacro:if value="${thruster_conf == 'H'}">

Commit message: Update wamv_gazebo.urdf.xacro file to use thruster yaml file if given

File: wamv_gazebo/urdf/wamv_gazebo.urdf.xacro (robot description, xacro)
@@ -11,6 +11,10 @@
   <xacro:arg name="ground_truth_enabled" default="false" />
   <xacro:arg name="vrx_sensors_enabled" default="false" />
+  <!-- Sensor yaml file -->
   <xacro:arg name="yaml_sensor_generation" default="false"/>
   <xacro:arg name="sensor_xacro_file" default = ""/>
+  <!-- Thruster yaml file -->
+  <xacro:arg name="yaml_thruster_generation" default="false"/>
+  <xacro:arg name="thruster_xacro_file" default = ""/>
   <!-- === The WAM-V platform === -->
   <xacro:include filename="$(find wamv_gazebo)/urdf/wamv_gazebo.xacro"/>
@@ -20,18 +24,26 @@
   <xacro:battery prefix="right" position="0 -1 0.45" orientation="0 0 0"/>
   <!-- === Thrusters === -->
-  <xacro:property name="thruster_conf" value="$(arg thruster_config)"/>
-  <!-- Default WAM-V with two aft thrusters -->
-  <xacro:if value="${thruster_conf == 'H'}">
-     <xacro:wamv_gazebo thruster_layout="$(find wamv_gazebo)/urdf/thruster_layouts/wamv_aft_thrusters.xacro"/>
+  <!-- Use thruster yaml file if given -->
+  <xacro:if value="$(arg yaml_thruster_generation)">
+    <xacro:include filename="$(arg thruster_xacro_file)"/>
+    <xacro:yaml_thrusters />
   </xacro:if>
-  <!-- WAMV with "T" thruster configuration -->
-  <xacro:if value="${thruster_conf == 'T'}">
-    <xacro:wamv_gazebo thruster_layout="$(find wamv_gazebo)/urdf/thruster_layouts/wamv_t_thrusters.xacro"/>
-  </xacro:if>
-  <!-- WAMV with "X" thruster configuration -->
-  <xacro:if value="${thruster_conf == 'X'}">
-    <xacro:wamv_gazebo thruster_layout="$(find wamv_gazebo)/urdf/thruster_layouts/wamv_x_thrusters.xacro"/>
-  </xacro:if>
-  <!-- Decide if we lock the robot to the world -->
+  <!-- Otherwise, add thrusters based on thruster_config variable -->
+  <xacro:unless value="$(arg yaml_thruster_generation)">
+    <xacro:property name="thruster_conf" value="$(arg thruster_config)"/>
+    <!-- Default WAM-V with two aft thrusters -->
+    <xacro:if value="${thruster_conf == 'H'}">
+       <xacro:wamv_gazebo thruster_layout="$(find wamv_gazebo)/urdf/thruster_layouts/wamv_aft_thrusters.xacro"/>
+    </xacro:if>
+    <!-- WAMV with "T" thruster configuration -->
+    <xacro:if value="${thruster_conf == 'T'}">
+      <xacro:wamv_gazebo thruster_layout="$(find wamv_gazebo)/urdf/thruster_layouts/wamv_t_thrusters.xacro"/>
+    </xacro:if>
+    <!-- WAMV with "X" thruster configuration -->
+    <xacro:if value="${thruster_conf == 'X'}">
+      <xacro:wamv_gazebo thruster_layout="$(find wamv_gazebo)/urdf/thruster_layouts/wamv_x_thrusters.xacro"/>
+    </xacro:if>
+  </xacro:unless>
+  <!-- === Decide if we lock the robot to the world === -->
   <xacro:if value="$(arg locked)">
     <gazebo>
@@ -60,8 +72,11 @@
     </gazebo>
   </xacro:if>
+  <!-- === Sensors === -->
+  <!-- Use sensor yaml file if given -->
   <xacro:if value="$(arg yaml_sensor_generation)">
     <xacro:include filename="$(arg sensor_xacro_file)"/>
     <xacro:yaml_sensors />
   </xacro:if>
+  <!-- Otherwise, add sensors based on enable variables -->
   <xacro:unless value="$(arg yaml_sensor_generation)">
     <!-- Add a front camera -->

Commit message: adding wamv/ prefix to base_link

File: wamv_gazebo/urdf/wamv_gazebo.urdf.xacro (robot description, xacro)
@@ -62,5 +62,5 @@
       <link name="wamv_external_link"/>
       <joint name="wamv_external_pivot_joint" type="universal">
-        <parent>wamv::base_link</parent>
+        <parent>wamv::wamv/base_link</parent>
         <child>wamv_external_link</child>
         <axis>
