Commit message: Testing
Signed-off-by: Carlos Agüero <caguero@openrobotics.org>

File: wamv_gazebo/urdf/macros.xacro (robot description, xacro)
@@ -14,3 +14,5 @@
   <xacro:include filename="$(find wamv_gazebo)/urdf/sensors/wamv_p3d.xacro" />
   <xacro:include filename="$(find wamv_gazebo)/urdf/sensors/wamv_pinger.xacro" />
+  <!-- Include ball shooter macros -->
+  <xacro:include filename="$(find wamv_gazebo)/urdf/ball_shooter/ball_shooter.xacro" />
 </robot>

File: wamv_gazebo/urdf/wamv_gazebo.urdf.xacro (robot description, xacro)
@@ -12,8 +12,10 @@
   <xacro:arg name="vrx_sensors_enabled" default="false" />
   <xacro:arg name="pinger_enabled" default="false" />
+  <xacro:arg name="ball_shooter_enabled" default="false" />
   <xacro:arg name="thruster_namespace" default="thrusters/"/>
   <xacro:arg name="camera_namespace" default="cameras/"/>
   <xacro:arg name="sensor_namespace" default="sensors/"/>
   <xacro:arg name="pinger_namespace" default="pingers/"/>
+  <xacro:arg name="shooter_namespace" default="shooters/"/>
   <!-- Note: this is only used for some sensors that do not correctly use the
   robotNamespace parameter -->
@@ -23,4 +25,5 @@
   <xacro:property name="sensor_namespace" value="$(arg sensor_namespace)" scope="global" />
   <xacro:property name="pinger_namespace" value="$(arg pinger_namespace)" scope="global" />
+  <xacro:property name="shooter_namespace" value="$(arg shooter_namespace)" scope="global" />
   <xacro:property name="namespace" value="$(arg namespace)" scope="global" />
   <!-- Sensor yaml file -->
@@ -119,4 +122,8 @@
       <xacro:wamv_pinger name="pinger" position="1.0 0 -1.0" />
     </xacro:if>
+    <!-- Add ball shooter -->
+    <xacro:if value="$(arg ball_shooter_enabled)">
+      <xacro:wamv_ball_shooter name="ball_shooter" position="2.0 0 -1.0" />
+    </xacro:if>
     <!-- ==== VRX sensor configuration ==== -->
     <xacro:if value="$(arg vrx_sensors_enabled)">
@@ -137,4 +144,6 @@
       <!-- Add pinger -->
       <xacro:wamv_pinger name="pinger" position="1.0 0 -1.0" />
+      <!-- Add ball shooter -->
+      <xacro:wamv_ball_shooter name="ball_shooter" position="0.55 0.35 1.4" />
     </xacro:if>
   </xacro:unless>
