Commit message: Add texture material to water

File: wave_gazebo/world_models/ocean_waves/model.xacro (robot description, xacro)
@@ -46,13 +46,13 @@
           <mesh>
             <uri>model://ocean_waves/meshes/mesh.dae</uri>
-            <scale>0.01 0.01 0.01</scale>
+            <!-- <scale>0.01 0.01 0.01</scale> -->
           </mesh>
         </geometry>
-        <material>
+        <!-- <material>
           <script>
             <uri>model://ocean_waves/materials/scripts/waves.material</uri>
             <name>reflection</name>
           </script>
-        </material>
+        </material> -->
         <laser_retro>-1</laser_retro>
       </visual>
@@ -62,13 +62,13 @@
           <mesh>
             <uri>model://ocean_waves/meshes/mesh_below.dae</uri>
-            <scale>0.1 0.1 0.1</scale>
+            <!-- <scale>0.1 0.1 0.1</scale> -->
           </mesh>
         </geometry>
-        <material>
+        <!-- <material>
           <script>
             <uri>model://ocean_waves/materials/scripts/waves.material</uri>
             <name>reflection</name>
           </script>
-        </material>
+        </material> -->
         <laser_retro>-1</laser_retro>
       </visual>

Commit message: Hide minimap, water constant texture, try get plane to be reflection, shows reflection but wrong geometry

File: wave_gazebo/world_models/ocean_waves/model.xacro (robot description, xacro)
@@ -49,10 +49,10 @@
           </mesh>
         </geometry>
-        <!-- <material>
+        <material>
           <script>
             <uri>model://ocean_waves/materials/scripts/waves.material</uri>
             <name>reflection</name>
           </script>
-        </material> -->
+        </material>
         <laser_retro>-1</laser_retro>
       </visual>
@@ -65,10 +65,10 @@
           </mesh>
         </geometry>
-        <!-- <material>
+        <material>
           <script>
             <uri>model://ocean_waves/materials/scripts/waves.material</uri>
             <name>reflection</name>
           </script>
-        </material> -->
+        </material>
         <laser_retro>-1</laser_retro>
       </visual>

Commit message: Refactor C++ code and change shaders to match version 130

File: wave_gazebo/world_models/ocean_waves/model.xacro (robot description, xacro)
@@ -44,33 +44,37 @@
         <plugin name="ocean_waves_visual_plugin" filename="libWavefieldVisualPlugin.so"/>
         <geometry>
-          <mesh>
-            <uri>model://ocean_waves/meshes/mesh.dae</uri>
-            <scale>0.01 0.01 0.01</scale>
-          </mesh>
+          <plane>$
+            <normal>0 0 1</normal>$
+            <size>1000 1000</size>$
+          </plane>$
         </geometry>
         <material>
           <script>
-            <uri>model://ocean_waves/materials/scripts/waves.material</uri>
-            <name>reflection</name>
+            <uri>model://ocean_waves/materials/scripts</uri>
+            <uri>model://ocean_waves/materials/programs</uri>
+            <uri>model://ocean_waves/materials/textures</uri>
+            <name>fresnel</name>
           </script>
         </material>
         <laser_retro>-1</laser_retro>
       </visual>
-      <visual name="ocean_waves_below_visual">
+      <!-- <visual name="ocean_waves_below_visual">
         <plugin name="ocean_waves_below_visual_plugin" filename="libWavefieldVisualPlugin.so"/>
         <geometry>
-          <mesh>
-            <uri>model://ocean_waves/meshes/mesh_below.dae</uri>
-            <scale>0.1 0.1 0.1</scale>
-          </mesh>
+          <plane>$
+            <normal>0 0 -1</normal>$
+            <size>1000 1000</size>$
+          </plane>$
         </geometry>
         <material>
           <script>
-            <uri>model://ocean_waves/materials/scripts/waves.material</uri>
-            <name>reflection</name>
+            <uri>model://ocean_waves/materials/scripts</uri>
+            <uri>model://ocean_waves/materials/programs</uri>
+            <uri>model://ocean_waves/materials/textures</uri>
+            <name>fresnel</name>
           </script>
         </material>
         <laser_retro>-1</laser_retro>
-      </visual>
+      </visual> -->
     </link>
   </model>

Commit message: Change mesh->plane and show pure reflection color on it, working well but need to switch back to mesh

File: wave_gazebo/world_models/ocean_waves/model.xacro (robot description, xacro)
@@ -57,7 +57,11 @@
         </plugin>
         <geometry>
-          <mesh>
+          <plane>
+            <normal>0 0 1</normal>
+            <size>1000 1000</size>
+          </plane>
+          <!-- <mesh>
             <uri>model://ocean_waves/meshes/mesh.dae</uri>
-          </mesh>
+          </mesh> -->
         </geometry>
         <material>
@@ -85,7 +89,11 @@
         </plugin>
         <geometry>
-          <mesh>
+          <plane>
+            <normal>0 0 1</normal>
+            <size>1000 1000</size>
+          </plane>
+          <!-- <mesh>
             <uri>model://ocean_waves/meshes/mesh_below.dae</uri>
-          </mesh>
+          </mesh> -->
         </geometry>
         <material>

Commit message: Change plane->mesh, still shows correct reflection texture but projected onto the mesh wrong

File: wave_gazebo/world_models/ocean_waves/model.xacro (robot description, xacro)
@@ -57,11 +57,11 @@
         </plugin>
         <geometry>
-          <plane>
+          <!-- <plane>
             <normal>0 0 1</normal>
             <size>1000 1000</size>
-          </plane>
-          <!-- <mesh>
+          </plane> -->
+          <mesh>
             <uri>model://ocean_waves/meshes/mesh.dae</uri>
-          </mesh> -->
+          </mesh>
         </geometry>
         <material>
@@ -89,11 +89,11 @@
         </plugin>
         <geometry>
-          <plane>
+          <!-- <plane>
             <normal>0 0 1</normal>
             <size>1000 1000</size>
-          </plane>
-          <!-- <mesh>
+          </plane> -->
+          <mesh>
             <uri>model://ocean_waves/meshes/mesh_below.dae</uri>
-          </mesh> -->
+          </mesh>
         </geometry>
         <material>

Commit message: Integrate reflection with Gerstner waves, working well

File: wave_gazebo/world_models/ocean_waves/model.xacro (robot description, xacro)
@@ -57,42 +57,6 @@
         </plugin>
         <geometry>
-          <!-- <plane>
-            <normal>0 0 1</normal>
-            <size>1000 1000</size>
-          </plane> -->
           <mesh>
             <uri>model://ocean_waves/meshes/mesh.dae</uri>
-          </mesh>
-        </geometry>
-        <material>
-          <script>
-            <uri>model://ocean_waves/materials/scripts/waves.material</uri>
-            <name>WaveSim/GerstnerWaves</name>
-          </script>
-        </material>
-        <laser_retro>-1</laser_retro>
-      </visual>
-      <visual name="ocean_waves_below_visual">
-        <plugin name="ocean_waves_below_visual_plugin" filename="libWavefieldVisualPlugin.so">
-          <wave>
-            <model>PMS</model>
-            <period>${period}</period>
-            <number>3</number>
-            <scale>1.5</scale>
-	    <gain>${gain}</gain>
-            <direction>${direction_x} ${direction_y}</direction>
-            <angle>${angle}</angle>
-            <tau>2.0</tau>
-            <amplitude>0.0</amplitude>  <!-- No effect for the PMS model -->
-            <steepness>0.0</steepness>
-          </wave>
-        </plugin>
-        <geometry>
-          <!-- <plane>
-            <normal>0 0 1</normal>
-            <size>1000 1000</size>
-          </plane> -->
-          <mesh>
-            <uri>model://ocean_waves/meshes/mesh_below.dae</uri>
           </mesh>
         </geometry>

Commit message: Add back ocean_waves_below_visual, without Visual Plugin, working as expected

File: wave_gazebo/world_models/ocean_waves/model.xacro (robot description, xacro)
@@ -71,4 +71,18 @@
         <laser_retro>-1</laser_retro>
       </visual>
+      <visual name="ocean_waves_below_visual">
+        <geometry>
+          <mesh>
+            <uri>model://ocean_waves/meshes/mesh_below.dae</uri>
+          </mesh>
+        </geometry>
+        <material>
+          <script>
+            <uri>model://ocean_waves/materials/scripts/waves.material</uri>
+            <name>WaveSim/GerstnerWaves</name>
+          </script>
+        </material>
+        <laser_retro>-1</laser_retro>
+      </visual>
     </link>
   </model>
