Commit message: thruster updates for VORC
Signed-off-by: Mabel Zhang <mabel@openrobotics.org>

File: wamv_gazebo/urdf/thruster_layouts/wamv_gazebo_thruster_config.xacro (robot description, xacro)
@@ -1,5 +1,5 @@
 <?xml version="1.0"?>
 <plugin xmlns:xacro="http://ros.org/wiki/xacro">
-  <xacro:macro  name="wamv_gazebo_thruster_config" params="name">
+  <xacro:macro  name="wamv_gazebo_thruster_config" params="name enable_angle:=true">
     <thruster>
       <!-- Required Parameters -->
@@ -9,5 +9,5 @@
       <cmdTopic>${thruster_namespace}${name}_thrust_cmd</cmdTopic>
       <angleTopic>${thruster_namespace}${name}_thrust_angle</angleTopic>
-      <enableAngle>true</enableAngle>
+      <enableAngle>${enable_angle}</enableAngle>
       <!-- Optional Parameters -->
       <mappingType>1</mappingType>
