Commit message: Reorganize assets by event and year.
Signed-off-by: Carlos Agüero <caguero@openrobotics.org>

File: vrx_gazebo/worlds/vrx/2019/dock.world.xacro (robot description, xacro)
@@ -3,5 +3,5 @@
 <sdf version="1.6" xmlns:xacro="http://ros.org/wiki/xacro">
   <world name="robotx_scan_and_dock">
-    <xacro:include filename="$(find vrx_gazebo)/worlds/sandisland.xacro" />
+    <xacro:include filename="$(find vrx_gazebo)/worlds/vrx/2019/sandisland.xacro" />
     <xacro:sandisland />
     <!--Waves-->
@@ -19,44 +19,9 @@
       </wind_objs>
     </xacro:usv_wind_gazebo>
-    <!-- The light buoy -->
-    <include>
-      <uri>model://robotx_light_buoy</uri>
-      <pose>90 70 0.25 0 0 0</pose>
-    </include>
     <!-- The 2018 dock with the two placards -->
     <include>
-      <uri>model://dock_2018</uri>
-      <pose>60 -2.75 0 0 0 0</pose>
+      <uri>model://dock_2018_dynamic</uri>
+      <pose>130 97 0 0 0 0</pose>
     </include>
-    <!-- Uncomment to visualize the bay #1 activation zone -->
-    <!-- <model name="activation_placard1">
-      <static>true</static>
-      <link name="link">
-        <visual name="visual">
-          <pose>72.75 0 0 0 0 0</pose>
-          <geometry>
-            <box>
-              <size>1.5 4 2</size>
-            </box>
-          </geometry>
-          <transparency>0.8</transparency>
-        </visual>
-      </link>
-    </model> -->
-    <!-- Uncomment to visualize the bay #2 activation zone -->
-    <!-- <model name="activation_placard2">
-      <static>true</static>
-      <link name="link">
-        <visual name="visual">
-          <pose>61.75 0 0 0 0 0</pose>
-          <geometry>
-            <box>
-              <size>1.5 4 2</size>
-            </box>
-          </geometry>
-          <transparency>0.8</transparency>
-        </visual>
-      </link>
-    </model> -->
     <!-- The scoring plugin -->
     <plugin name="scan_dock_scoring_plugin"
@@ -64,7 +29,7 @@
       <!-- Parameters for scoring_plugin -->
       <vehicle>wamv</vehicle>
-      <task_name>scan_and_dock</task_name>
-      <initial_state_duration>3</initial_state_duration>
-      <ready_state_duration>3</ready_state_duration>
+      <task_name>scan</task_name>
+      <initial_state_duration>10</initial_state_duration>
+      <ready_state_duration>10</ready_state_duration>
       <running_state_duration>300</running_state_duration>
       <release_joints>
@@ -78,27 +43,30 @@
       <!-- Color sequence checker -->
       <robot_namespace>vrx</robot_namespace>
+      <enable_color_checker>False</enable_color_checker>
       <color_sequence_service>scan_dock/color_sequence</color_sequence_service>
-      <color_1>blue</color_1>
+      <color_1>red</color_1>
       <color_2>green</color_2>
-      <color_3>red</color_3>
+      <color_3>blue</color_3>
       <!-- Dock checkers -->
       <bays>
         <bay>
           <name>bay1</name>
-          <internal_activation_topic>/vrx/dock_2018/bay_1/contain</internal_activation_topic>
-          <external_activation_topic>/vrx/dock_2018/bay_1_exterior/contain</external_activation_topic>
+          <internal_activation_topic>/vrx/dock_2018/bay_1_internal/contain</internal_activation_topic>
+          <external_activation_topic>/vrx/dock_2018/bay_1_external/contain</external_activation_topic>
           <symbol_topic>/vrx/dock_2018_placard1/symbol</symbol_topic>
-	        <min_dock_time>10.0</min_dock_time>
-	        <dock_allowed>false</dock_allowed>
-	        <symbol>red_circle</symbol>
+          <min_dock_time>10.0</min_dock_time>
+          <dock_allowed>false</dock_allowed>
+          <symbol>red_circle</symbol>
         </bay>
         <bay>
           <name>bay2</name>
-          <internal_activation_topic>/vrx/dock_2018/bay_2/contain</internal_activation_topic>
-          <external_activation_topic>/vrx/dock_2018/bay_2_exterior/contain</external_activation_topic>
+          <internal_activation_topic>/vrx/dock_2018/bay_2_internal/contain</internal_activation_topic>
+          <external_activation_topic>/vrx/dock_2018/bay_2_external/contain</external_activation_topic>
           <symbol_topic>/vrx/dock_2018_placard2/symbol</symbol_topic>
           <min_dock_time>10.0</min_dock_time>
-	        <dock_allowed>true</dock_allowed>
-	        <symbol>blue_circle</symbol>
+          <!-- Set this bay as the intended docking bay -->
+          <dock_allowed>true</dock_allowed>
+          <!-- Specify the visual symbol - should be same as announced -->
+          <symbol>red_cross</symbol>
         </bay>
       </bays>
@@ -107,5 +75,5 @@
     <plugin name="vehicle_docked_bay1" filename="libContainPlugin.so">
       <entity>wamv::base_link</entity>
-      <namespace>vrx/dock_2018/bay_1</namespace>
+      <namespace>vrx/dock_2018/bay_1_internal</namespace>
       <pose frame="robotx_dock_2018::dock_2018_placard1::placard::link">0 -5 -1.5 0 0 0</pose>
       <geometry>
@@ -115,8 +83,19 @@
       </geometry>
     </plugin>
+    <!-- Triggers a message when the vehicle enters and exits the bay #1 -->
+    <plugin name="vehicle_docked_bay1_exterior" filename="libContainPlugin.so">
+      <entity>wamv::base_link</entity>
+      <namespace>vrx/dock_2018/bay_1_external</namespace>
+      <pose frame="robotx_dock_2018::dock_2018_placard1::placard::link">0 -10 -1.5 0 0 0</pose>
+      <geometry>
+        <box>
+          <size>8 1.5 2</size>
+        </box>
+      </geometry>
+    </plugin>
     <!-- Triggers a message when the vehicle enters and exits the bay #2 -->
     <plugin name="vehicle_docked_bay2" filename="libContainPlugin.so">
       <entity>wamv::base_link</entity>
-      <namespace>vrx/dock_2018/bay_2</namespace>
+      <namespace>vrx/dock_2018/bay_2_internal</namespace>
       <pose frame="robotx_dock_2018::dock_2018_placard2::placard::link">0 5 -1.5 0 0 0</pose>
       <geometry>
@@ -126,4 +105,15 @@
       </geometry>
     </plugin>
+    <!-- Triggers a message when the vehicle enters and exits the bay #1 -->
+    <plugin name="vehicle_docked_bay2_exterior" filename="libContainPlugin.so">
+      <entity>wamv::base_link</entity>
+      <namespace>vrx/dock_2018/bay_2_external</namespace>
+      <pose frame="robotx_dock_2018::dock_2018_placard1::placard::link">0 10 -1.5 0 0 0</pose>
+      <geometry>
+        <box>
+          <size>8 1.5 2</size>
+        </box>
+      </geometry>
+    </plugin>
   </world>
 </sdf>

File: vrx_gazebo/worlds/vrx/2019/example_course_2019.world.xacro (robot description, xacro)
@@ -3,5 +3,5 @@
 <sdf version="1.6" xmlns:xacro="http://ros.org/wiki/xacro">
   <world name="robotx_example_course">
-    <xacro:include filename="$(find vrx_gazebo)/worlds/sandisland.xacro" />
+    <xacro:include filename="$(find vrx_gazebo)/worlds/vrx/2019/sandisland.xacro" />
     <xacro:sandisland />
     <!--Waves-->

File: vrx_gazebo/worlds/vrx/2019/navigation_task.world.xacro (robot description, xacro)
@@ -3,5 +3,5 @@
 <sdf version="1.6" xmlns:xacro="http://ros.org/wiki/xacro">
   <world name="robotx_example_course">
-    <xacro:include filename="$(find vrx_gazebo)/worlds/sandisland.xacro" />
+    <xacro:include filename="$(find vrx_gazebo)/worlds/vrx/2019/sandisland.xacro" />
     <xacro:sandisland />
     <!--Waves-->

File: vrx_gazebo/worlds/vrx/2019/sandisland.world.xacro (robot description, xacro)
@@ -1,11 +1,11 @@
 <?xml version="1.0" ?>
-<!-- World containing only sydneyregatta model -->
+<!-- World containing only sandisland model -->
 <sdf version="1.6" xmlns:xacro="http://ros.org/wiki/xacro">
-  <world name="sydneyregatta">
-    <xacro:include filename="$(find vrx_gazebo)/worlds/sydneyregatta.xacro" />
-    <xacro:sydneyregatta />
+  <world name="sandisland">
+    <xacro:include filename="$(find vrx_gazebo)/worlds/vrx/2019/sandisland.xacro" />
+    <xacro:sandisland />
     <!--Waves-->
     <xacro:include filename="$(find wave_gazebo)/world_models/ocean_waves/model.xacro"/>
-    <xacro:ocean_waves scale="2.5"/>
+    <xacro:ocean_waves/>
     <!--Wind for the WAM-V. Note, wind parameters are set in the plug.-->
     <xacro:include filename="$(find vrx_gazebo)/worlds/xacros/usv_wind_plugin.xacro"/>
@@ -14,5 +14,5 @@
         <wind_obj>
           <name>wamv</name>
-          <link_name>wamv/base_link</link_name>
+          <link_name>base_link</link_name>
           <coeff_vector>0.5 0.5 0.33</coeff_vector>
         </wind_obj>

File: vrx_gazebo/worlds/vrx/2019/scan_and_dock.world.xacro (robot description, xacro)
@@ -3,5 +3,5 @@
 <sdf version="1.6" xmlns:xacro="http://ros.org/wiki/xacro">
   <world name="robotx_scan_and_dock">
-    <xacro:include filename="$(find vrx_gazebo)/worlds/sandisland.xacro" />
+    <xacro:include filename="$(find vrx_gazebo)/worlds/vrx/2019/sandisland.xacro" />
     <xacro:sandisland />
     <!--Waves-->
@@ -19,9 +19,44 @@
       </wind_objs>
     </xacro:usv_wind_gazebo>
+    <!-- The light buoy -->
+    <include>
+      <uri>model://robotx_light_buoy</uri>
+      <pose>90 70 0.25 0 0 0</pose>
+    </include>
     <!-- The 2018 dock with the two placards -->
     <include>
-      <uri>model://dock_2018_dynamic</uri>
-      <pose>130 97 0 0 0 0</pose>
+      <uri>model://dock_2018</uri>
+      <pose>60 -2.75 0 0 0 0</pose>
     </include>
+    <!-- Uncomment to visualize the bay #1 activation zone -->
+    <!-- <model name="activation_placard1">
+      <static>true</static>
+      <link name="link">
+        <visual name="visual">
+          <pose>72.75 0 0 0 0 0</pose>
+          <geometry>
+            <box>
+              <size>1.5 4 2</size>
+            </box>
+          </geometry>
+          <transparency>0.8</transparency>
+        </visual>
+      </link>
+    </model> -->
+    <!-- Uncomment to visualize the bay #2 activation zone -->
+    <!-- <model name="activation_placard2">
+      <static>true</static>
+      <link name="link">
+        <visual name="visual">
+          <pose>61.75 0 0 0 0 0</pose>
+          <geometry>
+            <box>
+              <size>1.5 4 2</size>
+            </box>
+          </geometry>
+          <transparency>0.8</transparency>
+        </visual>
+      </link>
+    </model> -->
     <!-- The scoring plugin -->
     <plugin name="scan_dock_scoring_plugin"
@@ -29,7 +64,7 @@
       <!-- Parameters for scoring_plugin -->
       <vehicle>wamv</vehicle>
-      <task_name>scan</task_name>
-      <initial_state_duration>10</initial_state_duration>
-      <ready_state_duration>10</ready_state_duration>
+      <task_name>scan_and_dock</task_name>
+      <initial_state_duration>3</initial_state_duration>
+      <ready_state_duration>3</ready_state_duration>
       <running_state_duration>300</running_state_duration>
       <release_joints>
@@ -43,30 +78,27 @@
       <!-- Color sequence checker -->
       <robot_namespace>vrx</robot_namespace>
-      <enable_color_checker>False</enable_color_checker>
       <color_sequence_service>scan_dock/color_sequence</color_sequence_service>
-      <color_1>red</color_1>
+      <color_1>blue</color_1>
       <color_2>green</color_2>
-      <color_3>blue</color_3>
+      <color_3>red</color_3>
       <!-- Dock checkers -->
       <bays>
         <bay>
           <name>bay1</name>
-          <internal_activation_topic>/vrx/dock_2018/bay_1_internal/contain</internal_activation_topic>
-          <external_activation_topic>/vrx/dock_2018/bay_1_external/contain</external_activation_topic>
+          <internal_activation_topic>/vrx/dock_2018/bay_1/contain</internal_activation_topic>
+          <external_activation_topic>/vrx/dock_2018/bay_1_exterior/contain</external_activation_topic>
           <symbol_topic>/vrx/dock_2018_placard1/symbol</symbol_topic>
-          <min_dock_time>10.0</min_dock_time>
-          <dock_allowed>false</dock_allowed>
-          <symbol>red_circle</symbol>
+	        <min_dock_time>10.0</min_dock_time>
+	        <dock_allowed>false</dock_allowed>
+	        <symbol>red_circle</symbol>
         </bay>
         <bay>
           <name>bay2</name>
-          <internal_activation_topic>/vrx/dock_2018/bay_2_internal/contain</internal_activation_topic>
-          <external_activation_topic>/vrx/dock_2018/bay_2_external/contain</external_activation_topic>
+          <internal_activation_topic>/vrx/dock_2018/bay_2/contain</internal_activation_topic>
+          <external_activation_topic>/vrx/dock_2018/bay_2_exterior/contain</external_activation_topic>
           <symbol_topic>/vrx/dock_2018_placard2/symbol</symbol_topic>
           <min_dock_time>10.0</min_dock_time>
-          <!-- Set this bay as the intended docking bay -->
-          <dock_allowed>true</dock_allowed>
-          <!-- Specify the visual symbol - should be same as announced -->
-          <symbol>red_cross</symbol>
+	        <dock_allowed>true</dock_allowed>
+	        <symbol>blue_circle</symbol>
         </bay>
       </bays>
@@ -75,5 +107,5 @@
     <plugin name="vehicle_docked_bay1" filename="libContainPlugin.so">
       <entity>wamv::base_link</entity>
-      <namespace>vrx/dock_2018/bay_1_internal</namespace>
+      <namespace>vrx/dock_2018/bay_1</namespace>
       <pose frame="robotx_dock_2018::dock_2018_placard1::placard::link">0 -5 -1.5 0 0 0</pose>
       <geometry>
@@ -83,19 +115,8 @@
       </geometry>
     </plugin>
-    <!-- Triggers a message when the vehicle enters and exits the bay #1 -->
-    <plugin name="vehicle_docked_bay1_exterior" filename="libContainPlugin.so">
-      <entity>wamv::base_link</entity>
-      <namespace>vrx/dock_2018/bay_1_external</namespace>
-      <pose frame="robotx_dock_2018::dock_2018_placard1::placard::link">0 -10 -1.5 0 0 0</pose>
-      <geometry>
-        <box>
-          <size>8 1.5 2</size>
-        </box>
-      </geometry>
-    </plugin>
     <!-- Triggers a message when the vehicle enters and exits the bay #2 -->
     <plugin name="vehicle_docked_bay2" filename="libContainPlugin.so">
       <entity>wamv::base_link</entity>
-      <namespace>vrx/dock_2018/bay_2_internal</namespace>
+      <namespace>vrx/dock_2018/bay_2</namespace>
       <pose frame="robotx_dock_2018::dock_2018_placard2::placard::link">0 5 -1.5 0 0 0</pose>
       <geometry>
@@ -105,15 +126,4 @@
       </geometry>
     </plugin>
-    <!-- Triggers a message when the vehicle enters and exits the bay #1 -->
-    <plugin name="vehicle_docked_bay2_exterior" filename="libContainPlugin.so">
-      <entity>wamv::base_link</entity>
-      <namespace>vrx/dock_2018/bay_2_external</namespace>
-      <pose frame="robotx_dock_2018::dock_2018_placard1::placard::link">0 10 -1.5 0 0 0</pose>
-      <geometry>
-        <box>
-          <size>8 1.5 2</size>
-        </box>
-      </geometry>
-    </plugin>
   </world>
 </sdf>

File: vrx_gazebo/worlds/vrx/2019/wind_test.world.xacro (robot description, xacro)
@@ -2,5 +2,5 @@
 <sdf version="1.6" xmlns:xacro="http://ros.org/wiki/xacro">
   <world name="wind_test">
-    <xacro:include filename="$(find vrx_gazebo)/worlds/sandisland.xacro" />
+    <xacro:include filename="$(find vrx_gazebo)/worlds/vrx/2019/sandisland.xacro" />
     <xacro:sandisland />
     <!--Waves-->

File: vrx_gazebo/worlds/vrx/2022/example_course.world.xacro (robot description, xacro)
@@ -3,5 +3,5 @@
 <sdf version="1.6" xmlns:xacro="http://ros.org/wiki/xacro">
   <world name="robotx_example_course">
-    <xacro:include filename="$(find vrx_gazebo)/worlds/sydneyregatta.xacro" />
+    <xacro:include filename="$(find vrx_gazebo)/worlds/vrx/2022/sydneyregatta.xacro" />
     <xacro:sydneyregatta />
     <!--Waves-->

File: vrx_gazebo/worlds/vrx/2022/gymkhana.world.xacro (robot description, xacro)
@@ -3,5 +3,5 @@
 <sdf version="1.6" xmlns:xacro="http://ros.org/wiki/xacro">
   <world name="vrx_gymkhana">
-    <xacro:include filename="$(find vrx_gazebo)/worlds/sydneyregatta.xacro" />
+    <xacro:include filename="$(find vrx_gazebo)/worlds/vrx/2022/sydneyregatta.xacro" />
     <xacro:sydneyregatta />
     <!--Waves-->

File: vrx_gazebo/worlds/vrx/2022/perception_task.world.xacro (robot description, xacro)
@@ -3,5 +3,5 @@
 <sdf version="1.6" xmlns:xacro="http://ros.org/wiki/xacro">
   <world name="vrx_perception">
-    <xacro:include filename="$(find vrx_gazebo)/worlds/sydneyregatta.xacro" />
+    <xacro:include filename="$(find vrx_gazebo)/worlds/vrx/2022/sydneyregatta.xacro" />
     <xacro:sydneyregatta />
     <!--Waves-->

File: vrx_gazebo/worlds/vrx/2022/scan_dock_deliver.world.xacro (robot description, xacro)
@@ -3,5 +3,5 @@
 <sdf version="1.6" xmlns:xacro="http://ros.org/wiki/xacro">
   <world name="vrx_scan_dock_deliver">
-    <xacro:include filename="$(find vrx_gazebo)/worlds/sydneyregatta.xacro" />
+    <xacro:include filename="$(find vrx_gazebo)/worlds/vrx/2022/sydneyregatta.xacro" />
     <xacro:sydneyregatta />
     <!--Waves-->

File: vrx_gazebo/worlds/vrx/2022/stationkeeping_task.world.xacro (robot description, xacro)
@@ -2,6 +2,6 @@
 <!-- World containing sandisland model and some course challenges -->
 <sdf version="1.6" xmlns:xacro="http://ros.org/wiki/xacro">
-  <world name="vrx_wayfinding">
-    <xacro:include filename="$(find vrx_gazebo)/worlds/sydneyregatta.xacro" />
+  <world name="vrx_stationkeeping">
+    <xacro:include filename="$(find vrx_gazebo)/worlds/vrx/2022/sydneyregatta.xacro" />
     <xacro:sydneyregatta />
     <!--Waves-->
@@ -19,23 +19,10 @@
       </wind_objs>
     </xacro:usv_wind_gazebo>
-    <plugin name="wayfinding_scoring_plugin"
-            filename="libwayfinding_scoring_plugin.so">
+  <plugin name="stationkeeping_scoring_plugin"
+          filename="libstationkeeping_scoring_plugin.so">
       <vehicle>wamv</vehicle>
-      <task_name>wayfinding</task_name>
+      <task_name>stationkeeping</task_name>
       <!-- Goal as Latitude, Longitude, Yaw -->
-      <waypoints>
-        <!-- Approx. starting point of wamv -->
-        <waypoint>
-          <pose>-33.7226766699 150.6740630167 1.21756121843</pose>
-        </waypoint>
-        <!-- A waypoint -->
-        <waypoint>
-          <pose>-33.7220832884 150.67379127877 1.0</pose>
-        </waypoint>
-        <!-- Another waypoint -->
-        <waypoint>
-          <pose>-33.7226013209 150.67504609858 1.0</pose>
-        </waypoint>
-      </waypoints>
+      <goal_pose>-33.722702498 150.67402097002 3.14159 </goal_pose>
       <initial_state_duration>10</initial_state_duration>
       <ready_state_duration>10</ready_state_duration>

File: vrx_gazebo/worlds/vrx/2022/sydneyregatta.world.xacro (robot description, xacro)
@@ -1,11 +1,11 @@
 <?xml version="1.0" ?>
-<!-- World containing only sandisland model -->
+<!-- World containing only sydneyregatta model -->
 <sdf version="1.6" xmlns:xacro="http://ros.org/wiki/xacro">
-  <world name="sandisland">
-    <xacro:include filename="$(find vrx_gazebo)/worlds/sandisland.xacro" />
-    <xacro:sandisland />
+  <world name="sydneyregatta">
+    <xacro:include filename="$(find vrx_gazebo)/worlds/vrx/2022/sydneyregatta.xacro" />
+    <xacro:sydneyregatta />
     <!--Waves-->
     <xacro:include filename="$(find wave_gazebo)/world_models/ocean_waves/model.xacro"/>
-    <xacro:ocean_waves/>
+    <xacro:ocean_waves scale="2.5"/>
     <!--Wind for the WAM-V. Note, wind parameters are set in the plug.-->
     <xacro:include filename="$(find vrx_gazebo)/worlds/xacros/usv_wind_plugin.xacro"/>
@@ -14,5 +14,5 @@
         <wind_obj>
           <name>wamv</name>
-          <link_name>base_link</link_name>
+          <link_name>wamv/base_link</link_name>
           <coeff_vector>0.5 0.5 0.33</coeff_vector>
         </wind_obj>

File: vrx_gazebo/worlds/vrx/2022/wayfinding_task.world.xacro (robot description, xacro)
@@ -2,6 +2,6 @@
 <!-- World containing sandisland model and some course challenges -->
 <sdf version="1.6" xmlns:xacro="http://ros.org/wiki/xacro">
-  <world name="vrx_stationkeeping">
-    <xacro:include filename="$(find vrx_gazebo)/worlds/sydneyregatta.xacro" />
+  <world name="vrx_wayfinding">
+    <xacro:include filename="$(find vrx_gazebo)/worlds/vrx/2022/sydneyregatta.xacro" />
     <xacro:sydneyregatta />
     <!--Waves-->
@@ -19,10 +19,23 @@
       </wind_objs>
     </xacro:usv_wind_gazebo>
-  <plugin name="stationkeeping_scoring_plugin"
-          filename="libstationkeeping_scoring_plugin.so">
+    <plugin name="wayfinding_scoring_plugin"
+            filename="libwayfinding_scoring_plugin.so">
       <vehicle>wamv</vehicle>
-      <task_name>stationkeeping</task_name>
+      <task_name>wayfinding</task_name>
       <!-- Goal as Latitude, Longitude, Yaw -->
-      <goal_pose>-33.722702498 150.67402097002 3.14159 </goal_pose>
+      <waypoints>
+        <!-- Approx. starting point of wamv -->
+        <waypoint>
+          <pose>-33.7226766699 150.6740630167 1.21756121843</pose>
+        </waypoint>
+        <!-- A waypoint -->
+        <waypoint>
+          <pose>-33.7220832884 150.67379127877 1.0</pose>
+        </waypoint>
+        <!-- Another waypoint -->
+        <waypoint>
+          <pose>-33.7226013209 150.67504609858 1.0</pose>
+        </waypoint>
+      </waypoints>
       <initial_state_duration>10</initial_state_duration>
       <ready_state_duration>10</ready_state_duration>

File: vrx_gazebo/worlds/vrx/2022/wildlife_task.world.xacro (robot description, xacro)
@@ -3,5 +3,5 @@
 <sdf version="1.6" xmlns:xacro="http://ros.org/wiki/xacro">
   <world name="vrx_wildlife">
-    <xacro:include filename="$(find vrx_gazebo)/worlds/sydneyregatta.xacro" />
+    <xacro:include filename="$(find vrx_gazebo)/worlds/vrx/2022/sydneyregatta.xacro" />
     <xacro:sydneyregatta />
     <!--Waves-->

File: vrx_gazebo/worlds/xacros/include_all_xacros.xacro (robot description, xacro)
@@ -2,6 +2,7 @@
 <world xmlns:xacro="http://ros.org/wiki/xacro">
   <xacro:macro name="include_all_xacros">
-    <xacro:include filename="$(find vrx_gazebo)/worlds/sandisland.xacro" />
+    <xacro:include filename="$(find vrx_gazebo)/worlds/vrx/2019/sandisland.xacro" />
     <xacro:include filename="$(find vrx_gazebo)/worlds/xacros/sandisland_minus_scene.xacro" />
+    <xacro:include filename="$(find vrx_gazebo)/worlds/vrx/2022/sydneyregatta.xacro" />
     <xacro:include filename="$(find vrx_gazebo)/worlds/xacros/scene.xacro" />
     <xacro:include filename="$(find vrx_gazebo)/worlds/xacros/nav_challenge.xacro" />
