Commit message: Change boat

File: vrx_2019/worlds/example_course.world.xacro (robot description, xacro)
@@ -8,21 +8,4 @@
     <xacro:include filename="$(find wave_gazebo)/world_models/ocean_waves/model.xacro"/>
     <xacro:ocean_waves/>
-    <include>
-      <uri>model://robotx_navigation_challenge</uri>
-      <pose>58 68 2 0 0 0.4</pose>
-    </include>
-    <include>
-      <uri>model://robotx_light_buoy</uri>
-      <pose>110 28 0.25 0 0 0</pose>
-    </include>
-    <include>
-      <uri>model://robotx_2016_qualifying_pinger_transit</uri>
-      <pose>55 -50 0 0 0 -1.3</pose>
-    </include>
-    <!-- The 2016 dock with the three placards -->
-    <include>
-      <uri>model://dock_2016</uri>
-      <pose>75 22 0.0 0 0 -2.78</pose>
-    </include>
     <!-- The 2018 dock with the two placards -->
     <include>

File: vrx_2019/worlds/sandisland.xacro (robot description, xacro)
@@ -45,14 +45,4 @@
       <uri>model://post</uri>
     </include>
-    <include>
-      <name>post_1</name>
-      <pose>173.558 100.809 0.42 0.046 -0.157 0</pose>
-      <uri>model://post</uri>
-    </include>
-    <include>
-      <name>post_2</name>
-      <pose>177.64 90.86 0.3 0.046 -0.157 0</pose>
-      <uri>model://post</uri>
-    </include>
     <!-- Antenna for communication with the WAM-V -->
     <include>
@@ -66,39 +56,4 @@
       <uri>model://ground_station</uri>
     </include>
-    <include>
-      <name>ground_station_1</name>
-      <pose>179.16 113.73 1.55 0 0 3.54</pose>
-      <uri>model://ground_station</uri>
-    </include>
-    <include>
-      <name>ground_station_2</name>
-      <pose>180.61 110.31 1.55 0 0 3.54</pose>
-      <uri>model://ground_station</uri>
-    </include>
-    <include>
-      <name>ground_station_3</name>
-      <pose>182.05 106.83 1.55 0 0 3.54</pose>
-      <uri>model://ground_station</uri>
-    </include>
-    <include>
-      <name>ground_station_4</name>
-      <pose>183.71 103.14 1.55 0 0 3.54</pose>
-      <uri>model://ground_station</uri>
-    </include>
-    <include>
-      <name>ground_station_5</name>
-      <pose>185.28 99.51 1.55 0 0 3.54</pose>
-      <uri>model://ground_station</uri>
-    </include>
-    <include>
-      <name>ground_station_6</name>
-      <pose>186.80 96.02 1.55 0 0 3.54</pose>
-      <uri>model://ground_station</uri>
-    </include>
-    <include>
-      <name>ground_station_7</name>
-      <pose>188.17 92.45 1.55 0 0 3.54</pose>
-      <uri>model://ground_station</uri>
-    </include>
   </xacro:macro>
 </world>

File: wamv_description/urdf/thrusters/engine.xacro (robot description, xacro)
@@ -7,11 +7,11 @@
         <origin xyz="-0.16 0 -0.24" rpy="0 0 0" />
         <geometry>
-          <box size="0.2 0.15 0.83" />
+          <box size="0.01 0.01 0.01" />
         </geometry>
       </collision>
       <collision name="${prefix}_engine_rear_end_collision">
-        <origin xyz="-0.34 0 0.12" rpy="0 0 0" />
+        <origin xyz="-0.034 0 0.012" rpy="0 0 0" />
         <geometry>
-          <box size="0.12 0.15 0.12" />
+          <box size="0.012 0.015 0.012" />
         </geometry>
       </collision>
@@ -28,7 +28,7 @@
       </visual>
       <collision name="${prefix}_propeller_collision">
-        <origin xyz="-0.08 0 0" rpy="0 1.57 0" />
+        <origin xyz="-0.04 0 0" rpy="0 1.57 0" />
         <geometry>
-          <cylinder length="0.18" radius="0.24" />
+          <cylinder length="0.05" radius="0.1" />
         </geometry>
       </collision>

File: wamv_gazebo/urdf/components/wamv_camera.xacro (robot description, xacro)
@@ -1,5 +1,5 @@
 <?xml version="1.0"?>
 <robot xmlns:xacro="http://ros.org/wiki/xacro">
-  <xacro:macro name="wamv_camera" params="name x:=0.5 y:=0 z:=1.5 post_z_from:=1.2965 R:=0 P:=0 Y:=0 post_Y:=0 visualize:=False">
+  <xacro:macro name="wamv_camera" params="name x:=0.5 y:=0 z:=1.5 post_z_from:=1.2965 R:=0 P:=0 Y:=0 post_Y:=0 visualize:=true">
     <!-- Define length variables for link positioning -->
     <xacro:property name="platform_z" value="${post_z_from}"/>

File: wamv_gazebo/urdf/thruster_layouts/wamv_aft_thrusters.xacro (robot description, xacro)
@@ -2,9 +2,9 @@
 <robot xmlns:xacro="http://ros.org/wiki/xacro">
   <xacro:include filename="$(find wamv_description)/urdf/thrusters/engine.xacro" />
-  <xacro:engine prefix="left" position="-2.373776 1.027135 0.318237" />
-  <xacro:engine prefix="right" position="-2.373776 -1.027135 0.318237" />
+  <xacro:engine prefix="left" position="-0.75 0.647 0.365 "/>
+  <xacro:engine prefix="right" position="-0.75 -0.647 0.365" />
   <gazebo>
     <plugin name="wamv_gazebo_thrust" filename="libusv_gazebo_thrust_plugin.so">
-      <cmdTimeout>1.0</cmdTimeout>
+      <cmdTimeout>0.1</cmdTimeout>
       <publisherRate>100.0</publisherRate>
       <robotNamespace>${namespace}</robotNamespace>

File: wamv_gazebo/urdf/thruster_layouts/wamv_gazebo_thruster_config.xacro (robot description, xacro)
@@ -1,5 +1,5 @@
 <?xml version="1.0"?>
 <plugin xmlns:xacro="http://ros.org/wiki/xacro">
-  <xacro:macro  name="wamv_gazebo_thruster_config" params="name enable_angle:=true">
+  <xacro:macro  name="wamv_gazebo_thruster_config" params="name enable_angle:=false">
     <thruster>
       <!-- Required Parameters -->
@@ -14,5 +14,5 @@
       <maxCmd>1.0</maxCmd>
       <maxForceFwd>250.0</maxForceFwd>
-      <maxForceRev>-100.0</maxForceRev>
+      <maxForceRev>-200.0</maxForceRev>
       <maxAngle>${pi/2}</maxAngle>
     </thruster>

File: wamv_gazebo/urdf/wamv_gazebo.urdf.xacro (robot description, xacro)
@@ -35,8 +35,9 @@
   <!-- === The WAM-V platform === -->
   <xacro:include filename="$(find wamv_gazebo)/urdf/wamv_gazebo.xacro"/>
-  <!-- === Batteries === -->
+  <!-- === Batteries ===
   <xacro:include filename="$(find wamv_description)/urdf/battery.xacro"/>
   <xacro:battery prefix="left" position="0 1 0.45" orientation="0 0 0"/>
   <xacro:battery prefix="right" position="0 -1 0.45" orientation="0 0 0"/>
+	-->
   <!-- === Thrusters === -->
   <!-- Use thruster yaml file if given -->
