Commit message: Add ball shooter model.
Signed-off-by: Carlos Agüero <caguero@openrobotics.org>

File: wamv_gazebo/urdf/ball_shooter/ball_shooter.xacro (robot description, xacro)
@@ -4,11 +4,21 @@
     <link name="${namespace}/${name}_link">
       <visual name="${name}_visual">
-        <origin xyz="0 0 0" rpy="0 0 0" />
+        <!-- The cylinder has a -15deg pitch. We compensate for that here.
+             That way, if the user passes a 0 deg rotation the cylinder will
+             be parallel to the ground -->
+        <origin xyz="0 0 0" rpy="0 0.261799 0" />
         <geometry>
-          <box size="0.3 0.3 0.2" />
+          <mesh filename="package://vrx_gazebo/models/ball_shooter/meshes/ball_shooter.dae"/>
         </geometry>
       </visual>
+      <!-- Uncomment to see the pose where the ball is teleported -->
+      <!-- <visual name="${name}_visual_ball">
+        <origin xyz="0.14 0 0.09" rpy="0 0 0" />
+        <geometry>
+          <sphere radius="0.0285"/>
+        </geometry>
+      </visual> -->
       <collision name="${name}_collision">
-        <origin xyz="0 0 0" rpy="0 0 0" />
+        <origin xyz="0 0 0" rpy="0 0.261799 0" />
         <geometry>
           <box size="0.3 0.3 0.2" />
@@ -16,6 +26,6 @@
       </collision>
       <inertial>
-        <mass value="1"/>
-        <inertia ixx="0.006458" ixy="0.0" ixz="0.0" iyy="0.006458" iyz="0.0" izz="0.01125"/>
+        <mass value="0.5"/>
+        <inertia ixx="0.001779167" ixy="0.0" ixz="0.0" iyy="0.001779167" iyz="0.0" izz="0.000225"/>
       </inertial>
     </link>
@@ -33,5 +43,5 @@
           <link_name>link</link_name>
           <frame>wamv/ball_shooter_link</frame>
-          <pose>0.2 0 0 0 0 0</pose>
+          <pose>0.14 0 0.09 0 0 0</pose>
         </projectile>
         <shot_force>250</shot_force>

File: wamv_gazebo/urdf/wamv_gazebo.urdf.xacro (robot description, xacro)
@@ -122,7 +122,7 @@
       <xacro:wamv_pinger name="pinger" position="1.0 0 -1.0" />
     </xacro:if>
-    <!-- Add ball shooter -->
+    <!-- Add ball shooter (default pitch angle: -15 deg) -->
     <xacro:if value="$(arg ball_shooter_enabled)">
-      <xacro:wamv_ball_shooter name="ball_shooter" position="2.0 0 -1.0" />
+      <xacro:wamv_ball_shooter name="ball_shooter" position="0.54 0.30 1.296" orientation="0 0.436332 0"/>
     </xacro:if>
     <!-- ==== VRX sensor configuration ==== -->
@@ -144,6 +144,6 @@
       <!-- Add pinger -->
       <xacro:wamv_pinger name="pinger" position="1.0 0 -1.0" />
-      <!-- Add ball shooter -->
-      <xacro:wamv_ball_shooter name="ball_shooter" position="0.55 0.35 1.4" orientation="0 -1.0472 0"/>
+      <!-- Add ball shooter (default pitch angle: -15 deg) -->
+      <xacro:wamv_ball_shooter name="ball_shooter" position="0.54 0.30 1.296" orientation="0 -0.261799 0"/>
     </xacro:if>
   </xacro:unless>

Commit message: Fix ball shooter inertia in the WAM-V
Signed-off-by: Carlos Agüero <caguero@openrobotics.org>

File: wamv_gazebo/urdf/ball_shooter/ball_shooter.xacro (robot description, xacro)
@@ -26,4 +26,5 @@
       </collision>
       <inertial>
+        <origin xyz="0 0 0.08" rpy="0 -1.5708 0" />
         <mass value="0.5"/>
         <inertia ixx="0.001779167" ixy="0.0" ixz="0.0" iyy="0.001779167" iyz="0.0" izz="0.000225"/>

Commit message: Add ball shooter model (#316)
* Add ball shooter model.

Signed-off-by: Carlos Agüero <caguero@openrobotics.org>

File: wamv_gazebo/urdf/ball_shooter/ball_shooter.xacro (robot description, xacro)
@@ -4,11 +4,21 @@
     <link name="${namespace}/${name}_link">
       <visual name="${name}_visual">
-        <origin xyz="0 0 0" rpy="0 0 0" />
+        <!-- The cylinder has a -15deg pitch. We compensate for that here.
+             That way, if the user passes a 0 deg rotation the cylinder will
+             be parallel to the ground -->
+        <origin xyz="0 0 0" rpy="0 0.261799 0" />
         <geometry>
-          <box size="0.3 0.3 0.2" />
+          <mesh filename="package://vrx_gazebo/models/ball_shooter/meshes/ball_shooter.dae"/>
         </geometry>
       </visual>
+      <!-- Uncomment to see the pose where the ball is teleported -->
+      <!-- <visual name="${name}_visual_ball">
+        <origin xyz="0.14 0 0.09" rpy="0 0 0" />
+        <geometry>
+          <sphere radius="0.0285"/>
+        </geometry>
+      </visual> -->
       <collision name="${name}_collision">
-        <origin xyz="0 0 0" rpy="0 0 0" />
+        <origin xyz="0 0 0" rpy="0 0.261799 0" />
         <geometry>
           <box size="0.3 0.3 0.2" />
@@ -16,6 +26,7 @@
       </collision>
       <inertial>
-        <mass value="1"/>
-        <inertia ixx="0.006458" ixy="0.0" ixz="0.0" iyy="0.006458" iyz="0.0" izz="0.01125"/>
+        <origin xyz="0 0 0.08" rpy="0 -1.5708 0" />
+        <mass value="0.5"/>
+        <inertia ixx="0.001779167" ixy="0.0" ixz="0.0" iyy="0.001779167" iyz="0.0" izz="0.000225"/>
       </inertial>
     </link>
@@ -33,5 +44,5 @@
           <link_name>link</link_name>
           <frame>wamv/ball_shooter_link</frame>
-          <pose>0.2 0 0 0 0 0</pose>
+          <pose>0.14 0 0.09 0 0 0</pose>
         </projectile>
         <shot_force>250</shot_force>

File: wamv_gazebo/urdf/wamv_gazebo.urdf.xacro (robot description, xacro)
@@ -122,7 +122,7 @@
       <xacro:wamv_pinger name="pinger" position="1.0 0 -1.0" />
     </xacro:if>
-    <!-- Add ball shooter -->
+    <!-- Add ball shooter (default pitch angle: -15 deg) -->
     <xacro:if value="$(arg ball_shooter_enabled)">
-      <xacro:wamv_ball_shooter name="ball_shooter" position="2.0 0 -1.0" />
+      <xacro:wamv_ball_shooter name="ball_shooter" position="0.54 0.30 1.296" orientation="0 -0.261799 0"/>
     </xacro:if>
     <!-- ==== VRX sensor configuration ==== -->
@@ -144,6 +144,6 @@
       <!-- Add pinger -->
       <xacro:wamv_pinger name="pinger" position="1.0 0 -1.0" />
-      <!-- Add ball shooter -->
-      <xacro:wamv_ball_shooter name="ball_shooter" position="0.55 0.35 1.4" orientation="0 -1.0472 0"/>
+      <!-- Add ball shooter (default pitch angle: -15 deg) -->
+      <xacro:wamv_ball_shooter name="ball_shooter" position="0.54 0.30 1.296" orientation="0 -0.261799 0"/>
     </xacro:if>
   </xacro:unless>

Commit message: Migrated wamv_gazebo to ROS 2.

File: wamv_gazebo/urdf/ball_shooter/ball_shooter.xacro (robot description, xacro)
@@ -9,5 +9,5 @@
         <origin xyz="0 0 0" rpy="0 0.261799 0" />
         <geometry>
-          <mesh filename="package://vrx_gazebo/models/ball_shooter/meshes/ball_shooter.dae"/>
+          <mesh filename="file://$(find vrx_gazebo)/models/ball_shooter/meshes/ball_shooter.dae"/>
         </geometry>
       </visual>

File: wamv_gazebo/urdf/sensors/wamv_3d_lidar.xacro (robot description, xacro)
@@ -40,5 +40,5 @@
         <origin xyz="0 0 -0.035" rpy="0 0 0"/>
         <geometry>
-          <mesh filename="package://vrx_gazebo/models/3d_lidar/mesh/3d_lidar.dae"/>
+          <mesh filename="file://$(find vrx_gazebo)/models/3d_lidar/mesh/3d_lidar.dae"/>
         </geometry>
       </visual>
@@ -95,5 +95,5 @@
         <origin xyz="-0.038 0 -0.003" rpy="${radians(-60)} 0 ${-pi/2}"/>
         <geometry>
-          <mesh filename="package://vrx_gazebo/models/sensor_post/mesh/sensor_post_arm.dae"/>
+          <mesh filename="file://$(find vrx_gazebo)/models/sensor_post/mesh/sensor_post_arm.dae"/>
         </geometry>
       </visual>

File: wamv_gazebo/urdf/sensors/wamv_camera.xacro (robot description, xacro)
@@ -12,5 +12,5 @@
         <origin xyz="-0.033 0 0" rpy="0 0 ${pi/2}"/>
         <geometry>
-          <mesh filename="package://vrx_gazebo/models/mono_camera/mesh/mono_camera.dae"/>
+          <mesh filename="file://$(find vrx_gazebo)/models/mono_camera/mesh/mono_camera.dae"/>
         </geometry>
       </visual>
@@ -79,5 +79,5 @@
         <origin xyz="-0.038 0 -0.003" rpy="${radians(-60)} 0 ${-pi/2}"/>
         <geometry>
-          <mesh filename="package://vrx_gazebo/models/sensor_post/mesh/sensor_post_arm.dae"/>
+          <mesh filename="file://$(find vrx_gazebo)/models/sensor_post/mesh/sensor_post_arm.dae"/>
         </geometry>
       </visual>

File: wamv_gazebo/urdf/sensors/wamv_gps.xacro (robot description, xacro)
@@ -6,5 +6,5 @@
       <visual name="${name}_visual">
         <geometry>
-          <mesh filename="package://wamv_gazebo/models/gps/mesh/gps.dae"/>
+          <mesh filename="file://$(find wamv_gazebo)/models/gps/mesh/gps.dae"/>
         </geometry>
       </visual>

File: wamv_gazebo/urdf/thruster_layouts/wamv_gazebo_thruster_config.xacro (robot description, xacro)
@@ -7,6 +7,6 @@
       <propJointName>${namespace}/${name}_engine_propeller_joint</propJointName>
       <engineJointName>${namespace}/${name}_chasis_engine_joint</engineJointName>
-      <cmdTopic>${thruster_namespace}${name}_thrust_cmd</cmdTopic>
-      <angleTopic>${thruster_namespace}${name}_thrust_angle</angleTopic>
+      <cmdTopic>${namespace}/${thruster_namespace}${name}_thrust_cmd</cmdTopic>
+      <angleTopic>${namespace}/${thruster_namespace}${name}_thrust_angle</angleTopic>
       <enableAngle>${enable_angle}</enableAngle>
       <!-- Optional Parameters -->

Commit message: Tweak joint types.
Signed-off-by: Carlos Agüero <caguero@openrobotics.org>

File: wamv_gazebo/urdf/ball_shooter/ball_shooter.xacro (robot description, xacro)
@@ -31,7 +31,8 @@
       </inertial>
     </link>
-    <joint name="${namespace}/${name}_joint" type="revolute">
+    <!-- <joint name="${namespace}/${name}_joint" type="revolute"> -->
+    <joint name="${namespace}/${name}_joint" type="fixed">
       <axis xyz="0 0 1"/>
-      <limit effort="1000.0" lower="0.0" upper="0" velocity="0"/>
+      <!-- <limit effort="1000.0" lower="0.0" upper="0" velocity="0"/> -->
       <origin xyz="${position}" rpy="${orientation}"/>
       <parent link="${namespace}/base_link"/>

File: wamv_gazebo/urdf/sensors/wamv_gps.xacro (robot description, xacro)
@@ -27,7 +27,8 @@
       </inertial>
     </link>
-    <joint name="${namespace}/${name}_joint" type="revolute">
+    <!-- <joint name="${namespace}/${name}_joint" type="revolute"> -->
+    <joint name="${namespace}/${name}_joint" type="fixed">
       <axis xyz="0 0 1"/>
-      <limit effort="1000.0" lower="0.0" upper="0" velocity="0"/>
+      <!-- <limit effort="1000.0" lower="0.0" upper="0" velocity="0"/> -->
       <origin xyz="${x} ${y} ${z}" rpy="${R} ${P} ${Y}" />
       <parent link="${namespace}/base_link" />

File: wamv_gazebo/urdf/sensors/wamv_imu.xacro (robot description, xacro)
@@ -16,7 +16,8 @@
       </inertial>
     </link>
-    <joint name="${namespace}/${name}_joint" type="revolute">
+    <!-- <joint name="${namespace}/${name}_joint" type="revolute"> -->
+    <joint name="${namespace}/${name}_joint" type="fixed">
       <axis xyz="0 0 1"/>
-      <limit effort="1000.0" lower="0.0" upper="0" velocity="0"/>
+      <!-- <limit effort="1000.0" lower="0.0" upper="0" velocity="0"/> -->
       <origin xyz="${x} ${y} ${z}" rpy="${R} ${P} ${Y}"/>
       <parent link="${namespace}/base_link"/>

File: wamv_gazebo/urdf/wamv_gazebo.urdf.xacro (robot description, xacro)
@@ -145,5 +145,5 @@
       <xacro:wamv_pinger name="pinger" position="1.0 0 -1.0" />
       <!-- Add ball shooter (default pitch angle: ~-60 deg) -->
-      <xacro:wamv_ball_shooter name="ball_shooter" position="0.54 0.30 1.296" orientation="0 -1.04 0"/>
+      <!-- <xacro:wamv_ball_shooter name="ball_shooter" position="0.54 0.30 1.296" orientation="0 -1.04 0"/> -->
     </xacro:if>
   </xacro:unless>

Commit message: Update ball shooter.
Signed-off-by: Carlos Agüero <caguero@openrobotics.org>

File: wamv_gazebo/urdf/ball_shooter/ball_shooter.xacro (robot description, xacro)
@@ -1,18 +1,32 @@
 <?xml version="1.0"?>
 <robot xmlns:xacro="http://ros.org/wiki/xacro">
-  <xacro:macro name="wamv_ball_shooter" params="name:='ball_shooter' frameId:='wamv/ball_shooter' position:='0.55 0.35 1.4' orientation:='0 0 0'">
-    <link name="${namespace}/${name}_link">
-      <visual name="${name}_visual">
+  <xacro:macro name="wamv_ball_shooter" params="name:='ball_shooter' frameId:='wamv/ball_shooter' position:='0.55 0.35 1.4' pitch:='0' yaw:='0'">
+    <link name="${namespace}/${name}_base_link">
+      <visual name="${name}_base_visual">
+        <origin xyz="0 0 0" rpy="0 0 0" />
+        <geometry>
+          <mesh filename="package://vrx_gazebo/models/ball_shooter/meshes/ball_shooter_base.dae"/>
+        </geometry>
+      </visual>
+      <inertial>
+        <origin xyz="-0.02 0 0.05" rpy="0 0 0" />
+        <mass value="0.5"/>
+        <inertia ixx="0.00083" ixy="0.0" ixz="0.0" iyy="0.00052083" iyz="0.0" izz="0.00052083"/>
+      </inertial>
+    </link>
+    <link name="${namespace}/${name}_launcher_link">
+      <visual name="${name}_launcher_visual">
         <!-- The cylinder has a -15deg pitch. We compensate for that here.
              That way, if the user passes a 0 deg rotation the cylinder will
              be parallel to the ground -->
+        <!-- <origin xyz="-0.0204 0 0.107877" rpy="0 0.261799 0" /> -->
         <origin xyz="0 0 0" rpy="0 0.261799 0" />
         <geometry>
-          <mesh filename="package://vrx_gazebo/models/ball_shooter/meshes/ball_shooter.dae"/>
+          <mesh filename="package://vrx_gazebo/models/ball_shooter/meshes/ball_shooter_launcher.dae"/>
         </geometry>
       </visual>
       <!-- Uncomment to see the pose where the ball is teleported -->
       <!-- <visual name="${name}_visual_ball">
-        <origin xyz="0.14 0 0.09" rpy="0 0 0" />
+        <origin xyz="0.14 0 0" rpy="0 0 0" />
         <geometry>
           <sphere radius="0.0285"/>
@@ -26,15 +40,22 @@
       </collision>
       <inertial>
-        <origin xyz="0 0 0.08" rpy="0 -1.5708 0" />
+        <origin xyz="0 0 0" rpy="0 -1.5708 0" />
         <mass value="0.5"/>
         <inertia ixx="0.001779167" ixy="0.0" ixz="0.0" iyy="0.001779167" iyz="0.0" izz="0.000225"/>
       </inertial>
     </link>
-    <joint name="${namespace}/${name}_joint" type="revolute">
+    <joint name="${namespace}/${name}_base_joint" type="revolute">
       <axis xyz="0 0 1"/>
       <limit effort="1000.0" lower="0.0" upper="0" velocity="0"/>
-      <origin xyz="${position}" rpy="${orientation}"/>
+      <origin xyz="${position}" rpy="0 0 ${yaw}"/>
       <parent link="${namespace}/base_link"/>
-      <child link="${namespace}/${name}_link"/>
+      <child link="${namespace}/${name}_base_link"/>
+    </joint>
+    <joint name="${namespace}/${name}_launcher_joint" type="revolute">
+      <axis xyz="0 0 1"/>
+      <limit effort="1000.0" lower="0.0" upper="0" velocity="0"/>
+      <origin xyz="-0.0204 0 0.107877" rpy="0 ${pitch} 0"/>
+      <parent link="${namespace}/${name}_base_link"/>
+      <child link="${namespace}/${name}_launcher_link"/>
     </joint>
     <gazebo>
@@ -43,6 +64,6 @@
           <model_name>blue_projectile</model_name>
           <link_name>link</link_name>
-          <frame>wamv/ball_shooter_link</frame>
-          <pose>0.14 0 0.09 0 0 0</pose>
+          <frame>wamv/ball_shooter_launcher_link</frame>
+          <pose>0.14 0 0 0 0 0</pose>
         </projectile>
         <num_shots>4</num_shots>

File: wamv_gazebo/urdf/wamv_gazebo.urdf.xacro (robot description, xacro)
@@ -124,5 +124,5 @@
     <!-- Add ball shooter (default pitch angle: ~-60 deg) -->
     <xacro:if value="$(arg ball_shooter_enabled)">
-      <xacro:wamv_ball_shooter name="ball_shooter" position="0.54 0.30 1.296" orientation="0 -1.04 0"/>
+      <xacro:wamv_ball_shooter name="ball_shooter" position="0.54 0.30 1.296" pitch="-1.04"/>
     </xacro:if>
     <!-- ==== VRX sensor configuration ==== -->
@@ -145,5 +145,5 @@
       <xacro:wamv_pinger name="pinger" position="1.0 0 -1.0" />
       <!-- Add ball shooter (default pitch angle: ~-60 deg) -->
-      <xacro:wamv_ball_shooter name="ball_shooter" position="0.54 0.30 1.296" orientation="0 -1.04 0"/>
+      <xacro:wamv_ball_shooter name="ball_shooter" position="0.54 0.30 1.296" pitch="-1.04"/>
     </xacro:if>
   </xacro:unless>

Commit message: Corrected ball_shooter.xacro namespace change

File: wamv_gazebo/urdf/ball_shooter/ball_shooter.xacro (robot description, xacro)
@@ -49,5 +49,5 @@
       <limit effort="1000.0" lower="0.0" upper="0" velocity="0"/>
       <origin xyz="${position}" rpy="0 0 ${yaw}"/>
-      <parent link="wamv/base_link"/>
+      <parent link="${namespace}/base_link"/>
       <child link="${namespace}/${name}_base_link"/>
     </joint>
