Commit message: Added supporting files for sandwich, still needs adjustments to fit model

File: sandwich_description/urdf/sandwich.urdf.xacro (robot description, xacro)
@@ -1,4 +1,4 @@
 <?xml version="1.0"?>
-<robot xmlns:xacro="http://ros.org/wiki/xacro">
+<robot xmlns:xacro="http://ros.org/wiki/xacro" name="sandwich">
 	<!-- "Dummy" base link to eliminate root link inertia warning -->
 	<link name="sandwich/base_link"/>
@@ -15,5 +15,5 @@
 		<visual>
 			<origin xyz="0 0 0" rpy="0 0 0"/>
-			<goemetry>
+			<geometry>
 				<mesh filename="file://$(find sandwich_description)/models/sandwich_base/sandwich.dae" scale="1 1 1"/>
 			</geometry>

File: sandwich_description/urdf/sandwich.xacro (robot description, xacro)
@@ -4,8 +4,8 @@
 	<!-- Include macros for dynamics plugins -->
 	<!-- TODO -->
-	<!-- <xacro:include filename="(find sandwich_description)/urdf/macros.xacros"/> -->
+	<xacro:include filename="$(find sandwich_description)/urdf/macros.xacro"/>
 	<!-- Attach hydrodynamics plugin -->
 	<!-- TODO -->
-	<!-- <xacro:usv_dynamics_gazebo name="sandwich_dynamics_plugin"/> -->
+	<xacro:usv_dynamics_gazebo name="sandwich_dynamics_plugin"/>
 	<!-- Robot mesh -->
 	<xacro:include filename="$(find sandwich_description)/urdf/sandwich.urdf.xacro"/>
@@ -15,7 +15,7 @@
 	<!-- Thrusters -->
 	<!-- TODO -->
-	<!-- <xacro:arg name="thruster_namespace" default="thruster/"/> -->
-	<!-- <xacro:property name="thruster_namespace" value="$(arg thruster_namespace)" scope="global"/> -->
-	<!-- <xacro:include filename="$(find sandwich_description)/urdf/thruster.xacro"/> -->
+	<xacro:arg name="thruster_namespace" default="thruster/"/>
+	<xacro:property name="thruster_namespace" value="$(arg thruster_namespace)" scope="global"/>
+	<xacro:include filename="$(find sandwich_description)/urdf/thruster.xacro"/>
 	<!-- Decide if we lock the robot to the world -->
 	<xacro:if value="$(arg locked)">

File: wamv_gazebo/urdf/wamv_gazebo.urdf.xacro (robot description, xacro)
@@ -31,5 +31,5 @@
   <xacro:arg name="component_xacro_file" default = ""/>
   <!-- Thruster yaml file -->
-  <xacro:arg name="yaml_thruster_generation" default="true"/>
+  <xacro:arg name="yaml_thruster_generation" default="false"/>
   <xacro:arg name="thruster_xacro_file" default = ""/>
   <!-- === The WAM-V platform === -->
@@ -94,5 +94,5 @@
     <!-- Add CPU Cases -->
     <xacro:include filename="$(find wamv_description)/urdf/cpu_cases.xacro" />
-    <xacro:cpu_cases position="2.5 0 1.53" orientation="0 0 0"/>
+    <xacro:cpu_cases position="-0.15 0 1.53" orientation="0 0 0"/>
   </xacro:if>
   <!-- Otherwise, add sensors based on enable variables -->
