Commit message: add mesh geometry for buoyancy calculation

File: wamv_gazebo/urdf/buoyancy/wamv_buoyancy_plugin.xacro (robot description, xacro)
@@ -4,5 +4,5 @@
     <!--Gazebo Plugin for simulating WAM-V buoyancy-->
     <gazebo>
-      <plugin name="usv_buoyancy_${name}_hull_left" filename="libbuoyancy_gazebo_plugin.so">
+      <plugin name="usv_buoyancy_${name}" filename="libbuoyancy_gazebo_plugin.so">
         <!-- Wave model -->
         <wave_model>ocean_waves</wave_model>
@@ -13,30 +13,7 @@
         <buoyancy>
           <link_name>${namespace}/base_link</link_name>
-          <!-- pose info from wamv_base.urdf.xacro/${prefix}_float-->
-          <pose>0 -1.03 0.2 0 1.57 0</pose>
           <geometry>
-            <cylinder>
-              <radius>0.213</radius>
-              <length>${length}</length>
-            </cylinder>
-          </geometry>
-        </buoyancy>
-      </plugin>
-      <plugin name="usv_buoyancy_${name}_hull_right" filename="libbuoyancy_gazebo_plugin.so">
-        <!-- Wave model -->
-        <wave_model>ocean_waves</wave_model>
-        <fluid_density>997.8</fluid_density>
-        <fluid_level>0</fluid_level>
-        <linear_drag>0</linear_drag>
-        <angular_drag>0</angular_drag>
-        <buoyancy>
-          <link_name>${namespace}/base_link</link_name>
-          <!-- pose info from wamv_base.urdf.xacro/${prefix}_float-->
-          <pose>0 1.03 0.2 0 1.57 0</pose>
-          <geometry>
-            <cylinder>
-              <radius>0.213</radius>
-              <length>${length}</length>
-            </cylinder>
+            <!-- mesh from wamv_base.urdf.xacro/${namespace}/dummy_link -->
+            <mesh filename="package://wamv_description/models/WAM-V-Base/mesh/WAM-V-Base.dae"/>
           </geometry>
         </buoyancy>
