Commit message: Docking working.
Signed-off-by: Carlos Agüero <caguero@openrobotics.org>

File: vrx_urdf/wamv_description/urdf/cpu_cases.xacro (robot description, xacro)
@@ -3,10 +3,24 @@
 <xacro:macro name="cpu_cases" params="position:='0 0 0' orientation:='0 0 0'">
   <link name="${namespace}/cpu_cases_link">
-    <visual name="cpu_cases_visual">
+    <!-- <visual name="cpu_cases_visual">
       <origin xyz="0.073 0 -1.53" rpy="0 0 0"/>
       <geometry>
         <mesh filename="package://vrx_gazebo/models/cpu_cases/mesh/cpu_cases.dae"/>
       </geometry>
-    </visual>
+      <gazebo>
+        <material>
+          <diffuse>1.0 1.0 1.0</diffuse>
+          <specular>1.0 1.0 1.0</specular>
+          <pbr>
+            <metal>
+              <albedo_map>package://vrx_gazebo/models/cpu_cases/mesh/cpu_cases_Albedo.png</albedo_map>
+              <normal_map>package://vrx_gazebo/models/cpu_cases/mesh/cpu_cases_Normal.png</normal_map>
+              <roughness_map>package://vrx_gazebo/models/cpu_cases/mesh/cpu_cases_Roughness.png</roughness_map>
+              <metalness_map>package://vrx_gazebo/models/cpu_cases/mesh/cpu_cases_Metalness.png</metalness_map>
+            </metal>
+          </pbr>
+        </material>
+      </gazebo>
+    </visual> -->
     <collision name="cpu_case_1_collision">
       <origin xyz="0.185 0 0" rpy="0 0 0"/>
@@ -37,4 +51,26 @@
     <child link="${namespace}/cpu_cases_link"/>
   </joint>
+  <gazebo reference="${namespace}/cpu_cases_link">
+    <visual name="cpu_cases_visual">
+      <pose>0.073 0 -1.53 0 0 0</pose>
+      <geometry>
+        <mesh>
+          <uri>https://fuel.gazebosim.org/1.0/openrobotics/models/cpu_cases/mesh/cpu_cases.dae</uri>
+        </mesh>
+      </geometry>
+      <material>
+        <diffuse>1.0 1.0 1.0</diffuse>
+        <specular>1.0 1.0 1.0</specular>
+        <pbr>
+          <metal>
+            <albedo_map>https://fuel.gazebosim.org/1.0/openrobotics/models/cpu_cases/mesh/cpu_cases_Albedo.png</albedo_map>
+            <normal_map>https://fuel.gazebosim.org/1.0/openrobotics/models/cpu_cases/mesh/cpu_cases_Normal.png</normal_map>
+            <roughness_map>https://fuel.gazebosim.org/1.0/openrobotics/models/cpu_cases/mesh/cpu_cases_Roughness.png</roughness_map>
+            <metalness_map>https://fuel.gazebosim.org/1.0/openrobotics/models/cpu_cases/mesh/cpu_cases_Metalness.png</metalness_map>
+          </metal>
+        </pbr>
+      </material>
+    </visual>
+  </gazebo>
 </xacro:macro>
 </robot>

Commit message: Restore
Signed-off-by: Carlos Agüero <caguero@openrobotics.org>

File: vrx_urdf/wamv_description/urdf/cpu_cases.xacro (robot description, xacro)
@@ -3,24 +3,10 @@
 <xacro:macro name="cpu_cases" params="position:='0 0 0' orientation:='0 0 0'">
   <link name="${namespace}/cpu_cases_link">
-    <!-- <visual name="cpu_cases_visual">
+    <visual name="cpu_cases_visual">
       <origin xyz="0.073 0 -1.53" rpy="0 0 0"/>
       <geometry>
         <mesh filename="package://vrx_gazebo/models/cpu_cases/mesh/cpu_cases.dae"/>
       </geometry>
-      <gazebo>
-        <material>
-          <diffuse>1.0 1.0 1.0</diffuse>
-          <specular>1.0 1.0 1.0</specular>
-          <pbr>
-            <metal>
-              <albedo_map>package://vrx_gazebo/models/cpu_cases/mesh/cpu_cases_Albedo.png</albedo_map>
-              <normal_map>package://vrx_gazebo/models/cpu_cases/mesh/cpu_cases_Normal.png</normal_map>
-              <roughness_map>package://vrx_gazebo/models/cpu_cases/mesh/cpu_cases_Roughness.png</roughness_map>
-              <metalness_map>package://vrx_gazebo/models/cpu_cases/mesh/cpu_cases_Metalness.png</metalness_map>
-            </metal>
-          </pbr>
-        </material>
-      </gazebo>
-    </visual> -->
+    </visual>
     <collision name="cpu_case_1_collision">
       <origin xyz="0.185 0 0" rpy="0 0 0"/>
@@ -51,26 +37,4 @@
     <child link="${namespace}/cpu_cases_link"/>
   </joint>
-  <gazebo reference="${namespace}/cpu_cases_link">
-    <visual name="cpu_cases_visual">
-      <pose>0.073 0 -1.53 0 0 0</pose>
-      <geometry>
-        <mesh>
-          <uri>https://fuel.gazebosim.org/1.0/openrobotics/models/cpu_cases/mesh/cpu_cases.dae</uri>
-        </mesh>
-      </geometry>
-      <material>
-        <diffuse>1.0 1.0 1.0</diffuse>
-        <specular>1.0 1.0 1.0</specular>
-        <pbr>
-          <metal>
-            <albedo_map>https://fuel.gazebosim.org/1.0/openrobotics/models/cpu_cases/mesh/cpu_cases_Albedo.png</albedo_map>
-            <normal_map>https://fuel.gazebosim.org/1.0/openrobotics/models/cpu_cases/mesh/cpu_cases_Normal.png</normal_map>
-            <roughness_map>https://fuel.gazebosim.org/1.0/openrobotics/models/cpu_cases/mesh/cpu_cases_Roughness.png</roughness_map>
-            <metalness_map>https://fuel.gazebosim.org/1.0/openrobotics/models/cpu_cases/mesh/cpu_cases_Metalness.png</metalness_map>
-          </metal>
-        </pbr>
-      </material>
-    </visual>
-  </gazebo>
 </xacro:macro>
 </robot>

Commit message: Adding PBR to cpu cases.
Signed-off-by: Carlos Agüero <caguero@openrobotics.org>

File: vrx_urdf/wamv_description/urdf/cpu_cases.xacro (robot description, xacro)
@@ -3,5 +3,5 @@
 <xacro:macro name="cpu_cases" params="position:='0 0 0' orientation:='0 0 0'">
   <link name="${namespace}/cpu_cases_link">
-    <visual name="cpu_cases_visual">
+    <visual>
       <origin xyz="0.073 0 -1.53" rpy="0 0 0"/>
       <geometry>
@@ -37,4 +37,20 @@
     <child link="${namespace}/cpu_cases_link"/>
   </joint>
+  <gazebo reference="${namespace}/cpu_cases_link">
+    <visual>
+      <material>
+        <diffuse>1.0 1.0 1.0</diffuse>
+        <specular>1.0 1.0 1.0</specular>
+        <pbr>
+          <metal>
+            <albedo_map>model://vrx_gazebo/models/cpu_cases/mesh/cpu_cases_Albedo.png</albedo_map>
+            <normal_map>model://vrx_gazebo/models/cpu_cases/mesh/cpu_cases_Normal.png</normal_map>
+            <roughness_map>model://vrx_gazebo/models/cpu_cases/mesh/cpu_cases_Roughness.png</roughness_map>
+            <metalness_map>model://vrx_gazebo/models/cpu_cases/mesh/cpu_cases_Metalness.png</metalness_map>
+          </metal>
+        </pbr>
+      </material>
+    </visual>
+  </gazebo>
 </xacro:macro>
 </robot>
