Commit message: Battery PBR assets.
Signed-off-by: Carlos Agüero <caguero@openrobotics.org>

File: vrx_urdf/wamv_description/urdf/battery.xacro (robot description, xacro)
@@ -3,5 +3,5 @@
   <xacro:macro name="battery" params="prefix position:='0 0 0' orientation:='0 0 0'">
     <link name="${namespace}/${prefix}_battery_link">
-      <visual name="${prefix}_battery_visual">
+      <visual>
         <origin xyz="0 -1.03 -.45" rpy="0 0 0"/>
         <geometry>
@@ -32,4 +32,20 @@
       <child link="${namespace}/${prefix}_battery_link"/>
     </joint>
+    <gazebo reference="${namespace}/${prefix}_battery_link">
+      <visual>
+        <material>
+          <diffuse>1.0 1.0 1.0</diffuse>
+          <specular>1.0 1.0 1.0</specular>
+          <pbr>
+            <metal>
+              <albedo_map>model://vrx_gazebo/models/battery/mesh/battery_Albedo.png</albedo_map>
+              <normal_map>model://vrx_gazebo/models/battery/mesh/battery_Normal.png</normal_map>
+              <roughness_map>model://vrx_gazebo/models/battery/mesh/battery_Roughness.png</roughness_map>
+              <metalness_map>model://vrx_gazebo/models/battery/mesh/battery_Metalness.png</metalness_map>
+            </metal>
+          </pbr>
+        </material>
+      </visual>
+    </gazebo>
   </xacro:macro>
 </robot>
