Commit message: cleanup, contact sensor working, locked mode working
Signed-off-by: Ian Chen <ichen@openrobotics.org>

File: vrx_urdf/wamv_description/urdf/wamv_base.urdf.xacro (robot description, xacro)
@@ -86,5 +86,5 @@
   <link name="${namespace}/base_link">
   </link>
-  <joint name="${namespace}/dummy_joint" type = "fixed">
+  <joint name="${namespace}/dummy_joint" type="fixed">
     <parent link="${namespace}/base_link"/>
     <child link="${namespace}/dummy_link"/>
@@ -114,3 +114,20 @@
     </inertial>
   </link>
+  <gazebo reference="${namespace}/base_link">
+    <sensor type="contact" name="contact_sensor">
+      <contact>
+        <!-- collisions are renamed during urdf -> sdf fixed joint lumping -->
+        <collision>${namespace}/base_link_fixed_joint_lump__top_base_collision_41</collision>
+        <collision>${namespace}/base_link_fixed_joint_lump__left_float_collision_17</collision>
+        <collision>${namespace}/base_link_fixed_joint_lump__left_mid_float_collision_18</collision>
+        <collision>${namespace}/base_link_fixed_joint_lump__left_front_float_collision_19</collision>
+        <collision>${namespace}/base_link_fixed_joint_lump__right_float_collision_29</collision>
+        <collision>${namespace}/base_link_fixed_joint_lump__right_mid_float_collision_30</collision>
+        <collision>${namespace}/base_link_fixed_joint_lump__right_front_float_collision_31</collision>
+        <topic>/vrx/contacts</topic>
+      </contact>
+      <always_on>1</always_on>
+      <update_rate>5</update_rate>
+    </sensor>
+  </gazebo>
 </robot>

File: vrx_urdf/wamv_gazebo/urdf/components/wamv_3d_lidar.xacro (robot description, xacro)
@@ -164,19 +164,6 @@
           </noise>
         </ray>
-        <!--
-        <plugin name="${name}_plugin" filename="libgazebo_ros_velodyne_gpu_laser.so">
-          <topicName>${namespace}/${sensor_namespace}lidars/${name}/points</topicName>
-          <frameName>${namespace}/${name}_link</frameName>
-          <min_intensity>0</min_intensity>
-        </plugin>
-        -->
       </sensor>
     </gazebo>
-    <!-- Set color of post -->
-<!--
-    <gazebo reference="${namespace}/${name}_post_link">
-      <material>Gazebo/Black</material>
-    </gazebo>
--->
   </xacro:macro>
 </robot>

File: vrx_urdf/wamv_gazebo/urdf/components/wamv_camera.xacro (robot description, xacro)
@@ -154,28 +154,6 @@
           </noise>
         </camera>
-        <!--
-        <plugin name="camera_plugin_${name}" filename="libgazebo_ros_camera.so">
-          <alwaysOn>true</alwaysOn>
-          <updateRate>0.0</updateRate>
-          <cameraName>${namespace}/${sensor_namespace}${camera_namespace}${name}</cameraName>
-          <imageTopicName>image_raw</imageTopicName>
-          <cameraInfoTopicName>camera_info</cameraInfoTopicName>
-          <frameName>${namespace}/${name}_link_optical</frameName>
-          <hackBaseline>0.07</hackBaseline>
-          <distortionK1>0.0</distortionK1>
-          <distortionK2>0.0</distortionK2>
-          <distortionK3>0.0</distortionK3>
-          <distortionT1>0.0</distortionT1>
-          <distortionT2>0.0</distortionT2>
-        </plugin>
-        -->
-      </sensor>
+        </sensor>
     </gazebo>
-    <!-- Set color of post -->
-    <!--
-    <gazebo reference="${namespace}/${name}_post_link">
-      <material>Gazebo/Black</material>
-    </gazebo>
-    -->
   </xacro:macro>
 </robot>

File: vrx_urdf/wamv_gazebo/urdf/components/wamv_gps.xacro (robot description, xacro)
@@ -41,32 +41,4 @@
       </sensor>
     </gazebo>
-<!--
-    <gazebo>
-      <plugin name="gps_plugin_${name}" filename="libhector_gazebo_ros_gps.so">
-        <updateRate>${update_rate}</updateRate>
-        <alwaysOn>true</alwaysOn>
-        <bodyName>${namespace}/${name}_link</bodyName>
-        <frameId>${namespace}/${name}_link</frameId>
-        <topicName>${namespace}/${sensor_namespace}gps/gps/fix</topicName>
-        <velocityTopicName>${namespace}/${sensor_namespace}gps/gps/fix_velocity</velocityTopicName>
-	<useWorldSphericalCoordinates>true</useWorldSphericalCoordinates>
-        <offset>0.0 0.0 0.0</offset>
-        <drift>0.0 0.0 0.0</drift>
-        <gaussianNoise>0 0 0</gaussianNoise>
-        <velocityOffset>0.0 0.0 0.0</velocityOffset>
-        <velocityDrift>0.0 0.0 0.0</velocityDrift>
-        <velocityGaussianNoise>0.0 0.0 0.0</velocityGaussianNoise>
-      </plugin>
-    </gazebo>
--->
-        <!-- Note that the hector_gazebo_ros_gps plugin uses NWU coordinates
-             for reporting velocities.  This may cause problems if localization
-             requires velocity in ENU.
-             See Issue #64 in VRX project for details
-             https://bitbucket.org/osrf/vrx/issues/64 -->
-        <!-- Tell the plugin to use the spherical_coordiantes parameters
-	     from SDF.
-	     https://github.com/tu-darmstadt-ros-pkg/hector_gazebo/blob/melodic-devel/hector_gazebo_plugins/src/gazebo_ros_gps.cpp#L101
-	-->
   </xacro:macro>
 </robot>

File: vrx_urdf/wamv_gazebo/urdf/components/wamv_imu.xacro (robot description, xacro)
@@ -18,7 +18,4 @@
       <inertial>
         <mass value="0.1"/>
-        <!--
-        <inertia ixx="0.000083" ixy="0.0" ixz="0.0" iyy="0.000083" iyz="0.0" izz="0.0125"/>
-        -->
         <inertia ixx="0.00000542" ixy="0.0" ixz="0.0" iyy="0.00002104" iyz="0.0" izz="0.00002604"/>
       </inertial>
@@ -108,28 +105,4 @@
       </sensor>
     </gazebo>
-<!--
-    <gazebo>
-      <plugin name="imu_plugin_${name}" filename="libhector_gazebo_ros_imu.so">
-        <updateRate>${update_rate}</updateRate>
-        <bodyName>${namespace}/${name}_link</bodyName>
-        <topicName>${namespace}/${sensor_namespace}imu/imu/data</topicName>
-        <serviceName>${namespace}/${sensor_namespace}imu_service</serviceName>
-        <frameId>${namespace}/${name}_link</frameId>
-        <alwaysOn>true</alwaysOn>
-        <accelOffset>0.0 0.0 0.0</accelOffset>
-        <accelDrift>0.0 0.0 0.0</accelDrift>
-        <accelDriftFrequency>0.00027 0.00027 0.000027</accelDriftFrequency>
-        <accelGaussianNoise>0.0 0.0 0.0</accelGaussianNoise>
-        <rateOffset>0.0 0.0 0.0</rateOffset>
-        <rateDrift>0.0 0.0 0.0</rateDrift>
-        <rateDriftFrequency>0.00027 0.00027 0.000027</rateDriftFrequency>
-        <rateGaussianNoise>0.0 0.0 0.0</rateGaussianNoise>
-        <yawOffset>0.0</yawOffset>
-        <yawDrift>0.0</yawDrift>
-        <yawDriftFrequency>0.00027</yawDriftFrequency>
-        <yawGaussianNoise>0.0</yawGaussianNoise>
-      </plugin>
-    </gazebo>
--->
   </xacro:macro>
 </robot>

File: vrx_urdf/wamv_gazebo/urdf/components/wamv_p3d.xacro (robot description, xacro)
@@ -2,17 +2,4 @@
 <robot xmlns:xacro="http://ros.org/wiki/xacro">
   <xacro:macro name="wamv_p3d" params="name:=ground_truth_odometry">
-<!--
-    <gazebo>
-      <plugin name="p3d_plugin_${name}" filename="libgazebo_ros_p3d.so">
-        <bodyName>${namespace}/base_link</bodyName>
-        <frameName>map</frameName>
-        <updateRate>10.0</updateRate>
-        <topicName>${namespace}/${sensor_namespace}position/${name}</topicName>
-        <xyzOffset>0 0 0</xyzOffset>
-        <rpyOffset>0 0 0</rpyOffset>
-        <gaussianNoise>0</gaussianNoise>
-      </plugin>
-    </gazebo>
--->
     <gazebo>
       <plugin

File: vrx_urdf/wamv_gazebo/urdf/components/wamv_planar_lidar.xacro (robot description, xacro)
@@ -38,10 +38,4 @@
           </range>
         </ray>
-<!--
-        <plugin name="multibeam_simulator" filename="libgazebo_ros_gpu_laser.so">
-          <topicName>${namespace}/${sensor_namespace}lidars/${name}/scan</topicName>
-          <frameName>${namespace}/${name}_link</frameName>
-        </plugin>
--->
       </sensor>
     </gazebo>

File: vrx_urdf/wamv_gazebo/urdf/wamv_gazebo.urdf.xacro (robot description, xacro)
@@ -64,7 +64,8 @@
     <gazebo>
       <link name="wamv_external_link"/>
+      <link name="wamv_external_link_base"/>
       <joint name="wamv_external_pivot_joint" type="universal">
-        <parent>wamv::wamv/base_link</parent>
-        <child>wamv_external_link</child>
+        <parent>wamv_external_link</parent>
+        <child>wamv/base_link</child>
         <axis>
           <xyz>1 0 0</xyz>
@@ -75,5 +76,5 @@
       </joint>
       <joint name="wamv_external_riser" type="prismatic">
-        <parent>world</parent>
+        <parent>wamv_external_link_base</parent>
         <child>wamv_external_link</child>
         <axis>
@@ -85,4 +86,11 @@
         </axis>
       </joint>
+      <plugin filename="gz-sim-detachable-joint-system" name="gz::sim::systems::DetachableJoint">
+        <parent_link>wamv_external_link_base</parent_link>
+        <child_model>platform</child_model>
+        <child_link>dummy_base</child_link>
+        <topic>/vrx/release</topic>
+        <suppress_child_warning>true</suppress_child_warning>
+      </plugin>
     </gazebo>
   </xacro:if>
@@ -118,4 +126,24 @@
       <xacro:wamv_p3d name="p3d_wamv"/>
     </xacro:if>
+    <!-- Contact sensors -->
+<!--    <gazebo>
+      <experimental:params>
+        <sensor element_id="${namespace}/base_link" name='sensor_contacts' type='contact' action="add">
+          <contact>
+            <collision>top_base</collision>
+            <collision>left_float</collision>
+            <collision>left_mid_float</collision>
+            <collision>left_front_float</collision>
+            <collision>right_float</collision>
+            <collision>right_mid_float</collision>
+            <collision>right_front_float</collision>
+            <topic>/vrx/contacts</topic>
+          </contact>
+          <always_on>1</always_on>
+          <update_rate>5</update_rate>
+        </sensor>
+      </experimental:params>
+    </gazebo>
+-->
     <!-- Add pinger -->
     <xacro:if value="$(arg pinger_enabled)">

Commit message: WAM-V with PBR.
Signed-off-by: Carlos Agüero <caguero@osrfoundation.org>

File: vrx_urdf/wamv_description/urdf/wamv_base.urdf.xacro (robot description, xacro)
@@ -84,12 +84,6 @@
     </collision>
   </xacro:macro>
+  <!-- Basic model of the 16' WAM-V USV -->
   <link name="${namespace}/base_link">
-  </link>
-  <joint name="${namespace}/dummy_joint" type="fixed">
-    <parent link="${namespace}/base_link"/>
-    <child link="${namespace}/dummy_link"/>
-  </joint>
-  <!-- Basic model of the 16' WAM-V USV -->
-  <link name="${namespace}/dummy_link">
     <visual>
       <geometry>
@@ -115,4 +109,18 @@
   </link>
   <gazebo reference="${namespace}/base_link">
+    <visual>
+      <material>
+        <diffuse>1.0 1.0 1.0</diffuse>
+        <specular>1.0 1.0 1.0</specular>
+        <pbr>
+          <metal>
+            <albedo_map>model://wamv_description/models/WAM-V-Base/mesh/WAM-V_Albedo.png</albedo_map>
+            <!-- <normal_map>model://wamv_description/models/WAM-V-Base/mesh/WAM-V_Normal.png</normal_map> -->
+            <roughness_map>model://wamv_description/models/WAM-V-Base/mesh/WAM-V_Roughness.png</roughness_map>
+            <metalness_map>model://wamv_description/models/WAM-V-Base/mesh/WAM-V_Metalness.png</metalness_map>
+          </metal>
+        </pbr>
+      </material>
+    </visual>
     <sensor type="contact" name="contact_sensor">
       <contact>

Commit message: [Garden] Add PBR to the WAM-V base (#568)
* WAM-V with PBR.

Signed-off-by: Carlos Agüero <caguero@osrfoundation.org>

File: vrx_urdf/wamv_description/urdf/wamv_base.urdf.xacro (robot description, xacro)
@@ -84,12 +84,6 @@
     </collision>
   </xacro:macro>
+  <!-- Basic model of the 16' WAM-V USV -->
   <link name="${namespace}/base_link">
-  </link>
-  <joint name="${namespace}/dummy_joint" type="fixed">
-    <parent link="${namespace}/base_link"/>
-    <child link="${namespace}/dummy_link"/>
-  </joint>
-  <!-- Basic model of the 16' WAM-V USV -->
-  <link name="${namespace}/dummy_link">
     <visual>
       <geometry>
@@ -118,4 +112,18 @@
   </gazebo>
   <gazebo reference="${namespace}/base_link">
+    <visual>
+      <material>
+        <diffuse>1.0 1.0 1.0</diffuse>
+        <specular>1.0 1.0 1.0</specular>
+        <pbr>
+          <metal>
+            <albedo_map>model://wamv_description/models/WAM-V-Base/mesh/WAM-V_Albedo.png</albedo_map>
+            <normal_map>model://wamv_description/models/WAM-V-Base/mesh/WAM-V_Normal.png</normal_map>
+            <roughness_map>model://wamv_description/models/WAM-V-Base/mesh/WAM-V_Roughness.png</roughness_map>
+            <metalness_map>model://wamv_description/models/WAM-V-Base/mesh/WAM-V_Metalness.png</metalness_map>
+          </metal>
+        </pbr>
+      </material>
+    </visual>
     <sensor type="contact" name="contact_sensor">
       <contact>

Commit message: Restore collisions
Signed-off-by: Carlos Agüero <caguero@openrobotics.org>

File: vrx_urdf/wamv_description/urdf/wamv_base.urdf.xacro (robot description, xacro)
@@ -129,11 +129,11 @@
       <contact>
         <!-- collisions are renamed during urdf -> sdf fixed joint lumping -->
-        <collision>${namespace}/base_link_fixed_joint_lump__top_base_collision_41</collision>
-        <collision>${namespace}/base_link_fixed_joint_lump__left_float_collision_17</collision>
-        <collision>${namespace}/base_link_fixed_joint_lump__left_mid_float_collision_18</collision>
-        <collision>${namespace}/base_link_fixed_joint_lump__left_front_float_collision_19</collision>
-        <collision>${namespace}/base_link_fixed_joint_lump__right_float_collision_29</collision>
-        <collision>${namespace}/base_link_fixed_joint_lump__right_mid_float_collision_30</collision>
-        <collision>${namespace}/base_link_fixed_joint_lump__right_front_float_collision_31</collision>
+        <collision>${namespace}/base_link_fixed_joint_lump__top_base_collision_24</collision>
+        <collision>${namespace}/base_link_fixed_joint_lump__left_float_collision</collision>
+        <collision>${namespace}/base_link_fixed_joint_lump__left_mid_float_collision_1</collision>
+        <collision>${namespace}/base_link_fixed_joint_lump__left_front_float_collision_2</collision>
+        <collision>${namespace}/base_link_fixed_joint_lump__right_float_collision_12</collision>
+        <collision>${namespace}/base_link_fixed_joint_lump__right_mid_float_collision_13</collision>
+        <collision>${namespace}/base_link_fixed_joint_lump__right_front_float_collision_14</collision>
         <topic>/vrx/contacts</topic>
       </contact>
