Commit message: PBR camera and lidar.
Signed-off-by: Carlos Agüero <caguero@openrobotics.org>

File: vrx_urdf/wamv_gazebo/urdf/components/wamv_3d_lidar.xacro (robot description, xacro)
@@ -37,5 +37,5 @@
     <!-- 3d lidar sensor -->
     <link name="${namespace}/${name}_link">
-      <visual name="${name}_visual">
+      <visual>
         <origin xyz="0 0 -0.035" rpy="0 0 0"/>
         <geometry>
@@ -137,4 +137,18 @@
     </joint>
     <gazebo reference="${namespace}/${name}_link">
+      <visual>
+        <material>
+          <diffuse>1.0 1.0 1.0</diffuse>
+          <specular>1.0 1.0 1.0</specular>
+          <pbr>
+            <metal>
+              <albedo_map>model://vrx_gazebo/models/3d_lidar/mesh/3d_Lidar_Albedo.png</albedo_map>
+              <normal_map>model://vrx_gazebo/models/3d_lidar/mesh/3d_Lidar_Normal.png</normal_map>
+              <roughness_map>model://vrx_gazebo/models/3d_lidar/mesh/3d_Lidar_Roughness.png</roughness_map>
+              <metalness_map>model://vrx_gazebo/models/3d_lidar/mesh/3d_Lidar_Metalness.png</metalness_map>
+            </metal>
+          </pbr>
+        </material>
+      </visual>
       <sensor type="gpu_ray" name="${name}_sensor">
         <update_rate>${update_rate}</update_rate>

File: vrx_urdf/wamv_gazebo/urdf/components/wamv_camera.xacro (robot description, xacro)
@@ -9,5 +9,5 @@
     <!-- Monocular Camera -->
     <link name="${namespace}/${name}_link">
-      <visual name="${name}_visual">
+      <visual>
         <origin xyz="-0.033 0 0" rpy="0 0 ${pi/2}"/>
         <geometry>
@@ -129,4 +129,18 @@
     <!-- Gazebo camera setup -->
     <gazebo reference="${namespace}/${name}_link">
+      <visual>
+        <material>
+          <diffuse>1.0 1.0 1.0</diffuse>
+          <specular>1.0 1.0 1.0</specular>
+          <pbr>
+            <metal>
+              <albedo_map>model://vrx_gazebo/models/mono_camera/mesh/mono_camera_Albedo.png</albedo_map>
+              <normal_map>model://vrx_gazebo/models/mono_camera/mesh/mono_camera_Normal.png</normal_map>
+              <roughness_map>model://vrx_gazebo/models/mono_camera/mesh/mono_camera_Roughness.png</roughness_map>
+              <metalness_map>model://vrx_gazebo/models/mono_camera/mesh/mono_camera_Metalness.png</metalness_map>
+            </metal>
+          </pbr>
+        </material>
+      </visual>
       <sensor type="camera" name="${name}_sensor">
         <update_rate>30.0</update_rate>
