Commit message: Fix inertia and pinger visual.
Signed-off-by: Carlos Agüero <caguero@osrfoundation.org>

File: vrx_urdf/wamv_gazebo/urdf/components/wamv_pinger.xacro (robot description, xacro)
@@ -5,17 +5,11 @@
       <visual>
         <origin xyz="0 0 0" rpy="0 0 0" />
-        <geometry>
-          <box size="0.1 0.1 0.1" />
-        </geometry>
       </visual>
-      <collision name="${name}_collision">
-        <origin xyz="0 0 0" rpy="0 0 0" />
-        <geometry>
-          <box size="0.1 0.1 0.1" />
-        </geometry>
-      </collision>
+      <inertial>
+        <mass value="0.1"/>
+        <inertia ixx="0.00000542" ixy="0.0" ixz="0.0" iyy="0.00002104" iyz="0.0" izz="0.00002604"/>
+      </inertial>
     </link>
     <joint name="${namespace}/${name}_pinger_joint" type="fixed">
-      <origin xyz="${position}" rpy="${orientation}"/>
       <parent link="${namespace}/base_link"/>
       <child link="${namespace}/${name}"/>

File: vrx_urdf/wamv_gazebo/urdf/wamv_gazebo.urdf.xacro (robot description, xacro)
@@ -63,6 +63,30 @@
   <xacro:if value="$(arg locked)">
     <gazebo>
-      <link name="wamv_external_link"/>
-      <link name="wamv_external_link_base"/>
+      <link name="wamv_external_link">
+        <inertial>
+          <mass>0.001</mass>
+          <inertia>
+            <ixx>0.00000004</ixx>
+            <ixy>0</ixy>
+            <ixz>0</ixz>
+            <iyy>0.00000004</iyy>
+            <iyz>0</iyz>
+            <izz>0.00000004</izz>
+          </inertia>
+        </inertial>
+      </link>
+      <link name="wamv_external_link_base">
+        <inertial>
+          <mass>0.001</mass>
+          <inertia>
+            <ixx>0.00000004</ixx>
+            <ixy>0</ixy>
+            <ixz>0</ixz>
+            <iyy>0.00000004</iyy>
+            <iyz>0</iyz>
+            <izz>0.00000004</izz>
+          </inertia>
+        </inertial>
+      </link>
       <joint name="wamv_external_pivot_joint" type="universal">
         <parent>wamv_external_link</parent>

Commit message: Enable pinger link and visual
Signed-off-by: Carlos Agüero <caguero@openrobotics.org>

File: vrx_urdf/wamv_gazebo/urdf/components/wamv_pinger.xacro (robot description, xacro)
@@ -5,4 +5,7 @@
       <visual>
         <origin xyz="0 0 0" rpy="0 0 0" />
+        <geometry>
+          <sphere radius="0.01" />
+        </geometry>
       </visual>
       <inertial>
@@ -11,5 +14,8 @@
       </inertial>
     </link>
-    <joint name="${namespace}/${name}_pinger_joint" type="fixed">
+    <joint name="${namespace}/${name}_pinger_joint" type="revolute">
+      <axis xyz="0 0 1"/>
+      <limit effort="1000.0" lower="0.0" upper="0" velocity="0"/>
+      <origin xyz="0 0 0" rpy="0 0 0" />
       <parent link="${namespace}/base_link"/>
       <child link="${namespace}/${name}"/>

Commit message: Rename pinger topics.
Signed-off-by: Carlos Agüero <caguero@openrobotics.org>

File: vrx_urdf/wamv_gazebo/urdf/components/wamv_pinger.xacro (robot description, xacro)
@@ -1,6 +1,6 @@
 <?xml version="1.0"?>
 <robot xmlns:xacro="http://ros.org/wiki/xacro">
-  <xacro:macro name="wamv_pinger" params="name:='pinger' frameId:='wamv/pinger' position:='0 0 0' orientation:='0 0 0'">
-    <link name="${namespace}/${name}">
+  <xacro:macro name="wamv_pinger" params="pinger_name:='pinger' sensor_name:='receiver' frameId:='/pinger' position:='0 0 0' orientation:='0 0 0'">
+    <link name="${namespace}/${sensor_name}">
       <visual>
         <origin xyz="0 0 0" rpy="0 0 0" />
@@ -14,10 +14,10 @@
       </inertial>
     </link>
-    <joint name="${namespace}/${name}_pinger_joint" type="revolute">
+    <joint name="${namespace}/${sensor_name}_pinger_joint" type="revolute">
       <axis xyz="0 0 1"/>
       <limit effort="1000.0" lower="0.0" upper="0" velocity="0"/>
       <origin xyz="0 0 0" rpy="0 0 0" />
       <parent link="${namespace}/base_link"/>
-      <child link="${namespace}/${name}"/>
+      <child link="${namespace}/${sensor_name}"/>
     </joint>
     <gazebo>
@@ -26,8 +26,8 @@
         name="vrx::AcousticPingerPlugin">
         <position>${position}</position>
-        <topic>${namespace}/${pinger_namespace}${name}/range_bearing</topic>
-        <set_position_topic>${namespace}/${pinger_namespace}${name}/set_pinger_position
+        <topic>/${namespace}/${sensor_namespace}${acoustic_namespace}${sensor_name}/range_bearing</topic>
+        <set_position_topic>/${pinger_name}/set_pinger_position
         </set_position_topic>
-        <frame_id>${namespace}/${name}</frame_id>
+        <frame_id>${namespace}/${sensor_name}</frame_id>
         <range_noise>
           <noise>

File: vrx_urdf/wamv_gazebo/urdf/wamv_gazebo.urdf.xacro (robot description, xacro)
@@ -16,5 +16,5 @@
   <xacro:arg name="camera_namespace" default="cameras/"/>
   <xacro:arg name="sensor_namespace" default="sensors/"/>
-  <xacro:arg name="pinger_namespace" default="pingers/"/>
+  <xacro:arg name="acoustic_namespace" default="acoustics/"/>
   <xacro:arg name="shooter_namespace" default="shooters/"/>
   <!-- Note: this is only used for some sensors that do not correctly use the
@@ -24,5 +24,5 @@
   <xacro:property name="camera_namespace" value="$(arg camera_namespace)" scope="global" />
   <xacro:property name="sensor_namespace" value="$(arg sensor_namespace)" scope="global" />
-  <xacro:property name="pinger_namespace" value="$(arg pinger_namespace)" scope="global" />
+  <xacro:property name="acoustic_namespace" value="$(arg acoustic_namespace)" scope="global" />
   <xacro:property name="shooter_namespace" value="$(arg shooter_namespace)" scope="global" />
   <xacro:property name="namespace" value="$(arg namespace)" scope="global" />
@@ -168,5 +168,5 @@
     <!-- Add pinger -->
     <xacro:if value="$(arg pinger_enabled)">
-      <xacro:wamv_pinger name="pinger" position="-528 191 -2.0" />
+      <xacro:wamv_pinger sensor_name="receiver" position="-528 191 -2.0" />
     </xacro:if>
     <!-- Add ball shooter (default pitch angle: ~-60 deg) -->
@@ -191,5 +191,5 @@
       <xacro:lidar name="lidar_wamv" type="16_beam"/>
       <!-- Add pinger -->
-      <xacro:wamv_pinger name="pinger" position="-528 191 -2.0" />
+      <xacro:wamv_pinger sensor_name="receiver" position="-528 191 -2.0" />
       <!-- Add ball shooter (default pitch angle: ~-60 deg) -->
       <xacro:wamv_ball_shooter name="ball_shooter" x="0.54" y="0.30" z="1.296" pitch="-1.04"/>

Commit message: Fix issue #691 (#692)
* Rename pinger topics.

Signed-off-by: Carlos Agüero <caguero@openrobotics.org>
Co-authored-by: M1chaelM <M1chaelM@users.noreply.github.com>

File: vrx_urdf/wamv_gazebo/urdf/components/wamv_pinger.xacro (robot description, xacro)
@@ -1,6 +1,6 @@
 <?xml version="1.0"?>
 <robot xmlns:xacro="http://ros.org/wiki/xacro">
-  <xacro:macro name="wamv_pinger" params="name:='pinger' frameId:='wamv/pinger' position:='0 0 0' orientation:='0 0 0'">
-    <link name="${namespace}/${name}">
+  <xacro:macro name="wamv_pinger" params="pinger_name:='pinger' sensor_name:='receiver' frameId:='/pinger' position:='0 0 0' orientation:='0 0 0'">
+    <link name="${namespace}/${sensor_name}">
       <visual>
         <origin xyz="0 0 0" rpy="0 0 0" />
@@ -14,10 +14,10 @@
       </inertial>
     </link>
-    <joint name="${namespace}/${name}_pinger_joint" type="revolute">
+    <joint name="${namespace}/${sensor_name}_pinger_joint" type="revolute">
       <axis xyz="0 0 1"/>
       <limit effort="1000.0" lower="0.0" upper="0" velocity="0"/>
       <origin xyz="0 0 0" rpy="0 0 0" />
       <parent link="${namespace}/base_link"/>
-      <child link="${namespace}/${name}"/>
+      <child link="${namespace}/${sensor_name}"/>
     </joint>
     <gazebo>
@@ -26,8 +26,8 @@
         name="vrx::AcousticPingerPlugin">
         <position>${position}</position>
-        <topic>${namespace}/${pinger_namespace}${name}/range_bearing</topic>
-        <set_position_topic>${namespace}/${pinger_namespace}${name}/set_pinger_position
+        <topic>/${namespace}/${sensor_namespace}${acoustic_namespace}${sensor_name}/range_bearing</topic>
+        <set_position_topic>/${pinger_name}/set_pinger_position
         </set_position_topic>
-        <frame_id>${namespace}/${name}</frame_id>
+        <frame_id>${pinger_name}</frame_id>
         <range_noise>
           <noise>
