Commit message: updating plugins
Signed-off-by: Ian Chen <ichen@openrobotics.org>

File: vrx_urdf/wamv_gazebo/urdf/components/ball_shooter.xacro (robot description, xacro)
@@ -59,4 +59,5 @@
       <child link="${namespace}/${name}_launcher_link"/>
     </joint>
+<!--
     <gazebo>
       <plugin name="ball_shooter_plugin" filename="libball_shooter_plugin.so">
@@ -72,4 +73,5 @@
       </plugin>
     </gazebo>
+-->
   </xacro:macro>
 </robot>

File: vrx_urdf/wamv_gazebo/urdf/components/wamv_3d_lidar.xacro (robot description, xacro)
@@ -164,4 +164,5 @@
           </noise>
         </ray>
+        <!--
         <plugin name="${name}_plugin" filename="libgazebo_ros_velodyne_gpu_laser.so">
           <topicName>${namespace}/${sensor_namespace}lidars/${name}/points</topicName>
@@ -169,7 +170,9 @@
           <min_intensity>0</min_intensity>
         </plugin>
+        -->
       </sensor>
     </gazebo>
     <!-- Set color of post -->
+<!--
     <gazebo reference="${namespace}/${name}_post_link">
       <material>Gazebo/Black</material>

File: vrx_urdf/wamv_gazebo/urdf/components/wamv_camera.xacro (robot description, xacro)
@@ -154,4 +154,5 @@
           </noise>
         </camera>
+        <!--
         <plugin name="camera_plugin_${name}" filename="libgazebo_ros_camera.so">
           <alwaysOn>true</alwaysOn>
@@ -168,10 +169,13 @@
           <distortionT2>0.0</distortionT2>
         </plugin>
+        -->
       </sensor>
     </gazebo>
     <!-- Set color of post -->
+    <!--
     <gazebo reference="${namespace}/${name}_post_link">
       <material>Gazebo/Black</material>
     </gazebo>
+    -->
   </xacro:macro>
 </robot>

File: vrx_urdf/wamv_gazebo/urdf/components/wamv_gps.xacro (robot description, xacro)
@@ -34,4 +34,12 @@
       <child link="${namespace}/${name}_link" />
     </joint>
+    <gazebo reference="${namespace}/${name}_link">
+      <sensor name="navsat" type="navsat">
+        <always_on>1</always_on>
+        <update_rate>15</update_rate>
+        <topic>${namespace}/${sensor_namespace}gps/gps/fix</topic>
+      </sensor>
+    </gazebo>
+<!--
     <gazebo>
       <plugin name="gps_plugin_${name}" filename="libhector_gazebo_ros_gps.so">
@@ -39,17 +47,7 @@
         <alwaysOn>true</alwaysOn>
         <bodyName>${namespace}/${name}_link</bodyName>
-        <!-- Manually prepend namespace to tf frame. -->
         <frameId>${namespace}/${name}_link</frameId>
         <topicName>${namespace}/${sensor_namespace}gps/gps/fix</topicName>
-        <!-- Note that the hector_gazebo_ros_gps plugin uses NWU coordinates
-             for reporting velocities.  This may cause problems if localization
-             requires velocity in ENU.
-             See Issue #64 in VRX project for details
-             https://bitbucket.org/osrf/vrx/issues/64 -->
         <velocityTopicName>${namespace}/${sensor_namespace}gps/gps/fix_velocity</velocityTopicName>
-        <!-- Tell the plugin to use the spherical_coordiantes parameters
-	     from SDF.
-	     https://github.com/tu-darmstadt-ros-pkg/hector_gazebo/blob/melodic-devel/hector_gazebo_plugins/src/gazebo_ros_gps.cpp#L101
-	-->
 	<useWorldSphericalCoordinates>true</useWorldSphericalCoordinates>
         <offset>0.0 0.0 0.0</offset>
@@ -61,4 +59,14 @@
       </plugin>
     </gazebo>
+-->
+        <!-- Note that the hector_gazebo_ros_gps plugin uses NWU coordinates
+             for reporting velocities.  This may cause problems if localization
+             requires velocity in ENU.
+             See Issue #64 in VRX project for details
+             https://bitbucket.org/osrf/vrx/issues/64 -->
+        <!-- Tell the plugin to use the spherical_coordiantes parameters
+	     from SDF.
+	     https://github.com/tu-darmstadt-ros-pkg/hector_gazebo/blob/melodic-devel/hector_gazebo_plugins/src/gazebo_ros_gps.cpp#L101
+	-->
   </xacro:macro>
 </robot>

File: vrx_urdf/wamv_gazebo/urdf/components/wamv_imu.xacro (robot description, xacro)
@@ -23,4 +23,5 @@
       <child link="${namespace}/${name}_link"/>
     </joint>
+<!--
     <gazebo>
       <plugin name="imu_plugin_${name}" filename="libhector_gazebo_ros_imu.so">
@@ -29,5 +30,4 @@
         <topicName>${namespace}/${sensor_namespace}imu/imu/data</topicName>
         <serviceName>${namespace}/${sensor_namespace}imu_service</serviceName>
-        <!-- Manually prepend namespace to tf frame. -->
         <frameId>${namespace}/${name}_link</frameId>
         <alwaysOn>true</alwaysOn>
@@ -46,4 +46,5 @@
       </plugin>
     </gazebo>
+-->
   </xacro:macro>
 </robot>

File: vrx_urdf/wamv_gazebo/urdf/components/wamv_p3d.xacro (robot description, xacro)
@@ -2,4 +2,5 @@
 <robot xmlns:xacro="http://ros.org/wiki/xacro">
   <xacro:macro name="wamv_p3d" params="name:=ground_truth_odometry">
+<!--
     <gazebo>
       <plugin name="p3d_plugin_${name}" filename="libgazebo_ros_p3d.so">
@@ -13,4 +14,14 @@
       </plugin>
     </gazebo>
+-->
+    <gazebo>
+      <plugin
+        filename="gz-sim-odometry-publisher-system"
+        name="gz::sim::systems::OdometryPublisher_${name}">
+        <dimensions>3</dimensions>
+        <odom_publish_frequency>10.0</odom_publish_frequency>
+        <odom_frame>map</odom_frame>
+      </plugin>
+    </gazebo>
   </xacro:macro>
 </robot>

File: vrx_urdf/wamv_gazebo/urdf/components/wamv_pinger.xacro (robot description, xacro)
@@ -21,4 +21,5 @@
       <child link="${namespace}/${name}"/>
     </joint>
+<!--
     <gazebo>
       <plugin name="pinger_plugin" filename="libusv_gazebo_acoustic_pinger_plugin.so">
@@ -49,4 +50,5 @@
       </plugin>
     </gazebo>
+-->
   </xacro:macro>
 </robot>

File: vrx_urdf/wamv_gazebo/urdf/components/wamv_planar_lidar.xacro (robot description, xacro)
@@ -38,8 +38,10 @@
           </range>
         </ray>
+<!--
         <plugin name="multibeam_simulator" filename="libgazebo_ros_gpu_laser.so">
           <topicName>${namespace}/${sensor_namespace}lidars/${name}/scan</topicName>
           <frameName>${namespace}/${name}_link</frameName>
         </plugin>
+-->
       </sensor>
     </gazebo>

File: vrx_urdf/wamv_gazebo/urdf/dynamics/wamv_gazebo_dynamics_plugin.xacro (robot description, xacro)
@@ -1,5 +1,5 @@
 <?xml version="1.0"?>
 <robot xmlns:xacro="http://ros.org/wiki/xacro">
-  <xacro:macro name="usv_dynamics_gazebo" params="wavefield_size:=1000">
+  <xacro:macro name="usv_dynamics_gazebo" params="name wavefield_size:=1000">
     <!--Gazebo Plugin for simulating WAM-V dynamics-->
     <gazebo>
@@ -64,5 +64,5 @@
       <plugin
         filename="libSimpleHydrodynamics.so"
-        name="vrx::SimpleHydrodynamics">
+        name="vrx::SimpleHydrodynamics_${name}">
         <link_name>${namespace}/base_link</link_name>
         <!-- Added mass -->

File: vrx_urdf/wamv_gazebo/urdf/wamv_gazebo.xacro (robot description, xacro)
@@ -10,5 +10,5 @@
     <xacro:include filename="${thruster_layout}"/>
     <!-- Attach hydrodynamics plugin -->
-    <xacro:usv_dynamics_gazebo/>
+    <xacro:usv_dynamics_gazebo name="wamv_dynamics_plugin"/>
   </xacro:macro>
 </robot>

Commit message: Ball shooter PBR
Signed-off-by: Carlos Agüero <caguero@osrfoundation.org>

File: vrx_urdf/wamv_gazebo/urdf/components/ball_shooter.xacro (robot description, xacro)
@@ -3,5 +3,5 @@
   <xacro:macro name="wamv_ball_shooter" params="name:='ball_shooter' frameId:='wamv/ball_shooter' x:=0.55 y:=0.35 z:=1.4 pitch:='0' yaw:='0'">
     <link name="${namespace}/${name}_base_link">
-      <visual name="${name}_base_visual">
+      <visual>
         <origin xyz="0 0 0" rpy="0 0 0" />
         <geometry>
@@ -16,5 +16,5 @@
     </link>
     <link name="${namespace}/${name}_launcher_link">
-      <visual name="${name}_launcher_visual">
+      <visual>
         <!-- The cylinder has a -15deg pitch. We compensate for that here.
              That way, if the user passes a 0 deg rotation the cylinder will
@@ -59,4 +59,36 @@
       <child link="${namespace}/${name}_launcher_link"/>
     </joint>
+    <gazebo reference="${namespace}/${name}_base_link">
+      <visual>
+        <material>
+          <diffuse>1.0 1.0 1.0</diffuse>
+          <specular>1.0 1.0 1.0</specular>
+          <pbr>
+            <metal>
+              <albedo_map>model://vrx_gazebo/models/ball_shooter/materials/Textures/Launcher_Albedo.png</albedo_map>
+              <normal_map>model://vrx_gazebo/models/ball_shooter/materials/Textures/Launcher_Normal.png</normal_map>
+              <roughness_map>model://vrx_gazebo/models/ball_shooter/materials/Textures/Launcher_Roughness.png</roughness_map>
+              <metalness_map>model://vrx_gazebo/models/ball_shooter/materials/Textures/Launcher_Metalness.png</metalness_map>
+            </metal>
+          </pbr>
+        </material>
+      </visual>
+    </gazebo>
+    <gazebo reference="${namespace}/${name}_launcher_link">
+      <visual>
+        <material>
+          <diffuse>1.0 1.0 1.0</diffuse>
+          <specular>1.0 1.0 1.0</specular>
+          <pbr>
+            <metal>
+              <albedo_map>model://vrx_gazebo/models/ball_shooter/materials/Textures/Launcher_Albedo.png</albedo_map>
+              <normal_map>model://vrx_gazebo/models/ball_shooter/materials/Textures/Launcher_Normal.png</normal_map>
+              <roughness_map>model://vrx_gazebo/models/ball_shooter/materials/Textures/Launcher_Roughness.png</roughness_map>
+              <metalness_map>model://vrx_gazebo/models/ball_shooter/materials/Textures/Launcher_Metalness.png</metalness_map>
+            </metal>
+          </pbr>
+        </material>
+      </visual>
+    </gazebo>
     <gazebo>
       <plugin name="vrx::BallShooterPlugin" filename="libBallShooterPlugin.so">

Commit message: Make IMU, GPS, pinger and ball shooter joints fixed

File: vrx_urdf/wamv_gazebo/urdf/components/ball_shooter.xacro (robot description, xacro)
@@ -45,14 +45,10 @@
       </inertial>
     </link>
-    <joint name="${namespace}/${name}_base_joint" type="revolute">
-      <axis xyz="0 0 1"/>
-      <limit effort="1000.0" lower="0.0" upper="0" velocity="0"/>
+    <joint name="${namespace}/${name}_base_joint" type="fixed">
       <origin xyz="${x} ${y} ${z}" rpy="0 0 ${yaw}"/>
       <parent link="${namespace}/base_link"/>
       <child link="${namespace}/${name}_base_link"/>
     </joint>
-    <joint name="${namespace}/${name}_launcher_joint" type="revolute">
-      <axis xyz="0 0 1"/>
-      <limit effort="1000.0" lower="0.0" upper="0" velocity="0"/>
+    <joint name="${namespace}/${name}_launcher_joint" type="fixed">
       <origin xyz="-0.0204 0 0.107877" rpy="0 ${pitch} 0"/>
       <parent link="${namespace}/${name}_base_link"/>

File: vrx_urdf/wamv_gazebo/urdf/components/wamv_gps.xacro (robot description, xacro)
@@ -27,7 +27,5 @@
       </inertial>
     </link>
-    <joint name="${namespace}/${name}_joint" type="revolute">
-      <axis xyz="0 0 1"/>
-      <limit effort="1000.0" lower="0.0" upper="0" velocity="0"/>
+    <joint name="${namespace}/${name}_joint" type="fixed">
       <origin xyz="${x} ${y} ${z}" rpy="${R} ${P} ${Y}" />
       <parent link="${namespace}/base_link" />

File: vrx_urdf/wamv_gazebo/urdf/components/wamv_imu.xacro (robot description, xacro)
@@ -21,7 +21,5 @@
       </inertial>
     </link>
-    <joint name="${namespace}/${name}_joint" type="revolute">
-      <axis xyz="0 0 1"/>
-      <limit effort="1000.0" lower="0.0" upper="0" velocity="0"/>
+    <joint name="${namespace}/${name}_joint" type="fixed">
       <origin xyz="${x} ${y} ${z}" rpy="${R} ${P} ${Y}"/>
       <parent link="${namespace}/base_link"/>

File: vrx_urdf/wamv_gazebo/urdf/components/wamv_pinger.xacro (robot description, xacro)
@@ -14,7 +14,5 @@
       </inertial>
     </link>
-    <joint name="${namespace}/${sensor_name}_pinger_joint" type="revolute">
-      <axis xyz="0 0 1"/>
-      <limit effort="1000.0" lower="0.0" upper="0" velocity="0"/>
+    <joint name="${namespace}/${sensor_name}_pinger_joint" type="fixed">
       <origin xyz="0 0 0" rpy="0 0 0" />
       <parent link="${namespace}/base_link"/>
