Commit message: Refix engine.xacro to have revolute joint

File: wamv_description/urdf/thrusters/engine.xacro (robot description, xacro)
@@ -43,5 +43,7 @@
       </inertial>
     </link>
-    <joint name="${prefix}_chasis_engine_joint" type="fixed">
+    <joint name="${prefix}_chasis_engine_joint" type="revolute">
+      <axis xyz="0 0 1"/>
+      <limit lower="${-pi}" upper="${pi}" effort="10" velocity="10"/>
       <origin xyz="${position}" rpy="${orientation}"/>
       <parent link="base_link"/>

Commit message: Add support for namespaces This includes thruster, camera and sensor namespaces, as well as a global namespace allowing multiple vehicles to be created without causing interference.

File: wamv_description/urdf/thrusters/engine.xacro (robot description, xacro)
@@ -2,5 +2,5 @@
 <robot xmlns:xacro="http://ros.org/wiki/xacro" name="wam-v-two-engines">
   <!-- Macro for inserting an engine with its propeller. -->
-  <xacro:macro name="engine" params="prefix position:='0 0 0' orientation:='0 0 0'">
+  <xacro:macro name="engine" params="prefix position:='0 0 0' orientation:='0 0 0' namespace:='' thruster_namespace:=''">
     <link name="${prefix}_engine_link">
       <visual>

File: wamv_gazebo/urdf/sensors/wamv_3d_lidar.xacro (robot description, xacro)
@@ -164,5 +164,5 @@
         </ray>
         <plugin name="${name}_plugin" filename="libgazebo_ros_velodyne_gpu_laser.so">
-          <topicName>${name}/points</topicName>
+          <topicName>${namespace}${sensor_namespace}/${name}/points</topicName>
           <frameName>${name}_link</frameName>
           <min_intensity>0</min_intensity>

File: wamv_gazebo/urdf/sensors/wamv_camera.xacro (robot description, xacro)
@@ -1,5 +1,5 @@
 <?xml version="1.0"?>
 <robot xmlns:xacro="http://ros.org/wiki/xacro">
-  <xacro:macro name="wamv_camera" params="name x:=0.5 y:=0 z:=1.5 R:=0 P:=0 Y:=0 post_Y:=0">
+  <xacro:macro name="wamv_camera" params="name x:=0.5 y:=0 z:=1.5 R:=0 P:=0 Y:=0 post_Y:=0 ">
     <!-- Define length variables for link positioning -->
     <xacro:property name="platform_z" value="1.2965"/>
@@ -143,5 +143,5 @@
           <alwaysOn>true</alwaysOn>
           <updateRate>0.0</updateRate>
-          <cameraName>${name}</cameraName>
+          <cameraName>${namespace}${camera_namespace}/${name}</cameraName>
           <imageTopicName>image_raw</imageTopicName>
           <cameraInfoTopicName>camera_info</cameraInfoTopicName>

File: wamv_gazebo/urdf/sensors/wamv_gps.xacro (robot description, xacro)
@@ -36,6 +36,6 @@
         <bodyName>${name}_link</bodyName>
         <frameId>${name}_link</frameId>
-        <topicName>gps/fix</topicName>
-        <velocityTopicName>gps/fix_velocity</velocityTopicName>
+        <topicName>${namespace}${sensor_namespace}/gps/fix</topicName>
+        <velocityTopicName>${namespace}${sensor_namespace}/gps/fix_velocity</velocityTopicName>
         <!-- Location of origin of Gazebo Sand Island map -->
         <referenceLatitude>21.30996</referenceLatitude>

File: wamv_gazebo/urdf/sensors/wamv_imu.xacro (robot description, xacro)
@@ -21,6 +21,6 @@
         <updateRate>15.0</updateRate>
         <bodyName>${name}_link</bodyName>
-        <topicName>imu/data</topicName>
-        <serviceName>imu_service</serviceName>
+        <topicName>${namespace}${sensor_namespace}/imu/data</topicName>
+        <serviceName>${namespace}${sensor_namespace}/imu_service</serviceName>
         <frameId>${name}_link</frameId>
         <alwaysOn>true</alwaysOn>

File: wamv_gazebo/urdf/thruster_layouts/wamv_gazebo_thruster_config.xacro (robot description, xacro)
@@ -7,6 +7,6 @@
       <propJointName>${name}_engine_propeller_joint</propJointName>
       <engineJointName>${name}_chasis_engine_joint</engineJointName>
-      <cmdTopic>${name}_thrust_cmd</cmdTopic>
-      <angleTopic>${name}_thrust_angle</angleTopic>
+      <cmdTopic>${namespace}${thruster_namespace}/${name}_thrust_cmd</cmdTopic>
+      <angleTopic>${namespace}${thruster_namespace}/${name}_thrust_angle</angleTopic>
       <enableAngle>true</enableAngle>
       <!-- Optional Parameters -->

File: wamv_gazebo/urdf/wamv_gazebo.urdf.xacro (robot description, xacro)
@@ -11,4 +11,12 @@
   <xacro:arg name="ground_truth_enabled" default="false" />
   <xacro:arg name="vrx_sensors_enabled" default="false" />
+  <xacro:arg name="namespace" default="/wamv"/>
+  <xacro:arg name="thruster_namespace" default="/thrusters"/>
+  <xacro:arg name="camera_namespace" default="/cameras"/>
+  <xacro:arg name="sensor_namespace" default="/sensors"/>
+  <xacro:property name="namespace" value="$(arg namespace)" scope="global" />
+  <xacro:property name="thruster_namespace" value="$(arg thruster_namespace)" scope="global" />
+  <xacro:property name="camera_namespace" value="$(arg camera_namespace)" scope="global" />
+  <xacro:property name="sensor_namespace" value="$(arg sensor_namespace)" scope="global" />
   <!-- Sensor yaml file -->
   <xacro:arg name="yaml_sensor_generation" default="false"/>

Commit message: Add sensor namepsace to planar lidar Remove gloabl namespace

File: wamv_description/urdf/thrusters/engine.xacro (robot description, xacro)
@@ -2,5 +2,5 @@
 <robot xmlns:xacro="http://ros.org/wiki/xacro" name="wam-v-two-engines">
   <!-- Macro for inserting an engine with its propeller. -->
-  <xacro:macro name="engine" params="prefix position:='0 0 0' orientation:='0 0 0' namespace:='' thruster_namespace:=''">
+  <xacro:macro name="engine" params="prefix position:='0 0 0' orientation:='0 0 0'">
     <link name="${prefix}_engine_link">
       <visual>

File: wamv_gazebo/urdf/sensors/wamv_3d_lidar.xacro (robot description, xacro)
@@ -164,5 +164,5 @@
         </ray>
         <plugin name="${name}_plugin" filename="libgazebo_ros_velodyne_gpu_laser.so">
-          <topicName>${namespace}${sensor_namespace}/${name}/points</topicName>
+          <topicName>${sensor_namespace}/${name}/points</topicName>
           <frameName>${name}_link</frameName>
           <min_intensity>0</min_intensity>

File: wamv_gazebo/urdf/sensors/wamv_camera.xacro (robot description, xacro)
@@ -1,5 +1,5 @@
 <?xml version="1.0"?>
 <robot xmlns:xacro="http://ros.org/wiki/xacro">
-  <xacro:macro name="wamv_camera" params="name x:=0.5 y:=0 z:=1.5 R:=0 P:=0 Y:=0 post_Y:=0 ">
+  <xacro:macro name="wamv_camera" params="name x:=0.5 y:=0 z:=1.5 R:=0 P:=0 Y:=0 post_Y:=0">
     <!-- Define length variables for link positioning -->
     <xacro:property name="platform_z" value="1.2965"/>
@@ -143,5 +143,5 @@
           <alwaysOn>true</alwaysOn>
           <updateRate>0.0</updateRate>
-          <cameraName>${namespace}${camera_namespace}/${name}</cameraName>
+          <cameraName>${camera_namespace}/${name}</cameraName>
           <imageTopicName>image_raw</imageTopicName>
           <cameraInfoTopicName>camera_info</cameraInfoTopicName>

File: wamv_gazebo/urdf/sensors/wamv_gps.xacro (robot description, xacro)
@@ -36,6 +36,6 @@
         <bodyName>${name}_link</bodyName>
         <frameId>${name}_link</frameId>
-        <topicName>${namespace}${sensor_namespace}/gps/fix</topicName>
-        <velocityTopicName>${namespace}${sensor_namespace}/gps/fix_velocity</velocityTopicName>
+        <topicName>${sensor_namespace}/gps/fix</topicName>
+        <velocityTopicName>${sensor_namespace}/gps/fix_velocity</velocityTopicName>
         <!-- Location of origin of Gazebo Sand Island map -->
         <referenceLatitude>21.30996</referenceLatitude>

File: wamv_gazebo/urdf/sensors/wamv_imu.xacro (robot description, xacro)
@@ -21,6 +21,6 @@
         <updateRate>15.0</updateRate>
         <bodyName>${name}_link</bodyName>
-        <topicName>${namespace}${sensor_namespace}/imu/data</topicName>
-        <serviceName>${namespace}${sensor_namespace}/imu_service</serviceName>
+        <topicName>${sensor_namespace}/imu/data</topicName>
+        <serviceName>${sensor_namespace}/imu_service</serviceName>
         <frameId>${name}_link</frameId>
         <alwaysOn>true</alwaysOn>

File: wamv_gazebo/urdf/sensors/wamv_planar_lidar.xacro (robot description, xacro)
@@ -39,5 +39,5 @@
         </ray>
         <plugin name="multibeam_simulator" filename="libgazebo_ros_gpu_laser.so">
-          <topicName>${name}/scan</topicName>
+          <topicName>${sensor_namespace}/${name}/scan</topicName>
           <frameName>${name}_link</frameName>
         </plugin>

File: wamv_gazebo/urdf/thruster_layouts/wamv_gazebo_thruster_config.xacro (robot description, xacro)
@@ -7,6 +7,6 @@
       <propJointName>${name}_engine_propeller_joint</propJointName>
       <engineJointName>${name}_chasis_engine_joint</engineJointName>
-      <cmdTopic>${namespace}${thruster_namespace}/${name}_thrust_cmd</cmdTopic>
-      <angleTopic>${namespace}${thruster_namespace}/${name}_thrust_angle</angleTopic>
+      <cmdTopic>${thruster_namespace}/${name}_thrust_cmd</cmdTopic>
+      <angleTopic>${thruster_namespace}/${name}_thrust_angle</angleTopic>
       <enableAngle>true</enableAngle>
       <!-- Optional Parameters -->

File: wamv_gazebo/urdf/wamv_gazebo.urdf.xacro (robot description, xacro)
@@ -11,9 +11,7 @@
   <xacro:arg name="ground_truth_enabled" default="false" />
   <xacro:arg name="vrx_sensors_enabled" default="false" />
-  <xacro:arg name="namespace" default="/wamv"/>
   <xacro:arg name="thruster_namespace" default="/thrusters"/>
   <xacro:arg name="camera_namespace" default="/cameras"/>
   <xacro:arg name="sensor_namespace" default="/sensors"/>
-  <xacro:property name="namespace" value="$(arg namespace)" scope="global" />
   <xacro:property name="thruster_namespace" value="$(arg thruster_namespace)" scope="global" />
   <xacro:property name="camera_namespace" value="$(arg camera_namespace)" scope="global" />

Commit message: Fully functional solution, with urdf file modified when calling spawn_wamv.bash and giving proper model dirs to wamv_gazebo and wamv_description

File: wamv_description/urdf/thrusters/engine.xacro (robot description, xacro)
@@ -6,5 +6,5 @@
       <visual>
         <geometry>
-          <mesh filename="package://wamv_description/mesh/engine.dae"/>
+          <mesh filename="package://wamv_description/models/engine/mesh/engine.dae"/>
         </geometry>
       </visual>
@@ -29,5 +29,5 @@
       <visual>
         <geometry>
-          <mesh filename="package://wamv_description/mesh/propeller.dae"/>
+          <mesh filename="package://wamv_description/models/propeller/mesh/propeller.dae"/>
         </geometry>
       </visual>

File: wamv_description/urdf/wamv_base.urdf.xacro (robot description, xacro)
@@ -91,5 +91,5 @@
     <visual>
       <geometry>
-        <mesh filename="package://wamv_description/mesh/WAM-V-Base.dae"/>
+        <mesh filename="package://wamv_description/models/WAM-V-Base/mesh/WAM-V-Base.dae"/>
       </geometry>
     </visual>

File: wamv_gazebo/urdf/sensors/wamv_gps.xacro (robot description, xacro)
@@ -5,5 +5,5 @@
       <visual name="${name}_visual">
         <geometry>
-          <mesh filename="package://wamv_gazebo/mesh/gps.dae"/>
+          <mesh filename="package://wamv_gazebo/models/gps/mesh/gps.dae"/>
         </geometry>
       </visual>

Commit message: Added engine and thruster namespace prefix

File: wamv_description/urdf/thrusters/engine.xacro (robot description, xacro)
@@ -3,5 +3,5 @@
   <!-- Macro for inserting an engine with its propeller. -->
   <xacro:macro name="engine" params="prefix position:='0 0 0' orientation:='0 0 0'">
-    <link name="${prefix}_engine_link">
+    <link name="${namespace}/${prefix}_engine_link">
       <visual>
         <geometry>
@@ -26,5 +26,5 @@
       </inertial>
     </link>
-    <link name="${prefix}_propeller_link">
+    <link name="${namespace}/${prefix}_propeller_link">
       <visual>
         <geometry>
@@ -43,15 +43,15 @@
       </inertial>
     </link>
-    <joint name="${prefix}_chasis_engine_joint" type="revolute">
+    <joint name="${namespace}/${prefix}_chasis_engine_joint" type="revolute">
       <axis xyz="0 0 1"/>
       <limit lower="${-pi}" upper="${pi}" effort="10" velocity="10"/>
       <origin xyz="${position}" rpy="${orientation}"/>
       <parent link="base_link"/>
-      <child link="${prefix}_engine_link"/>
+      <child link="${namespace}/${prefix}_engine_link"/>
     </joint>
-    <joint name="${prefix}_engine_propeller_joint" type="continuous">
+    <joint name="${namespace}/${prefix}_engine_propeller_joint" type="continuous">
       <axis rpy="0 0 0" xyz="1 0 0"/>
-      <parent link="${prefix}_engine_link"/>
-      <child link="${prefix}_propeller_link"/>
+      <parent link="${namespace}/${prefix}_engine_link"/>
+      <child link="${namespace}/${prefix}_propeller_link"/>
       <origin rpy="0 0 0" xyz="-0.278156 0 -0.509371"/>
       <limit effort="100" velocity="100" />

File: wamv_gazebo/urdf/thruster_layouts/wamv_gazebo_thruster_config.xacro (robot description, xacro)
@@ -4,7 +4,7 @@
     <thruster>
       <!-- Required Parameters -->
-      <linkName>${name}_propeller_link</linkName>
-      <propJointName>${name}_engine_propeller_joint</propJointName>
-      <engineJointName>${name}_chasis_engine_joint</engineJointName>
+      <linkName>${namespace}/${name}_propeller_link</linkName>
+      <propJointName>${namespace}/${name}_engine_propeller_joint</propJointName>
+      <engineJointName>${namespace}/${name}_chasis_engine_joint</engineJointName>
       <cmdTopic>${thruster_namespace}${name}_thrust_cmd</cmdTopic>
       <angleTopic>${thruster_namespace}${name}_thrust_angle</angleTopic>

Commit message: Updates boat

File: wamv_description/urdf/thrusters/engine.xacro (robot description, xacro)
@@ -4,9 +4,4 @@
   <xacro:macro name="engine" params="prefix position:='0 0 0' orientation:='0 0 0'">
     <link name="${namespace}/${prefix}_engine_link">
-      <visual>
-        <geometry>
-          <mesh filename="package://wamv_description/models/engine/mesh/engine.dae"/>
-        </geometry>
-      </visual>
       <collision name="${prefix}_engine_vertical_axis_collision">
         <origin xyz="-0.16 0 -0.24" rpy="0 0 0" />
@@ -29,5 +24,5 @@
       <visual>
         <geometry>
-          <mesh filename="package://wamv_description/models/propeller/mesh/propeller.dae"/>
+          <mesh filename="package://wamv_description/models/propeller/mesh/propeller.dae" scale="0.42 0.42 0.42"/>
         </geometry>
       </visual>

File: wamv_description/urdf/wamv_base.urdf.xacro (robot description, xacro)
@@ -7,78 +7,8 @@
   <xacro:macro name="main_collisions" params="prefix reflect:=1">
     <!-- Main float -->
-    <collision name="${prefix}_float">
-      <origin xyz="-0.4 ${1.03*reflect} 0.2" rpy="${0*reflect} 1.57 0" />
+    <collision name="rear_${prefix}_beam_upper">
+        <origin xyz="0 -0 0" rpy="0 0 3.1416" />
       <geometry>
-        <cylinder length="4" radius="0.2" />
-      </geometry>
-    </collision>
-    <collision name="${prefix}_mid_float">
-      <origin xyz="1.85 ${1.03*reflect} 0.3" rpy="${0*reflect} 1.38 0" />
-      <geometry>
-        <cylinder length="0.5" radius="0.17" />
-      </geometry>
-    </collision>
-    <collision name="${prefix}_front_float">
-      <origin xyz="2.3 ${1.03*reflect} 0.4" rpy="${0*reflect} 1.3 0" />
-      <geometry>
-        <cylinder length="0.45" radius="0.12" />
-      </geometry>
-    </collision>
-    <!-- Front beam -->
-    <collision name="front_${prefix}_beam_lower">
-      <origin xyz="0.9 ${0.85*reflect} 1" rpy="${0.78*reflect} 0 0" />
-      <geometry>
-        <cylinder length="0.5" radius="0.04" />
-      </geometry>
-    </collision>
-    <collision name="front_${prefix}_beam_upper">
-      <origin xyz="0.9 ${0.6*reflect} 1.18" rpy="${1.35*reflect} 0 0" />
-      <geometry>
-        <cylinder length="0.2" radius="0.04" />
-      </geometry>
-    </collision>
-    <!-- Mid beam -->
-    <collision name="mid_${prefix}_beam_lower">
-      <origin xyz="-0.65 ${0.99*reflect} 0.7" rpy="${0.1*reflect} 0.25 0" />
-      <geometry>
-        <cylinder length="0.45" radius="0.03" />
-      </geometry>
-    </collision>
-    <collision name="mid_${prefix}_beam_medium">
-      <origin xyz="-0.57 ${0.87*reflect} 1.05" rpy="${0.75*reflect} 0.25 0" />
-      <geometry>
-        <cylinder length="0.32" radius="0.03" />
-      </geometry>
-    </collision>
-    <collision name="mid_${prefix}_beam_upper">
-      <origin xyz="-0.55 ${0.65*reflect} 1.17" rpy="${1.35*reflect} 0.25 0" />
-      <geometry>
-        <cylinder length="0.3" radius="0.03" />
-      </geometry>
-    </collision>
-    <!-- Rear beam -->
-    <collision name="rear_${prefix}_beam_lower">
-      <origin xyz="-0.74 ${1.03*reflect} 0.7" rpy="${0*reflect} -0.15 0" />
-      <geometry>
-        <cylinder length="0.45" radius="0.03" />
-      </geometry>
-    </collision>
-    <collision name="rear_${prefix}_beam_medium">
-      <origin xyz="-0.79 ${0.91*reflect} 1.05" rpy="${0.75*reflect} -0.15 0" />
-      <geometry>
-        <cylinder length="0.32" radius="0.03" />
-      </geometry>
-    </collision>
-    <collision name="rear_${prefix}_beam_upper">
-      <origin xyz="-0.81 ${0.67*reflect} 1.18" rpy="${1.45*reflect} -0.15 0" />
-      <geometry>
-        <cylinder length="0.3" radius="0.03" />
-      </geometry>
-    </collision>
-    <!-- Joint -->
-    <collision name="${prefix}_joint">
-      <origin xyz="0.58 ${1.03*reflect} 0.6" rpy="${0*reflect} -0.6 0" />
-      <geometry>
-        <box size="0.65 0.2 0.1" />
+        <mesh filename="package://wamv_description/models/WAM-V-Base/mesh/Balsa.dae" scale="0.15 0.15 015" />
       </geometry>
     </collision>
@@ -90,10 +20,24 @@
     <child link="${namespace}/dummy_link"/>
   </joint>
+  <joint name="${namespace}/dummy2_joint" type = "fixed">
+    <parent link="${namespace}/base_link"/>
+    <child link="${namespace}/dummy2_link"/>
+  </joint>
+  <joint name="${namespace}/dummy3_joint" type = "fixed">
+    <parent link="${namespace}/base_link"/>
+    <child link="${namespace}/dummy3_link"/>
+  </joint>
+    <joint name="${namespace}/imu_joint" type="fixed">
+    <parent link="${namespace}/dummy_link"/>
+    <child link="${namespace}/imu_link"/>
+    <origin rpy="0 0 0" xyz="0 0 0" />
+  </joint>
   <!-- Basic model of the 16' WAM-V USV -->
   <link name="${namespace}/dummy_link">
     <visual>
       <geometry>
-        <mesh filename="package://wamv_description/models/WAM-V-Base/mesh/WAM-V-Base.dae"/>
+        <mesh filename="package://wamv_description/models/WAM-V-Base/mesh/Balsa.dae" scale="0.1 0.1 0.1" />
       </geometry>
+      <origin xyz="0 -0 0" rpy="0 0 3.1416" />
     </visual>
     <!-- Left base collisions -->
@@ -101,11 +45,4 @@
     <!-- Right side collisions -->
     <xacro:main_collisions prefix="right" reflect="-1" />
-     <!-- Top base -->
-    <collision name="top_base">
-      <origin xyz="0 -0 1.25" rpy="0 0 0" />
-      <geometry>
-        <box size="1.85 1 0.1" />
-      </geometry>
-    </collision>
     <inertial>
       <!-- From WAM-V spec sheet -->
@@ -114,3 +51,84 @@
     </inertial>
   </link>
+  <link name="${namespace}/dummy2_link">
+    <visual >
+        <origin xyz="-0.7 0.75 0.26" rpy="0 1.6 0" />
+      <geometry>
+        <cylinder length="0.4" radius="0.04"/>
+      </geometry>
+    </visual>
+    <visual >
+        <origin xyz="-0.7 -0.75 0.26" rpy="0 1.6 0" />
+      <geometry>
+        <cylinder length="0.4" radius="0.04"/>
+      </geometry>
+    </visual>
+    <visual >
+        <origin xyz="0.1 -0.75 0.26" rpy="0 1.6 0" />
+      <geometry>
+        <cylinder length="0.4" radius="0.04"/>
+      </geometry>
+    </visual>
+    <visual >
+      <origin xyz="0.1 0.75 0.26" rpy="0 1.6 0" />
+      <geometry>
+        <cylinder length="0.4" radius="0.04"/>
+      </geometry>
+    </visual>
+    <inertial>
+      <!-- From WAM-V spec sheet -->
+      <mass value="0.1"/>
+      <inertia ixx="120.0" ixy="0.0" ixz="0.0" iyy="393" iyz="0.0" izz="446.0"/>
+    </inertial>
+  </link>
+  <link name="${namespace}/dummy3_link">
+    <visual >
+        <origin xyz="-0.7 0 0.26" rpy="0 0 0" />
+      <geometry>
+        <box size="0.8 0.7 0.1"/>
+      </geometry>
+    </visual>
+    <inertial>
+      <!-- From WAM-V spec sheet -->
+      <mass value="0.1"/>
+      <inertia ixx="120.0" ixy="0.0" ixz="0.0" iyy="393" iyz="0.0" izz="446.0"/>
+    </inertial>
+  </link>
+  <link name="${namespace}/imu_link">
+    <visual>
+      <geometry>
+        <box size="0.01 0.01 0.01" />
+      </geometry>
+    </visual>
+    <collision>
+      <origin rpy="0 0 0" xyz="0 0 0" />
+      <geometry>
+        <box size="0.01 0.01 0.01" />
+      </geometry>
+    </collision>
+  </link>
+ <gazebo reference="${namespace}/dummy_link">
+    <material>Gazebo/Green</material>
+  </gazebo>
+  <gazebo reference="${namespace}/dummy2_link">
+    <material>Gazebo/Black</material>
+  </gazebo>
+  <gazebo reference="${namespace}/dummy3_link">
+    <material>Gazebo/White</material>
+  </gazebo>
+<gazebo reference="${namespace}/imu_link">
+<plugin name="gazebo_imu_plugin" filename="libgazebo_imu_plugin.so">
+      <robotNamespace></robotNamespace>
+      <linkName>${namespace}/imu_link</linkName>
+      <imuTopic>/imu</imuTopic>
+      <gyroscopeNoiseDensity>0.0003394</gyroscopeNoiseDensity>
+      <gyroscopeRandomWalk>3.8785e-05</gyroscopeRandomWalk>
+      <gyroscopeBiasCorrelationTime>1000.0</gyroscopeBiasCorrelationTime>
+      <gyroscopeTurnOnBiasSigma>0.0087</gyroscopeTurnOnBiasSigma>
+      <accelerometerNoiseDensity>0.004</accelerometerNoiseDensity>
+      <accelerometerRandomWalk>0.006</accelerometerRandomWalk>
+      <accelerometerBiasCorrelationTime>300.0</accelerometerBiasCorrelationTime>
+      <accelerometerTurnOnBiasSigma>0.196</accelerometerTurnOnBiasSigma>
+  </plugin>
+</gazebo>
 </robot>
