Commit message: Bug solution multi-vehicles in wamv_gazebo.urdf.xacro
When trying to launch a second vessel with the name wamv2, the following error message was shown
"[ERROR] [launch]: Caught exception in launch (see debug for traceback): Error Code 20: Msg: Child frame with name[wamv/base_link] specified by joint with name[wamv_external_pivot_joint] not found in model with name[WAM-V]"
The problem was found in line 103 of the wamv_gazebo.urdf.xacro file, in which the namespace was not properly referenced to the namespace but only to the standard topic namespace of "wamv/base_link". As a result without changing the child to "$(arg namespace)/base_link, it is not possible to spawn a second vehicle with a different namespace. Therefor, without the change, it would not be possible to control the vessels independent of each other, as both subscribe to the same topic.

File: vrx_urdf/wamv_gazebo/urdf/wamv_gazebo.urdf.xacro (robot description, xacro)
@@ -91,5 +91,5 @@
       <joint name="wamv_external_pivot_joint" type="universal">
         <parent>wamv_external_link</parent>
-        <child>wamv/base_link</child>
+        <child>$(arg namespace)/base_link</child>
         <axis>
           <xyz>1 0 0</xyz>

Commit message: Move the extra links to [un]lock the WAM-V out of the model and into the platforms.
Signed-off-by: Carlos Agüero <caguero@openrobotics.org>

File: vrx_urdf/wamv_gazebo/urdf/wamv_gazebo.urdf.xacro (robot description, xacro)
@@ -60,63 +60,14 @@
     </xacro:if>
   </xacro:unless>
-  <!-- === Decide if we lock the robot to the world === -->
-  <xacro:if value="$(arg locked)">
-    <gazebo>
-      <link name="wamv_external_link">
-        <inertial>
-          <mass>0.001</mass>
-          <inertia>
-            <ixx>0.00000004</ixx>
-            <ixy>0</ixy>
-            <ixz>0</ixz>
-            <iyy>0.00000004</iyy>
-            <iyz>0</iyz>
-            <izz>0.00000004</izz>
-          </inertia>
-        </inertial>
-      </link>
-      <link name="wamv_external_link_base">
-        <inertial>
-          <mass>0.001</mass>
-          <inertia>
-            <ixx>0.00000004</ixx>
-            <ixy>0</ixy>
-            <ixz>0</ixz>
-            <iyy>0.00000004</iyy>
-            <iyz>0</iyz>
-            <izz>0.00000004</izz>
-          </inertia>
-        </inertial>
-      </link>
-      <joint name="wamv_external_pivot_joint" type="universal">
-        <parent>wamv_external_link</parent>
-        <child>$(arg namespace)/base_link</child>
-        <axis>
-          <xyz>1 0 0</xyz>
-        </axis>
-        <axis2>
-          <xyz>0 1 0</xyz>
-        </axis2>
-      </joint>
-      <joint name="wamv_external_riser" type="prismatic">
-        <parent>wamv_external_link_base</parent>
-        <child>wamv_external_link</child>
-        <axis>
-          <limit>
-            <lower>-3</lower>
-            <upper>3</upper>
-          </limit>
-          <xyz>0 0 1</xyz>
-        </axis>
-      </joint>
-      <plugin filename="gz-sim-detachable-joint-system" name="gz::sim::systems::DetachableJoint">
-        <parent_link>wamv_external_link_base</parent_link>
-        <child_model>platform</child_model>
-        <child_link>dummy_base</child_link>
-        <topic>/vrx/release</topic>
-        <suppress_child_warning>true</suppress_child_warning>
-      </plugin>
-    </gazebo>
-  </xacro:if>
+  <!-- === [Un]lock the robot to the world === -->
+  <gazebo>
+    <plugin filename="gz-sim-detachable-joint-system" name="gz::sim::systems::DetachableJoint">
+      <parent_link>$(arg namespace)/base_link</parent_link>
+      <child_model>platform</child_model>
+      <child_link>dummy_upper</child_link>
+      <topic>/vrx/release</topic>
+      <suppress_child_warning>true</suppress_child_warning>
+    </plugin>
+  </gazebo>
   <!-- === TF === -->
   <!-- Publish robot state information -->
