Commit message: Fix issue #690 (#706)
* Move the extra links to [un]lock the WAM-V out of the model and into the platforms.

Signed-off-by: Carlos Agüero <caguero@openrobotics.org>

File: vrx_urdf/wamv_gazebo/urdf/dynamics/wamv_gazebo_dynamics_plugin.xacro (robot description, xacro)
@@ -45,13 +45,15 @@
         <nDotR>0.0</nDotR>
         <!-- Linear and quadratic drag -->
-        <xU>51.3</xU>
-        <xUU>72.4</xUU>
-        <yV>40.0</yV>
-        <yVV>0.0</yVV>
+        <xU>100.0</xU>
+        <xUU>150.0</xUU>
+        <yV>100.0</yV>
+        <yVV>100.0</yVV>
         <zW>500.0</zW>
-        <kP>100.0</kP>
-        <mQ>100.0</mQ>
-        <nR>400.0</nR>
-        <nRR>0.0</nRR>
+        <kP>300.0</kP>
+        <kPP>600.0</kPP>
+        <mQ>900.0</mQ>
+        <mQQ>900.0</mQQ>
+        <nR>800.0</nR>
+        <nRR>800.0</nRR>
       </plugin>
     </gazebo>

File: vrx_urdf/wamv_gazebo/urdf/wamv_gazebo.urdf.xacro (robot description, xacro)
@@ -60,63 +60,14 @@
     </xacro:if>
   </xacro:unless>
-  <!-- === Decide if we lock the robot to the world === -->
-  <xacro:if value="$(arg locked)">
-    <gazebo>
-      <link name="wamv_external_link">
-        <inertial>
-          <mass>0.001</mass>
-          <inertia>
-            <ixx>0.00000004</ixx>
-            <ixy>0</ixy>
-            <ixz>0</ixz>
-            <iyy>0.00000004</iyy>
-            <iyz>0</iyz>
-            <izz>0.00000004</izz>
-          </inertia>
-        </inertial>
-      </link>
-      <link name="wamv_external_link_base">
-        <inertial>
-          <mass>0.001</mass>
-          <inertia>
-            <ixx>0.00000004</ixx>
-            <ixy>0</ixy>
-            <ixz>0</ixz>
-            <iyy>0.00000004</iyy>
-            <iyz>0</iyz>
-            <izz>0.00000004</izz>
-          </inertia>
-        </inertial>
-      </link>
-      <joint name="wamv_external_pivot_joint" type="universal">
-        <parent>wamv_external_link</parent>
-        <child>$(arg namespace)/base_link</child>
-        <axis>
-          <xyz>1 0 0</xyz>
-        </axis>
-        <axis2>
-          <xyz>0 1 0</xyz>
-        </axis2>
-      </joint>
-      <joint name="wamv_external_riser" type="prismatic">
-        <parent>wamv_external_link_base</parent>
-        <child>wamv_external_link</child>
-        <axis>
-          <limit>
-            <lower>-3</lower>
-            <upper>3</upper>
-          </limit>
-          <xyz>0 0 1</xyz>
-        </axis>
-      </joint>
-      <plugin filename="gz-sim-detachable-joint-system" name="gz::sim::systems::DetachableJoint">
-        <parent_link>wamv_external_link_base</parent_link>
-        <child_model>platform</child_model>
-        <child_link>dummy_base</child_link>
-        <topic>/vrx/release</topic>
-        <suppress_child_warning>true</suppress_child_warning>
-      </plugin>
-    </gazebo>
-  </xacro:if>
+  <!-- === [Un]lock the robot to the world === -->
+  <gazebo>
+    <plugin filename="gz-sim-detachable-joint-system" name="gz::sim::systems::DetachableJoint">
+      <parent_link>$(arg namespace)/base_link</parent_link>
+      <child_model>platform</child_model>
+      <child_link>dummy_upper</child_link>
+      <topic>/vrx/release</topic>
+      <suppress_child_warning>true</suppress_child_warning>
+    </plugin>
+  </gazebo>
   <!-- === TF === -->
   <!-- Publish robot state information -->
